File: l2_dev_board/Design/Buffering.sch (KiCad schematic (older format))
At the start: 20 parts, among them U302 NC7WZ17, U303 NC7WZ17, U304 NC7WZ17, U305 NC7WZ17, U306 NC7WZ17, U307 NC7WZ17, U308 NC7WZ17, U309 NC7WZ17, U310 NC7WZ17, U311 NC7WZ17

Commit message: Isolated L1 stuff (inc. JTAG) in single sheet. Added buffered for the L2's JTAG control signals.
Parts:
- removed U308: NC7WZ17, symbol NC7WZ17
- added R? (x10): 10K, symbol R
- added U? (x4): NC7WZ07, symbol NC7WZ07
Connections:
- net labels added: MSEL_N, MSEL_N_BUF_0, MSEL_N_BUF_1, MSEL_N_BUF_2, MSEL_N_BUF_3, RST_N_BUF_0, RST_N_BUF_1
- net labels removed: MSEL_BUF_2
- wire segments 113 -> 125
Other:
- note added: "L2 \nJTAG TCK TMS Buffering"
- note added: "L2\nJTAG RST_N MSEL_N L2 Buffering"
- moved on the sheet: U309

Commit message: removing old buffering and wanted to check point
Parts:
- removed U309: NC7WZ17, symbol NC7WZ17
- gave numbers to parts that had none: 14
Other:
- moved on the sheet: R303, R305, R307, R309, R318, R319, R320, R321, U304, U305, U310, U311

Commit message: missing header connector for 2 L2s. Find space!
Parts:
- removed R303, R305, R307, R309, R318, R319, R320, R321: 10K, symbol R
- removed U304, U305, U310, U311: NC7WZ17, symbol NC7WZ17
Other:
- note removed: "JTAG L1 Buffering"
- note removed: "JTAG L2 Buffering"

Commit message: new design with heirachial and new libraries
Parts:
- renumbered R306 to R201, R308 to R202, R202 to R203, R203 to R204, R204 to R205, R205 to R206, R206 to R207, R207 to R208, R208 to R209, R209 to R210, R210 to R211, R211 to R212, U302 to U201, U303 to U202, U306 to U203, U307 to U204, U202 to U205, U203 to U206, U204 to U207, U205 to U208
Changed lines of the file:
@@
-EESchema Schematic File Version 2  date 29/07/2011 09:19:43
+EESchema Schematic File Version 2  date 29/07/2011 14:29:23
 LIBS:power
 LIBS:device
@@
 +3V3
 $Comp
-L R R211
+L R R212
 U 1 1 4E3161E2
 P 5890 4030
-F 0 "R211" V 5940 3830 50  0000 C CNN
+F 0 "R212" V 5940 3830 50  0000 C CNN
 F 1 "10K" V 5890 4030 50  0000 C CNN
 	1    5890 4030
@@
 $EndComp
 $Comp
-L R R207
+L R R208
 U 1 1 4E3161E1
 P 5770 4030
-F 0 "R207" V 5820 3830 50  0000 C CNN
+F 0 "R208" V 5820 3830 50  0000 C CNN
 F 1 "10K" V 5770 4030 50  0000 C CNN
 	1    5770 4030
@@
 $EndComp
 $Comp
-L R R206
+L R R207
 U 1 1 4E3161D3
 P 5770 3030
-F 0 "R206" V 5820 2830 50  0000 C CNN
+F 0 "R207" V 5820 2830 50  0000 C CNN
 F 1 "10K" V 5770 3030 50  0000 C CNN
 	1    5770 3030
@@
 $EndComp
 $Comp
-L R R210
+L R R211
 U 1 1 4E3161D2
 P 5890 3030
-F 0 "R210" V 5940 2830 50  0000 C CNN
+F 0 "R211" V 5940 2830 50  0000 C CNN
 F 1 "10K" V 5890 3030 50  0000 C CNN
 	1    5890 3030
@@
 +3V3
 $Comp
-L R R209
+L R R210
 U 1 1 4E3161B2
 P 5890 2030
-F 0 "R209" V 5940 1830 50  0000 C CNN
+F 0 "R210" V 5940 1830 50  0000 C CNN
 F 1 "10K" V 5890 2030 50  0000 C CNN
 	1    5890 2030
@@
 $EndComp
 $Comp
-L R R205
+L R R206
 U 1 1 4E3161B1
 P 5770 2030
-F 0 "R205" V 5820 1830 50  0000 C CNN
+F 0 "R206" V 5820 1830 50  0000 C CNN
 F 1 "10K" V 5770 2030 50  0000 C CNN
 	1    5770 2030
@@
 RST_N_BUF_2
 $Comp
-L R R204
+L R R205
 U 1 1 4E316108
 P 5770 1030
-F 0 "R204" V 5820 830 50  0000 C CNN
+F 0 "R205" V 5820 830 50  0000 C CNN
 F 1 "10K" V 5770 1030 50  0000 C CNN
 	1    5770 1030
@@
 $EndComp
 $Comp
-L R R208
+L R R209
 U 1 1 4E316107
 P 5890 1030
-F 0 "R208" V 5940 830 50  0000 C CNN
+F 0 "R209" V 5940 830 50  0000 C CNN
 F 1 "10K" V 5890 1030 50  0000 C CNN
 	1    5890 1030
@@
 +3V3
 $Comp
-L GND #PWR018
+L GND #PWR020
 U 1 1 4E315D30
 P 5400 4790
-F 0 "#PWR018" H 5400 4790 30  0001 C CNN
+F 0 "#PWR020" H 5400 4790 30  0001 C CNN
 F 1 "GND" H 5400 4720 30  0001 C CNN
 	1    5400 4790
@@
 MSEL_N_BUF_3
 $Comp
-L NC7WZ07 U205
+L NC7WZ07 U208
 U 1 1 4E315D2F
 P 4750 4440
-F 0 "U205" H 4450 4840 60  0000 C CNN
+F 0 "U208" H 4450 4840 60  0000 C CNN
 F 1 "NC7WZ07" H 4600 4040 60  0000 C CNN
 	1    4750 4440
@@
 $EndComp
 $Comp
-L GND #PWR019
+L GND #PWR021
 U 1 1 4E315D25
 P 5400 3790
-F 0 "#PWR019" H 5400 3790 30  0001 C CNN
+F 0 "#PWR021" H 5400 3790 30  0001 C CNN
 F 1 "GND" H 5400 3720 30  0001 C CNN
 	1    5400 3790
@@
 MSEL_N_BUF_2
 $Comp
-L NC7WZ07 U204
+L NC7WZ07 U207
 U 1 1 4E315D24
 P 4750 3440
-F 0 "U204" H 4450 3840 60  0000 C CNN
+F 0 "U207" H 4450 3840 60  0000 C CNN
 F 1 "NC7WZ07" H 4600 3040 60  0000 C CNN
 	1    4750 3440
@@
 $EndComp
 $Comp
-L GND #PWR020
+L GND #PWR022
 U 1 1 4E315D05
 P 5400 2790
-F 0 "#PWR020" H 5400 2790 30  0001 C CNN
+F 0 "#PWR022" H 5400 2790 30  0001 C CNN
 F 1 "GND" H 5400 2720 30  0001 C CNN
 	1    5400 2790
@@
 MSEL_N_BUF_1
 $Comp
-L NC7WZ07 U203
+L NC7WZ07 U206
 U 1 1 4E315D04
 P 4750 2440
-F 0 "U203" H 4450 2840 60  0000 C CNN
+F 0 "U206" H 4450 2840 60  0000 C CNN
 F 1 "NC7WZ07" H 4600 2040 60  0000 C CNN
 	1    4750 2440
@@
 $EndComp
 $Comp
-L R R202
+L R R203
 U 1 1 4E315C86
 P 3910 1030
-F 0 "R202" V 3960 830 50  0000 C CNN
+F 0 "R203" V 3960 830 50  0000 C CNN
 F 1 "10K" V 3910 1030 50  0000 C CNN
 	1    3910 1030
@@
 $EndComp
 $Comp
-L R R203
+L R R204
 U 1 1 4E315C85
 P 4030 1030
-F 0 "R203" V 4080 830 50  0000 C CNN
+F 0 "R204" V 4080 830 50  0000 C CNN
 F 1 "10K" V 4030 1030 50  0000 C CNN
 	1    4030 1030
@@
 $EndComp
 $Comp
-L NC7WZ07 U202
+L NC7WZ07 U205
 U 1 1 4E315966
 P 4750 1440
-F 0 "U202" H 4450 1840 60  0000 C CNN
+F 0 "U205" H 4450 1840 60  0000 C CNN
 F 1 "NC7WZ07" H 4600 1040 60  0000 C CNN
 	1    4750 1440
@@
 +3V3
 $Comp
-L GND #PWR021
+L GND #PWR023
 U 1 1 4E3155B0
 P 2670 4790
-F 0 "#PWR021" H 2670 4790 30  0001 C CNN
+F 0 "#PWR023" H 2670 4790 30  0001 C CNN
 F 1 "GND" H 2670 4720 30  0001 C CNN
 	1    2670 4790
@@
 +3V3
 $Comp
-L GND #PWR022
+L GND #PWR024
 U 1 1 4E31557E
 P 2670 3790
-F 0 "#PWR022" H 2670 3790 30  0001 C CNN
+F 0 "#PWR024" H 2670 3790 30  0001 C CNN
 F 1 "GND" H 2670 3720 30  0001 C CNN
 	1    2670 3790
@@
 +3V3
 $Comp
-L GND #PWR023
+L GND #PWR025
 U 1 1 4E302B4C
 P 5400 1790
-F 0 "#PWR023" H 5400 1790 30  0001 C CNN
+F 0 "#PWR025" H 5400 1790 30  0001 C CNN
 F 1 "GND" H 5400 1720 30  0001 C CNN
 	1    5400 1790
@@
 $EndComp
 $Comp
-L NC7WZ17 U307
+L NC7WZ17 U204
 U 1 1 4E302B33
 P 2020 4440
-F 0 "U307" H 1720 4840 60  0000 C CNN
+F 0 "U204" H 1720 4840 60  0000 C CNN
 F 1 "NC7WZ17" H 1870 4040 60  0000 C CNN
 	1    2020 4440
@@
 $EndComp
 $Comp
-L NC7WZ17 U306
+L NC7WZ17 U203
 U 1 1 4E302B32
 P 2020 3440
-F 0 "U306" H 1720 3840 60  0000 C CNN
+F 0 "U203" H 1720 3840 60  0000 C CNN
 F 1 "NC7WZ17" H 1870 3040 60  0000 C CNN
 	1    2020 3440
@@
 $EndComp
 $Comp
-L NC7WZ17 U302
+L NC7WZ17 U201
 U 1 1 4E302A25
 P 2020 1440
-F 0 "U302" H 1720 1840 60  0000 C CNN
+F 0 "U201" H 1720 1840 60  0000 C CNN
 F 1 "NC7WZ17" H 1870 1040 60  0000 C CNN
 	1    2020 1440
@@
 $EndComp
 $Comp
-L NC7WZ17 U303
+L NC7WZ17 U202
 U 1 1 4E302A24
 P 2020 2440
-F 0 "U303" H 1720 2840 60  0000 C CNN
+F 0 "U202" H 1720 2840 60  0000 C CNN
 F 1 "NC7WZ17" H 1870 2040 60  0000 C CNN
 	1    2020 2440
@@
 +3V3
 $Comp
-L GND #PWR024
+L GND #PWR026
 U 1 1 4E302A23
 P 2670 1790
-F 0 "#PWR024" H 2670 1790 30  0001 C CNN
+F 0 "#PWR026" H 2670 1790 30  0001 C CNN
 F 1 "GND" H 2670 1720 30  0001 C CNN
 	1    2670 1790
@@
 $EndComp
 $Comp
-L GND #PWR025
+L GND #PWR027
 U 1 1 4E302A22
 P 2670 2790
-F 0 "#PWR025" H 2670 2790 30  0001 C CNN
+F 0 "#PWR027" H 2670 2790 30  0001 C CNN
 F 1 "GND" H 2670 2720 30  0001 C CNN
 	1    2670 2790
@@
 +3V3
 $Comp
-L R R308
+L R R202
 U 1 1 4E302A21
 P 1300 1030
-F 0 "R308" V 1350 830 50  0000 C CNN
+F 0 "R202" V 1350 830 50  0000 C CNN
 F 1 "10K" V 1300 1030 50  0000 C CNN
 	1    1300 1030
@@
 $EndComp
 $Comp
-L R R306
+L R R201
 U 1 1 4E302A20
 P 1180 1030
-F 0 "R306" V 1230 830 50  0000 C CNN
+F 0 "R201" V 1230 830 50  0000 C CNN
 F 1 "10K" V 1180 1030 50  0000 C CNN
 	1    1180 1030
