File: l2_dev_board/Design/L1_Power.sch (KiCad schematic (older format))
At the start: 18 parts

Commit message: squash and back to work!
Parts:
- gave numbers to parts that had none: 18
Changed lines of the file:
@@
-EESchema Schematic File Version 2  date 27/07/2011 16:09:28
+EESchema Schematic File Version 2  date 27/07/2011 16:56:06
 LIBS:power
 LIBS:device
@@
 $EndDescr
 $Comp
-L NCP1521B U?
+L NCP1521B U403
 U 1 1 4E3022F0
 P 2650 3400
-F 0 "U?" H 2650 3350 60  0000 C CNN
+F 0 "U403" H 2650 3350 60  0000 C CNN
 F 1 "NCP1521B" H 2650 3450 60  0000 C CNN
 	1    2650 3400
@@
 +5V
 $Comp
-L C C?
+L C C413
 U 1 1 4E301C8E
 P 1750 3250
-F 0 "C?" H 1800 3350 50  0000 L CNN
+F 0 "C413" H 1800 3350 50  0000 L CNN
 F 1 "10uF" H 1800 3150 50  0000 L CNN
 	1    1750 3250
@@
 $EndComp
 $Comp
-L GND #PWR?
+L GND #PWR018
 U 1 1 4E301C8D
 P 1750 3450
-F 0 "#PWR?" H 1750 3450 30  0001 C CNN
+F 0 "#PWR018" H 1750 3450 30  0001 C CNN
 F 1 "GND" H 1750 3380 30  0001 C CNN
 	1    1750 3450
@@
 $EndComp
 $Comp
-L GND #PWR?
+L GND #PWR019
 U 1 1 4E301C8C
 P 2650 4050
-F 0 "#PWR?" H 2650 4050 30  0001 C CNN
+F 0 "#PWR019" H 2650 4050 30  0001 C CNN
 F 1 "GND" H 2650 3980 30  0001 C CNN
 	1    2650 4050
@@
 $EndComp
 $Comp
-L INDUCTOR L?
+L INDUCTOR L402
 U 1 1 4E301C8B
 P 3700 3050
-F 0 "L?" V 3650 3050 40  0000 C CNN
+F 0 "L402" V 3650 3050 40  0000 C CNN
 F 1 "2u2H" V 3800 3050 40  0000 C CNN
 	1    3700 3050
@@
 $EndComp
 $Comp
-L C C?
+L C C415
 U 1 1 4E301C8A
 P 4250 3350
-F 0 "C?" H 4300 3450 50  0000 L CNN
+F 0 "C415" H 4300 3450 50  0000 L CNN
 F 1 "33pF" H 4300 3250 50  0000 L CNN
 	1    4250 3350
@@
 $EndComp
 $Comp
-L R R?
+L R R404
 U 1 1 4E301C89
 P 4000 3350
-F 0 "R?" V 4080 3350 50  0000 C CNN
+F 0 "R404" V 4080 3350 50  0000 C CNN
 F 1 "68k" V 4000 3350 50  0000 C CNN
 	1    4000 3350
@@
 $EndComp
 $Comp
-L R R?
+L R R405
 U 1 1 4E301C88
 P 4000 3900
-F 0 "R?" V 4080 3900 50  0000 C CNN
+F 0 "R405" V 4080 3900 50  0000 C CNN
 F 1 "100k" V 4000 3900 50  0000 C CNN
 	1    4000 3900
@@
 $EndComp
 $Comp
-L C C?
+L C C417
 U 1 1 4E301C87
 P 4550 3250
-F 0 "C?" H 4600 3350 50  0000 L CNN
+F 0 "C417" H 4600 3350 50  0000 L CNN
 F 1 "10uF" H 4600 3150 50  0000 L CNN
 	1    4550 3250
@@
 $EndComp
 $Comp
-L GND #PWR?
+L GND #PWR020
 U 1 1 4E301C86
 P 4000 4150
-F 0 "#PWR?" H 4000 4150 30  0001 C CNN
+F 0 "#PWR020" H 4000 4150 30  0001 C CNN
 F 1 "GND" H 4000 4080 30  0001 C CNN
 	1    4000 4150
@@
 $EndComp
 $Comp
-L GND #PWR?
+L GND #PWR021
 U 1 1 4E301C85
 P 4550 3450
-F 0 "#PWR?" H 4550 3450 30  0001 C CNN
+F 0 "#PWR021" H 4550 3450 30  0001 C CNN
 F 1 "GND" H 4550 3380 30  0001 C CNN
 	1    4550 3450
@@
 	5150 4250 1100 4250
 Wire Wire Line
-	4250 3650 4250 3550
+	4250 3550 4250 3650
 Connection ~ 4550 3050
 Wire Wire Line
-	4000 3050 4650 3050
-Wire Wire Line
-	4000 3100 4000 3050
+	4650 3050 4000 3050
+Wire Wire Line
+	4000 3050 4000 3100
 Wire Wire Line
 	1900 3650 1750 3650
@@
 Connection ~ 1750 3050
 Wire Wire Line
-	3400 3650 4250 3650
+	4250 3650 3400 3650
 Connection ~ 4000 3650
 Wire Wire Line
@@
 	4000 3600 4000 3650
 Wire Notes Line
-	5150 2850 5150 4250
-Wire Notes Line
-	1100 2850 5150 2850
+	5150 4250 5150 2850
+Wire Notes Line
+	5150 2850 1100 2850
 Wire Notes Line
 	1100 2850 1100 4250
@@
 +3V3
 $Comp
-L NCP1529 U?
+L NCP1529 U402
 U 1 1 4E3018CD
 P 2500 1700
-F 0 "U?" H 2500 1650 60  0000 C CNN
+F 0 "U402" H 2500 1650 60  0000 C CNN
 F 1 "NCP1529" H 2500 1750 60  0000 C CNN
 	1    2500 1700
@@
 +5V
 $Comp
-L C C?
+L C C412
 U 1 1 4E3018CC
 P 1600 1550
-F 0 "C?" H 1650 1650 50  0000 L CNN
+F 0 "C412" H 1650 1650 50  0000 L CNN
 F 1 "10uF" H 1650 1450 50  0000 L CNN
 	1    1600 1550
@@
 $EndComp
 $Comp
-L GND #PWR?
+L GND #PWR022
 U 1 1 4E3018CB
 P 1600 1750
-F 0 "#PWR?" H 1600 1750 30  0001 C CNN
+F 0 "#PWR022" H 1600 1750 30  0001 C CNN
 F 1 "GND" H 1600 1680 30  0001 C CNN
 	1    1600 1750
@@
 $EndComp
 $Comp
-L GND #PWR?
+L GND #PWR023
 U 1 1 4E3018CA
 P 2500 2350
-F 0 "#PWR?" H 2500 2350 30  0001 C CNN
+F 0 "#PWR023" H 2500 2350 30  0001 C CNN
 F 1 "GND" H 2500 2280 30  0001 C CNN
 	1    2500 2350
@@
 $EndComp
 $Comp
-L INDUCTOR L?
+L INDUCTOR L401
 U 1 1 4E3018C9
 P 3550 1350
-F 0 "L?" V 3500 1350 40  0000 C CNN
+F 0 "L401" V 3500 1350 40  0000 C CNN
 F 1 "2u2H" V 3650 1350 40  0000 C CNN
 	1    3550 1350
@@
 $EndComp
 $Comp
-L C C?
+L C C414
 U 1 1 4E3018C8
 P 4100 1650
-F 0 "C?" H 4150 1750 50  0000 L CNN
+F 0 "C414" H 4150 1750 50  0000 L CNN
 F 1 "33pF" H 4150 1550 50  0000 L CNN
 	1    4100 1650
@@
 $EndComp
 $Comp
-L R R?
+L R R402
 U 1 1 4E3018C7
 P 3850 1650
-F 0 "R?" V 3930 1650 50  0000 C CNN
+F 0 "R402" V 3930 1650 50  0000 C CNN
 F 1 "68k" V 3850 1650 50  0000 C CNN
 	1    3850 1650
@@
 $EndComp
 $Comp
-L R R?
+L R R403
 U 1 1 4E3018C6
 P 3850 2200
-F 0 "R?" V 3930 2200 50  0000 C CNN
+F 0 "R403" V 3930 2200 50  0000 C CNN
 F 1 "15k" V 3850 2200 50  0000 C CNN
 	1    3850 2200
@@
 $EndComp
 $Comp
-L C C?
+L C C416
 U 1 1 4E3018C5
 P 4400 1550
-F 0 "C?" H 4450 1650 50  0000 L CNN
+F 0 "C416" H 4450 1650 50  0000 L CNN
 F 1 "10uF" H 4450 1450 50  0000 L CNN
 	1    4400 1550
@@
 $EndComp
 $Comp
-L GND #PWR?
+L GND #PWR024
 U 1 1 4E3018C4
 P 3850 2450
-F 0 "#PWR?" H 3850 2450 30  0001 C CNN
+F 0 "#PWR024" H 3850 2450 30  0001 C CNN
 F 1 "GND" H 3850 2380 30  0001 C CNN
 	1    3850 2450
@@
 $EndComp
 $Comp
-L GND #PWR?
+L GND #PWR025
 U 1 1 4E3018C3
 P 4400 1750
-F 0 "#PWR?" H 4400 1750 30  0001 C CNN
+F 0 "#PWR025" H 4400 1750 30  0001 C CNN
 F 1 "GND" H 4400 1680 30  0001 C CNN
 	1    4400 1750
@@
 3.3V 1A Power Island\nFor L1 + extras
 $Comp
-L APX803 U?
+L APX803 U405
 U 1 1 4E3018C2
 P 7300 1850
-F 0 "U?" H 7050 2100 39  0000 C CNN
+F 0 "U405" H 7050 2100 39  0000 C CNN
 F 1 "APX803" H 7100 1600 39  0000 C CNN
 F 2 "SOT23R" H 7100 1750 20  0001 C CNN
@@
 $EndComp
 $Comp
-L APX803 U?
+L APX803 U404
 U 1 1 4E3018C1
 P 6150 1850
-F 0 "U?" H 5900 2100 39  0000 C CNN
+F 0 "U404" H 5900 2100 39  0000 C CNN
 F 1 "APX803" H 5950 1600 39  0000 C CNN
 F 2 "SOT23R" H 5950 1750 20  0001 C CNN
@@
 +3V3
 $Comp
-L R R?
+L R R406
 U 1 1 4E3018C0
 P 6800 1500
-F 0 "R?" V 6880 1500 50  0000 C CNN
+F 0 "R406" V 6880 1500 50  0000 C CNN
 F 1 "1K" V 6800 1500 50  0000 C CNN
 	1    6800 1500
@@
 +3V3
 $Comp
-L R R?
+L R R407
 U 1 1 4E3018BF
 P 7800 1500
-F 0 "R?" V 7880 1500 50  0000 C CNN
+F 0 "R407" V 7880 1500 50  0000 C CNN
 F 1 "10K" V 7800 1500 50  0000 C CNN
 	1    7800 1500
@@
 RST_N_BUF_L1
 $Comp
-L GND #PWR?
+L GND #PWR026
 U 1 1 4E3018BE
 P 6150 2250
-F 0 "#PWR?" H 6150 2250 30  0001 C CNN
+F 0 "#PWR026" H 6150 2250 30  0001 C CNN
 F 1 "GND" H 6150 2180 30  0001 C CNN
 	1    6150 2250
@@
 $EndComp
 $Comp
-L GND #PWR?
+L GND #PWR027
 U 1 1 4E3018BD
 P 7300 2250
-F 0 "#PWR?" H 7300 2250 30  0001 C CNN
+F 0 "#PWR027" H 7300 2250 30  0001 C CNN
 F 1 "GND" H 7300 2180 30  0001 C CNN
 	1    7300 2250
