File: l2_dev_board/Design/L2.sch (KiCad schematic (older format))
At the start: 13 parts, among them U201 XS1_L2

Commit message: Started adding tracks
Parts:
- C209: footprint (none) -> X-0402
Changed lines of the file:
@@
-EESchema Schematic File Version 2  date 22/07/2011 14:08:59
+EESchema Schematic File Version 2  date 25/07/2011 13:55:09
 LIBS:power
 LIBS:device
@@
 LIBS:contrib
 LIBS:valves
-LIBS:LT3480
-LIBS:ncp1529
-LIBS:ncp303
-LIBS:nc7wz17
 LIBS:apx803
 LIBS:ase_20mhz
+LIBS:brooktre
+LIBS:cmos_ieee
 LIBS:Dmitri_Belimovl
 LIBS:EECV
+LIBS:elec-unifil
 LIBS:ft232r
+LIBS:gennum
+LIBS:graphic
+LIBS:LT3480
+LIBS:microchip1
+LIBS:nc7wz17
+LIBS:ncp303
+LIBS:ncp1529
+LIBS:pspice
 LIBS:SymbolsSimilarEN60617+oldDIN617
+LIBS:transf
+LIBS:ttl_ieee
+LIBS:video
 LIBS:xmos_capacitors
 LIBS:xmos_resistors
@@
 LIBS:xs1
 LIBS:XS1_L2_V2
-LIBS:L2DevBoard-cache
 EELAYER 25  0
 EELAYER END
 $Descr A4 11700 8267
 encoding utf-8
-Sheet 6 10
+Sheet 9 10
 Title ""
-Date "22 jul 2011"
+Date "25 jul 2011"
 Rev ""
 Comp ""
@@
 AR Path="/4E1ACC57/4E282660" Ref="U801"  Part="1"
 AR Path="/4E146472/4E282660" Ref="U901"  Part="1"
-F 0 "U701" H 3200 3800 50  0000 C CNN
+F 0 "U901" H 3200 3800 50  0000 C CNN
 F 1 "XS1_L2" H 3200 3900 50  0000 C CNN
 F 2 "124" H 3200 3700 60  0000 C CNN
@@
 AR Path="/4E1ACC57/4E17143C" Ref="#PWR030"  Part="1"
 AR Path="/4E146472/4E17143C" Ref="#PWR034"  Part="1"
-F 0 "#PWR026" H 2650 6450 30  0001 C CNN
+F 0 "#PWR034" H 2650 6450 30  0001 C CNN
 F 1 "GND" H 2650 6380 30  0001 C CNN
 	1    2650 6450
@@
 AR Path="/4E1ACC57/4E171407" Ref="#PWR031"  Part="1"
 AR Path="/4E146472/4E171407" Ref="#PWR035"  Part="1"
-F 0 "#PWR027" H 950 6450 30  0001 C CNN
+F 0 "#PWR035" H 950 6450 30  0001 C CNN
 F 1 "GND" H 950 6380 30  0001 C CNN
 	1    950  6450
@@
 AR Path="/4E1ACC57/4E1713E0" Ref="C811"  Part="1"
 AR Path="/4E146472/4E1713E0" Ref="C911"  Part="1"
-F 0 "C711" H 3700 6250 25  0000 L CNN
+F 0 "C911" H 3700 6250 25  0000 L CNN
 F 1 "10uF" H 3700 6050 25  0000 L CNN
 	1    3650 6150
@@
 AR Path="/4E1ACC57/4E1713DF" Ref="C810"  Part="1"
 AR Path="/4E146472/4E1713DF" Ref="C910"  Part="1"
-F 0 "C710" H 3450 6250 25  0000 L CNN
+F 0 "C910" H 3450 6250 25  0000 L CNN
 F 1 "100nF" H 3450 6050 25  0000 L CNN
 	1    3400 6150
@@
 AR Path="/4E1ACC57/4E1713DE" Ref="C808"  Part="1"
 AR Path="/4E146472/4E1713DE" Ref="C908"  Part="1"
-F 0 "C708" H 3200 6250 25  0000 L CNN
+F 0 "C908" H 3200 6250 25  0000 L CNN
 F 1 "100nF" H 3200 6050 25  0000 L CNN
 	1    3150 6150
@@
 AR Path="/4E1ACC57/4E1713DD" Ref="C807"  Part="1"
 AR Path="/4E146472/4E1713DD" Ref="C907"  Part="1"
-F 0 "C707" H 2950 6250 25  0000 L CNN
+F 0 "C907" H 2950 6250 25  0000 L CNN
 F 1 "100nF" H 2950 6050 25  0000 L CNN
 	1    2900 6150
@@
 AR Path="/4E1ACC57/4E1713DB" Ref="C806"  Part="1"
 AR Path="/4E146472/4E1713DB" Ref="C906"  Part="1"
-F 0 "C706" H 2700 6250 25  0000 L CNN
+F 0 "C906" H 2700 6250 25  0000 L CNN
 F 1 "100nF" H 2700 6050 25  0000 L CNN
 	1    2650 6150
@@
 AR Path="/4E1ACC57/4E1713D9" Ref="C805"  Part="1"
 AR Path="/4E146472/4E1713D9" Ref="C905"  Part="1"
-F 0 "C705" H 2000 6250 25  0000 L CNN
+F 0 "C905" H 2000 6250 25  0000 L CNN
 F 1 "10uF" H 2000 6050 25  0000 L CNN
 	1    1950 6150
@@
 AR Path="/4E1ACC57/4E1713D8" Ref="C804"  Part="1"
 AR Path="/4E146472/4E1713D8" Ref="C904"  Part="1"
-F 0 "C704" H 1750 6250 25  0000 L CNN
+F 0 "C904" H 1750 6250 25  0000 L CNN
 F 1 "100nF" H 1750 6050 25  0000 L CNN
 	1    1700 6150
@@
 AR Path="/4E1ACC57/4E1713D6" Ref="C803"  Part="1"
 AR Path="/4E146472/4E1713D6" Ref="C903"  Part="1"
-F 0 "C703" H 1500 6250 25  0000 L CNN
+F 0 "C903" H 1500 6250 25  0000 L CNN
 F 1 "100nF" H 1500 6050 25  0000 L CNN
 	1    1450 6150
@@
 AR Path="/4E1ACC57/4E1713D4" Ref="C802"  Part="1"
 AR Path="/4E146472/4E1713D4" Ref="C902"  Part="1"
-F 0 "C702" H 1250 6250 25  0000 L CNN
+F 0 "C902" H 1250 6250 25  0000 L CNN
 F 1 "100nF" H 1250 6050 25  0000 L CNN
 	1    1200 6150
@@
 AR Path="/4E1ACC57/4E1713B5" Ref="C801"  Part="1"
 AR Path="/4E146472/4E1713B5" Ref="C901"  Part="1"
-F 0 "C701" H 1000 6250 25  0000 L CNN
+F 0 "C901" H 1000 6250 25  0000 L CNN
 F 1 "100nF" H 1000 6050 25  0000 L CNN
 	1    950  6150
@@
 AR Path="/4E1ACC57/4E15B90D" Ref="R801"  Part="1"
 AR Path="/4E146472/4E15B90D" Ref="R901"  Part="1"
-F 0 "R701" V 3480 4000 50  0000 C CNN
+F 0 "R901" V 3480 4000 50  0000 C CNN
 F 1 "2R2" V 3400 4000 50  0000 C CNN
 	1    3400 4000
@@
 AR Path="/4E1ACC57/4E15B90C" Ref="C809"  Part="1"
 AR Path="/4E146472/4E15B90C" Ref="C909"  Part="1"
-F 0 "C709" H 3450 4650 50  0000 L CNN
+F 0 "C909" H 3450 4650 50  0000 L CNN
 F 1 "1uF" H 3450 4450 50  0000 L CNN
+F 2 "X-0402" H 3400 4550 60  0001 C CNN
 	1    3400 4550
 	1    0    0    -1
@@
 AR Path="/4E1ACC57/4E15B90B" Ref="#PWR032"  Part="1"
 AR Path="/4E146472/4E15B90B" Ref="#PWR036"  Part="1"
-F 0 "#PWR028" H 3400 5050 30  0001 C CNN
+F 0 "#PWR036" H 3400 5050 30  0001 C CNN
 F 1 "GND" H 3400 4980 30  0001 C CNN
 	1    3400 5050
@@
 AR Path="/4E1ACC57/4E15B90A" Ref="#PWR033"  Part="1"
 AR Path="/4E146472/4E15B90A" Ref="#PWR037"  Part="1"
-F 0 "#PWR029" H 3000 5050 30  0001 C CNN
+F 0 "#PWR037" H 3000 5050 30  0001 C CNN
 F 1 "GND" H 3000 4980 30  0001 C CNN
 	1    3000 5050

Commit message: Added appropriate sepearte power modules. Moved buffering to hiearchial sheet Buffering per 2 L2s due to harsh pull down on pads moved pins from global labels to heirachial
Connections:
- net +3V3 renamed +3V3_L2

Commit message: squash and back to work!
Connections:
- no-connect marks 2 -> 52
Other:
- note removed: "TODO: FIND OUT WHAT BOOT MODES WE WANT!"
Changed lines of the file:
@@
-EESchema Schematic File Version 2  date 27/07/2011 16:09:28
+EESchema Schematic File Version 2  date 27/07/2011 16:56:06
 LIBS:power
 LIBS:device
@@
 $Descr A4 11700 8267
 encoding utf-8
-Sheet 11 13
+Sheet 2 13
 Title ""
 Date "27 jul 2011"
@@
 Comment4 ""
 $EndDescr
-Text HLabel 2100 2300 0    39   Input ~ 0
-TCK_BUF
-Text HLabel 2100 2200 0    39   Input ~ 0
-TMS_BUF
+NoConn ~ 2300 1450
+NoConn ~ 2300 1350
+NoConn ~ 2300 1250
+NoConn ~ 2300 1150
+NoConn ~ 2300 1050
+NoConn ~ 7450 850
+NoConn ~ 7450 1950
+NoConn ~ 7450 2050
+NoConn ~ 7450 3150
+NoConn ~ 7450 3250
+NoConn ~ 7450 3350
+NoConn ~ 7450 3450
+NoConn ~ 7450 3550
+NoConn ~ 7450 3650
+NoConn ~ 7450 3750
+NoConn ~ 7450 3850
+NoConn ~ 7450 3950
+NoConn ~ 7450 4050
+NoConn ~ 7450 4150
+NoConn ~ 7450 4250
+NoConn ~ 7450 4350
+NoConn ~ 7450 4450
+NoConn ~ 7450 4550
+NoConn ~ 7450 4650
+NoConn ~ 7450 4750
+NoConn ~ 7450 4850
+NoConn ~ 7450 4950
+NoConn ~ 7450 5050
+NoConn ~ 7450 5150
+NoConn ~ 5150 5000
+NoConn ~ 5150 4900
+NoConn ~ 5150 4800
+NoConn ~ 5150 4700
+NoConn ~ 5150 4600
+NoConn ~ 5150 4500
+NoConn ~ 5150 4400
+NoConn ~ 5150 4300
+NoConn ~ 5150 4200
+NoConn ~ 5150 4100
+NoConn ~ 5150 4000
+NoConn ~ 5150 3900
+NoConn ~ 5150 3800
+NoConn ~ 5150 3700
+NoConn ~ 5150 3600
+NoConn ~ 5150 3600
+NoConn ~ 5150 3500
+NoConn ~ 5150 3400
+NoConn ~ 5150 2300
+NoConn ~ 5150 2200
+NoConn ~ 5150 1100
 Wire Notes Line
 	750  5500 750  6600
@@
 Wire Notes Line
 	4000 6600 4000 5500
+Text HLabel 2100 2300 0    39   Input ~ 0
+TCK_BUF
+Text HLabel 2100 2200 0    39   Input ~ 0
+TMS_BUF
 $Comp
 L XS1_L2 U201
@@
 AR Path="/4E1ACC57/4E282660" Ref="U801"  Part="1"
 AR Path="/4E146472/4E282660" Ref="U901"  Part="1"
-F 0 "U901" H 3200 3800 50  0000 C CNN
+F 0 "U201" H 3200 3800 50  0000 C CNN
 F 1 "XS1_L2" H 3200 3900 50  0000 C CNN
 F 2 "124" H 3200 3700 60  0000 C CNN
@@
 Decoupling Caps
 $Comp
-L GND #PWR302
+L GND #PWR04
 U 1 1 4E17143C
 P 2650 6450
-AR Path="/4E1B01C1/4E17143C" Ref="#PWR302"  Part="1"
-AR Path="/4E1B01C0/4E17143C" Ref="#PWR402"  Part="1"
-AR Path="/4E1B01BF/4E17143C" Ref="#PWR502"  Part="1"
-AR Path="/4E1B01BE/4E17143C" Ref="#PWR602"  Part="1"
-AR Path="/4E1ACC75/4E17143C" Ref="#PWR702"  Part="1"
-AR Path="/4E1ACC74/4E17143C" Ref="#PWR802"  Part="1"
-AR Path="/4E1ACC57/4E17143C" Ref="#PWR902"  Part="1"
-AR Path="/4E146472/4E17143C" Ref="#PWR1002"  Part="1"
-F 0 "#PWR1002" H 2650 6450 30  0001 C CNN
+AR Path="/4E1B01C1/4E17143C" Ref="#PWR04"  Part="1"
+AR Path="/4E1B01C0/4E17143C" Ref="#PWR034"  Part="1"
+AR Path="/4E1B01BF/4E17143C" Ref="#PWR038"  Part="1"
+AR Path="/4E1B01BE/4E17143C" Ref="#PWR042"  Part="1"
+AR Path="/4E1ACC75/4E17143C" Ref="#PWR046"  Part="1"
+AR Path="/4E1ACC74/4E17143C" Ref="#PWR050"  Part="1"
+AR Path="/4E1ACC57/4E17143C" Ref="#PWR054"  Part="1"
+AR Path="/4E146472/4E17143C" Ref="#PWR058"  Part="1"
+F 0 "#PWR04" H 2650 6450 30  0001 C CNN
 F 1 "GND" H 2650 6380 30  0001 C CNN
 	1    2650 6450
@@
 +3V3_L2
 $Comp
-L GND #PWR301
+L GND #PWR05
 U 1 1 4E171407
 P 950 6450
-AR Path="/4E1B01C1/4E171407" Ref="#PWR301"  Part="1"
-AR Path="/4E1B01C0/4E171407" Ref="#PWR401"  Part="1"
-AR Path="/4E1B01BF/4E171407" Ref="#PWR501"  Part="1"
-AR Path="/4E1B01BE/4E171407" Ref="#PWR601"  Part="1"
-AR Path="/4E1ACC75/4E171407" Ref="#PWR701"  Part="1"
-AR Path="/4E1ACC74/4E171407" Ref="#PWR801"  Part="1"
-AR Path="/4E1ACC57/4E171407" Ref="#PWR901"  Part="1"
-AR Path="/4E146472/4E171407" Ref="#PWR1001"  Part="1"
-F 0 "#PWR1001" H 950 6450 30  0001 C CNN
+AR Path="/4E1B01C1/4E171407" Ref="#PWR05"  Part="1"
+AR Path="/4E1B01C0/4E171407" Ref="#PWR035"  Part="1"
+AR Path="/4E1B01BF/4E171407" Ref="#PWR039"  Part="1"
+AR Path="/4E1B01BE/4E171407" Ref="#PWR043"  Part="1"
+AR Path="/4E1ACC75/4E171407" Ref="#PWR047"  Part="1"
+AR Path="/4E1ACC74/4E171407" Ref="#PWR051"  Part="1"
+AR Path="/4E1ACC57/4E171407" Ref="#PWR055"  Part="1"
+AR Path="/4E146472/4E171407" Ref="#PWR059"  Part="1"
+F 0 "#PWR05" H 950 6450 30  0001 C CNN
 F 1 "GND" H 950 6380 30  0001 C CNN
 	1    950  6450
@@
 AR Path="/4E1ACC57/4E1713E0" Ref="C811"  Part="1"
 AR Path="/4E146472/4E1713E0" Ref="C911"  Part="1"
-F 0 "C911" H 3700 6250 25  0000 L CNN
+F 0 "C211" H 3700 6250 25  0000 L CNN
 F 1 "10uF" H 3700 6050 25  0000 L CNN
 	1    3650 6150
@@
 AR Path="/4E1ACC57/4E1713DF" Ref="C810"  Part="1"
 AR Path="/4E146472/4E1713DF" Ref="C910"  Part="1"
-F 0 "C910" H 3450 6250 25  0000 L CNN
+F 0 "C210" H 3450 6250 25  0000 L CNN
 F 1 "100nF" H 3450 6050 25  0000 L CNN
 	1    3400 6150
@@
 AR Path="/4E1ACC57/4E1713DE" Ref="C808"  Part="1"
 AR Path="/4E146472/4E1713DE" Ref="C908"  Part="1"
-F 0 "C908" H 3200 6250 25  0000 L CNN
+F 0 "C208" H 3200 6250 25  0000 L CNN
 F 1 "100nF" H 3200 6050 25  0000 L CNN
 	1    3150 6150
@@
 AR Path="/4E1ACC57/4E1713DD" Ref="C807"  Part="1"
 AR Path="/4E146472/4E1713DD" Ref="C907"  Part="1"
-F 0 "C907" H 2950 6250 25  0000 L CNN
+F 0 "C207" H 2950 6250 25  0000 L CNN
 F 1 "100nF" H 2950 6050 25  0000 L CNN
 	1    2900 6150
@@
 AR Path="/4E1ACC57/4E1713DB" Ref="C806"  Part="1"
 AR Path="/4E146472/4E1713DB" Ref="C906"  Part="1"
-F 0 "C906" H 2700 6250 25  0000 L CNN
+F 0 "C206" H 2700 6250 25  0000 L CNN
 F 1 "100nF" H 2700 6050 25  0000 L CNN
 	1    2650 6150
@@
 AR Path="/4E1ACC57/4E1713D9" Ref="C805"  Part="1"
 AR Path="/4E146472/4E1713D9" Ref="C905"  Part="1"
-F 0 "C905" H 2000 6250 25  0000 L CNN
+F 0 "C205" H 2000 6250 25  0000 L CNN
 F 1 "10uF" H 2000 6050 25  0000 L CNN
 	1    1950 6150
@@
 AR Path="/4E1ACC57/4E1713D8" Ref="C804"  Part="1"
 AR Path="/4E146472/4E1713D8" Ref="C904"  Part="1"
-F 0 "C904" H 1750 6250 25  0000 L CNN
+F 0 "C204" H 1750 6250 25  0000 L CNN
 F 1 "100nF" H 1750 6050 25  0000 L CNN
 	1    1700 6150
@@
 AR Path="/4E1ACC57/4E1713D6" Ref="C803"  Part="1"
 AR Path="/4E146472/4E1713D6" Ref="C903"  Part="1"
-F 0 "C903" H 1500 6250 25  0000 L CNN
+F 0 "C203" H 1500 6250 25  0000 L CNN
 F 1 "100nF" H 1500 6050 25  0000 L CNN
 	1    1450 6150
@@
 AR Path="/4E1ACC57/4E1713D4" Ref="C802"  Part="1"
 AR Path="/4E146472/4E1713D4" Ref="C902"  Part="1"
-F 0 "C902" H 1250 6250 25  0000 L CNN
+F 0 "C202" H 1250 6250 25  0000 L CNN
 F 1 "100nF" H 1250 6050 25  0000 L CNN
 	1    1200 6150
@@
 AR Path="/4E1ACC57/4E1713B5" Ref="C801"  Part="1"
 AR Path="/4E146472/4E1713B5" Ref="C901"  Part="1"
-F 0 "C901" H 1000 6250 25  0000 L CNN
+F 0 "C201" H 1000 6250 25  0000 L CNN
 F 1 "100nF" H 1000 6050 25  0000 L CNN
 	1    950  6150
@@
 Text GLabel 3000 4150 2    39   Input ~ 0
 CLK_20M
-Text Notes 700  1350 0    39   ~ 0
-TODO: FIND OUT WHAT BOOT MODES WE WANT!
 Text GLabel 2100 1850 0    39   Input ~ 0
 CLK_20M
@@
 AR Path="/4E1ACC57/4E15B90D" Ref="R801"  Part="1"
 AR Path="/4E146472/4E15B90D" Ref="R901"  Part="1"
-F 0 "R901" V 3480 4000 50  0000 C CNN
+F 0 "R201" V 3480 4000 50  0000 C CNN
 F 1 "2R2" V 3400 4000 50  0000 C CNN
 	1    3400 4000
@@
 AR Path="/4E1ACC57/4E15B90C" Ref="C809"  Part="1"
 AR Path="/4E146472/4E15B90C" Ref="C909"  Part="1"
-F 0 "C909" H 3450 4650 50  0000 L CNN
+F 0 "C209" H 3450 4650 50  0000 L CNN
 F 1 "1uF" H 3450 4450 50  0000 L CNN
 F 2 "X-0402" H 3400 4550 60  0001 C CNN
@@
 $EndComp
 $Comp
-L GND #PWR304
+L GND #PWR06
 U 1 1 4E15B90B
 P 3400 5050
-AR Path="/4E1B01C1/4E15B90B" Ref="#PWR304"  Part="1"
-AR Path="/4E1B01C0/4E15B90B" Ref="#PWR404"  Part="1"
-AR Path="/4E1B01BF/4E15B90B" Ref="#PWR504"  Part="1"
-AR Path="/4E1B01BE/4E15B90B" Ref="#PWR604"  Part="1"
-AR Path="/4E1ACC75/4E15B90B" Ref="#PWR704"  Part="1"
-AR Path="/4E1ACC74/4E15B90B" Ref="#PWR804"  Part="1"
-AR Path="/4E1ACC57/4E15B90B" Ref="#PWR904"  Part="1"
-AR Path="/4E146472/4E15B90B" Ref="#PWR1004"  Part="1"
-F 0 "#PWR1004" H 3400 5050 30  0001 C CNN
+AR Path="/4E1B01C1/4E15B90B" Ref="#PWR06"  Part="1"
+AR Path="/4E1B01C0/4E15B90B" Ref="#PWR036"  Part="1"
+AR Path="/4E1B01BF/4E15B90B" Ref="#PWR040"  Part="1"
+AR Path="/4E1B01BE/4E15B90B" Ref="#PWR044"  Part="1"
+AR Path="/4E1ACC75/4E15B90B" Ref="#PWR048"  Part="1"
+AR Path="/4E1ACC74/4E15B90B" Ref="#PWR052"  Part="1"
+AR Path="/4E1ACC57/4E15B90B" Ref="#PWR056"  Part="1"
+AR Path="/4E146472/4E15B90B" Ref="#PWR060"  Part="1"
+F 0 "#PWR06" H 3400 5050 30  0001 C CNN
 F 1 "GND" H 3400 4980 30  0001 C CNN
 	1    3400 5050
@@
 $EndComp
 $Comp
-L GND #PWR303
+L GND #PWR07
 U 1 1 4E15B90A
 P 3000 5050
-AR Path="/4E1B01C1/4E15B90A" Ref="#PWR303"  Part="1"
-AR Path="/4E1B01C0/4E15B90A" Ref="#PWR403"  Part="1"
-AR Path="/4E1B01BF/4E15B90A" Ref="#PWR503"  Part="1"
-AR Path="/4E1B01BE/4E15B90A" Ref="#PWR603"  Part="1"
-AR Path="/4E1ACC75/4E15B90A" Ref="#PWR703"  Part="1"
-AR Path="/4E1ACC74/4E15B90A" Ref="#PWR803"  Part="1"
-AR Path="/4E1ACC57/4E15B90A" Ref="#PWR903"  Part="1"
-AR Path="/4E146472/4E15B90A" Ref="#PWR1003"  Part="1"
-F 0 "#PWR1003" H 3000 5050 30  0001 C CNN
+AR Path="/4E1B01C1/4E15B90A" Ref="#PWR07"  Part="1"
+AR Path="/4E1B01C0/4E15B90A" Ref="#PWR037"  Part="1"
+AR Path="/4E1B01BF/4E15B90A" Ref="#PWR041"  Part="1"
+AR Path="/4E1B01BE/4E15B90A" Ref="#PWR045"  Part="1"
+AR Path="/4E1ACC75/4E15B90A" Ref="#PWR049"  Part="1"
+AR Path="/4E1ACC74/4E15B90A" Ref="#PWR053"  Part="1"
+AR Path="/4E1ACC57/4E15B90A" Ref="#PWR057"  Part="1"
+AR Path="/4E146472/4E15B90A" Ref="#PWR061"  Part="1"
+F 0 "#PWR07" H 3000 5050 30  0001 C CNN
 F 1 "GND" H 3000 4980 30  0001 C CNN
 	1    3000 5050

Commit message: more buffers and added connectors for end
Connections:
- net GND: now also U201.A35 (MODE4)
- net +3V3: now reaches U201.B33 (MODE0)
- net +3V3: now also U201.B34 (MODE1)
- net MSEL: now reaches U201.B35 (MODE2)
- net MSEL: now also U201.B36 (MODE3)
- no-connect marks 52 -> 47

Commit message: Isolated L1 stuff (inc. JTAG) in single sheet. Added buffered for the L2's JTAG control signals.
Changed lines of the file:
@@
-EESchema Schematic File Version 2  date 28/07/2011 13:33:42
+EESchema Schematic File Version 2  date 28/07/2011 16:32:29
 LIBS:power
 LIBS:device
@@
 $Descr A4 11700 8267
 encoding utf-8
-Sheet 12 13
+Sheet 9 12
 Title ""
 Date "28 jul 2011"
@@
 U 1 1 4E314D6E
 P 2150 1500
+AR Path="/4E146472/4E314D6E" Ref="#PWR?"  Part="1"
+AR Path="/4E1B01BF/4E314D6E" Ref="#PWR?"  Part="1"
+AR Path="/4E1ACC75/4E314D6E" Ref="#PWR?"  Part="1"
 F 0 "#PWR?" H 2150 1500 30  0001 C CNN
 F 1 "GND" H 2150 1430 30  0001 C CNN
@@
 AR Path="/4E1ACC57/4E282660" Ref="U801"  Part="1"
 AR Path="/4E146472/4E282660" Ref="U901"  Part="1"
-F 0 "U901" H 3200 3800 50  0000 C CNN
+F 0 "U601" H 3200 3800 50  0000 C CNN
 F 1 "XS1_L2" H 3200 3900 50  0000 C CNN
 F 2 "124" H 3200 3700 60  0000 C CNN
@@
 AR Path="/4E1ACC57/4E17143C" Ref="#PWR054"  Part="1"
 AR Path="/4E146472/4E17143C" Ref="#PWR058"  Part="1"
-F 0 "#PWR058" H 2650 6450 30  0001 C CNN
+F 0 "#PWR046" H 2650 6450 30  0001 C CNN
 F 1 "GND" H 2650 6380 30  0001 C CNN
 	1    2650 6450
@@
 AR Path="/4E1ACC57/4E171407" Ref="#PWR055"  Part="1"
 AR Path="/4E146472/4E171407" Ref="#PWR059"  Part="1"
-F 0 "#PWR059" H 950 6450 30  0001 C CNN
+F 0 "#PWR047" H 950 6450 30  0001 C CNN
 F 1 "GND" H 950 6380 30  0001 C CNN
 	1    950  6450
@@
 AR Path="/4E1ACC57/4E1713E0" Ref="C811"  Part="1"
 AR Path="/4E146472/4E1713E0" Ref="C911"  Part="1"
-F 0 "C911" H 3700 6250 25  0000 L CNN
+F 0 "C611" H 3700 6250 25  0000 L CNN
 F 1 "10uF" H 3700 6050 25  0000 L CNN
 	1    3650 6150
@@
 AR Path="/4E1ACC57/4E1713DF" Ref="C810"  Part="1"
 AR Path="/4E146472/4E1713DF" Ref="C910"  Part="1"
-F 0 "C910" H 3450 6250 25  0000 L CNN
+F 0 "C610" H 3450 6250 25  0000 L CNN
 F 1 "100nF" H 3450 6050 25  0000 L CNN
 	1    3400 6150
@@
 AR Path="/4E1ACC57/4E1713DE" Ref="C808"  Part="1"
 AR Path="/4E146472/4E1713DE" Ref="C908"  Part="1"
-F 0 "C908" H 3200 6250 25  0000 L CNN
+F 0 "C608" H 3200 6250 25  0000 L CNN
 F 1 "100nF" H 3200 6050 25  0000 L CNN
 	1    3150 6150
@@
 AR Path="/4E1ACC57/4E1713DD" Ref="C807"  Part="1"
 AR Path="/4E146472/4E1713DD" Ref="C907"  Part="1"
-F 0 "C907" H 2950 6250 25  0000 L CNN
+F 0 "C607" H 2950 6250 25  0000 L CNN
 F 1 "100nF" H 2950 6050 25  0000 L CNN
 	1    2900 6150
@@
 AR Path="/4E1ACC57/4E1713DB" Ref="C806"  Part="1"
 AR Path="/4E146472/4E1713DB" Ref="C906"  Part="1"
-F 0 "C906" H 2700 6250 25  0000 L CNN
+F 0 "C606" H 2700 6250 25  0000 L CNN
 F 1 "100nF" H 2700 6050 25  0000 L CNN
 	1    2650 6150
@@
 AR Path="/4E1ACC57/4E1713D9" Ref="C805"  Part="1"
 AR Path="/4E146472/4E1713D9" Ref="C905"  Part="1"
-F 0 "C905" H 2000 6250 25  0000 L CNN
+F 0 "C605" H 2000 6250 25  0000 L CNN
 F 1 "10uF" H 2000 6050 25  0000 L CNN
 	1    1950 6150
@@
 AR Path="/4E1ACC57/4E1713D8" Ref="C804"  Part="1"
 AR Path="/4E146472/4E1713D8" Ref="C904"  Part="1"
-F 0 "C904" H 1750 6250 25  0000 L CNN
+F 0 "C604" H 1750 6250 25  0000 L CNN
 F 1 "100nF" H 1750 6050 25  0000 L CNN
 	1    1700 6150
@@
 AR Path="/4E1ACC57/4E1713D6" Ref="C803"  Part="1"
 AR Path="/4E146472/4E1713D6" Ref="C903"  Part="1"
-F 0 "C903" H 1500 6250 25  0000 L CNN
+F 0 "C603" H 1500 6250 25  0000 L CNN
 F 1 "100nF" H 1500 6050 25  0000 L CNN
 	1    1450 6150
@@
 AR Path="/4E1ACC57/4E1713D4" Ref="C802"  Part="1"
 AR Path="/4E146472/4E1713D4" Ref="C902"  Part="1"
-F 0 "C902" H 1250 6250 25  0000 L CNN
+F 0 "C602" H 1250 6250 25  0000 L CNN
 F 1 "100nF" H 1250 6050 25  0000 L CNN
 	1    1200 6150
@@
 AR Path="/4E1ACC57/4E1713B5" Ref="C801"  Part="1"
 AR Path="/4E146472/4E1713B5" Ref="C901"  Part="1"
-F 0 "C901" H 1000 6250 25  0000 L CNN
+F 0 "C601" H 1000 6250 25  0000 L CNN
 F 1 "100nF" H 1000 6050 25  0000 L CNN
 	1    950  6150
@@
 AR Path="/4E1ACC57/4E15B90D" Ref="R801"  Part="1"
 AR Path="/4E146472/4E15B90D" Ref="R901"  Part="1"
-F 0 "R901" V 3480 4000 50  0000 C CNN
+F 0 "R601" V 3480 4000 50  0000 C CNN
 F 1 "2R2" V 3400 4000 50  0000 C CNN
 	1    3400 4000
@@
 AR Path="/4E1ACC57/4E15B90C" Ref="C809"  Part="1"
 AR Path="/4E146472/4E15B90C" Ref="C909"  Part="1"
-F 0 "C909" H 3450 4650 50  0000 L CNN
+F 0 "C609" H 3450 4650 50  0000 L CNN
 F 1 "1uF" H 3450 4450 50  0000 L CNN
 F 2 "X-0402" H 3400 4550 60  0001 C CNN
@@
 AR Path="/4E1ACC57/4E15B90B" Ref="#PWR056"  Part="1"
 AR Path="/4E146472/4E15B90B" Ref="#PWR060"  Part="1"
-F 0 "#PWR060" H 3400 5050 30  0001 C CNN
+F 0 "#PWR048" H 3400 5050 30  0001 C CNN
 F 1 "GND" H 3400 4980 30  0001 C CNN
 	1    3400 5050
@@
 AR Path="/4E1ACC57/4E15B90A" Ref="#PWR057"  Part="1"
 AR Path="/4E146472/4E15B90A" Ref="#PWR061"  Part="1"
-F 0 "#PWR061" H 3000 5050 30  0001 C CNN
+F 0 "#PWR049" H 3000 5050 30  0001 C CNN
 F 1 "GND" H 3000 4980 30  0001 C CNN
 	1    3000 5050
