File: l2_dev_board/Design/L2.sch (KiCad schematic (older format))
At the start: 13 parts, among them U201 XS1_L2

Commit message: removing old buffering and wanted to check point
Changed lines of the file:
@@
-EESchema Schematic File Version 2  date 28/07/2011 16:32:29
+EESchema Schematic File Version 2  date 28/07/2011 17:12:08
 LIBS:power
 LIBS:device
@@
 $Descr A4 11700 8267
 encoding utf-8
-Sheet 9 12
+Sheet 11 12
 Title ""
 Date "28 jul 2011"
@@
 Text HLabel 2100 1750 0    39   Input ~ 0
 RST_N_BUF
-Text HLabel 2000 1250 0    60   Input ~ 0
+Text HLabel 2000 1250 0    39   Input ~ 0
 MSEL
 $Comp
-L GND #PWR?
+L GND #PWR083
 U 1 1 4E314D6E
 P 2150 1500
-AR Path="/4E146472/4E314D6E" Ref="#PWR?"  Part="1"
-AR Path="/4E1B01BF/4E314D6E" Ref="#PWR?"  Part="1"
-AR Path="/4E1ACC75/4E314D6E" Ref="#PWR?"  Part="1"
-F 0 "#PWR?" H 2150 1500 30  0001 C CNN
+AR Path="/4E146472/4E314D6E" Ref="#PWR083"  Part="1"
+AR Path="/4E1B01BF/4E314D6E" Ref="#PWR058"  Part="1"
+AR Path="/4E1ACC75/4E314D6E" Ref="#PWR068"  Part="1"
+AR Path="/4E1ACC57/4E314D6E" Ref="#PWR078"  Part="1"
+AR Path="/4E1B01C1/4E314D6E" Ref="#PWR031"  Part="1"
+AR Path="/4E1B01C0/4E314D6E" Ref="#PWR053"  Part="1"
+AR Path="/4E1B01BE/4E314D6E" Ref="#PWR063"  Part="1"
+AR Path="/4E1ACC74/4E314D6E" Ref="#PWR073"  Part="1"
+F 0 "#PWR083" H 2150 1500 30  0001 C CNN
 F 1 "GND" H 2150 1430 30  0001 C CNN
 	1    2150 1500
@@
 AR Path="/4E1ACC57/4E282660" Ref="U801"  Part="1"
 AR Path="/4E146472/4E282660" Ref="U901"  Part="1"
-F 0 "U601" H 3200 3800 50  0000 C CNN
+F 0 "U901" H 3200 3800 50  0000 C CNN
 F 1 "XS1_L2" H 3200 3900 50  0000 C CNN
 F 2 "124" H 3200 3700 60  0000 C CNN
@@
 Decoupling Caps
 $Comp
-L GND #PWR04
+L GND #PWR032
 U 1 1 4E17143C
 P 2650 6450
-AR Path="/4E1B01C1/4E17143C" Ref="#PWR04"  Part="1"
-AR Path="/4E1B01C0/4E17143C" Ref="#PWR034"  Part="1"
-AR Path="/4E1B01BF/4E17143C" Ref="#PWR038"  Part="1"
-AR Path="/4E1B01BE/4E17143C" Ref="#PWR042"  Part="1"
-AR Path="/4E1ACC75/4E17143C" Ref="#PWR046"  Part="1"
-AR Path="/4E1ACC74/4E17143C" Ref="#PWR050"  Part="1"
-AR Path="/4E1ACC57/4E17143C" Ref="#PWR054"  Part="1"
-AR Path="/4E146472/4E17143C" Ref="#PWR058"  Part="1"
-F 0 "#PWR046" H 2650 6450 30  0001 C CNN
+AR Path="/4E1B01C1/4E17143C" Ref="#PWR032"  Part="1"
+AR Path="/4E1B01C0/4E17143C" Ref="#PWR054"  Part="1"
+AR Path="/4E1B01BF/4E17143C" Ref="#PWR059"  Part="1"
+AR Path="/4E1B01BE/4E17143C" Ref="#PWR064"  Part="1"
+AR Path="/4E1ACC75/4E17143C" Ref="#PWR069"  Part="1"
+AR Path="/4E1ACC74/4E17143C" Ref="#PWR074"  Part="1"
+AR Path="/4E1ACC57/4E17143C" Ref="#PWR079"  Part="1"
+AR Path="/4E146472/4E17143C" Ref="#PWR084"  Part="1"
+F 0 "#PWR084" H 2650 6450 30  0001 C CNN
 F 1 "GND" H 2650 6380 30  0001 C CNN
 	1    2650 6450
@@
 +3V3_L2
 $Comp
-L GND #PWR05
+L GND #PWR033
 U 1 1 4E171407
 P 950 6450
-AR Path="/4E1B01C1/4E171407" Ref="#PWR05"  Part="1"
-AR Path="/4E1B01C0/4E171407" Ref="#PWR035"  Part="1"
-AR Path="/4E1B01BF/4E171407" Ref="#PWR039"  Part="1"
-AR Path="/4E1B01BE/4E171407" Ref="#PWR043"  Part="1"
-AR Path="/4E1ACC75/4E171407" Ref="#PWR047"  Part="1"
-AR Path="/4E1ACC74/4E171407" Ref="#PWR051"  Part="1"
-AR Path="/4E1ACC57/4E171407" Ref="#PWR055"  Part="1"
-AR Path="/4E146472/4E171407" Ref="#PWR059"  Part="1"
-F 0 "#PWR047" H 950 6450 30  0001 C CNN
+AR Path="/4E1B01C1/4E171407" Ref="#PWR033"  Part="1"
+AR Path="/4E1B01C0/4E171407" Ref="#PWR055"  Part="1"
+AR Path="/4E1B01BF/4E171407" Ref="#PWR060"  Part="1"
+AR Path="/4E1B01BE/4E171407" Ref="#PWR065"  Part="1"
+AR Path="/4E1ACC75/4E171407" Ref="#PWR070"  Part="1"
+AR Path="/4E1ACC74/4E171407" Ref="#PWR075"  Part="1"
+AR Path="/4E1ACC57/4E171407" Ref="#PWR080"  Part="1"
+AR Path="/4E146472/4E171407" Ref="#PWR085"  Part="1"
+F 0 "#PWR085" H 950 6450 30  0001 C CNN
 F 1 "GND" H 950 6380 30  0001 C CNN
 	1    950  6450
@@
 AR Path="/4E1ACC57/4E1713E0" Ref="C811"  Part="1"
 AR Path="/4E146472/4E1713E0" Ref="C911"  Part="1"
-F 0 "C611" H 3700 6250 25  0000 L CNN
+F 0 "C911" H 3700 6250 25  0000 L CNN
 F 1 "10uF" H 3700 6050 25  0000 L CNN
 	1    3650 6150
@@
 AR Path="/4E1ACC57/4E1713DF" Ref="C810"  Part="1"
 AR Path="/4E146472/4E1713DF" Ref="C910"  Part="1"
-F 0 "C610" H 3450 6250 25  0000 L CNN
+F 0 "C910" H 3450 6250 25  0000 L CNN
 F 1 "100nF" H 3450 6050 25  0000 L CNN
 	1    3400 6150
@@
 AR Path="/4E1ACC57/4E1713DE" Ref="C808"  Part="1"
 AR Path="/4E146472/4E1713DE" Ref="C908"  Part="1"
-F 0 "C608" H 3200 6250 25  0000 L CNN
+F 0 "C908" H 3200 6250 25  0000 L CNN
 F 1 "100nF" H 3200 6050 25  0000 L CNN
 	1    3150 6150
@@
 AR Path="/4E1ACC57/4E1713DD" Ref="C807"  Part="1"
 AR Path="/4E146472/4E1713DD" Ref="C907"  Part="1"
-F 0 "C607" H 2950 6250 25  0000 L CNN
+F 0 "C907" H 2950 6250 25  0000 L CNN
 F 1 "100nF" H 2950 6050 25  0000 L CNN
 	1    2900 6150
@@
 AR Path="/4E1ACC57/4E1713DB" Ref="C806"  Part="1"
 AR Path="/4E146472/4E1713DB" Ref="C906"  Part="1"
-F 0 "C606" H 2700 6250 25  0000 L CNN
+F 0 "C906" H 2700 6250 25  0000 L CNN
 F 1 "100nF" H 2700 6050 25  0000 L CNN
 	1    2650 6150
@@
 AR Path="/4E1ACC57/4E1713D9" Ref="C805"  Part="1"
 AR Path="/4E146472/4E1713D9" Ref="C905"  Part="1"
-F 0 "C605" H 2000 6250 25  0000 L CNN
+F 0 "C905" H 2000 6250 25  0000 L CNN
 F 1 "10uF" H 2000 6050 25  0000 L CNN
 	1    1950 6150
@@
 AR Path="/4E1ACC57/4E1713D8" Ref="C804"  Part="1"
 AR Path="/4E146472/4E1713D8" Ref="C904"  Part="1"
-F 0 "C604" H 1750 6250 25  0000 L CNN
+F 0 "C904" H 1750 6250 25  0000 L CNN
 F 1 "100nF" H 1750 6050 25  0000 L CNN
 	1    1700 6150
@@
 AR Path="/4E1ACC57/4E1713D6" Ref="C803"  Part="1"
 AR Path="/4E146472/4E1713D6" Ref="C903"  Part="1"
-F 0 "C603" H 1500 6250 25  0000 L CNN
+F 0 "C903" H 1500 6250 25  0000 L CNN
 F 1 "100nF" H 1500 6050 25  0000 L CNN
 	1    1450 6150
@@
 AR Path="/4E1ACC57/4E1713D4" Ref="C802"  Part="1"
 AR Path="/4E146472/4E1713D4" Ref="C902"  Part="1"
-F 0 "C602" H 1250 6250 25  0000 L CNN
+F 0 "C902" H 1250 6250 25  0000 L CNN
 F 1 "100nF" H 1250 6050 25  0000 L CNN
 	1    1200 6150
@@
 AR Path="/4E1ACC57/4E1713B5" Ref="C801"  Part="1"
 AR Path="/4E146472/4E1713B5" Ref="C901"  Part="1"
-F 0 "C601" H 1000 6250 25  0000 L CNN
+F 0 "C901" H 1000 6250 25  0000 L CNN
 F 1 "100nF" H 1000 6050 25  0000 L CNN
 	1    950  6150
@@
 AR Path="/4E1ACC57/4E15B90D" Ref="R801"  Part="1"
 AR Path="/4E146472/4E15B90D" Ref="R901"  Part="1"
-F 0 "R601" V 3480 4000 50  0000 C CNN
+F 0 "R901" V 3480 4000 50  0000 C CNN
 F 1 "2R2" V 3400 4000 50  0000 C CNN
 	1    3400 4000
@@
 AR Path="/4E1ACC57/4E15B90C" Ref="C809"  Part="1"
 AR Path="/4E146472/4E15B90C" Ref="C909"  Part="1"
-F 0 "C609" H 3450 4650 50  0000 L CNN
+F 0 "C909" H 3450 4650 50  0000 L CNN
 F 1 "1uF" H 3450 4450 50  0000 L CNN
 F 2 "X-0402" H 3400 4550 60  0001 C CNN
@@
 $EndComp
 $Comp
-L GND #PWR06
+L GND #PWR034
 U 1 1 4E15B90B
 P 3400 5050
-AR Path="/4E1B01C1/4E15B90B" Ref="#PWR06"  Part="1"
-AR Path="/4E1B01C0/4E15B90B" Ref="#PWR036"  Part="1"
-AR Path="/4E1B01BF/4E15B90B" Ref="#PWR040"  Part="1"
-AR Path="/4E1B01BE/4E15B90B" Ref="#PWR044"  Part="1"
-AR Path="/4E1ACC75/4E15B90B" Ref="#PWR048"  Part="1"
-AR Path="/4E1ACC74/4E15B90B" Ref="#PWR052"  Part="1"
-AR Path="/4E1ACC57/4E15B90B" Ref="#PWR056"  Part="1"
-AR Path="/4E146472/4E15B90B" Ref="#PWR060"  Part="1"
-F 0 "#PWR048" H 3400 5050 30  0001 C CNN
+AR Path="/4E1B01C1/4E15B90B" Ref="#PWR034"  Part="1"
+AR Path="/4E1B01C0/4E15B90B" Ref="#PWR056"  Part="1"
+AR Path="/4E1B01BF/4E15B90B" Ref="#PWR061"  Part="1"
+AR Path="/4E1B01BE/4E15B90B" Ref="#PWR066"  Part="1"
+AR Path="/4E1ACC75/4E15B90B" Ref="#PWR071"  Part="1"
+AR Path="/4E1ACC74/4E15B90B" Ref="#PWR076"  Part="1"
+AR Path="/4E1ACC57/4E15B90B" Ref="#PWR081"  Part="1"
+AR Path="/4E146472/4E15B90B" Ref="#PWR086"  Part="1"
+F 0 "#PWR086" H 3400 5050 30  0001 C CNN
 F 1 "GND" H 3400 4980 30  0001 C CNN
 	1    3400 5050
@@
 $EndComp
 $Comp
-L GND #PWR07
+L GND #PWR035
 U 1 1 4E15B90A
 P 3000 5050
-AR Path="/4E1B01C1/4E15B90A" Ref="#PWR07"  Part="1"
-AR Path="/4E1B01C0/4E15B90A" Ref="#PWR037"  Part="1"
-AR Path="/4E1B01BF/4E15B90A" Ref="#PWR041"  Part="1"
-AR Path="/4E1B01BE/4E15B90A" Ref="#PWR045"  Part="1"
-AR Path="/4E1ACC75/4E15B90A" Ref="#PWR049"  Part="1"
-AR Path="/4E1ACC74/4E15B90A" Ref="#PWR053"  Part="1"
-AR Path="/4E1ACC57/4E15B90A" Ref="#PWR057"  Part="1"
-AR Path="/4E146472/4E15B90A" Ref="#PWR061"  Part="1"
-F 0 "#PWR049" H 3000 5050 30  0001 C CNN
+AR Path="/4E1B01C1/4E15B90A" Ref="#PWR035"  Part="1"
+AR Path="/4E1B01C0/4E15B90A" Ref="#PWR057"  Part="1"
+AR Path="/4E1B01BF/4E15B90A" Ref="#PWR062"  Part="1"
+AR Path="/4E1B01BE/4E15B90A" Ref="#PWR067"  Part="1"
+AR Path="/4E1ACC75/4E15B90A" Ref="#PWR072"  Part="1"
+AR Path="/4E1ACC74/4E15B90A" Ref="#PWR077"  Part="1"
+AR Path="/4E1ACC57/4E15B90A" Ref="#PWR082"  Part="1"
+AR Path="/4E146472/4E15B90A" Ref="#PWR087"  Part="1"
+F 0 "#PWR087" H 3000 5050 30  0001 C CNN
 F 1 "GND" H 3000 4980 30  0001 C CNN
 	1    3000 5050
