File: l2_dev_board/Design/L2.sch (KiCad schematic (older format))
At the start: 13 parts, among them U201 XS1_L2

Commit message: new design with heirachial and new libraries
Parts:
- renumbered C201 to C301, C202 to C302, C203 to C303, C204 to C304, C205 to C305, C206 to C306, C207 to C307, C208 to C308, C209 to C309, C210 to C310, C211 to C311, R201 to R301, U201 to U301
