File: l2_dev_board/Design/L2DevBoard.sch (KiCad schematic (older format))
At the start: 10 parts, among them P101 CONN_10X2, U101 ASE_20MHZ, U102 NC7WZ17, U103 NC7WZ17

Commit message: Started adding tracks
Changed lines of the file:
@@
-EESchema Schematic File Version 2  date 22/07/2011 14:08:59
+EESchema Schematic File Version 2  date 25/07/2011 13:55:09
 LIBS:power
 LIBS:device
@@
 LIBS:contrib
 LIBS:valves
-LIBS:LT3480
-LIBS:ncp1529
-LIBS:ncp303
-LIBS:nc7wz17
 LIBS:apx803
 LIBS:ase_20mhz
+LIBS:brooktre
+LIBS:cmos_ieee
 LIBS:Dmitri_Belimovl
 LIBS:EECV
+LIBS:elec-unifil
 LIBS:ft232r
+LIBS:gennum
+LIBS:graphic
+LIBS:LT3480
+LIBS:microchip1
+LIBS:nc7wz17
+LIBS:ncp303
+LIBS:ncp1529
+LIBS:pspice
 LIBS:SymbolsSimilarEN60617+oldDIN617
+LIBS:transf
+LIBS:ttl_ieee
+LIBS:video
 LIBS:xmos_capacitors
 LIBS:xmos_resistors
@@
 LIBS:xs1
 LIBS:XS1_L2_V2
-LIBS:L2DevBoard-cache
 EELAYER 25  0
 EELAYER END
@@
 Sheet 1 10
 Title ""
-Date "22 jul 2011"
+Date "25 jul 2011"
 Rev ""
 Comp ""
@@
 $EndDescr
 Wire Wire Line
+	11940 5030 13970 5030
+Wire Wire Line
+	11940 4870 13970 4870
+Wire Wire Line
+	11940 4710 13970 4710
+Wire Wire Line
+	11940 4520 13970 4520
+Wire Wire Line
+	11940 4360 13970 4360
+Wire Wire Line
 	1950 1550 2200 1550
 Wire Wire Line
@@
 	15760 7280 15760 3870
 Wire Wire Line
-	11940 5030 13970 5030
-Wire Wire Line
 	6790 2020 13140 2020
 Wire Wire Line
@@
 Wire Wire Line
 	15160 3120 15950 3120
-Wire Wire Line
-	11940 4950 13970 4950
-Wire Wire Line
-	11940 4790 13970 4790
-Wire Wire Line
-	11940 4600 13970 4600
-Wire Wire Line
-	11940 4440 13970 4440
-Wire Wire Line
-	11940 4280 13970 4280
 Wire Wire Line
 	13970 3120 13310 3120
@@
 	6640 3200 6190 3200
 Wire Wire Line
-	13970 4360 11940 4360
-Wire Wire Line
-	13970 4520 11940 4520
-Wire Wire Line
-	13970 4710 11940 4710
-Wire Wire Line
-	13970 4870 11940 4870
-Wire Wire Line
 	15930 3200 15160 3200
 Wire Wire Line
@@
 Wire Wire Line
 	4650 5910 5000 5910
+Wire Wire Line
+	13970 4280 11940 4280
+Wire Wire Line
+	13970 4440 11940 4440
+Wire Wire Line
+	13970 4600 11940 4600
+Wire Wire Line
+	13970 4790 11940 4790
+Wire Wire Line
+	13970 4950 11940 4950
 Text GLabel 4650 5230 0    39   Input ~ 0
 TDI
@@
 F33 "X0_XLB_3o" I R 9160 7950 60
 F34 "X0_XLB_4o" I R 9160 8030 60
-F35 "X0_XLA_4i" I L 7970 6870 60
-F36 "X0_XLA_3i" I L 7970 6790 60
-F37 "X0_XLA_2i" I L 7970 6710 60
-F38 "X0_XLA_1i" I L 7970 6630 60
-F39 "X0_XLA_0i" I L 7970 6550 60
-F40 "X0_XLA_0o" I L 7970 6440 60
-F41 "X0_XLA_1o" I L 7970 6360 60
-F42 "X0_XLA_2o" I L 7970 6280 60
-F43 "X0_XLA_3o" I L 7970 6200 60
-F44 "X0_XLA_4o" I L 7970 6120 60
+F35 "X0_XLA_4i" I L 7970 6120 60
+F36 "X0_XLA_3i" I L 7970 6200 60
+F37 "X0_XLA_2i" I L 7970 6280 60
+F38 "X0_XLA_1i" I L 7970 6360 60
+F39 "X0_XLA_0i" I L 7970 6440 60
+F40 "X0_XLA_0o" I L 7970 6550 60
+F41 "X0_XLA_1o" I L 7970 6630 60
+F42 "X0_XLA_2o" I L 7970 6710 60
+F43 "X0_XLA_3o" I L 7970 6790 60
+F44 "X0_XLA_4o" I L 7970 6870 60
 $EndSheet
 $Sheet
@@
 F13 "X1_XLB_3o" I R 15160 3790 60
 F14 "X1_XLB_4o" I R 15160 3870 60
-F15 "X1_XLA_4i" I L 13970 4280 60
-F16 "X1_XLA_3i" I L 13970 4360 60
-F17 "X1_XLA_2i" I L 13970 4440 60
-F18 "X1_XLA_1i" I L 13970 4520 60
-F19 "X1_XLA_0i" I L 13970 4600 60
-F20 "X1_XLA_0o" I L 13970 4710 60
-F21 "X1_XLA_1o" I L 13970 4790 60
-F22 "X1_XLA_2o" I L 13970 4870 60
-F23 "X1_XLA_3o" I L 13970 4950 60
-F24 "X1_XLA_4o" I L 13970 5030 60
+F15 "X1_XLA_4i" I L 13970 5030 60
+F16 "X1_XLA_3i" I L 13970 4950 60
+F17 "X1_XLA_2i" I L 13970 4870 60
+F18 "X1_XLA_1i" I L 13970 4790 60
+F19 "X1_XLA_0i" I L 13970 4710 60
+F20 "X1_XLA_0o" I L 13970 4600 60
+F21 "X1_XLA_1o" I L 13970 4520 60
+F22 "X1_XLA_2o" I L 13970 4440 60
+F23 "X1_XLA_3o" I L 13970 4360 60
+F24 "X1_XLA_4o" I L 13970 4280 60
 F25 "X0_XLB_4i" I L 13970 3870 60
 F26 "X0_XLB_3i" I L 13970 3790 60

Commit message: Added appropriate sepearte power modules. Moved buffering to hiearchial sheet Buffering per 2 L2s due to harsh pull down on pads moved pins from global labels to heirachial
Parts:
- removed R102, R103, R104, R105: 10K, symbol R
- removed U102, U103: NC7WZ17, symbol NC7WZ17
Other:
- note removed: "JTAG Buffering"

Commit message: more buffers and added connectors for end
Parts:
- added P? (x2): CONN_20, symbol CONN_20
- added P? (x10): CONN_10X2, symbol CONN_10X2
Connections:
- net labels added: L2_0_TCK, L2_0_TMS, L2_1_TCK, L2_1_TMS, L2_2_TCK, L2_2_TMS, L2_3_TCK, L2_3_TMS
- net labels removed: 123
- wire segments 346 -> 602

Commit message: Isolated L1 stuff (inc. JTAG) in single sheet. Added buffered for the L2's JTAG control signals.
Parts:
- removed P? (x2): CONN_20, symbol CONN_20
- added P? (x4): CONN_10X2, symbol CONN_10X2
Connections:
- net labels added: L2_MSEL_0, L2_MSEL_1, L2_MSEL_2, L2_MSEL_3, L2_RST_0, L2_RST_1, L2_RST_2, L2_RST_3, MSEL_N
- net labels removed: MSEL
- wire segments 602 -> 726

Commit message: removing old buffering and wanted to check point
Parts:
- gave numbers to parts that had none: 14
Other:
- moved on the sheet: P106, P107, P110, P111

Commit message: missing header connector for 2 L2s. Find space!
Parts:
- added P?: CONN_10X2, symbol CONN_10X2
Connections:
- net GND: now also P102.19 (P19), P103.19 (P19), P108.19 (P19), P112.19 (P19), P113.11 (P11), P113.13 (P13), P113.15 (P15), P113.17 (P17), P113.19 (P19), P113.3 (P3), P113.5 (P5), P113.7 (P7), P113.9 (P9), P114.19 (P19), P115.1 (P1), P?.1 (P1), P?.11 (P11), P?.13 (P13), P?.15 (P15), P?.17 (P17), P?.19 (P19), P?.3 (P3), P?.5 (P5), P?.7 (P7), P?.9 (P9)
Other:
- moved on the sheet: P112, P113

Commit message: workaround found for headers problem. Early start, good progess!
Parts:
- added P?: CONN_10X2, symbol CONN_10X2
Connections:
- net L2_2/X1_XLA_0i: now also P?.10 (P10)
- net L2_2/X1_XLA_0o: now also P?.12 (P12)
- net L2_2/X1_XLA_1i: now also P?.8 (P8)
- net L2_2/X1_XLA_1o: now also P?.14 (P14)
- net L2_2/X1_XLA_2i: now also P?.6 (P6)
- net L2_2/X1_XLA_2o: now also P?.16 (P16)
- net L2_2/X1_XLA_3i: now also P?.4 (P4)
- net L2_2/X1_XLA_3o: now also P?.18 (P18)
- net L2_2/X1_XLA_4i: now also P?.2 (P2)
- net L2_2/X1_XLA_4o: now also P?.20 (P20)
- net L2_5/X1_XLA_0i: now also P?.12 (P12)
- net L2_5/X1_XLA_0o: now also P?.10 (P10)
- net L2_5/X1_XLA_1i: now also P?.14 (P14)
- net L2_5/X1_XLA_1o: now also P?.8 (P8)
- net L2_5/X1_XLA_2i: now also P?.16 (P16)
- net L2_5/X1_XLA_2o: now also P?.6 (P6)
- net L2_5/X1_XLA_3i: now also P?.18 (P18)
- net L2_5/X1_XLA_3o: now also P?.4 (P4)
- net L2_5/X1_XLA_4i: now also P?.20 (P20)
- net L2_5/X1_XLA_4o: now also P?.2 (P2)
- new net: P?.1 (P1), P?.11 (P11), P?.13 (P13), P?.15 (P15), P?.17 (P17), P?.19 (P19), P?.3 (P3), P?.5 (P5), P?.7 (P7), P?.9 (P9)
Other:
- moved on the sheet: P113, P114, P115, P?
