File: l2_dev_board/Design/power.sch (KiCad schematic (older format))
At the start: 49 parts, among them U1001 LT3480, U1002 NCP1529, U1003 NCP1529, U1004 NCP1529, U1005 APX803-SR, U1006 NCP1529, U1007 NCP1529, U1008 APX803-SR

Commit message: new design with heirachial and new libraries
Parts:
- renumbered C1001 to C1201, C1002 to C1202, C1005 to C1203, C1003 to C1204, C1004 to C1205, C1006 to C1206, C1007 to C1207, C1010 to C1208, C1008 to C1209, C1009 to C1210, C1013 to C1211, C1011 to C1212, C1012 to C1213, C1014 to C1214, C1015 to C1215, C1016 to C1216, C1017 to C1217, C1018 to C1218, C1019 to C1219, D1001 to D1201, L1001 to L1201, L1004 to L1202, L1002 to L1203, L1003 to L1204, L1005 to L1205, L1006 to L1206, R1001 to R1201, R1002 to R1202, R1003 to R1203, R1004 to R1204, R1009 to R1205, R1010 to R1206, R1005 to R1207, R1006 to R1208, R1007 to R1209, R1008 to R1210, R1011 to R1211, R1013 to R1212, R1014 to R1213, R1015 to R1214, R1016 to R1215, U1001 to U1201, U1004 to U1202, U1002 to U1203, U1003 to U1204, U1005 to U1205, U1006 to U1206, U1007 to U1207, U1008 to U1208
Other:
- moved on the sheet: C1201, C1202, C1206, C1207, D1201, L1201, R1201, R1202, R1203, R1204, U1201
