File: l2_dev_clean/l1.sch (KiCad schematic (older format))
At the start: 38 parts

Commit message: just need adc and done...hopefully
Parts:
- gave numbers to parts that had none: 34
