File: l2_dev_clean/l1.sch (KiCad schematic (older format))
At the start: 34 parts, among them U1401 NC7WZ17, U1402 NC7WZ07, U1403 NCP1529, U1404 NCP1521B, U1405 APX803-SR, U1406 APX803-SR, U1407 XS1-L1-128

Commit message: added extra buffers to remove lengthy lines. Also looking and audio board for L1 layout!
Parts:
- added R1409: R, symbol R
Connections:
- net +3.3V: now also R1409.1
- net DEBUG_N: now also R1409.2
