File: l2_dev_clean/l2.sch (KiCad schematic (older format))
At the start: 16 parts

Commit message: just need adc and done...hopefully
Parts:
- gave numbers to parts that had none: 13
Connections:
- net +1V0: now also U301.A19 (VDD_A19), U301.A34 (VDD_A34), U301.A53 (VDD_A53), U301.A68 (VDD_A68), U301.B15 (VDD_B15), U301.B28 (VDD_B28), U301.B43 (VDD_B43), U301.B5 (PCU_VDD), U301.B56 (VDD_B56); no longer U301.A19 (VDD_A19), U301.A34 (VDD_A34), U301.A53 (VDD_A53), U301.A68 (VDD_A68), U301.B15 (VDD_B15), U301.B28 (VDD_B28), U301.B43 (VDD_B43), U301.B5 (PCU_VDD), U301.B56 (VDD_B56)
- net +3V3: now also U301.A17 (VDDIO_A17), U301.A2 (VDDIO_A2), U301.A36 (VDDIO_A36), U301.A51 (VDDIO_51), U301.B1 (VDDIO_B1), U301.B14 (VDDIO_B14), U301.B29 (VDDIO_B29), U301.B32 (OTP_VDDIO), U301.B33 (MODE0), U301.B34 (MODE1), U301.B4 (PCU_VDDIO), U301.B42 (VDDIO_B42); no longer U301.A17 (VDDIO_A17), U301.A2 (VDDIO_A2), U301.A36 (VDDIO_A36), U301.A51 (VDDIO_51), U301.B1 (VDDIO_B1), U301.B14 (VDDIO_B14), U301.B29 (VDDIO_B29), U301.B32 (OTP_VDDIO), U301.B33 (MODE0), U301.B34 (MODE1), U301.B4 (PCU_VDDIO), U301.B42 (VDDIO_B42)
- net CLK: now also U301.B6 (PCU_CLK), U301.B7 (CLK); no longer U301.B6 (PCU_CLK), U301.B7 (CLK)
- net DEBUG_N: now also U301.B37 (DEBUG); no longer U301.B37 (DEBUG)
- net GND: now also U301.A1 (GND_A1), U301.A18 (GND_A18), U301.A35 (MODE4), U301.A37 (PLL_AVGND), U301.A52 (GND_A52), U301.GND (GND_PAD); no longer U301.A1 (GND_A1), U301.A18 (GND_A18), U301.A35 (MODE4), U301.A37 (PLL_AVGND), U301.A52 (GND_A52), U301.GND (GND_PAD)
- net MSEL: now also U301.B35 (MODE2), U301.B36 (MODE3); no longer U301.B35 (MODE2), U301.B36 (MODE3)
- net RST_N: now also U301.B13 (TRST_N), U301.B8 (RST_N); no longer U301.B13 (TRST_N), U301.B8 (RST_N)
- net TCK: now also U301.B10 (TCK); no longer U301.B10 (TCK)
- net TDI: now also U301.B12 (TDI); no longer U301.B12 (TDI)
- net TDO: now also U301.B9 (TDO); no longer U301.B9 (TDO)
- net TMS: now also U301.B11 (TMS); no longer U301.B11 (TMS)
- net at C301.1, R301.2: now also U301.A38 (PLL_AVDD); no longer U301.A38 (PLL_AVDD)
Other:
- moved on the sheet: C301, R301
