File: l2_dev_clean/l2_dev_board.sch (KiCad schematic (older format))
At the start: 15 parts

Commit message: Schematics back to previous progress but with better layout and heirarchial structure. Also created switch and rotary dip layout.
Parts:
- removed C? (x2): 4.7uF, symbol C
- removed L?: 4.7uH, symbol INDUCTOR
- removed U?: MCP1603, symbol MCP1603
- added C? (x2): 10uF, symbol C
- added C?: 33pF, symbol C
- added L?: 2u2H, symbol INDUCTOR
- added P? (x10): CONN_30, symbol CONN_30
- added R?: 100k, symbol R
- added R?: 453k, symbol R
- added R?: 10k, symbol R
- added U?: NCP1529, symbol NCP1529
- added U? (x2): APX803-SR, symbol APX803-SR
Connections:
- net labels added: +3V3_L2, +3V3_PG, DEBUG_N_B, DEBUG_N_L, DEBUG_N_R, DEBUG_N_TOP, L1_DEBUG_N_B, L1_DEBUG_N_L, L1_DEBUG_N_R, L1_DEBUG_N_TOP, L1_RST_N_B, L1_RST_N_L, L1_RST_N_R, L1_RST_N_TOP, L1_TCK_B, L1_TCK_TOP, L1_TDI_B, L1_TDI_L, L1_TDI_R, L1_TDI_TOP, L1_TDO_B, L1_TDO_L, L1_TDO_R, L1_TDO_TOP, L1_TMS_B, L1_TMS_TOP, L1_TRST_N_B, L1_TRST_N_L, L1_TRST_N_R, L1_TRST_N_TOP, L1_XLINK_0i_B, L1_XLINK_0i_L, L1_XLINK_0i_R, L1_XLINK_0i_TOP, L1_XLINK_0o_B, L1_XLINK_0o_L, L1_XLINK_0o_R, L1_XLINK_0o_TOP, L1_XLINK_1i_B, L1_XLINK_1i_L, L1_XLINK_1i_R, L1_XLINK_1i_TOP, L1_XLINK_1o_B, L1_XLINK_1o_L, L1_XLINK_1o_R, L1_XLINK_1o_TOP, RST_N_B, RST_N_L, RST_N_R, RST_N_SPVSR, RST_N_TOP, TCK_B, TCK_L, TCK_R, TCK_TOP, TDI_B, TDI_L, TDI_R, TDI_TOP, TDO_B, TDO_L, TDO_R, TDO_TOP, TMS_B, TMS_L, TMS_R, TMS_TOP, TRST_N_B, TRST_N_L, TRST_N_R, TRST_N_TOP
- net labels removed: +3.3V
- wire segments 41 -> 710
Other:
- note added: "5V to 3V3 @ 1A"
- note removed: "5V to 3V3 @ 0.5A"
- moved on the sheet: C?, D?, L?, R?, U?

Commit message: added switch and some logic to adjust JTAG. Need to confirm timing operations :s
Parts:
- added R? (x6): 10k, symbol R
- added U?: A6RS-161RF, symbol A6RS-161RF
- added U? (x2): SN74CBTD3861, symbol SN74CBTD3861
- added U? (x4): SN74LVC1G18, symbol SN74LVC1G18
- added U?: 74AHC1GU04, symbol 74AHC1GU04
- added U?: NC7SZ157, symbol NC7SZ157
Connections:
- net DEBUG_N_TOP is gone; now on net GND: P?.8 (P8)
- net L1_DEBUG_N_TOP is gone; now on net GND: P?.16 (P16)
- net L1_TDI_TOP is gone; now on net L2_PAIR/T_X0_XLB_4o: P?.28 (P28)
- net L1_TDO_TOP is gone; now on net GND: P?.30 (P30)
- net L1_TRST_N_TOP is gone; now on net GND: P?.15 (P15)
- net L1_XLINK_1o_TOP is gone; now on net GND: P?.22 (P22)
- net L2_PAIR/BL_X0_XLA_0i is gone; now on net L2_PAIR/BL_X0_XLA_0i: P?.7 (P7)
- net L2_PAIR/BL_X0_XLA_0o is gone; now on net L2_PAIR/BL_X0_XLA_0o: P?.10 (P10)
- net L2_PAIR/BL_X0_XLA_1i is gone; now on net L2_PAIR/BL_X0_XLA_1i: P?.6 (P6)
- net L2_PAIR/BL_X0_XLA_1o is gone; now on net L2_PAIR/BL_X0_XLA_1o: P?.11 (P11)
- net L2_PAIR/BL_X0_XLA_2i is gone; now on net L2_PAIR/BL_X0_XLA_2i: P?.5 (P5)
- net L2_PAIR/BL_X0_XLA_2o is gone; now on net L2_PAIR/BL_X0_XLA_2o: P?.12 (P12)
- net L2_PAIR/BL_X0_XLA_3i is gone; now on net L2_PAIR/BL_X0_XLA_3i: P?.4 (P4)
- net L2_PAIR/BL_X0_XLA_3o is gone; now on net L2_PAIR/BL_X0_XLA_3o: P?.13 (P13)
- net L2_PAIR/BL_X0_XLA_4i is gone; now on net L2_PAIR/BL_X0_XLA_4i: P?.3 (P3)
- net L2_PAIR/BL_X0_XLA_4o is gone; now on net L2_PAIR/BL_X0_XLA_4o: P?.14 (P14)
- net L2_PAIR/BR_X1_XLA_0i is gone; now on net L2_PAIR/BR_X1_XLA_0i: P?.9 (P9)
- net L2_PAIR/BR_X1_XLA_0o is gone; now on net L2_PAIR/BR_X1_XLA_0o: P?.6 (P6)
- net L2_PAIR/BR_X1_XLA_1i is gone; now on net L2_PAIR/BR_X1_XLA_1i: P?.10 (P10)
- net L2_PAIR/BR_X1_XLA_1o is gone; now on net L2_PAIR/BR_X1_XLA_1o: P?.5 (P5)
- net L2_PAIR/BR_X1_XLA_2i is gone; now on net L2_PAIR/BR_X1_XLA_2i: P?.11 (P11)
- net L2_PAIR/BR_X1_XLA_2o is gone; now on net L2_PAIR/BR_X1_XLA_2o: P?.4 (P4)
- net L2_PAIR/BR_X1_XLA_3i is gone; now on net L2_PAIR/BR_X1_XLA_3i: P?.2 (P2)
- net L2_PAIR/BR_X1_XLA_3o is gone; now on net L2_PAIR/BR_X1_XLA_3o: P?.3 (P3)
- net L2_PAIR/BR_X1_XLA_4i is gone; now on net L2_PAIR/BR_X1_XLA_4i: P?.3 (P3)
- net L2_PAIR/BR_X1_XLA_4o is gone; now on net L2_PAIR/BR_X1_XLA_4o: P?.2 (P2)
- net L2_PAIR/B_X1_XLB_0i is gone; now on net L1_XLINK_1i_B: P?.21 (P21)
- net L2_PAIR/B_X1_XLB_0i is gone; now on net TRST_N_B: P?.7 (P7)
- net L2_PAIR/B_X1_XLB_0o is gone; now on net L1_TMS_B: P?.10 (P10)
- net L2_PAIR/B_X1_XLB_0o is gone; now on net TDO_B: P?.24 (P24)
- net L2_PAIR/B_X1_XLB_1i is gone; now on net GND: P?.20 (P20)
- net L2_PAIR/B_X1_XLB_1i is gone; now on net RST_N_B: P?.6 (P6)
- net L2_PAIR/B_X1_XLB_1o is gone; now on net GND: P?.11 (P11)
- net L2_PAIR/B_X1_XLB_1o is gone; now on net GND: P?.25 (P25)
- net L2_PAIR/B_X1_XLB_2i is gone; now on net L1_XLINK_1o_B: P?.19 (P19)
- net L2_PAIR/B_X1_XLB_2i is gone; now on net GND: P?.5 (P5)
- net L2_PAIR/B_X1_XLB_2o is gone; now on net L1_TCK_B: P?.12 (P12)
- net L2_PAIR/B_X1_XLB_2o is gone; now on net TDI_B: P?.26 (P26)
- net L2_PAIR/B_X1_XLB_3i is gone; now on net L1_XLINK_0o_B: P?.18 (P18)
- net L2_PAIR/B_X1_XLB_3i is gone; now on net TCK_B: P?.4 (P4)
- net L2_PAIR/B_X1_XLB_3o is gone; now on net GND: P?.13 (P13)
- net L2_PAIR/B_X1_XLB_3o is gone; now on net GND: P?.27 (P27)
- net L2_PAIR/B_X1_XLB_4i is gone; now on net GND: P?.17 (P17)
- net L2_PAIR/B_X1_XLB_4i is gone; now on net GND: P?.3 (P3)
- net L2_PAIR/B_X1_XLB_4o is gone; now on net L1_RST_N_B: P?.14 (P14)
- net L2_PAIR/B_X1_XLB_4o is gone; now on net L1_TDO_B: P?.28 (P28)
- net L2_PAIR/TL_X0_XLA_0i is gone; now on net L2_PAIR/TL_X0_XLA_0i: P?.21 (P21)
- net L2_PAIR/TL_X0_XLA_0o is gone; now on net L2_PAIR/TL_X0_XLA_0o: P?.24 (P24)
- net L2_PAIR/TL_X0_XLA_1i is gone; now on net L2_PAIR/TL_X0_XLA_1i: P?.20 (P20)
- net L2_PAIR/TL_X0_XLA_1o is gone; now on net L2_PAIR/TL_X0_XLA_1o: P?.25 (P25)
- net L2_PAIR/TL_X0_XLA_2i is gone; now on net L2_PAIR/TL_X0_XLA_2i: P?.19 (P19)
- net L2_PAIR/TL_X0_XLA_2o is gone; now on net L2_PAIR/TL_X0_XLA_2o: P?.26 (P26)
- net L2_PAIR/TL_X0_XLA_3i is gone; now on net L2_PAIR/TL_X0_XLA_3i: P?.18 (P18)
- net L2_PAIR/TL_X0_XLA_3o is gone; now on net L2_PAIR/TL_X0_XLA_3o: P?.27 (P27)
- net L2_PAIR/TL_X0_XLA_4i is gone; now on net L2_PAIR/TL_X0_XLA_4i: P?.17 (P17)
- net L2_PAIR/TL_X0_XLA_4o is gone; now on net L2_PAIR/TL_X0_XLA_4o: P?.28 (P28)
- net L2_PAIR/TR_X1_XLA_0i is gone; now on net L2_PAIR/TR_X1_XLA_0i: P?.13 (P13)
- net L2_PAIR/TR_X1_XLA_0o is gone; now on net L2_PAIR/TR_X1_XLA_0o: P?.10 (P10)
- net L2_PAIR/TR_X1_XLA_1i is gone; now on net L2_PAIR/TR_X1_XLA_1i: P?.14 (P14)
- net L2_PAIR/TR_X1_XLA_1o is gone; now on net L2_PAIR/TR_X1_XLA_1o: P?.9 (P9)
- net L2_PAIR/TR_X1_XLA_2i is gone; now on net L2_PAIR/TR_X1_XLA_2i: P?.15 (P15)
- net L2_PAIR/TR_X1_XLA_2o is gone; now on net L2_PAIR/TR_X1_XLA_2o: P?.8 (P8)
- net L2_PAIR/TR_X1_XLA_3i is gone; now on net L2_PAIR/TR_X1_XLA_3i: P?.16 (P16)
- net L2_PAIR/TR_X1_XLA_3o is gone; now on net L2_PAIR/TR_X1_XLA_3o: P?.7 (P7)
- net L2_PAIR/TR_X1_XLA_4i is gone; now on net L2_PAIR/TR_X1_XLA_4i: P?.17 (P17)
- net L2_PAIR/TR_X1_XLA_4o is gone; now on net L2_PAIR/TR_X1_XLA_4o: P?.6 (P6)
- net L2_PAIR/T_X0_XLB_1o is gone; now on net GND: P?.25 (P25)
- net L2_PAIR/T_X0_XLB_2i is gone; now on net GND: P?.5 (P5)
- net L2_PAIR/T_X0_XLB_3o is gone; now on net GND: P?.27 (P27)
- net L2_PAIR/T_X0_XLB_4i is gone; now on net GND: P?.3 (P3)
- net RST_N_TOP is gone; now on net L2_PAIR/T_X0_XLB_1i: P?.6 (P6)
- net TCK_TOP is gone; now on net L2_PAIR/T_X0_XLB_3i: P?.4 (P4)
- net TDI_TOP is gone; now on net L2_PAIR/T_X0_XLB_0o: P?.24 (P24)
- net TDO_TOP is gone; now on net L2_PAIR/T_X0_XLB_2o: P?.26 (P26)
- net TRST_N_TOP is gone; now on net L2_PAIR/T_X0_XLB_0i: P?.7 (P7)
- net +5V: now also U?.24 (VCC), U?.24 (VCC), U?.5 (VCC), U?.5 (VCC), U?.5 (VCC), U?.5 (VCC)
- net DEBUG_N_B: now also P?.8 (P8); no longer P?.8 (P8)
- net DEBUG_N_L: now also U?.2 (A1)
- net GND: now also P?.11 (P11), P?.13 (P13), P?.17 (P17), P?.2 (P2), P?.20 (P20), R?.2, R?.2, R?.2, R?.2, U?.12 (GND), U?.12 (GND), U?.2 (GND), U?.2 (GND), U?.2 (GND), U?.2 (GND), U?.2 (GND), U?.3 (GND); no longer P?.1 (P1), P?.11 (P11), P?.11 (P11), P?.13 (P13), P?.13 (P13), P?.15 (P15), P?.15 (P15), P?.16 (P16), P?.16 (P16), P?.17 (P17), P?.17 (P17), P?.2 (P2), P?.2 (P2), P?.20 (P20), P?.20 (P20), P?.22 (P22), P?.22 (P22), P?.23 (P23), P?.25 (P25), P?.25 (P25), P?.27 (P27), P?.27 (P27), P?.29 (P29), P?.3 (P3), P?.3 (P3), P?.30 (P30), P?.30 (P30), P?.5 (P5), P?.5 (P5), P?.8 (P8), P?.8 (P8), P?.9 (P9)
- net L1_DEBUG_N_B: now also P?.16 (P16); no longer P?.16 (P16)
- net L1_DEBUG_N_L: now also U?.7 (A6)
- net L1_RST_N_B: no longer P?.14 (P14)
- net L1_RST_N_L: now also U?.9 (A8)
- net L1_TCK_B: no longer P?.12 (P12)
- net L1_TDI_B: now also P?.30 (P30); no longer P?.30 (P30)
- net L1_TDO_B: no longer P?.28 (P28)
- net L1_TMS_B: no longer P?.10 (P10)
- net L1_TRST_N_B: now also P?.15 (P15); no longer P?.15 (P15)
- net L1_TRST_N_L: now also U?.8 (A7)
- net L1_XLINK_0i_B: now also P?.22 (P22); no longer P?.22 (P22)
- net L1_XLINK_0o_B: no longer P?.18 (P18)
- net L1_XLINK_1i_B: no longer P?.21 (P21)
- net L1_XLINK_1o_B: no longer P?.19 (P19)
- net L2_PAIR/BR_X1_XLA_0i: no longer P?.10 (P10)
- net L2_PAIR/BR_X1_XLA_0o: no longer P?.7 (P7)
- net L2_PAIR/BR_X1_XLA_1i: no longer P?.11 (P11)
- net L2_PAIR/BR_X1_XLA_1o: no longer P?.6 (P6)
- net L2_PAIR/BR_X1_XLA_2i: no longer P?.12 (P12)
- net L2_PAIR/BR_X1_XLA_2o: no longer P?.5 (P5)
- net L2_PAIR/BR_X1_XLA_3i: no longer P?.13 (P13)
- net L2_PAIR/BR_X1_XLA_3o: no longer P?.4 (P4)
- net L2_PAIR/BR_X1_XLA_4i: no longer P?.14 (P14)
- net L2_PAIR/BR_X1_XLA_4o: no longer P?.3 (P3)
- net L2_PAIR/B_X1_XLB_0i: now also P?.7 (P7)
- net L2_PAIR/B_X1_XLB_0o: now also P?.24 (P24)
- net L2_PAIR/B_X1_XLB_1i: now also P?.6 (P6)
- net L2_PAIR/B_X1_XLB_1o: now also P?.25 (P25)
- net L2_PAIR/B_X1_XLB_2i: now also P?.5 (P5)
- net L2_PAIR/B_X1_XLB_2o: now also P?.26 (P26)
- net L2_PAIR/B_X1_XLB_3i: now also P?.4 (P4)
- net L2_PAIR/B_X1_XLB_3o: now also P?.27 (P27)
- net L2_PAIR/B_X1_XLB_4i: now also P?.3 (P3)
- net L2_PAIR/B_X1_XLB_4o: now also P?.28 (P28)
- net L2_PAIR/TR_X1_XLA_0i: no longer P?.24 (P24)
- net L2_PAIR/TR_X1_XLA_0o: no longer P?.21 (P21)
- net L2_PAIR/TR_X1_XLA_1i: no longer P?.25 (P25)
- net L2_PAIR/TR_X1_XLA_1o: no longer P?.20 (P20)
- net L2_PAIR/TR_X1_XLA_2i: no longer P?.26 (P26)
- net L2_PAIR/TR_X1_XLA_2o: no longer P?.19 (P19)
- net L2_PAIR/TR_X1_XLA_3i: no longer P?.27 (P27)
- net L2_PAIR/TR_X1_XLA_3o: no longer P?.18 (P18)
- net L2_PAIR/TR_X1_XLA_4i: no longer P?.28 (P28)
- net L2_PAIR/TR_X1_XLA_4o: no longer P?.17 (P17)
- net L2_PAIR/T_X0_XLB_0i: no longer P?.21 (P21)
- net L2_PAIR/T_X0_XLB_0o: no longer P?.10 (P10)
- net L2_PAIR/T_X0_XLB_1i: no longer P?.20 (P20)
- net L2_PAIR/T_X0_XLB_1o: now also P?.25 (P25); no longer P?.11 (P11)
- net L2_PAIR/T_X0_XLB_2i: now also P?.5 (P5); no longer P?.19 (P19)
- net L2_PAIR/T_X0_XLB_2o: no longer P?.12 (P12)
- net L2_PAIR/T_X0_XLB_3i: no longer P?.18 (P18)
- net L2_PAIR/T_X0_XLB_3o: now also P?.27 (P27); no longer P?.13 (P13)
- net L2_PAIR/T_X0_XLB_4i: now also P?.3 (P3); no longer P?.17 (P17)
- net L2_PAIR/T_X0_XLB_4o: no longer P?.14 (P14)
- net RST_N_B: no longer P?.6 (P6)
- net RST_N_L: now also U?.4 (A3)
- net TCK_B: no longer P?.4 (P4)
- net TCK_L: now also U?.10 (A9), U?.5 (A4); no longer P?.22 (P22)
- net TCK_R: no longer P?.22 (P22)
- net TDI_B: no longer P?.26 (P26)
- net TDO_B: no longer P?.24 (P24)
- net TMS_B: now also P?.2 (P2); no longer P?.2 (P2)
- net TMS_L: now also U?.11 (A10), U?.6 (A5); no longer P?.20 (P20)
- net TMS_R: no longer P?.20 (P20)
- net TMS_TOP: now also P?.2 (P2); no longer P?.2 (P2)
- net TRST_N_B: no longer P?.7 (P7)
- net TRST_N_L: now also U?.3 (A2)
- net L1_RST_N_TOP renamed L2_PAIR/T_X0_XLB_4o
- net L1_TCK_TOP renamed L2_PAIR/T_X0_XLB_2o
- net L1_TMS_TOP renamed L2_PAIR/T_X0_XLB_0o
- net L1_XLINK_0i_TOP renamed L2_PAIR/T_X0_XLB_2i
- net L1_XLINK_0o_TOP renamed L2_PAIR/T_X0_XLB_0i
- net L1_XLINK_1i_TOP renamed L2_PAIR/T_X0_XLB_3i
- net L2_PAIR/T_X0_XLB_0i renamed TRST_N_T
- net TRST_N_T: now also U?.3 (A2)
- net L2_PAIR/T_X0_XLB_0o renamed TDI_T
- net L2_PAIR/T_X0_XLB_1i renamed RST_N_T
- net RST_N_T: now also U?.4 (A3)
- net L2_PAIR/T_X0_XLB_2o renamed TDO_T
- net L2_PAIR/T_X0_XLB_3i renamed TCK_T
- net TCK_T: now also U?.10 (A9), U?.5 (A4)
- net L2_PAIR/T_X0_XLB_4o renamed L1_TDI_T
- net RST_N_SPVSR renamed RST_N
- net RST_N: now also R?.2, U?.20 (B3), U?.20 (B3)
- new net: U?.2 (A), U?.23 (OE), U?.4 (A)
- new net: U?.23 (OE), U?.4 (Y)
- new net +3.3V: R?.1, R?.1, U?.5 (VCC), U?.5 (VCC), U?.C
- new net DEBUG_N: U?.22 (B1), U?.22 (B1)
- new net DEBUG_N_T: P?.8 (P8), U?.2 (A1)
- new net L1_DEBUG_N: U?.17 (B6), U?.17 (B6)
- new net L1_DEBUG_N_T: P?.16 (P16), U?.7 (A6)
- new net L1_RST_N: U?.15 (B8), U?.15 (B8)
- new net L1_RST_N_T: P?.14 (P14), U?.9 (A8)
- new net L1_TCK_L: P?.22 (P22)
- new net L1_TCK_R: P?.22 (P22)
- new net L1_TCK_T: P?.12 (P12)
- new net L1_TDO_T: P?.30 (P30)
- new net L1_TMS_L: P?.20 (P20)
- new net L1_TMS_R: P?.20 (P20)
- new net L1_TMS_T: P?.10 (P10)
- new net L1_TRST_N: U?.16 (B7), U?.16 (B7)
- new net L1_TRST_N_T: P?.15 (P15), U?.8 (A7)
- new net L1_XLINK_0i_T: P?.19 (P19)
- new net L1_XLINK_0o_T: P?.21 (P21)
- new net L1_XLINK_1i_T: P?.18 (P18)
- new net L1_XLINK_1o_T: P?.22 (P22)
- new net L2_PAIR/BR_X1_XLA_0i: P?.10 (P10)
- new net L2_PAIR/BR_X1_XLA_0o: P?.7 (P7)
- new net L2_PAIR/BR_X1_XLA_1i: P?.11 (P11)
- new net L2_PAIR/BR_X1_XLA_1o: P?.6 (P6)
- new net L2_PAIR/BR_X1_XLA_2i: P?.12 (P12)
- new net L2_PAIR/BR_X1_XLA_2o: P?.5 (P5)
- new net L2_PAIR/BR_X1_XLA_3i: P?.13 (P13)
- new net L2_PAIR/BR_X1_XLA_3o: P?.4 (P4)
- new net L2_PAIR/BR_X1_XLA_4i: P?.14 (P14)
- new net L2_PAIR/BR_X1_XLA_4o: P?.3 (P3)
- new net L2_PAIR/B_X1_XLB_0i: P?.21 (P21)
- new net L2_PAIR/B_X1_XLB_0o: P?.10 (P10)
- new net L2_PAIR/B_X1_XLB_1i: P?.20 (P20)
- new net L2_PAIR/B_X1_XLB_1o: P?.11 (P11)
- new net L2_PAIR/B_X1_XLB_2i: P?.19 (P19)
- new net L2_PAIR/B_X1_XLB_2o: P?.12 (P12)
- new net L2_PAIR/B_X1_XLB_3i: P?.18 (P18)
- new net L2_PAIR/B_X1_XLB_3o: P?.13 (P13)
- new net L2_PAIR/B_X1_XLB_4i: P?.17 (P17)
- new net L2_PAIR/B_X1_XLB_4o: P?.14 (P14)
- new net L2_PAIR/TR_X1_XLA_0i: P?.24 (P24)
- new net L2_PAIR/TR_X1_XLA_0o: P?.21 (P21)
- new net L2_PAIR/TR_X1_XLA_1i: P?.25 (P25)
- new net L2_PAIR/TR_X1_XLA_1o: P?.20 (P20)
- new net L2_PAIR/TR_X1_XLA_2i: P?.26 (P26)
- new net L2_PAIR/TR_X1_XLA_2o: P?.19 (P19)
- new net L2_PAIR/TR_X1_XLA_3i: P?.27 (P27)
- new net L2_PAIR/TR_X1_XLA_3o: P?.18 (P18)
- new net L2_PAIR/TR_X1_XLA_4i: P?.28 (P28)
- new net L2_PAIR/TR_X1_XLA_4o: P?.17 (P17)
- new net L2_PAIR/T_X0_XLB_1i: P?.20 (P20)
- new net L2_PAIR/T_X0_XLB_1o: P?.11 (P11)
- new net L2_PAIR/T_X0_XLB_3o: P?.13 (P13)
- new net L2_PAIR/T_X0_XLB_4i: P?.17 (P17)
- new net SWT_1: R?.1, U?.1, U?.1 (S), U?.6 (S)
- new net SWT_2: R?.1, U?.1 (S), U?.2, U?.3 (I0)
- new net SWT_3: R?.1, U?.1 (I1), U?.1 (S), U?.3 (4)
- new net SWT_4: R?.1, U?.1 (S), U?.4 (8)
- new net TCK: U?.14 (B9), U?.14 (B9), U?.19 (B4), U?.19 (B4)
- new net TDO_Q1: U?.3 (A)
- new net TDO_Q2: U?.3 (A)
- new net TDO_Q3: U?.3 (A)
- new net TDO_Q4: U?.3 (A)
- new net TMS: U?.13 (B10), U?.13 (B10), U?.18 (B5), U?.18 (B5)
- new net TMS_T: U?.11 (A10), U?.6 (A5)
- new net TRST_N: R?.2, U?.21 (B2), U?.21 (B2)
Other:
- note added: "JTAG SIGNAL SWITCHES"
- note added: "L2 MESH AND EDGE CONNECTORS"
- note added: "L2 TDI/TDO SELECTORS"
- note added: "REFERENCE PAIR - Q1"
- note added: "REFERENCE PAIR - Q2\n"
- note added: "REFERENCE PAIR - Q3"
- note added: "REFERENCE PAIR - Q4"
- note added: "RST_N AND\nTRST_N\n\nPULL UPS"

Commit message: generated ps and pdfs
Connections:
- net L2_PAIR/BL_X0_XLA_0i is gone; now on net L2_PAIR/BL_X0_XLA_0i: P?.7 (P7)
- net L2_PAIR/BL_X0_XLA_0o is gone; now on net L2_PAIR/BL_X0_XLA_0o: P?.10 (P10)
- net L2_PAIR/BL_X0_XLA_1i is gone; now on net L2_PAIR/BL_X0_XLA_1i: P?.6 (P6)
- net L2_PAIR/BL_X0_XLA_1o is gone; now on net L2_PAIR/BL_X0_XLA_1o: P?.11 (P11)
- net L2_PAIR/BL_X0_XLA_2i is gone; now on net L2_PAIR/BL_X0_XLA_2i: P?.5 (P5)
- net L2_PAIR/BL_X0_XLA_2o is gone; now on net L2_PAIR/BL_X0_XLA_2o: P?.12 (P12)
- net L2_PAIR/BL_X0_XLA_3i is gone; now on net L2_PAIR/BL_X0_XLA_3i: P?.4 (P4)
- net L2_PAIR/BL_X0_XLA_3o is gone; now on net L2_PAIR/BL_X0_XLA_3o: P?.13 (P13)
- net L2_PAIR/BL_X0_XLA_4i is gone; now on net L2_PAIR/BL_X0_XLA_4i: P?.3 (P3)
- net L2_PAIR/BL_X0_XLA_4o is gone; now on net L2_PAIR/BL_X0_XLA_4o: P?.14 (P14)
- net L2_PAIR/BR_X1_XLA_0i is gone; now on net L2_PAIR/BR_X1_XLA_0i: P?.9 (P9)
- net L2_PAIR/BR_X1_XLA_0o is gone; now on net L2_PAIR/BR_X1_XLA_0o: P?.6 (P6)
- net L2_PAIR/BR_X1_XLA_1i is gone; now on net L2_PAIR/BR_X1_XLA_1i: P?.10 (P10)
- net L2_PAIR/BR_X1_XLA_1o is gone; now on net L2_PAIR/BR_X1_XLA_1o: P?.5 (P5)
- net L2_PAIR/BR_X1_XLA_2i is gone; now on net L2_PAIR/BR_X1_XLA_2i: P?.11 (P11)
- net L2_PAIR/BR_X1_XLA_2o is gone; now on net L2_PAIR/BR_X1_XLA_2o: P?.4 (P4)
- net L2_PAIR/BR_X1_XLA_3i is gone; now on net L2_PAIR/BR_X1_XLA_3i: P?.2 (P2)
- net L2_PAIR/BR_X1_XLA_3o is gone; now on net L2_PAIR/BR_X1_XLA_3o: P?.3 (P3)
- net L2_PAIR/BR_X1_XLA_4i is gone; now on net L2_PAIR/BR_X1_XLA_4i: P?.3 (P3)
- net L2_PAIR/BR_X1_XLA_4o is gone; now on net L2_PAIR/BR_X1_XLA_4o: P?.2 (P2)
- net L2_PAIR/B_X1_XLB_0i is gone; now on net L2_PAIR/B_X1_XLB_0i: P?.7 (P7)
- net L2_PAIR/B_X1_XLB_0o is gone; now on net L2_PAIR/B_X1_XLB_0o: P?.24 (P24)
- net L2_PAIR/B_X1_XLB_1i is gone; now on net L2_PAIR/B_X1_XLB_1i: P?.6 (P6)
- net L2_PAIR/B_X1_XLB_1o is gone; now on net L2_PAIR/B_X1_XLB_1o: P?.25 (P25)
- net L2_PAIR/B_X1_XLB_2i is gone; now on net L2_PAIR/B_X1_XLB_2i: P?.5 (P5)
- net L2_PAIR/B_X1_XLB_2o is gone; now on net L2_PAIR/B_X1_XLB_2o: P?.26 (P26)
- net L2_PAIR/B_X1_XLB_3i is gone; now on net L2_PAIR/B_X1_XLB_3i: P?.4 (P4)
- net L2_PAIR/B_X1_XLB_3o is gone; now on net L2_PAIR/B_X1_XLB_3o: P?.27 (P27)
- net L2_PAIR/B_X1_XLB_4i is gone; now on net L2_PAIR/B_X1_XLB_4i: P?.3 (P3)
- net L2_PAIR/B_X1_XLB_4o is gone; now on net L2_PAIR/B_X1_XLB_4o: P?.28 (P28)
- net L2_PAIR/TL_X0_XLA_0i is gone; now on net L2_PAIR/TL_X0_XLA_0i: P?.21 (P21)
- net L2_PAIR/TL_X0_XLA_0o is gone; now on net L2_PAIR/TL_X0_XLA_0o: P?.24 (P24)
- net L2_PAIR/TL_X0_XLA_1i is gone; now on net L2_PAIR/TL_X0_XLA_1i: P?.20 (P20)
- net L2_PAIR/TL_X0_XLA_1o is gone; now on net L2_PAIR/TL_X0_XLA_1o: P?.25 (P25)
- net L2_PAIR/TL_X0_XLA_2i is gone; now on net L2_PAIR/TL_X0_XLA_2i: P?.19 (P19)
- net L2_PAIR/TL_X0_XLA_2o is gone; now on net L2_PAIR/TL_X0_XLA_2o: P?.26 (P26)
- net L2_PAIR/TL_X0_XLA_3i is gone; now on net L2_PAIR/TL_X0_XLA_3i: P?.18 (P18)
- net L2_PAIR/TL_X0_XLA_3o is gone; now on net L2_PAIR/TL_X0_XLA_3o: P?.27 (P27)
- net L2_PAIR/TL_X0_XLA_4i is gone; now on net L2_PAIR/TL_X0_XLA_4i: P?.17 (P17)
- net L2_PAIR/TL_X0_XLA_4o is gone; now on net L2_PAIR/TL_X0_XLA_4o: P?.28 (P28)
- net L2_PAIR/TR_X1_XLA_0i is gone; now on net L2_PAIR/TR_X1_XLA_0i: P?.13 (P13)
- net L2_PAIR/TR_X1_XLA_0o is gone; now on net L2_PAIR/TR_X1_XLA_0o: P?.10 (P10)
- net L2_PAIR/TR_X1_XLA_1i is gone; now on net L2_PAIR/TR_X1_XLA_1i: P?.14 (P14)
- net L2_PAIR/TR_X1_XLA_1o is gone; now on net L2_PAIR/TR_X1_XLA_1o: P?.9 (P9)
- net L2_PAIR/TR_X1_XLA_2i is gone; now on net L2_PAIR/TR_X1_XLA_2i: P?.15 (P15)
- net L2_PAIR/TR_X1_XLA_2o is gone; now on net L2_PAIR/TR_X1_XLA_2o: P?.8 (P8)
- net L2_PAIR/TR_X1_XLA_3i is gone; now on net L2_PAIR/TR_X1_XLA_3i: P?.16 (P16)
- net L2_PAIR/TR_X1_XLA_3o is gone; now on net L2_PAIR/TR_X1_XLA_3o: P?.7 (P7)
- net L2_PAIR/TR_X1_XLA_4i is gone; now on net L2_PAIR/TR_X1_XLA_4i: P?.17 (P17)
- net L2_PAIR/TR_X1_XLA_4o is gone; now on net L2_PAIR/TR_X1_XLA_4o: P?.6 (P6)
- net L2_PAIR/T_X0_XLB_0i is gone; now on net L2_PAIR/T_X0_XLB_0i: P?.7 (P7)
- net L2_PAIR/T_X0_XLB_0o is gone; now on net L2_PAIR/T_X0_XLB_0o: P?.24 (P24)
- net L2_PAIR/T_X0_XLB_1i is gone; now on net L2_PAIR/T_X0_XLB_1i: P?.6 (P6)
- net L2_PAIR/T_X0_XLB_1o is gone; now on net L2_PAIR/T_X0_XLB_1o: P?.25 (P25)
- net L2_PAIR/T_X0_XLB_2i is gone; now on net L2_PAIR/T_X0_XLB_2i: P?.5 (P5)
- net L2_PAIR/T_X0_XLB_2o is gone; now on net L2_PAIR/T_X0_XLB_2o: P?.26 (P26)
- net L2_PAIR/T_X0_XLB_3i is gone; now on net L2_PAIR/T_X0_XLB_3i: P?.4 (P4)
- net L2_PAIR/T_X0_XLB_3o is gone; now on net L2_PAIR/T_X0_XLB_3o: P?.27 (P27)
- net L2_PAIR/T_X0_XLB_4i is gone; now on net L2_PAIR/T_X0_XLB_4i: P?.3 (P3)
- net L2_PAIR/T_X0_XLB_4o is gone; now on net L2_PAIR/T_X0_XLB_4o: P?.28 (P28)
- net GND: now also P?.1 (P1), P?.15 (P15), P?.16 (P16), P?.2 (P2), P?.22 (P22), P?.23 (P23), P?.29 (P29), P?.30 (P30), P?.8 (P8), P?.9 (P9)
- net L2_PAIR/BR_X1_XLA_0i: no longer P?.10 (P10)
- net L2_PAIR/BR_X1_XLA_0o: no longer P?.7 (P7)
- net L2_PAIR/BR_X1_XLA_1i: no longer P?.11 (P11)
- net L2_PAIR/BR_X1_XLA_1o: no longer P?.6 (P6)
- net L2_PAIR/BR_X1_XLA_2i: no longer P?.12 (P12)
- net L2_PAIR/BR_X1_XLA_2o: no longer P?.5 (P5)
- net L2_PAIR/BR_X1_XLA_3i: no longer P?.13 (P13)
- net L2_PAIR/BR_X1_XLA_3o: no longer P?.4 (P4)
- net L2_PAIR/BR_X1_XLA_4i: no longer P?.14 (P14)
- net L2_PAIR/BR_X1_XLA_4o: no longer P?.3 (P3)
- net L2_PAIR/TR_X1_XLA_0i: no longer P?.24 (P24)
- net L2_PAIR/TR_X1_XLA_0o: no longer P?.21 (P21)
- net L2_PAIR/TR_X1_XLA_1i: no longer P?.25 (P25)
- net L2_PAIR/TR_X1_XLA_1o: no longer P?.20 (P20)
- net L2_PAIR/TR_X1_XLA_2i: no longer P?.26 (P26)
- net L2_PAIR/TR_X1_XLA_2o: no longer P?.19 (P19)
- net L2_PAIR/TR_X1_XLA_3i: no longer P?.27 (P27)
- net L2_PAIR/TR_X1_XLA_3o: no longer P?.18 (P18)
- net L2_PAIR/TR_X1_XLA_4i: no longer P?.28 (P28)
- net L2_PAIR/TR_X1_XLA_4o: no longer P?.17 (P17)
- net L2_PAIR/T_X0_XLB_0i: no longer P?.21 (P21)
- net L2_PAIR/T_X0_XLB_0o: no longer P?.10 (P10)
- net L2_PAIR/T_X0_XLB_1i: no longer P?.20 (P20)
- net L2_PAIR/T_X0_XLB_1o: no longer P?.11 (P11)
- net L2_PAIR/T_X0_XLB_2i: no longer P?.19 (P19)
- net L2_PAIR/T_X0_XLB_2o: no longer P?.12 (P12)
- net L2_PAIR/T_X0_XLB_3i: no longer P?.18 (P18)
- net L2_PAIR/T_X0_XLB_3o: no longer P?.13 (P13)
- net L2_PAIR/T_X0_XLB_4i: no longer P?.17 (P17)
- net L2_PAIR/T_X0_XLB_4o: no longer P?.14 (P14)
- new net L2_PAIR/BR_X1_XLA_0i: P?.10 (P10)
- new net L2_PAIR/BR_X1_XLA_0o: P?.7 (P7)
- new net L2_PAIR/BR_X1_XLA_1i: P?.11 (P11)
- new net L2_PAIR/BR_X1_XLA_1o: P?.6 (P6)
- new net L2_PAIR/BR_X1_XLA_2i: P?.12 (P12)
- new net L2_PAIR/BR_X1_XLA_2o: P?.5 (P5)
- new net L2_PAIR/BR_X1_XLA_3i: P?.13 (P13)
- new net L2_PAIR/BR_X1_XLA_3o: P?.4 (P4)
- new net L2_PAIR/BR_X1_XLA_4i: P?.14 (P14)
- new net L2_PAIR/BR_X1_XLA_4o: P?.3 (P3)
- new net L2_PAIR/TR_X1_XLA_0i: P?.24 (P24)
- new net L2_PAIR/TR_X1_XLA_0o: P?.21 (P21)
- new net L2_PAIR/TR_X1_XLA_1i: P?.25 (P25)
- new net L2_PAIR/TR_X1_XLA_1o: P?.20 (P20)
- new net L2_PAIR/TR_X1_XLA_2i: P?.26 (P26)
- new net L2_PAIR/TR_X1_XLA_2o: P?.19 (P19)
- new net L2_PAIR/TR_X1_XLA_3i: P?.27 (P27)
- new net L2_PAIR/TR_X1_XLA_3o: P?.18 (P18)
- new net L2_PAIR/TR_X1_XLA_4i: P?.28 (P28)
- new net L2_PAIR/TR_X1_XLA_4o: P?.17 (P17)
- new net L2_PAIR/T_X0_XLB_0i: P?.21 (P21)
- new net L2_PAIR/T_X0_XLB_0o: P?.10 (P10)
- new net L2_PAIR/T_X0_XLB_1i: P?.20 (P20)
- new net L2_PAIR/T_X0_XLB_1o: P?.11 (P11)
- new net L2_PAIR/T_X0_XLB_2i: P?.19 (P19)
- new net L2_PAIR/T_X0_XLB_2o: P?.12 (P12)
- new net L2_PAIR/T_X0_XLB_3i: P?.18 (P18)
- new net L2_PAIR/T_X0_XLB_3o: P?.13 (P13)
- new net L2_PAIR/T_X0_XLB_4i: P?.17 (P17)
- new net L2_PAIR/T_X0_XLB_4o: P?.14 (P14)
Other:
- note added: "SWITCH FOR JTAG BOARD CONFIG"
- note added: "TL- POS = 1\nML- POS = 8\nBL- POS = 5\nMI- POS = C\nRI- POS = 7"
- moved on the sheet: R?, U?
