File: l2_dev_clean/l2_dev_board.sch (KiCad schematic (older format))
At the start: 55 parts

Commit message: added L1 links and JTAG signals. I think a mux can buffer...
Connections:
- net L1_TDO_Q3 is gone; now on net L1_TDI_R: U?.3 (A)
- net L1_TDO_Q4 is gone; now on net L1_TDI_B: U?.3 (A)
- net L2_PAIR/BL_X0_XLA_0i is gone; now on net L2_PAIR/BL_X0_XLA_0i: P?.7 (P7)
- net L2_PAIR/BL_X0_XLA_0o is gone; now on net L2_PAIR/BL_X0_XLA_0o: P?.10 (P10)
- net L2_PAIR/BL_X0_XLA_1i is gone; now on net L2_PAIR/BL_X0_XLA_1i: P?.6 (P6)
- net L2_PAIR/BL_X0_XLA_1o is gone; now on net L2_PAIR/BL_X0_XLA_1o: P?.11 (P11)
- net L2_PAIR/BL_X0_XLA_2i is gone; now on net L2_PAIR/BL_X0_XLA_2i: P?.5 (P5)
- net L2_PAIR/BL_X0_XLA_2o is gone; now on net L2_PAIR/BL_X0_XLA_2o: P?.12 (P12)
- net L2_PAIR/BL_X0_XLA_3i is gone; now on net L2_PAIR/BL_X0_XLA_3i: P?.4 (P4)
- net L2_PAIR/BL_X0_XLA_3o is gone; now on net L2_PAIR/BL_X0_XLA_3o: P?.13 (P13)
- net L2_PAIR/BL_X0_XLA_4i is gone; now on net L2_PAIR/BL_X0_XLA_4i: P?.3 (P3)
- net L2_PAIR/BL_X0_XLA_4o is gone; now on net L2_PAIR/BL_X0_XLA_4o: P?.14 (P14)
- net L2_PAIR/BR_X1_XLA_0i is gone; now on net L2_PAIR/BR_X1_XLA_0i: P?.9 (P9)
- net L2_PAIR/BR_X1_XLA_0o is gone; now on net L2_PAIR/BR_X1_XLA_0o: P?.6 (P6)
- net L2_PAIR/BR_X1_XLA_1i is gone; now on net L2_PAIR/BR_X1_XLA_1i: P?.10 (P10)
- net L2_PAIR/BR_X1_XLA_1o is gone; now on net L2_PAIR/BR_X1_XLA_1o: P?.5 (P5)
- net L2_PAIR/BR_X1_XLA_2i is gone; now on net L2_PAIR/BR_X1_XLA_2i: P?.11 (P11)
- net L2_PAIR/BR_X1_XLA_2o is gone; now on net L2_PAIR/BR_X1_XLA_2o: P?.4 (P4)
- net L2_PAIR/BR_X1_XLA_3i is gone; now on net L2_PAIR/BR_X1_XLA_3i: P?.2 (P2)
- net L2_PAIR/BR_X1_XLA_3o is gone; now on net L2_PAIR/BR_X1_XLA_3o: P?.3 (P3)
- net L2_PAIR/BR_X1_XLA_4i is gone; now on net L2_PAIR/BR_X1_XLA_4i: P?.3 (P3)
- net L2_PAIR/BR_X1_XLA_4o is gone; now on net L2_PAIR/BR_X1_XLA_4o: P?.2 (P2)
- net L2_PAIR/B_X1_XLB_0i is gone; now on net L2_PAIR/B_X1_XLB_0i: P?.7 (P7)
- net L2_PAIR/B_X1_XLB_0o is gone; now on net L2_PAIR/B_X1_XLB_0o: P?.24 (P24)
- net L2_PAIR/B_X1_XLB_1i is gone; now on net L2_PAIR/B_X1_XLB_1i: P?.6 (P6)
- net L2_PAIR/B_X1_XLB_1o is gone; now on net L2_PAIR/B_X1_XLB_1o: P?.25 (P25)
- net L2_PAIR/B_X1_XLB_2i is gone; now on net L2_PAIR/B_X1_XLB_2i: P?.5 (P5)
- net L2_PAIR/B_X1_XLB_2o is gone; now on net L2_PAIR/B_X1_XLB_2o: P?.26 (P26)
- net L2_PAIR/B_X1_XLB_3i is gone; now on net L2_PAIR/B_X1_XLB_3i: P?.4 (P4)
- net L2_PAIR/B_X1_XLB_3o is gone; now on net L2_PAIR/B_X1_XLB_3o: P?.27 (P27)
- net L2_PAIR/B_X1_XLB_4i is gone; now on net L2_PAIR/B_X1_XLB_4i: P?.3 (P3)
- net L2_PAIR/B_X1_XLB_4o is gone; now on net L2_PAIR/B_X1_XLB_4o: P?.28 (P28)
- net L2_PAIR/TL_X0_XLA_0i is gone; now on net L2_PAIR/TL_X0_XLA_0i: P?.21 (P21)
- net L2_PAIR/TL_X0_XLA_0o is gone; now on net L2_PAIR/TL_X0_XLA_0o: P?.24 (P24)
- net L2_PAIR/TL_X0_XLA_1i is gone; now on net L2_PAIR/TL_X0_XLA_1i: P?.20 (P20)
- net L2_PAIR/TL_X0_XLA_1o is gone; now on net L2_PAIR/TL_X0_XLA_1o: P?.25 (P25)
- net L2_PAIR/TL_X0_XLA_2i is gone; now on net L2_PAIR/TL_X0_XLA_2i: P?.19 (P19)
- net L2_PAIR/TL_X0_XLA_2o is gone; now on net L2_PAIR/TL_X0_XLA_2o: P?.26 (P26)
- net L2_PAIR/TL_X0_XLA_3i is gone; now on net L2_PAIR/TL_X0_XLA_3i: P?.18 (P18)
- net L2_PAIR/TL_X0_XLA_3o is gone; now on net L2_PAIR/TL_X0_XLA_3o: P?.27 (P27)
- net L2_PAIR/TL_X0_XLA_4i is gone; now on net L2_PAIR/TL_X0_XLA_4i: P?.17 (P17)
- net L2_PAIR/TL_X0_XLA_4o is gone; now on net L2_PAIR/TL_X0_XLA_4o: P?.28 (P28)
- net L2_PAIR/TR_X1_XLA_0i is gone; now on net L2_PAIR/TR_X1_XLA_0i: P?.13 (P13)
- net L2_PAIR/TR_X1_XLA_0o is gone; now on net L2_PAIR/TR_X1_XLA_0o: P?.10 (P10)
- net L2_PAIR/TR_X1_XLA_1i is gone; now on net L2_PAIR/TR_X1_XLA_1i: P?.14 (P14)
- net L2_PAIR/TR_X1_XLA_1o is gone; now on net L2_PAIR/TR_X1_XLA_1o: P?.9 (P9)
- net L2_PAIR/TR_X1_XLA_2i is gone; now on net L2_PAIR/TR_X1_XLA_2i: P?.15 (P15)
- net L2_PAIR/TR_X1_XLA_2o is gone; now on net L2_PAIR/TR_X1_XLA_2o: P?.8 (P8)
- net L2_PAIR/TR_X1_XLA_3i is gone; now on net L2_PAIR/TR_X1_XLA_3i: P?.16 (P16)
- net L2_PAIR/TR_X1_XLA_3o is gone; now on net L2_PAIR/TR_X1_XLA_3o: P?.7 (P7)
- net L2_PAIR/TR_X1_XLA_4i is gone; now on net L2_PAIR/TR_X1_XLA_4i: P?.17 (P17)
- net L2_PAIR/TR_X1_XLA_4o is gone; now on net L2_PAIR/TR_X1_XLA_4o: P?.6 (P6)
- net L2_PAIR/T_X0_XLB_0i is gone; now on net L2_PAIR/T_X0_XLB_0i: P?.7 (P7)
- net L2_PAIR/T_X0_XLB_0o is gone; now on net L2_PAIR/T_X0_XLB_0o: P?.24 (P24)
- net L2_PAIR/T_X0_XLB_1i is gone; now on net L2_PAIR/T_X0_XLB_1i: P?.6 (P6)
- net L2_PAIR/T_X0_XLB_1o is gone; now on net L2_PAIR/T_X0_XLB_1o: P?.25 (P25)
- net L2_PAIR/T_X0_XLB_2i is gone; now on net L2_PAIR/T_X0_XLB_2i: P?.5 (P5)
- net L2_PAIR/T_X0_XLB_2o is gone; now on net L2_PAIR/T_X0_XLB_2o: P?.26 (P26)
- net L2_PAIR/T_X0_XLB_3i is gone; now on net L2_PAIR/T_X0_XLB_3i: P?.4 (P4)
- net L2_PAIR/T_X0_XLB_3o is gone; now on net L2_PAIR/T_X0_XLB_3o: P?.27 (P27)
- net L2_PAIR/T_X0_XLB_4i is gone; now on net L2_PAIR/T_X0_XLB_4i: P?.3 (P3)
- net L2_PAIR/T_X0_XLB_4o is gone; now on net L2_PAIR/T_X0_XLB_4o: P?.28 (P28)
- net L1_TDI_B: now also U?.4 (Y1)
- net L1_TDI_L: now also U?.4 (Y1)
- net L1_TDI_R: now also U?.4 (Y1)
- net L1_TDI_T: now also U?.4 (Y1)
- net L1_TDO_B: now also U?.6 (Y0)
- net L1_TDO_L: now also U?.6 (Y0)
- net L1_TDO_R: now also U?.6 (Y0)
- net L1_TDO_T: now also U?.6 (Y0)
- net L2_PAIR/BR_X1_XLA_0i: no longer P?.10 (P10)
- net L2_PAIR/BR_X1_XLA_0o: no longer P?.7 (P7)
- net L2_PAIR/BR_X1_XLA_1i: no longer P?.11 (P11)
- net L2_PAIR/BR_X1_XLA_1o: no longer P?.6 (P6)
- net L2_PAIR/BR_X1_XLA_2i: no longer P?.12 (P12)
- net L2_PAIR/BR_X1_XLA_2o: no longer P?.5 (P5)
- net L2_PAIR/BR_X1_XLA_3i: no longer P?.13 (P13)
- net L2_PAIR/BR_X1_XLA_3o: no longer P?.4 (P4)
- net L2_PAIR/BR_X1_XLA_4i: no longer P?.14 (P14)
- net L2_PAIR/BR_X1_XLA_4o: no longer P?.3 (P3)
- net L2_PAIR/TR_X1_XLA_0i: no longer P?.24 (P24)
- net L2_PAIR/TR_X1_XLA_0o: no longer P?.21 (P21)
- net L2_PAIR/TR_X1_XLA_1i: no longer P?.25 (P25)
- net L2_PAIR/TR_X1_XLA_1o: no longer P?.20 (P20)
- net L2_PAIR/TR_X1_XLA_2i: no longer P?.26 (P26)
- net L2_PAIR/TR_X1_XLA_2o: no longer P?.19 (P19)
- net L2_PAIR/TR_X1_XLA_3i: no longer P?.27 (P27)
- net L2_PAIR/TR_X1_XLA_3o: no longer P?.18 (P18)
- net L2_PAIR/TR_X1_XLA_4i: no longer P?.28 (P28)
- net L2_PAIR/TR_X1_XLA_4o: no longer P?.17 (P17)
- net L2_PAIR/T_X0_XLB_0i: no longer P?.21 (P21)
- net L2_PAIR/T_X0_XLB_0o: no longer P?.10 (P10)
- net L2_PAIR/T_X0_XLB_1i: no longer P?.20 (P20)
- net L2_PAIR/T_X0_XLB_1o: no longer P?.11 (P11)
- net L2_PAIR/T_X0_XLB_2i: no longer P?.19 (P19)
- net L2_PAIR/T_X0_XLB_2o: no longer P?.12 (P12)
- net L2_PAIR/T_X0_XLB_3i: no longer P?.18 (P18)
- net L2_PAIR/T_X0_XLB_3o: no longer P?.13 (P13)
- net L2_PAIR/T_X0_XLB_4i: no longer P?.17 (P17)
- net L2_PAIR/T_X0_XLB_4o: no longer P?.14 (P14)
- net TDI_B: now also U?.4 (Y1)
- net TDI_L: now also U?.4 (Y1)
- net TDI_R: now also U?.4 (Y1)
- net TDI_T: now also U?.4 (Y1)
- net TDO_B: now also U?.6 (Y0)
- net TDO_L: now also U?.6 (Y0)
- net TDO_R: now also U?.6 (Y0)
- net TDO_T: now also U?.6 (Y0)
- new net L2_PAIR/BR_X1_XLA_0i: P?.10 (P10)
- new net L2_PAIR/BR_X1_XLA_0o: P?.7 (P7)
- new net L2_PAIR/BR_X1_XLA_1i: P?.11 (P11)
- new net L2_PAIR/BR_X1_XLA_1o: P?.6 (P6)
- new net L2_PAIR/BR_X1_XLA_2i: P?.12 (P12)
- new net L2_PAIR/BR_X1_XLA_2o: P?.5 (P5)
- new net L2_PAIR/BR_X1_XLA_3i: P?.13 (P13)
- new net L2_PAIR/BR_X1_XLA_3o: P?.4 (P4)
- new net L2_PAIR/BR_X1_XLA_4i: P?.14 (P14)
- new net L2_PAIR/BR_X1_XLA_4o: P?.3 (P3)
- new net L2_PAIR/TR_X1_XLA_0i: P?.24 (P24)
- new net L2_PAIR/TR_X1_XLA_0o: P?.21 (P21)
- new net L2_PAIR/TR_X1_XLA_1i: P?.25 (P25)
- new net L2_PAIR/TR_X1_XLA_1o: P?.20 (P20)
- new net L2_PAIR/TR_X1_XLA_2i: P?.26 (P26)
- new net L2_PAIR/TR_X1_XLA_2o: P?.19 (P19)
- new net L2_PAIR/TR_X1_XLA_3i: P?.27 (P27)
- new net L2_PAIR/TR_X1_XLA_3o: P?.18 (P18)
- new net L2_PAIR/TR_X1_XLA_4i: P?.28 (P28)
- new net L2_PAIR/TR_X1_XLA_4o: P?.17 (P17)
- new net L2_PAIR/T_X0_XLB_0i: P?.21 (P21)
- new net L2_PAIR/T_X0_XLB_0o: P?.10 (P10)
- new net L2_PAIR/T_X0_XLB_1i: P?.20 (P20)
- new net L2_PAIR/T_X0_XLB_1o: P?.11 (P11)
- new net L2_PAIR/T_X0_XLB_2i: P?.19 (P19)
- new net L2_PAIR/T_X0_XLB_2o: P?.12 (P12)
- new net L2_PAIR/T_X0_XLB_3i: P?.18 (P18)
- new net L2_PAIR/T_X0_XLB_3o: P?.13 (P13)
- new net L2_PAIR/T_X0_XLB_4i: P?.17 (P17)
- new net L2_PAIR/T_X0_XLB_4o: P?.14 (P14)
Other:
- note added: "JTAG SIGNAL BUFFERS"
- note added: "L1 MODULE"
- note removed: "JTAG SINGNAL BUFFERS"
- moved on the sheet: U?

Commit message: just need adc and done...hopefully
Parts:
- gave numbers to parts that had none: 55
Connections:
- net DEBUG_N_BUF is gone; now on net DEBUG_N_B: U118.6 (Y1)
- net DEBUG_N_R is gone; now on net DEBUG_N_B: P108.25 (P25)
- net L1_DEBUG_N_BUF is gone; now on net L1_DEBUG_N_B: U120.4 (Y2)
- net L1_DEBUG_N_R is gone; now on net L1_DEBUG_N_B: P109.25 (P25)
- net L1_RST_N_BUF is gone; now on net L1_RST_N_B: U121.4 (Y2)
- net L1_RST_N_R is gone; now on net L1_RST_N_B: P109.23 (P23)
- net L1_TCK_BUF is gone; now on net L1_TCK_B: U122.6 (Y1)
- net L1_TCK_R is gone; now on net L1_TCK_B: P109.22 (P22)
- net L1_TMS_BUF is gone; now on net L1_TMS_B: U122.4 (Y2)
- net L1_TMS_R is gone; now on net L1_TMS_B: P109.20 (P20)
- net L1_TRST_N_BUF is gone; now on net L1_TRST_N_B: U121.6 (Y1)
- net L1_TRST_N_R is gone; now on net L1_TRST_N_B: P109.24 (P24)
- net RST_N_BUF is gone; now on net RST_N_B: U119.6 (Y1)
- net RST_N_R is gone; now on net RST_N_B: P108.23 (P23)
- net TCK_BUF is gone; now on net TCK_B: U119.4 (Y2)
- net TCK_R is gone; now on net TCK_B: P108.21 (P21)
- net TMS_BUF is gone; now on net TMS_B: U120.6 (Y1)
- net TMS_R is gone; now on net TMS_B: P108.19 (P19)
- net TMS_TOP is gone; now on net TMS_T: P104.2 (P2)
- net TRST_N_BUF is gone; now on net TRST_N_B: U118.4 (Y2)
- net TRST_N_R is gone; now on net TRST_N_B: P108.24 (P24)
- net L2_PAIR/BL_X0_XLA_0i renamed L2_PAIR_Q1/BL_X0_XLA_0i
- net L2_PAIR/BL_X0_XLA_0i renamed L2_PAIR_Q4/BL_X0_XLA_0i
- net L2_PAIR/BL_X0_XLA_0o renamed L2_PAIR_Q1/BL_X0_XLA_0o
- net L2_PAIR/BL_X0_XLA_0o renamed L2_PAIR_Q4/BL_X0_XLA_0o
- net L2_PAIR/BL_X0_XLA_1i renamed L2_PAIR_Q1/BL_X0_XLA_1i
- net L2_PAIR/BL_X0_XLA_1i renamed L2_PAIR_Q4/BL_X0_XLA_1i
- net L2_PAIR/BL_X0_XLA_1o renamed L2_PAIR_Q1/BL_X0_XLA_1o
- net L2_PAIR/BL_X0_XLA_1o renamed L2_PAIR_Q4/BL_X0_XLA_1o
- net L2_PAIR/BL_X0_XLA_2i renamed L2_PAIR_Q1/BL_X0_XLA_2i
- net L2_PAIR/BL_X0_XLA_2i renamed L2_PAIR_Q4/BL_X0_XLA_2i
- net L2_PAIR/BL_X0_XLA_2o renamed L2_PAIR_Q1/BL_X0_XLA_2o
- net L2_PAIR/BL_X0_XLA_2o renamed L2_PAIR_Q4/BL_X0_XLA_2o
- net L2_PAIR/BL_X0_XLA_3i renamed L2_PAIR_Q1/BL_X0_XLA_3i
- net L2_PAIR/BL_X0_XLA_3i renamed L2_PAIR_Q4/BL_X0_XLA_3i
- net L2_PAIR/BL_X0_XLA_3o renamed L2_PAIR_Q1/BL_X0_XLA_3o
- net L2_PAIR/BL_X0_XLA_3o renamed L2_PAIR_Q4/BL_X0_XLA_3o
- net L2_PAIR/BL_X0_XLA_4i renamed L2_PAIR_Q1/BL_X0_XLA_4i
- net L2_PAIR/BL_X0_XLA_4i renamed L2_PAIR_Q4/BL_X0_XLA_4i
- net L2_PAIR/BL_X0_XLA_4o renamed L2_PAIR_Q1/BL_X0_XLA_4o
- net L2_PAIR/BL_X0_XLA_4o renamed L2_PAIR_Q4/BL_X0_XLA_4o
- net L2_PAIR/BR_X1_XLA_0i renamed L2_PAIR_Q3/BR_X1_XLA_0i
- net L2_PAIR/BR_X1_XLA_0i renamed L2_PAIR_Q2/BR_X1_XLA_0i
- net L2_PAIR/BR_X1_XLA_0o renamed L2_PAIR_Q3/BR_X1_XLA_0o
- net L2_PAIR/BR_X1_XLA_0o renamed L2_PAIR_Q2/BR_X1_XLA_0o
- net L2_PAIR/BR_X1_XLA_1i renamed L2_PAIR_Q3/BR_X1_XLA_1i
- net L2_PAIR/BR_X1_XLA_1i renamed L2_PAIR_Q2/BR_X1_XLA_1i
- net L2_PAIR/BR_X1_XLA_1o renamed L2_PAIR_Q3/BR_X1_XLA_1o
- net L2_PAIR/BR_X1_XLA_1o renamed L2_PAIR_Q2/BR_X1_XLA_1o
- net L2_PAIR/BR_X1_XLA_2i renamed L2_PAIR_Q3/BR_X1_XLA_2i
- net L2_PAIR/BR_X1_XLA_2i renamed L2_PAIR_Q2/BR_X1_XLA_2i
- net L2_PAIR/BR_X1_XLA_2o renamed L2_PAIR_Q3/BR_X1_XLA_2o
- net L2_PAIR/BR_X1_XLA_2o renamed L2_PAIR_Q2/BR_X1_XLA_2o
- net L2_PAIR/BR_X1_XLA_3i renamed L2_PAIR_Q3/BR_X1_XLA_3i
- net L2_PAIR/BR_X1_XLA_3i renamed L2_PAIR_Q2/BR_X1_XLA_3i
- net L2_PAIR/BR_X1_XLA_3o renamed L2_PAIR_Q3/BR_X1_XLA_3o
- net L2_PAIR/BR_X1_XLA_3o renamed L2_PAIR_Q2/BR_X1_XLA_3o
- net L2_PAIR/BR_X1_XLA_4i renamed L2_PAIR_Q3/BR_X1_XLA_4i
- net L2_PAIR/BR_X1_XLA_4i renamed L2_PAIR_Q2/BR_X1_XLA_4i
- net L2_PAIR/BR_X1_XLA_4o renamed L2_PAIR_Q3/BR_X1_XLA_4o
- net L2_PAIR/BR_X1_XLA_4o renamed L2_PAIR_Q2/BR_X1_XLA_4o
- net L2_PAIR/B_X1_XLB_0i renamed L2_PAIR_Q3/B_X1_XLB_0i
- net L2_PAIR/B_X1_XLB_0i renamed L2_PAIR_Q4/B_X1_XLB_0i
- net L2_PAIR/B_X1_XLB_0o renamed L2_PAIR_Q4/B_X1_XLB_0o
- net L2_PAIR/B_X1_XLB_0o renamed L2_PAIR_Q3/B_X1_XLB_0o
- net L2_PAIR/B_X1_XLB_1i renamed L2_PAIR_Q3/B_X1_XLB_1i
- net L2_PAIR/B_X1_XLB_1i renamed L2_PAIR_Q4/B_X1_XLB_1i
- net L2_PAIR/B_X1_XLB_1o renamed L2_PAIR_Q4/B_X1_XLB_1o
- net L2_PAIR/B_X1_XLB_1o renamed L2_PAIR_Q3/B_X1_XLB_1o
- net L2_PAIR/B_X1_XLB_2i renamed L2_PAIR_Q3/B_X1_XLB_2i
- net L2_PAIR/B_X1_XLB_2i renamed L2_PAIR_Q4/B_X1_XLB_2i
- net L2_PAIR/B_X1_XLB_2o renamed L2_PAIR_Q4/B_X1_XLB_2o
- net L2_PAIR/B_X1_XLB_2o renamed L2_PAIR_Q3/B_X1_XLB_2o
- net L2_PAIR/B_X1_XLB_3i renamed L2_PAIR_Q3/B_X1_XLB_3i
- net L2_PAIR/B_X1_XLB_3i renamed L2_PAIR_Q4/B_X1_XLB_3i
- net L2_PAIR/B_X1_XLB_3o renamed L2_PAIR_Q4/B_X1_XLB_3o
- net L2_PAIR/B_X1_XLB_3o renamed L2_PAIR_Q3/B_X1_XLB_3o
- net L2_PAIR/B_X1_XLB_4i renamed L2_PAIR_Q3/B_X1_XLB_4i
- net L2_PAIR/B_X1_XLB_4i renamed L2_PAIR_Q4/B_X1_XLB_4i
- net L2_PAIR/B_X1_XLB_4o renamed L2_PAIR_Q4/B_X1_XLB_4o
- net L2_PAIR/B_X1_XLB_4o renamed L2_PAIR_Q3/B_X1_XLB_4o
- net L2_PAIR/TL_X0_XLA_0i renamed L2_PAIR_Q1/TL_X0_XLA_0i
- net L2_PAIR/TL_X0_XLA_0i renamed L2_PAIR_Q4/TL_X0_XLA_0i
- net L2_PAIR/TL_X0_XLA_0o renamed L2_PAIR_Q1/TL_X0_XLA_0o
- net L2_PAIR/TL_X0_XLA_0o renamed L2_PAIR_Q4/TL_X0_XLA_0o
- net L2_PAIR/TL_X0_XLA_1i renamed L2_PAIR_Q1/TL_X0_XLA_1i
- net L2_PAIR/TL_X0_XLA_1i renamed L2_PAIR_Q4/TL_X0_XLA_1i
- net L2_PAIR/TL_X0_XLA_1o renamed L2_PAIR_Q1/TL_X0_XLA_1o
- net L2_PAIR/TL_X0_XLA_1o renamed L2_PAIR_Q4/TL_X0_XLA_1o
- net L2_PAIR/TL_X0_XLA_2i renamed L2_PAIR_Q1/TL_X0_XLA_2i
- net L2_PAIR/TL_X0_XLA_2i renamed L2_PAIR_Q4/TL_X0_XLA_2i
- net L2_PAIR/TL_X0_XLA_2o renamed L2_PAIR_Q1/TL_X0_XLA_2o
- net L2_PAIR/TL_X0_XLA_2o renamed L2_PAIR_Q4/TL_X0_XLA_2o
- net L2_PAIR/TL_X0_XLA_3i renamed L2_PAIR_Q1/TL_X0_XLA_3i
- net L2_PAIR/TL_X0_XLA_3i renamed L2_PAIR_Q4/TL_X0_XLA_3i
- net L2_PAIR/TL_X0_XLA_3o renamed L2_PAIR_Q1/TL_X0_XLA_3o
- net L2_PAIR/TL_X0_XLA_3o renamed L2_PAIR_Q4/TL_X0_XLA_3o
- net L2_PAIR/TL_X0_XLA_4i renamed L2_PAIR_Q1/TL_X0_XLA_4i
- net L2_PAIR/TL_X0_XLA_4i renamed L2_PAIR_Q4/TL_X0_XLA_4i
- net L2_PAIR/TL_X0_XLA_4o renamed L2_PAIR_Q1/TL_X0_XLA_4o
- net L2_PAIR/TL_X0_XLA_4o renamed L2_PAIR_Q4/TL_X0_XLA_4o
- net L2_PAIR/TR_X1_XLA_0i renamed L2_PAIR_Q3/TR_X1_XLA_0i
- net L2_PAIR/TR_X1_XLA_0i renamed L2_PAIR_Q2/TR_X1_XLA_0i
- net L2_PAIR/TR_X1_XLA_0o renamed L2_PAIR_Q3/TR_X1_XLA_0o
- net L2_PAIR/TR_X1_XLA_0o renamed L2_PAIR_Q2/TR_X1_XLA_0o
- net L2_PAIR/TR_X1_XLA_1i renamed L2_PAIR_Q3/TR_X1_XLA_1i
- net L2_PAIR/TR_X1_XLA_1i renamed L2_PAIR_Q2/TR_X1_XLA_1i
- net L2_PAIR/TR_X1_XLA_1o renamed L2_PAIR_Q3/TR_X1_XLA_1o
- net L2_PAIR/TR_X1_XLA_1o renamed L2_PAIR_Q2/TR_X1_XLA_1o
- net L2_PAIR/TR_X1_XLA_2i renamed L2_PAIR_Q3/TR_X1_XLA_2i
- net L2_PAIR/TR_X1_XLA_2i renamed L2_PAIR_Q2/TR_X1_XLA_2i
- net L2_PAIR/TR_X1_XLA_2o renamed L2_PAIR_Q3/TR_X1_XLA_2o
- net L2_PAIR/TR_X1_XLA_2o renamed L2_PAIR_Q2/TR_X1_XLA_2o
- net L2_PAIR/TR_X1_XLA_3i renamed L2_PAIR_Q3/TR_X1_XLA_3i
- net L2_PAIR/TR_X1_XLA_3i renamed L2_PAIR_Q2/TR_X1_XLA_3i
- net L2_PAIR/TR_X1_XLA_3o renamed L2_PAIR_Q3/TR_X1_XLA_3o
- net L2_PAIR/TR_X1_XLA_3o renamed L2_PAIR_Q2/TR_X1_XLA_3o
- net L2_PAIR/TR_X1_XLA_4i renamed L2_PAIR_Q3/TR_X1_XLA_4i
- net L2_PAIR/TR_X1_XLA_4i renamed L2_PAIR_Q2/TR_X1_XLA_4i
- net L2_PAIR/TR_X1_XLA_4o renamed L2_PAIR_Q3/TR_X1_XLA_4o
- net L2_PAIR/TR_X1_XLA_4o renamed L2_PAIR_Q2/TR_X1_XLA_4o
- net L2_PAIR/T_X0_XLB_0i renamed L2_PAIR_Q2/T_X0_XLB_0i
- net L2_PAIR/T_X0_XLB_0i renamed L2_PAIR_Q1/T_X0_XLB_0i
- net L2_PAIR/T_X0_XLB_0o renamed L2_PAIR_Q1/T_X0_XLB_0o
- net L2_PAIR/T_X0_XLB_0o renamed L2_PAIR_Q2/T_X0_XLB_0o
- net L2_PAIR/T_X0_XLB_1i renamed L2_PAIR_Q2/T_X0_XLB_1i
- net L2_PAIR/T_X0_XLB_1i renamed L2_PAIR_Q1/T_X0_XLB_1i
- net L2_PAIR/T_X0_XLB_1o renamed L2_PAIR_Q1/T_X0_XLB_1o
- net L2_PAIR/T_X0_XLB_1o renamed L2_PAIR_Q2/T_X0_XLB_1o
- net L2_PAIR/T_X0_XLB_2i renamed L2_PAIR_Q2/T_X0_XLB_2i
- net L2_PAIR/T_X0_XLB_2i renamed L2_PAIR_Q1/T_X0_XLB_2i
- net L2_PAIR/T_X0_XLB_2o renamed L2_PAIR_Q1/T_X0_XLB_2o
- net L2_PAIR/T_X0_XLB_2o renamed L2_PAIR_Q2/T_X0_XLB_2o
- net L2_PAIR/T_X0_XLB_3i renamed L2_PAIR_Q2/T_X0_XLB_3i
- net L2_PAIR/T_X0_XLB_3i renamed L2_PAIR_Q1/T_X0_XLB_3i
- net L2_PAIR/T_X0_XLB_3o renamed L2_PAIR_Q1/T_X0_XLB_3o
- net L2_PAIR/T_X0_XLB_3o renamed L2_PAIR_Q2/T_X0_XLB_3o
- net L2_PAIR/T_X0_XLB_4i renamed L2_PAIR_Q2/T_X0_XLB_4i
- net L2_PAIR/T_X0_XLB_4i renamed L2_PAIR_Q1/T_X0_XLB_4i
- net L2_PAIR/T_X0_XLB_4o renamed L2_PAIR_Q1/T_X0_XLB_4o
- net L2_PAIR/T_X0_XLB_4o renamed L2_PAIR_Q2/T_X0_XLB_4o
Other:
- note added: "JTAG SPLIT B+R"
- note added: "KiCad ERC FIX"
- moved on the sheet: P101, P102, P103, P104, P105, P106, P107, P108, P109, P110, R112, R113

Commit message: Laying out things. This is tedious work!
Parts:
- added C108: 0.1uF, symbol C
- added U123: ASE_CLK, symbol ASE_CLK
- C104: value 22uF -> 47uF
- L101: value 6.8uH -> 2.2uH
- R102: value 40.2k -> 11.5k
Connections:
- net +3.3V: now also C108.1, U123.1 (EN), U123.4 (VDD)
- net GND: now also C108.2, U123.2 (GND)
- new net 20M_CLK: U123.3 (OUTPUT)
Other:
- note added: "GLOBAL 20MHz CLK GENERATION"
