File: l2_dev_clean/l2_dev_board.sch (KiCad schematic (older format))
At the start: 57 parts, among them P101 CONN_30, P102 CONN_30, P103 CONN_30, P104 CONN_30, P105 CONN_30, P106 CONN_30, P107 CONN_30, P108 CONN_30, P109 CONN_30, P110 CONN_30, U101 APX803-SR, U102 NC7SZ157, U103 A6RS-161RF, U104 SN74LVC1G18, U105 SN74LVC1G18, U106 SN74LVC1G18, U107 SN74LVC1G18, U108 SN74CBTD3861, U109 LT3480, U110 APX803-SR, U111 74AHC1GU04, U112 SN74LVC1G18, U113 SN74LVC1G18, U114 SN74LVC1G18, U115 SN74LVC1G18, U116 SN74CBTD3861, U117 NCP1529, U118 NC7WZ17, U119 NC7WZ17, U120 NC7WZ17, U121 NC7WZ17, U122 NC7WZ17, U123 ASE_CLK

Commit message: If you don't want power sensing you can make the board smaller! added the JTAG signals with buffers
Connections:
- net L1_TRST_N: no longer U108.16 (B7), U116.21 (B2)
- net MSEL_N: now also U108.21 (B2), U116.16 (B7)
- net TRST_N: no longer U108.21 (B2), U116.16 (B7)
- new net L1_MSEL_N: U108.16 (B7), U116.21 (B2)

Commit message: started buffers for DEBUG signal
Parts:
- added U? (x2): NC7WZ17, symbol NC7WZ17
Connections:
- net +3.3V: now also U?.5 (VCC), U?.5 (VCC)
- net GND: now also U?.2 (GND), U?.2 (GND)
- net L1_MSEL_N: now also U121.1 (A1)
- net L1_TRST_N: no longer U121.1 (A1)
- net MSEL_N: now also U118.3 (A2)
- net TRST_N: no longer U118.3 (A2)
Other:
- moved on the sheet: C108, U123

Commit message: added extra buffers to remove lengthy lines. Also looking and audio board for L1 layout!
Parts:
- removed U? (x2): NC7WZ17, symbol NC7WZ17
- added U124, U125, U131: NC7WZ07, symbol NC7WZ07
- added U126, U127, U128, U129, U130: NC7WZ17, symbol NC7WZ17
Connections:
- net +3.3V: now also U124.5 (VCC), U125.5 (VCC), U126.5 (VCC), U127.5 (VCC), U128.5 (VCC), U129.5 (VCC), U130.5 (VCC), U131.5 (VCC)
- net DEBUG_N: now also U120.1 (A1), U124.1 (A1), U124.3 (A2), U125.1 (A1), U125.3 (A2), U126.1 (A1); no longer U118.1 (A1)
- net GND: now also U124.2 (GND), U125.2 (GND), U126.2 (GND), U127.2 (GND), U128.2 (GND), U129.2 (GND), U130.2 (GND), U131.2 (GND)
- net L1_DEBUG_N: now also U122.3 (A2), U128.3 (A2), U131.1 (A1); no longer U120.3 (A2)
- net L1_MSEL_N: now also U122.1 (A1), U129.1 (A1); no longer U121.1 (A1)
- net L1_RST_N: now also U129.3 (A2)
- net L1_TCK: now also U121.1 (A1), U130.1 (A1); no longer U122.1 (A1)
- net L1_TMS: now also U130.3 (A2), U131.3 (A2); no longer U122.3 (A2)
- net MSEL_N: now also U119.3 (A2), U126.3 (A2); no longer U118.3 (A2)
- net RST_N: now also U127.1 (A1)
- net TCK: now also U118.3 (A2), U127.3 (A2); no longer U119.3 (A2)
- net TMS: now also U118.1 (A1), U128.1 (A1); no longer U120.1 (A1)
- removed net DEBUG_N_B: P105.23 (P23), P108.6 (P6), U118.6 (Y1)
- removed net L1_DEBUG_N_B: P105.15 (P15), P109.17 (P17), U120.4 (Y2)
- net L1_RST_N_B renamed L1_RST_N_BUF_R
- net L1_RST_N_BUF_R: no longer P105.17 (P17)
- removed net L1_TCK_B: P105.19 (P19), P109.20 (P20), U122.6 (Y1)
- removed net L1_TMS_B: P105.21 (P21), P109.22 (P22), U122.4 (Y2)
- removed net L1_TRST_N_B: P105.16 (P16), P109.18 (P18), U121.6 (Y1)
- net RST_N_B renamed RST_N_BUF_R
- net RST_N_BUF_R: no longer P105.25 (P25)
- removed net TCK_B: P105.27 (P27), P108.10 (P10), U119.4 (Y2)
- removed net TMS_B: P105.29 (P29), P108.12 (P12), U120.6 (Y1)
- removed net TRST_N_B: P105.24 (P24), P108.7 (P7), U118.4 (Y2)
- new net DEBUG_N_BUF_B: P105.23 (P23), U126.6 (Y1)
- new net DEBUG_N_BUF_R: P108.6 (P6), U120.6 (Y1)
- new net DEBUG_N_Q1: U124.6 (Y1)
- new net DEBUG_N_Q2: U124.4 (Y2)
- new net DEBUG_N_Q3: U125.6 (Y1)
- new net DEBUG_N_Q4: U125.4 (Y2)
- new net L1_DEBUG_N_BUF: U131.6 (Y1)
- new net L1_DEBUG_N_BUF_B: P105.15 (P15), U128.4 (Y2)
- new net L1_DEBUG_N_BUF_R: P109.17 (P17), U122.4 (Y2)
- new net L1_RST_N_BUF_B: P105.17 (P17), U129.4 (Y2)
- new net L1_TCK_BUF_B: P105.19 (P19), U130.6 (Y1)
- new net L1_TCK_BUF_R: P109.20 (P20), U121.6 (Y1)
- new net L1_TMS_BUF_B: P105.21 (P21), U130.4 (Y2)
- new net L1_TMS_BUF_R: P109.22 (P22), U131.4 (Y2)
- new net L1_TRST_N_BUF_B: P105.16 (P16), U129.6 (Y1)
- new net L1_TRST_N_BUF_R: P109.18 (P18), U122.6 (Y1)
- new net RST_N_BUF_B: P105.25 (P25), U127.6 (Y1)
- new net TCK_BUF_B: P105.27 (P27), U127.4 (Y2)
- new net TCK_BUF_R: P108.10 (P10), U118.4 (Y2)
- new net TMS_BUF_B: P105.29 (P29), U128.6 (Y1)
- new net TMS_BUF_R: P108.12 (P12), U118.6 (Y1)
- new net TRST_N_BUF_B: P105.24 (P24), U126.4 (Y2)
- new net TRST_N_BUF_R: P108.7 (P7), U119.4 (Y2)
Other:
- note removed: "JTAG SPLIT B+R"
