File: l2_dev_clean/l2_pair.sch (KiCad schematic (older format))
At the start: 11 parts

Commit message: Schematics back to previous progress but with better layout and heirarchial structure. Also created switch and rotary dip layout.
Other:
- note added: "5V to 1V @ 1A"
- note removed: "5V to 1V 1A Regulator"
Changed lines of the file:
@@
-EESchema Schematic File Version 2  date 01/08/2011 00:22:28
+EESchema Schematic File Version 2  date 01/08/2011 18:10:28
 LIBS:power
 LIBS:device
@@
 LIBS:valves
 LIBS:xmos_custom_library
+LIBS:XS1-L1-128
 LIBS:l2_dev_board-cache
 EELAYER 25  0
@@
 $Descr A4 11700 8267
 encoding utf-8
-Sheet 2 4
+Sheet 8 14
 Title ""
-Date "31 jul 2011"
+Date "1 aug 2011"
 Rev ""
 Comp ""
@@
 U 1 1 4E35DB88
 P 2890 3300
+AR Path="/4E32CDCE/4E35DB88" Ref="#PWR?"  Part="1"
+AR Path="/4E36B740/4E35DB88" Ref="#PWR?"  Part="1"
 F 0 "#PWR?" H 2890 3260 30  0001 C CNN
 F 1 "+3.3V" H 2890 3410 30  0000 C CNN
@@
 U 1 1 4E35DB40
 P 2710 3550
+AR Path="/4E32CDCE/4E35DB40" Ref="R?"  Part="1"
+AR Path="/4E36B740/4E35DB40" Ref="R?"  Part="1"
 F 0 "R?" V 2790 3550 50  0000 C CNN
 F 1 "10k" V 2710 3550 50  0000 C CNN
@@
 U 1 1 4E35DB38
 P 2530 3550
+AR Path="/4E32CDCE/4E35DB38" Ref="R?"  Part="1"
+AR Path="/4E36B740/4E35DB38" Ref="R?"  Part="1"
 F 0 "R?" V 2610 3550 50  0000 C CNN
 F 1 "10k" V 2530 3550 50  0000 C CNN
@@
 U 1 1 4E35D9C0
 P 2340 4500
+AR Path="/4E32CDCE/4E35D9C0" Ref="#PWR?"  Part="1"
+AR Path="/4E36B740/4E35D9C0" Ref="#PWR?"  Part="1"
 F 0 "#PWR?" H 2340 4500 30  0001 C CNN
 F 1 "GND" H 2340 4430 30  0001 C CNN
@@
 U 1 1 4E35D9AA
 P 2340 3180
+AR Path="/4E32CDCE/4E35D9AA" Ref="#PWR?"  Part="1"
+AR Path="/4E36B740/4E35D9AA" Ref="#PWR?"  Part="1"
 F 0 "#PWR?" H 2340 3180 30  0001 C CNN
 F 1 "GND" H 2340 3110 30  0001 C CNN
@@
 U 1 1 4E35D9A0
 P 2340 3570
+AR Path="/4E32CDCE/4E35D9A0" Ref="#PWR?"  Part="1"
+AR Path="/4E36B740/4E35D9A0" Ref="#PWR?"  Part="1"
 F 0 "#PWR?" H 2340 3530 30  0001 C CNN
 F 1 "+3.3V" H 2340 3680 30  0000 C CNN
@@
 U 1 1 4E35D98B
 P 2340 2250
+AR Path="/4E32CDCE/4E35D98B" Ref="#PWR?"  Part="1"
+AR Path="/4E36B740/4E35D98B" Ref="#PWR?"  Part="1"
 F 0 "#PWR?" H 2340 2210 30  0001 C CNN
 F 1 "+3.3V" H 2340 2360 30  0000 C CNN
@@
 U 1 1 4E35D8BD
 P 1690 2730
+AR Path="/4E32CDCE/4E35D8BD" Ref="U?"  Part="1"
+AR Path="/4E36B740/4E35D8BD" Ref="U?"  Part="1"
 F 0 "U?" H 1390 3130 60  0000 C CNN
 F 1 "NC7WZ17" H 1540 2330 60  0000 C CNN
@@
 U 1 1 4E35D8B1
 P 1690 4050
+AR Path="/4E32CDCE/4E35D8B1" Ref="U?"  Part="1"
+AR Path="/4E36B740/4E35D8B1" Ref="U?"  Part="1"
 F 0 "U?" H 1390 4450 60  0000 C CNN
 F 1 "NC7WZ07" H 1540 3650 60  0000 C CNN
@@
 $EndComp
 Text Notes 1320 720  0    60   ~ 0
-5V to 1V 1A Regulator
+5V to 1V @ 1A
 Text Label 3880 830  1    60   ~ 0
 +1V0
@@
 U 1 1 4E35D6A2
 P 3800 1190
+AR Path="/4E32CDCE/4E35D6A2" Ref="C?"  Part="1"
+AR Path="/4E36B740/4E35D6A2" Ref="C?"  Part="1"
 F 0 "C?" H 3850 1290 50  0000 L CNN
 F 1 "10uF" H 3850 1090 50  0000 L CNN
@@
 U 1 1 4E35D649
 P 3500 1190
+AR Path="/4E32CDCE/4E35D649" Ref="C?"  Part="1"
+AR Path="/4E36B740/4E35D649" Ref="C?"  Part="1"
 F 0 "C?" H 3510 1290 50  0000 L CNN
 F 1 "33pF" H 3510 1100 50  0000 L CNN
@@
 U 1 1 4E35D5DA
 P 3230 1700
+AR Path="/4E32CDCE/4E35D5DA" Ref="R?"  Part="1"
+AR Path="/4E36B740/4E35D5DA" Ref="R?"  Part="1"
 F 0 "R?" V 3310 1700 50  0000 C CNN
 F 1 "100k" V 3230 1700 50  0000 C CNN
@@
 U 1 1 4E35D5C1
 P 3230 1170
+AR Path="/4E32CDCE/4E35D5C1" Ref="R?"  Part="1"
+AR Path="/4E36B740/4E35D5C1" Ref="R?"  Part="1"
 F 0 "R?" V 3310 1170 50  0000 C CNN
 F 1 "68k" V 3230 1170 50  0000 C CNN
@@
 U 1 1 4E35D5AC
 P 2840 920
+AR Path="/4E32CDCE/4E35D5AC" Ref="L?"  Part="1"
+AR Path="/4E36B740/4E35D5AC" Ref="L?"  Part="1"
 F 0 "L?" V 2790 920 40  0000 C CNN
 F 1 "INDUCTOR" V 2940 920 40  0000 C CNN
@@
 U 1 1 4E3545A6
 P 1740 1980
+AR Path="/4E32CDCE/4E3545A6" Ref="#PWR?"  Part="1"
+AR Path="/4E36B740/4E3545A6" Ref="#PWR?"  Part="1"
 F 0 "#PWR?" H 1740 1980 30  0001 C CNN
 F 1 "GND" H 1740 1910 30  0001 C CNN
@@
 U 1 1 4E354587
 P 690 1150
+AR Path="/4E32CDCE/4E354587" Ref="C?"  Part="1"
+AR Path="/4E36B740/4E354587" Ref="C?"  Part="1"
 F 0 "C?" H 740 1250 50  0000 L CNN
 F 1 "10uF" H 740 1050 50  0000 L CNN
@@
 U 1 1 4E35455A
 P 690 750
+AR Path="/4E32CDCE/4E35455A" Ref="#PWR?"  Part="1"
+AR Path="/4E36B740/4E35455A" Ref="#PWR?"  Part="1"
 F 0 "#PWR?" H 690 840 20  0001 C CNN
 F 1 "+5V" H 690 840 30  0000 C CNN
@@
 U 1 1 4E354532
 P 1740 1270
+AR Path="/4E32CDCE/4E354532" Ref="U?"  Part="1"
+AR Path="/4E36B740/4E354532" Ref="U?"  Part="1"
 F 0 "U?" H 1740 1220 60  0000 C CNN
 F 1 "NCP1529" H 1740 1320 60  0000 C CNN

Commit message: just need adc and done...hopefully
Parts:
- gave numbers to parts that had none: 11

Commit message: Laying out things. This is tedious work!
Parts:
- L201: value INDUCTOR -> 2u2H
Changed lines of the file:
@@
-EESchema Schematic File Version 2  date 03/08/2011 15:13:20
+EESchema Schematic File Version 2  date 08/08/2011 15:20:43
 LIBS:power
 LIBS:device
@@
 $Descr A4 11700 8267
 encoding utf-8
-Sheet 2 14
+Sheet 11 14
 Title ""
-Date "3 aug 2011"
+Date "8 aug 2011"
 Rev ""
 Comp ""
@@
 +1V0
 $Comp
-L +3.3V #PWR0163
+L +3.3V #PWR0166
 U 1 1 4E35DB88
 P 2890 3300
-AR Path="/4E36B777/4E35DB88" Ref="#PWR0163"  Part="1"
-AR Path="/4E36B760/4E35DB88" Ref="#PWR0180"  Part="1"
-AR Path="/4E36B740/4E35DB88" Ref="#PWR0197"  Part="1"
-AR Path="/4E32CDCE/4E35DB88" Ref="#PWR0214"  Part="1"
-F 0 "#PWR0214" H 2890 3260 30  0001 C CNN
+AR Path="/4E36B777/4E35DB88" Ref="#PWR0166"  Part="1"
+AR Path="/4E36B760/4E35DB88" Ref="#PWR0183"  Part="1"
+AR Path="/4E36B740/4E35DB88" Ref="#PWR0200"  Part="1"
+AR Path="/4E32CDCE/4E35DB88" Ref="#PWR0217"  Part="1"
+F 0 "#PWR0217" H 2890 3260 30  0001 C CNN
 F 1 "+3.3V" H 2890 3410 30  0000 C CNN
 	1    2890 3300
@@
 AR Path="/4E36B740/4E35DB40" Ref="R802"  Part="1"
 AR Path="/4E32CDCE/4E35DB40" Ref="R1102"  Part="1"
-F 0 "R202" V 2790 3550 50  0000 C CNN
+F 0 "R1102" V 2790 3550 50  0000 C CNN
 F 1 "10k" V 2710 3550 50  0000 C CNN
 	1    2710 3550
@@
 AR Path="/4E36B740/4E35DB38" Ref="R801"  Part="1"
 AR Path="/4E32CDCE/4E35DB38" Ref="R1101"  Part="1"
-F 0 "R201" V 2610 3550 50  0000 C CNN
+F 0 "R1101" V 2610 3550 50  0000 C CNN
 F 1 "10k" V 2530 3550 50  0000 C CNN
 	1    2530 3550
@@
 TCK
 $Comp
-L GND #PWR0164
+L GND #PWR0167
 U 1 1 4E35D9C0
 P 2340 4500
-AR Path="/4E36B777/4E35D9C0" Ref="#PWR0164"  Part="1"
-AR Path="/4E36B760/4E35D9C0" Ref="#PWR0181"  Part="1"
-AR Path="/4E36B740/4E35D9C0" Ref="#PWR0198"  Part="1"
-AR Path="/4E32CDCE/4E35D9C0" Ref="#PWR0215"  Part="1"
-F 0 "#PWR0215" H 2340 4500 30  0001 C CNN
+AR Path="/4E36B777/4E35D9C0" Ref="#PWR0167"  Part="1"
+AR Path="/4E36B760/4E35D9C0" Ref="#PWR0184"  Part="1"
+AR Path="/4E36B740/4E35D9C0" Ref="#PWR0201"  Part="1"
+AR Path="/4E32CDCE/4E35D9C0" Ref="#PWR0218"  Part="1"
+F 0 "#PWR0218" H 2340 4500 30  0001 C CNN
 F 1 "GND" H 2340 4430 30  0001 C CNN
 	1    2340 4500
@@
 $EndComp
 $Comp
-L GND #PWR0165
+L GND #PWR0168
 U 1 1 4E35D9AA
 P 2340 3180
-AR Path="/4E36B777/4E35D9AA" Ref="#PWR0165"  Part="1"
-AR Path="/4E36B760/4E35D9AA" Ref="#PWR0182"  Part="1"
-AR Path="/4E36B740/4E35D9AA" Ref="#PWR0199"  Part="1"
-AR Path="/4E32CDCE/4E35D9AA" Ref="#PWR0216"  Part="1"
-F 0 "#PWR0216" H 2340 3180 30  0001 C CNN
+AR Path="/4E36B777/4E35D9AA" Ref="#PWR0168"  Part="1"
+AR Path="/4E36B760/4E35D9AA" Ref="#PWR0185"  Part="1"
+AR Path="/4E36B740/4E35D9AA" Ref="#PWR0202"  Part="1"
+AR Path="/4E32CDCE/4E35D9AA" Ref="#PWR0219"  Part="1"
+F 0 "#PWR0219" H 2340 3180 30  0001 C CNN
 F 1 "GND" H 2340 3110 30  0001 C CNN
 	1    2340 3180
@@
 $EndComp
 $Comp
-L +3.3V #PWR0166
+L +3.3V #PWR0169
 U 1 1 4E35D9A0
 P 2340 3570
-AR Path="/4E36B777/4E35D9A0" Ref="#PWR0166"  Part="1"
-AR Path="/4E36B760/4E35D9A0" Ref="#PWR0183"  Part="1"
-AR Path="/4E36B740/4E35D9A0" Ref="#PWR0200"  Part="1"
-AR Path="/4E32CDCE/4E35D9A0" Ref="#PWR0217"  Part="1"
-F 0 "#PWR0217" H 2340 3530 30  0001 C CNN
+AR Path="/4E36B777/4E35D9A0" Ref="#PWR0169"  Part="1"
+AR Path="/4E36B760/4E35D9A0" Ref="#PWR0186"  Part="1"
+AR Path="/4E36B740/4E35D9A0" Ref="#PWR0203"  Part="1"
+AR Path="/4E32CDCE/4E35D9A0" Ref="#PWR0220"  Part="1"
+F 0 "#PWR0220" H 2340 3530 30  0001 C CNN
 F 1 "+3.3V" H 2340 3680 30  0000 C CNN
 	1    2340 3570
@@
 $EndComp
 $Comp
-L +3.3V #PWR0167
+L +3.3V #PWR0170
 U 1 1 4E35D98B
 P 2340 2250
-AR Path="/4E36B777/4E35D98B" Ref="#PWR0167"  Part="1"
-AR Path="/4E36B760/4E35D98B" Ref="#PWR0184"  Part="1"
-AR Path="/4E36B740/4E35D98B" Ref="#PWR0201"  Part="1"
-AR Path="/4E32CDCE/4E35D98B" Ref="#PWR0218"  Part="1"
-F 0 "#PWR0218" H 2340 2210 30  0001 C CNN
+AR Path="/4E36B777/4E35D98B" Ref="#PWR0170"  Part="1"
+AR Path="/4E36B760/4E35D98B" Ref="#PWR0187"  Part="1"
+AR Path="/4E36B740/4E35D98B" Ref="#PWR0204"  Part="1"
+AR Path="/4E32CDCE/4E35D98B" Ref="#PWR0221"  Part="1"
+F 0 "#PWR0221" H 2340 2210 30  0001 C CNN
 F 1 "+3.3V" H 2340 2360 30  0000 C CNN
 	1    2340 2250
@@
 AR Path="/4E36B740/4E35D8BD" Ref="U801"  Part="1"
 AR Path="/4E32CDCE/4E35D8BD" Ref="U1101"  Part="1"
-F 0 "U201" H 1390 3130 60  0000 C CNN
+F 0 "U1101" H 1390 3130 60  0000 C CNN
 F 1 "NC7WZ17" H 1540 2330 60  0000 C CNN
 	1    1690 2730
@@
 AR Path="/4E36B740/4E35D8B1" Ref="U802"  Part="1"
 AR Path="/4E32CDCE/4E35D8B1" Ref="U1102"  Part="1"
-F 0 "U202" H 1390 4450 60  0000 C CNN
+F 0 "U1102" H 1390 4450 60  0000 C CNN
 F 1 "NC7WZ07" H 1540 3650 60  0000 C CNN
 	1    1690 4050
@@
 AR Path="/4E36B740/4E35D6A2" Ref="C803"  Part="1"
 AR Path="/4E32CDCE/4E35D6A2" Ref="C1103"  Part="1"
-F 0 "C203" H 3850 1290 50  0000 L CNN
+F 0 "C1103" H 3850 1290 50  0000 L CNN
 F 1 "10uF" H 3850 1090 50  0000 L CNN
 	1    3800 1190
@@
 AR Path="/4E36B740/4E35D649" Ref="C802"  Part="1"
 AR Path="/4E32CDCE/4E35D649" Ref="C1102"  Part="1"
-F 0 "C202" H 3510 1290 50  0000 L CNN
+F 0 "C1102" H 3510 1290 50  0000 L CNN
 F 1 "33pF" H 3510 1100 50  0000 L CNN
 	1    3500 1190
@@
 AR Path="/4E36B740/4E35D5DA" Ref="R804"  Part="1"
 AR Path="/4E32CDCE/4E35D5DA" Ref="R1104"  Part="1"
-F 0 "R204" V 3310 1700 50  0000 C CNN
+F 0 "R1104" V 3310 1700 50  0000 C CNN
 F 1 "100k" V 3230 1700 50  0000 C CNN
 	1    3230 1700
@@
 AR Path="/4E36B740/4E35D5C1" Ref="R803"  Part="1"
 AR Path="/4E32CDCE/4E35D5C1" Ref="R1103"  Part="1"
-F 0 "R203" V 3310 1170 50  0000 C CNN
+F 0 "R1103" V 3310 1170 50  0000 C CNN
 F 1 "68k" V 3230 1170 50  0000 C CNN
 	1    3230 1170
@@
 AR Path="/4E36B740/4E35D5AC" Ref="L801"  Part="1"
 AR Path="/4E32CDCE/4E35D5AC" Ref="L1101"  Part="1"
-F 0 "L201" V 2790 920 40  0000 C CNN
-F 1 "INDUCTOR" V 2940 920 40  0000 C CNN
+F 0 "L1101" V 2790 920 40  0000 C CNN
+F 1 "2u2H" V 2940 920 40  0000 C CNN
 	1    2840 920
 	0    -1   -1   0
 $EndComp
 $Comp
-L GND #PWR0168
+L GND #PWR0171
 U 1 1 4E3545A6
 P 1740 1980
-AR Path="/4E36B777/4E3545A6" Ref="#PWR0168"  Part="1"
-AR Path="/4E36B760/4E3545A6" Ref="#PWR0185"  Part="1"
-AR Path="/4E36B740/4E3545A6" Ref="#PWR0202"  Part="1"
-AR Path="/4E32CDCE/4E3545A6" Ref="#PWR0219"  Part="1"
-F 0 "#PWR0219" H 1740 1980 30  0001 C CNN
+AR Path="/4E36B777/4E3545A6" Ref="#PWR0171"  Part="1"
+AR Path="/4E36B760/4E3545A6" Ref="#PWR0188"  Part="1"
+AR Path="/4E36B740/4E3545A6" Ref="#PWR0205"  Part="1"
+AR Path="/4E32CDCE/4E3545A6" Ref="#PWR0222"  Part="1"
+F 0 "#PWR0222" H 1740 1980 30  0001 C CNN
 F 1 "GND" H 1740 1910 30  0001 C CNN
 	1    1740 1980
@@
 AR Path="/4E36B740/4E354587" Ref="C801"  Part="1"
 AR Path="/4E32CDCE/4E354587" Ref="C1101"  Part="1"
-F 0 "C201" H 740 1250 50  0000 L CNN
+F 0 "C1101" H 740 1250 50  0000 L CNN
 F 1 "10uF" H 740 1050 50  0000 L CNN
 	1    690  1150
@@
 $EndComp
 $Comp
-L +5V #PWR0169
+L +5V #PWR0172
 U 1 1 4E35455A
 P 690 750
-AR Path="/4E36B777/4E35455A" Ref="#PWR0169"  Part="1"
-AR Path="/4E36B760/4E35455A" Ref="#PWR0186"  Part="1"
-AR Path="/4E36B740/4E35455A" Ref="#PWR0203"  Part="1"
-AR Path="/4E32CDCE/4E35455A" Ref="#PWR0220"  Part="1"
-F 0 "#PWR0220" H 690 840 20  0001 C CNN
+AR Path="/4E36B777/4E35455A" Ref="#PWR0172"  Part="1"
+AR Path="/4E36B760/4E35455A" Ref="#PWR0189"  Part="1"
+AR Path="/4E36B740/4E35455A" Ref="#PWR0206"  Part="1"
+AR Path="/4E32CDCE/4E35455A" Ref="#PWR0223"  Part="1"
+F 0 "#PWR0223" H 690 840 20  0001 C CNN
 F 1 "+5V" H 690 840 30  0000 C CNN
 	1    690  750
@@
 AR Path="/4E36B740/4E354532" Ref="U803"  Part="1"
 AR Path="/4E32CDCE/4E354532" Ref="U1103"  Part="1"
-F 0 "U203" H 1740 1220 60  0000 C CNN
+F 0 "U1103" H 1740 1220 60  0000 C CNN
 F 1 "NCP1529" H 1740 1320 60  0000 C CNN
 	1    1740 1270
