File: l2_dev_clean/l2_pair.sch (KiCad schematic (older format))
At the start: 11 parts, among them U201 NC7WZ17, U202 NC7WZ07, U203 NCP1529

Commit message: added extra buffers to remove lengthy lines. Also looking and audio board for L1 layout!
Changed lines of the file:
@@
-EESchema Schematic File Version 2  date Tue 16 Aug 2011 19:18:59 BST
+EESchema Schematic File Version 2  date 17/08/2011 16:55:33
 LIBS:power
 LIBS:device
@@
 Sheet 2 14
 Title ""
-Date "16 aug 2011"
+Date "17 aug 2011"
 Rev ""
 Comp ""
@@
 +1V0
 $Comp
-L +3.3V #PWR0183
+L +3.3V #PWR0199
 U 1 1 4E35DB88
 P 2890 3300
-AR Path="/4E36B777/4E35DB88" Ref="#PWR0183"  Part="1"
-AR Path="/4E36B760/4E35DB88" Ref="#PWR0200"  Part="1"
-AR Path="/4E36B740/4E35DB88" Ref="#PWR0217"  Part="1"
-AR Path="/4E32CDCE/4E35DB88" Ref="#PWR0166"  Part="1"
-F 0 "#PWR0217" H 2890 3260 30  0001 C CNN
+AR Path="/4E36B777/4E35DB88" Ref="#PWR0199"  Part="1"
+AR Path="/4E36B760/4E35DB88" Ref="#PWR0216"  Part="1"
+AR Path="/4E36B740/4E35DB88" Ref="#PWR0233"  Part="1"
+AR Path="/4E32CDCE/4E35DB88" Ref="#PWR0182"  Part="1"
+F 0 "#PWR0233" H 2890 3260 30  0001 C CNN
 F 1 "+3.3V" H 2890 3410 30  0000 C CNN
 	1    2890 3300
@@
 AR Path="/4E36B740/4E35DB40" Ref="R802"  Part="1"
 AR Path="/4E32CDCE/4E35DB40" Ref="R1102"  Part="1"
-F 0 "R1102" V 2790 3550 50  0000 C CNN
+F 0 "R802" V 2790 3550 50  0000 C CNN
 F 1 "10k" V 2710 3550 50  0000 C CNN
 	1    2710 3550
@@
 AR Path="/4E36B740/4E35DB38" Ref="R801"  Part="1"
 AR Path="/4E32CDCE/4E35DB38" Ref="R1101"  Part="1"
-F 0 "R1101" V 2610 3550 50  0000 C CNN
+F 0 "R801" V 2610 3550 50  0000 C CNN
 F 1 "10k" V 2530 3550 50  0000 C CNN
 	1    2530 3550
@@
 TCK
 $Comp
-L GND #PWR0184
+L GND #PWR0200
 U 1 1 4E35D9C0
 P 2340 4500
-AR Path="/4E36B777/4E35D9C0" Ref="#PWR0184"  Part="1"
-AR Path="/4E36B760/4E35D9C0" Ref="#PWR0201"  Part="1"
-AR Path="/4E36B740/4E35D9C0" Ref="#PWR0218"  Part="1"
-AR Path="/4E32CDCE/4E35D9C0" Ref="#PWR0167"  Part="1"
-F 0 "#PWR0218" H 2340 4500 30  0001 C CNN
+AR Path="/4E36B777/4E35D9C0" Ref="#PWR0200"  Part="1"
+AR Path="/4E36B760/4E35D9C0" Ref="#PWR0217"  Part="1"
+AR Path="/4E36B740/4E35D9C0" Ref="#PWR0234"  Part="1"
+AR Path="/4E32CDCE/4E35D9C0" Ref="#PWR0183"  Part="1"
+F 0 "#PWR0234" H 2340 4500 30  0001 C CNN
 F 1 "GND" H 2340 4430 30  0001 C CNN
 	1    2340 4500
@@
 $EndComp
 $Comp
-L GND #PWR0185
+L GND #PWR0201
 U 1 1 4E35D9AA
 P 2340 3180
-AR Path="/4E36B777/4E35D9AA" Ref="#PWR0185"  Part="1"
-AR Path="/4E36B760/4E35D9AA" Ref="#PWR0202"  Part="1"
-AR Path="/4E36B740/4E35D9AA" Ref="#PWR0219"  Part="1"
-AR Path="/4E32CDCE/4E35D9AA" Ref="#PWR0168"  Part="1"
-F 0 "#PWR0219" H 2340 3180 30  0001 C CNN
+AR Path="/4E36B777/4E35D9AA" Ref="#PWR0201"  Part="1"
+AR Path="/4E36B760/4E35D9AA" Ref="#PWR0218"  Part="1"
+AR Path="/4E36B740/4E35D9AA" Ref="#PWR0235"  Part="1"
+AR Path="/4E32CDCE/4E35D9AA" Ref="#PWR0184"  Part="1"
+F 0 "#PWR0235" H 2340 3180 30  0001 C CNN
 F 1 "GND" H 2340 3110 30  0001 C CNN
 	1    2340 3180
@@
 $EndComp
 $Comp
-L +3.3V #PWR0186
+L +3.3V #PWR0202
 U 1 1 4E35D9A0
 P 2340 3570
-AR Path="/4E36B777/4E35D9A0" Ref="#PWR0186"  Part="1"
-AR Path="/4E36B760/4E35D9A0" Ref="#PWR0203"  Part="1"
-AR Path="/4E36B740/4E35D9A0" Ref="#PWR0220"  Part="1"
-AR Path="/4E32CDCE/4E35D9A0" Ref="#PWR0169"  Part="1"
-F 0 "#PWR0220" H 2340 3530 30  0001 C CNN
+AR Path="/4E36B777/4E35D9A0" Ref="#PWR0202"  Part="1"
+AR Path="/4E36B760/4E35D9A0" Ref="#PWR0219"  Part="1"
+AR Path="/4E36B740/4E35D9A0" Ref="#PWR0236"  Part="1"
+AR Path="/4E32CDCE/4E35D9A0" Ref="#PWR0185"  Part="1"
+F 0 "#PWR0236" H 2340 3530 30  0001 C CNN
 F 1 "+3.3V" H 2340 3680 30  0000 C CNN
 	1    2340 3570
@@
 $EndComp
 $Comp
-L +3.3V #PWR0187
+L +3.3V #PWR0203
 U 1 1 4E35D98B
 P 2340 2250
-AR Path="/4E36B777/4E35D98B" Ref="#PWR0187"  Part="1"
-AR Path="/4E36B760/4E35D98B" Ref="#PWR0204"  Part="1"
-AR Path="/4E36B740/4E35D98B" Ref="#PWR0221"  Part="1"
-AR Path="/4E32CDCE/4E35D98B" Ref="#PWR0170"  Part="1"
-F 0 "#PWR0221" H 2340 2210 30  0001 C CNN
+AR Path="/4E36B777/4E35D98B" Ref="#PWR0203"  Part="1"
+AR Path="/4E36B760/4E35D98B" Ref="#PWR0220"  Part="1"
+AR Path="/4E36B740/4E35D98B" Ref="#PWR0237"  Part="1"
+AR Path="/4E32CDCE/4E35D98B" Ref="#PWR0186"  Part="1"
+F 0 "#PWR0237" H 2340 2210 30  0001 C CNN
 F 1 "+3.3V" H 2340 2360 30  0000 C CNN
 	1    2340 2250
@@
 AR Path="/4E36B740/4E35D8BD" Ref="U801"  Part="1"
 AR Path="/4E32CDCE/4E35D8BD" Ref="U1101"  Part="1"
-F 0 "U1101" H 1390 3130 60  0000 C CNN
+F 0 "U801" H 1390 3130 60  0000 C CNN
 F 1 "NC7WZ17" H 1540 2330 60  0000 C CNN
 	1    1690 2730
@@
 AR Path="/4E36B740/4E35D8B1" Ref="U802"  Part="1"
 AR Path="/4E32CDCE/4E35D8B1" Ref="U1102"  Part="1"
-F 0 "U1102" H 1390 4450 60  0000 C CNN
+F 0 "U802" H 1390 4450 60  0000 C CNN
 F 1 "NC7WZ07" H 1540 3650 60  0000 C CNN
 	1    1690 4050
@@
 AR Path="/4E36B740/4E35D6A2" Ref="C803"  Part="1"
 AR Path="/4E32CDCE/4E35D6A2" Ref="C1103"  Part="1"
-F 0 "C1103" H 3850 1290 50  0000 L CNN
+F 0 "C803" H 3850 1290 50  0000 L CNN
 F 1 "10uF" H 3850 1090 50  0000 L CNN
 	1    3800 1190
@@
 AR Path="/4E36B740/4E35D649" Ref="C802"  Part="1"
 AR Path="/4E32CDCE/4E35D649" Ref="C1102"  Part="1"
-F 0 "C1102" H 3510 1290 50  0000 L CNN
+F 0 "C802" H 3510 1290 50  0000 L CNN
 F 1 "33pF" H 3510 1100 50  0000 L CNN
 	1    3500 1190
@@
 AR Path="/4E36B740/4E35D5DA" Ref="R804"  Part="1"
 AR Path="/4E32CDCE/4E35D5DA" Ref="R1104"  Part="1"
-F 0 "R1104" V 3310 1700 50  0000 C CNN
+F 0 "R804" V 3310 1700 50  0000 C CNN
 F 1 "100k" V 3230 1700 50  0000 C CNN
 	1    3230 1700
@@
 AR Path="/4E36B740/4E35D5C1" Ref="R803"  Part="1"
 AR Path="/4E32CDCE/4E35D5C1" Ref="R1103"  Part="1"
-F 0 "R1103" V 3310 1170 50  0000 C CNN
+F 0 "R803" V 3310 1170 50  0000 C CNN
 F 1 "68k" V 3230 1170 50  0000 C CNN
 	1    3230 1170
@@
 AR Path="/4E36B740/4E35D5AC" Ref="L801"  Part="1"
 AR Path="/4E32CDCE/4E35D5AC" Ref="L1101"  Part="1"
-F 0 "L1101" V 2790 920 40  0000 C CNN
+F 0 "L801" V 2790 920 40  0000 C CNN
 F 1 "2u2H" V 2940 920 40  0000 C CNN
 	1    2840 920
@@
 $EndComp
 $Comp
-L GND #PWR0188
+L GND #PWR0204
 U 1 1 4E3545A6
 P 1740 1980
-AR Path="/4E36B777/4E3545A6" Ref="#PWR0188"  Part="1"
-AR Path="/4E36B760/4E3545A6" Ref="#PWR0205"  Part="1"
-AR Path="/4E36B740/4E3545A6" Ref="#PWR0222"  Part="1"
-AR Path="/4E32CDCE/4E3545A6" Ref="#PWR0171"  Part="1"
-F 0 "#PWR0222" H 1740 1980 30  0001 C CNN
+AR Path="/4E36B777/4E3545A6" Ref="#PWR0204"  Part="1"
+AR Path="/4E36B760/4E3545A6" Ref="#PWR0221"  Part="1"
+AR Path="/4E36B740/4E3545A6" Ref="#PWR0238"  Part="1"
+AR Path="/4E32CDCE/4E3545A6" Ref="#PWR0187"  Part="1"
+F 0 "#PWR0238" H 1740 1980 30  0001 C CNN
 F 1 "GND" H 1740 1910 30  0001 C CNN
 	1    1740 1980
@@
 AR Path="/4E36B740/4E354587" Ref="C801"  Part="1"
 AR Path="/4E32CDCE/4E354587" Ref="C1101"  Part="1"
-F 0 "C1101" H 740 1250 50  0000 L CNN
+F 0 "C801" H 740 1250 50  0000 L CNN
 F 1 "10uF" H 740 1050 50  0000 L CNN
 	1    690  1150
@@
 $EndComp
 $Comp
-L +5V #PWR0189
+L +5V #PWR0205
 U 1 1 4E35455A
 P 690 750
-AR Path="/4E36B777/4E35455A" Ref="#PWR0189"  Part="1"
-AR Path="/4E36B760/4E35455A" Ref="#PWR0206"  Part="1"
-AR Path="/4E36B740/4E35455A" Ref="#PWR0223"  Part="1"
-AR Path="/4E32CDCE/4E35455A" Ref="#PWR0172"  Part="1"
-F 0 "#PWR0223" H 690 840 20  0001 C CNN
+AR Path="/4E36B777/4E35455A" Ref="#PWR0205"  Part="1"
+AR Path="/4E36B760/4E35455A" Ref="#PWR0222"  Part="1"
+AR Path="/4E36B740/4E35455A" Ref="#PWR0239"  Part="1"
+AR Path="/4E32CDCE/4E35455A" Ref="#PWR0188"  Part="1"
+F 0 "#PWR0239" H 690 840 20  0001 C CNN
 F 1 "+5V" H 690 840 30  0000 C CNN
 	1    690  750
@@
 AR Path="/4E36B740/4E354532" Ref="U803"  Part="1"
 AR Path="/4E32CDCE/4E354532" Ref="U1103"  Part="1"
-F 0 "U1103" H 1740 1220 60  0000 C CNN
+F 0 "U803" H 1740 1220 60  0000 C CNN
 F 1 "NCP1529" H 1740 1320 60  0000 C CNN
 	1    1740 1270
