File: l2_dev_alternative/l2_dev_board.sch (KiCad schematic (older format))
At the start: 70 parts, among them P101 CONN_30, P102 CONN_30, P103 CONN_30, P104 CONN_30, P105 CONN_30, P106 CONN_30, P107 CONN_30, P108 CONN_30, P109 CONN_30, P110 CONN_30, U101 APX803-SR, U102 NC7SZ157, U103 A6RS-161RF, U104 SN74LVC1G18, U105 SN74LVC1G18, U106 SN74LVC1G18, U107 SN74LVC1G18, U108 SN74CBTD3861, U109 LT3480, U110 APX803-SR, U111 74AHC1GU04, U112 SN74LVC1G18, U113 SN74LVC1G18, U114 SN74LVC1G18, U115 SN74LVC1G18, U116 SN74CBTD3861, U117 NCP1529, U118 NC7WZ17, U119 NC7WZ17, U120 NC7WZ17, U121 NC7WZ17, U122 NC7WZ17, U123 ASE_CLK, U124 NC7WZ07, U125 NC7WZ07, U126 NC7WZ17, U127 NC7WZ17, U128 NC7WZ17, U129 NC7WZ17, U130 NC7WZ17, U131 NC7WZ07, U132 INA219

Commit message: buffers are in and BOM started. Changed open drain buffers for normal buffers and added pull ups to the _N JTAG signals
Parts:
- removed U124, U125, U131: NC7WZ07, symbol NC7WZ07
- added R117, R118, R119, R120: 10k, symbol R
- added U124, U125, U131: NC7WZ17, symbol NC7WZ17
Connections:
- net TRST_N is gone; now on net MSEL_N: R112.2
- net +3.3V: now also R117.1, R118.1, R119.1, R120.1, U124.5 (VCC), U125.5 (VCC), U131.5 (VCC)
- net DEBUG_N: now also R117.2, U125.1 (A1), U125.3 (A2), U131.1 (A1), U131.3 (A2)
- net DEBUG_N_BUF_B: now also P107.23 (P23); no longer P105.23 (P23)
- net DEBUG_N_Q1: now also U125.6 (Y1)
- net DEBUG_N_Q2: now also U125.4 (Y2)
- net DEBUG_N_Q3: now also U131.6 (Y1)
- net DEBUG_N_Q4: now also U131.4 (Y2)
- net DEBUG_N_T: now also P106.8 (P8); no longer P104.8 (P8)
- net GND: now also P104.14 (P14), P104.15 (P15), P104.21 (P21), P104.22 (P22), P104.24 (P24), P104.26 (P26), P104.28 (P28), P104.30 (P30), P104.4 (P4), P104.7 (P7), P104.8 (P8), P105.1 (P1), P105.10 (P10), P105.16 (P16), P105.17 (P17), P105.23 (P23), P105.24 (P24), P105.27 (P27), P105.3 (P3), P105.5 (P5), P105.7 (P7), P105.9 (P9), P106.11 (P11), P106.13 (P13), P106.17 (P17), P106.24 (P24), P106.3 (P3), P106.5 (P5), P107.14 (P14), P107.18 (P18), P107.20 (P20), P107.26 (P26), P107.28 (P28), P107.7 (P7), U124.2 (GND), U125.2 (GND), U131.2 (GND); no longer P104.11 (P11), P104.13 (P13), P104.17 (P17), P104.20 (P20), P104.23 (P23), P104.25 (P25), P104.27 (P27), P104.29 (P29), P104.3 (P3), P104.5 (P5), P104.9 (P9), P105.11 (P11), P105.14 (P14), P105.18 (P18), P105.2 (P2), P105.20 (P20), P105.22 (P22), P105.26 (P26), P105.28 (P28), P105.4 (P4), P105.6 (P6), P105.8 (P8), P106.15 (P15), P106.16 (P16), P106.2 (P2), P106.22 (P22), P106.29 (P29), P106.8 (P8), P107.15 (P15), P107.16 (P16), P107.2 (P2), P107.23 (P23), P107.29 (P29), P107.9 (P9)
- net L1_DEBUG_N: now also R118.2, U124.1 (A1)
- net L1_DEBUG_N_BUF: now also U124.6 (Y1)
- net L1_DEBUG_N_BUF_B: now also P107.15 (P15); no longer P105.15 (P15)
- net L1_DEBUG_N_T: now also P106.16 (P16); no longer P104.16 (P16)
- net L1_MSEL_N: now also R120.2
- net L1_RST_N: now also R119.2
- net L1_RST_N_BUF_B: now also P107.17 (P17); no longer P105.17 (P17)
- net L1_RST_N_T: now also P106.14 (P14); no longer P104.14 (P14)
- net L1_TCK_BUF_B: now also P107.19 (P19); no longer P105.19 (P19)
- net L1_TCK_T: now also P106.12 (P12); no longer P104.12 (P12)
- net L1_TDI_B: now also P105.2 (P2); no longer P105.1 (P1)
- net L1_TDI_T: now also P104.27 (P27); no longer P104.28 (P28)
- net L1_TDO_B: now also P105.4 (P4); no longer P105.3 (P3)
- net L1_TDO_T: now also P104.29 (P29); no longer P104.30 (P30)
- net L1_TMS: now also U124.3 (A2)
- net L1_TMS_BUF_B: now also P107.21 (P21); no longer P105.21 (P21)
- net L1_TMS_BUF_R: now also U124.4 (Y2)
- net L1_TMS_T: now also P106.10 (P10); no longer P104.10 (P10)
- net L1_TRST_N_BUF_B: now also P107.16 (P16); no longer P105.16 (P16)
- net L1_TRST_N_T: now also P106.15 (P15); no longer P104.15 (P15)
- net L1_XLINK_0i_B: now also P105.26 (P26); no longer P105.9 (P9)
- net L1_XLINK_0i_T: now also P104.3 (P3); no longer P104.19 (P19)
- net L1_XLINK_0o_B: now also P105.28 (P28); no longer P105.13 (P13)
- net L1_XLINK_0o_T: now also P104.5 (P5); no longer P104.21 (P21)
- net L1_XLINK_1i_B: now also P105.25 (P25); no longer P105.10 (P10)
- net L1_XLINK_1i_T: now also P104.2 (P2); no longer P104.18 (P18)
- net L1_XLINK_1o_B: now also P105.29 (P29); no longer P105.12 (P12)
- net L1_XLINK_1o_T: now also P104.6 (P6); no longer P104.22 (P22)
- net L2_PAIR_Q1/T_X0_XLB_0i: now also P104.13 (P13); no longer P106.7 (P7)
- net L2_PAIR_Q1/T_X0_XLB_0o: now also P104.16 (P16); no longer P106.10 (P10)
- net L2_PAIR_Q1/T_X0_XLB_1i: now also P104.12 (P12); no longer P106.6 (P6)
- net L2_PAIR_Q1/T_X0_XLB_1o: now also P104.17 (P17); no longer P106.11 (P11)
- net L2_PAIR_Q1/T_X0_XLB_2i: now also P104.11 (P11); no longer P106.5 (P5)
- net L2_PAIR_Q1/T_X0_XLB_2o: now also P104.18 (P18); no longer P106.12 (P12)
- net L2_PAIR_Q1/T_X0_XLB_3i: now also P104.10 (P10); no longer P106.4 (P4)
- net L2_PAIR_Q1/T_X0_XLB_3o: now also P104.19 (P19); no longer P106.13 (P13)
- net L2_PAIR_Q1/T_X0_XLB_4i: now also P104.9 (P9); no longer P106.3 (P3)
- net L2_PAIR_Q1/T_X0_XLB_4o: now also P104.20 (P20); no longer P106.14 (P14)
- net L2_PAIR_Q2/T_X0_XLB_0i: now also P106.22 (P22); no longer P106.21 (P21)
- net L2_PAIR_Q2/T_X0_XLB_0o: now also P106.25 (P25); no longer P106.24 (P24)
- net L2_PAIR_Q2/T_X0_XLB_1i: now also P106.21 (P21); no longer P106.20 (P20)
- net L2_PAIR_Q2/T_X0_XLB_1o: now also P106.26 (P26); no longer P106.25 (P25)
- net L2_PAIR_Q2/T_X0_XLB_2i: now also P106.20 (P20); no longer P106.19 (P19)
- net L2_PAIR_Q2/T_X0_XLB_2o: now also P106.27 (P27); no longer P106.26 (P26)
- net L2_PAIR_Q2/T_X0_XLB_3i: now also P106.19 (P19); no longer P106.18 (P18)
- net L2_PAIR_Q2/T_X0_XLB_3o: now also P106.28 (P28); no longer P106.27 (P27)
- net L2_PAIR_Q2/T_X0_XLB_4i: now also P106.18 (P18); no longer P106.17 (P17)
- net L2_PAIR_Q2/T_X0_XLB_4o: now also P106.29 (P29); no longer P106.28 (P28)
- net L2_PAIR_Q3/B_X1_XLB_0i: now also P107.6 (P6); no longer P107.7 (P7)
- net L2_PAIR_Q3/B_X1_XLB_0o: now also P107.9 (P9); no longer P107.10 (P10)
- net L2_PAIR_Q3/B_X1_XLB_1i: now also P107.5 (P5); no longer P107.6 (P6)
- net L2_PAIR_Q3/B_X1_XLB_1o: now also P107.10 (P10); no longer P107.11 (P11)
- net L2_PAIR_Q3/B_X1_XLB_2i: now also P107.4 (P4); no longer P107.5 (P5)
- net L2_PAIR_Q3/B_X1_XLB_2o: now also P107.11 (P11); no longer P107.12 (P12)
- net L2_PAIR_Q3/B_X1_XLB_3i: now also P107.3 (P3); no longer P107.4 (P4)
- net L2_PAIR_Q3/B_X1_XLB_3o: now also P107.12 (P12); no longer P107.13 (P13)
- net L2_PAIR_Q3/B_X1_XLB_4i: now also P107.2 (P2); no longer P107.3 (P3)
- net L2_PAIR_Q3/B_X1_XLB_4o: now also P107.13 (P13); no longer P107.14 (P14)
- net L2_PAIR_Q4/B_X1_XLB_0i: now also P105.15 (P15); no longer P107.21 (P21)
- net L2_PAIR_Q4/B_X1_XLB_0o: now also P105.18 (P18); no longer P107.24 (P24)
- net L2_PAIR_Q4/B_X1_XLB_1i: now also P105.14 (P14); no longer P107.20 (P20)
- net L2_PAIR_Q4/B_X1_XLB_1o: now also P105.19 (P19); no longer P107.25 (P25)
- net L2_PAIR_Q4/B_X1_XLB_2i: now also P105.13 (P13); no longer P107.19 (P19)
- net L2_PAIR_Q4/B_X1_XLB_2o: now also P105.20 (P20); no longer P107.26 (P26)
- net L2_PAIR_Q4/B_X1_XLB_3i: now also P105.12 (P12); no longer P107.18 (P18)
- net L2_PAIR_Q4/B_X1_XLB_3o: now also P105.21 (P21); no longer P107.27 (P27)
- net L2_PAIR_Q4/B_X1_XLB_4i: now also P105.11 (P11); no longer P107.17 (P17)
- net L2_PAIR_Q4/B_X1_XLB_4o: now also P105.22 (P22); no longer P107.28 (P28)
- net RST_N_BUF_B: now also P107.25 (P25); no longer P105.25 (P25)
- net RST_N_T: now also P106.6 (P6); no longer P104.6 (P6)
- net TCK_BUF_B: now also P107.27 (P27); no longer P105.27 (P27)
- net TCK_T: now also P106.4 (P4); no longer P104.4 (P4)
- net TDI_B: now also P105.6 (P6); no longer P105.5 (P5)
- net TDI_T: now also P104.23 (P23); no longer P104.24 (P24)
- net TDO_B: now also P105.8 (P8); no longer P105.7 (P7)
- net TDO_T: now also P104.25 (P25); no longer P104.26 (P26)
- net TMS_BUF_B: now also P107.29 (P29); no longer P105.29 (P29)
- net TMS_T: now also P106.2 (P2); no longer P104.2 (P2)
- net TRST_N_BUF_B: now also P107.24 (P24); no longer P105.24 (P24)
- net TRST_N_T: now also P106.7 (P7); no longer P104.7 (P7)
Other:
- note added: "\n"
- note removed: "RST_N AND\nTRST_N\n\nPULL UPS"
