File: l2_dev_alternative/l2_dev_board.sch (KiCad schematic (older format))
At the start: 74 parts, among them P101 CONN_30, P102 CONN_30, P103 CONN_30, P104 CONN_30, P105 CONN_30, P106 CONN_30, P107 CONN_30, P108 CONN_30, P109 CONN_30, P110 CONN_30, U101 APX803-SR, U102 NC7SZ157, U103 A6RS-161RF, U104 SN74LVC1G18, U105 SN74LVC1G18, U106 SN74LVC1G18, U107 SN74LVC1G18, U108 SN74CBTD3861, U109 LT3480, U110 APX803-SR, U111 74AHC1GU04, U112 SN74LVC1G18, U113 SN74LVC1G18, U114 SN74LVC1G18, U115 SN74LVC1G18, U116 SN74CBTD3861, U117 NCP1529, U118 NC7WZ17, U119 NC7WZ17, U120 NC7WZ17, U121 NC7WZ17, U122 NC7WZ17, U123 ASE_CLK, U124 NC7WZ17, U125 NC7WZ17, U126 NC7WZ17, U127 NC7WZ17, U128 NC7WZ17, U129 NC7WZ17, U130 NC7WZ17, U131 NC7WZ17, U132 INA219

Commit message: Most of the components now in. About to try finalise the size!
Parts:
- added R121, R122, R123, R124, R125, R126, R127, R128, R129: 33R, symbol R
- added U133, U134: NB3N551, symbol NB3N551
Connections:
- net +3.3V: now also U133.7 (VDD), U134.7 (VDD)
- net DEBUG_N: now also U126.3 (A2); no longer U126.1 (A1)
- net DEBUG_N_BUF_B: now also U126.4 (Y2); no longer U126.6 (Y1)
- net DEBUG_N_Q1: now also U125.4 (Y2); no longer U125.6 (Y1)
- net DEBUG_N_Q2: now also U131.4 (Y2); no longer U125.4 (Y2)
- net DEBUG_N_Q4: now also U125.6 (Y1); no longer U131.4 (Y2)
- net GND: now also U133.6 (GND), U134.6 (GND)
- net L1_DEBUG_N: now also U122.1 (A1), U129.1 (A1); no longer U122.3 (A2), U128.3 (A2)
- net L1_DEBUG_N_BUF_B: now also U129.6 (Y1); no longer U128.4 (Y2)
- net L1_DEBUG_N_BUF_R: now also U122.6 (Y1); no longer U122.4 (Y2)
- net L1_MSEL_N: now also U122.3 (A2), U129.3 (A2); no longer U122.1 (A1), U129.1 (A1)
- net L1_RST_N: now also U121.1 (A1), U130.1 (A1); no longer U121.3 (A2), U129.3 (A2)
- net L1_RST_N_BUF_B: now also U130.6 (Y1); no longer U129.4 (Y2)
- net L1_RST_N_BUF_R: now also U121.6 (Y1); no longer U121.4 (Y2)
- net L1_TCK: now also U121.3 (A2), U130.3 (A2); no longer U121.1 (A1), U130.1 (A1)
- net L1_TCK_BUF_B: now also U130.4 (Y2); no longer U130.6 (Y1)
- net L1_TCK_BUF_R: now also U121.4 (Y2); no longer U121.6 (Y1)
- net L1_TMS: now also U126.1 (A1); no longer U130.3 (A2)
- net L1_TMS_BUF_B: now also U126.6 (Y1); no longer U130.4 (Y2)
- net L1_TRST_N_BUF_B: now also U129.4 (Y2); no longer U129.6 (Y1)
- net L1_TRST_N_BUF_R: now also U122.4 (Y2); no longer U122.6 (Y1)
- net MSEL_N: now also U119.1 (A1), U127.1 (A1); no longer U119.3 (A2), U126.3 (A2)
- net RST_N: now also U119.3 (A2), U127.3 (A2); no longer U119.1 (A1), U127.1 (A1)
- net RST_N_BUF_B: now also U127.4 (Y2); no longer U127.6 (Y1)
- net RST_N_BUF_R: now also U119.4 (Y2); no longer U119.6 (Y1)
- net TCK: now also U118.1 (A1), U128.1 (A1); no longer U118.3 (A2), U127.3 (A2)
- net TCK_BUF_B: now also U128.6 (Y1); no longer U127.4 (Y2)
- net TCK_BUF_R: now also U118.6 (Y1); no longer U118.4 (Y2)
- net TMS: now also U118.3 (A2), U128.3 (A2); no longer U118.1 (A1), U128.1 (A1)
- net TMS_BUF_B: now also U128.4 (Y2); no longer U128.6 (Y1)
- net TMS_BUF_R: now also U118.4 (Y2); no longer U118.6 (Y1)
- net TRST_N_BUF_B: now also U127.6 (Y1); no longer U126.4 (Y2)
- net TRST_N_BUF_R: now also U119.6 (Y1); no longer U119.4 (Y2)
- net 20M_CLK: no longer names the net of U123.3 (OUTPUT)
- net 20M_CLK: now also R121.2
- new net: R122.2, U133.2 (Q1)
- new net: R123.2, U133.3 (Q2)
- new net: R124.2, U133.4 (Q3)
- new net: R125.2, U133.5 (Q4)
- new net: R126.2, U134.2 (Q1)
- new net: R127.2, U134.3 (Q2)
- new net: R128.2, U134.4 (Q3)
- new net: R129.2, U134.5 (Q4)
- new net CLK_20M: U133.1 (ICLK), U134.1 (ICLK)
- new net CLK_20M_BUF_1: R122.1
- new net CLK_20M_BUF_2: R123.1
- new net CLK_20M_BUF_3: R124.1
- new net CLK_20M_BUF_4: R125.1
- new net CLK_20M_BUF_5: R126.1
- new net CLK_20M_BUF_6: R127.1
- new net CLK_20M_BUF_7: R128.1
- new net CLK_20M_BUF_8: R129.1
- no-connect marks 2 -> 4
Other:
- moved on the sheet: C108, U123, U124

Commit message: adding links, looking full in the middle!
Connections:
- net DEBUG_N_BUF_R: now also P108.20 (P20); no longer P108.6 (P6)
- net DEBUG_N_L: now also P101.11 (P11); no longer P101.25 (P25)
- net GND: now also P101.14 (P14), P101.16 (P16), P101.17 (P17), P101.23 (P23), P101.24 (P24), P101.6 (P6), P101.8 (P8), P108.14 (P14), P108.15 (P15), P108.17 (P17), P108.23 (P23), P108.25 (P25), P108.7 (P7), P108.8 (P8); no longer P101.11 (P11), P101.18 (P18), P101.20 (P20), P101.22 (P22), P101.26 (P26), P101.28 (P28), P101.5 (P5), P108.11 (P11), P108.13 (P13), P108.20 (P20), P108.26 (P26), P108.3 (P3), P108.5 (P5), P108.9 (P9)
- net L2_PAIR_Q1/TL_X0_XLA_0i: now also P101.22 (P22); no longer P101.10 (P10)
- net L2_PAIR_Q1/TL_X0_XLA_0o: now also P101.25 (P25); no longer P101.13 (P13)
- net L2_PAIR_Q1/TL_X0_XLA_1i: now also P101.21 (P21); no longer P101.9 (P9)
- net L2_PAIR_Q1/TL_X0_XLA_1o: now also P101.26 (P26); no longer P101.14 (P14)
- net L2_PAIR_Q1/TL_X0_XLA_2i: now also P101.20 (P20); no longer P101.8 (P8)
- net L2_PAIR_Q1/TL_X0_XLA_2o: now also P101.27 (P27); no longer P101.15 (P15)
- net L2_PAIR_Q1/TL_X0_XLA_3i: now also P101.19 (P19); no longer P101.7 (P7)
- net L2_PAIR_Q1/TL_X0_XLA_3o: now also P101.28 (P28); no longer P101.16 (P16)
- net L2_PAIR_Q1/TL_X0_XLA_4i: now also P101.18 (P18); no longer P101.6 (P6)
- net L2_PAIR_Q1/TL_X0_XLA_4o: now also P101.29 (P29); no longer P101.17 (P17)
- net L2_PAIR_Q2/TR_X1_XLA_0i: now also P108.6 (P6); no longer P108.18 (P18)
- net L2_PAIR_Q2/TR_X1_XLA_0o: now also P108.9 (P9); no longer P108.21 (P21)
- net L2_PAIR_Q2/TR_X1_XLA_1i: now also P108.5 (P5); no longer P108.17 (P17)
- net L2_PAIR_Q2/TR_X1_XLA_1o: now also P108.10 (P10); no longer P108.22 (P22)
- net L2_PAIR_Q2/TR_X1_XLA_2i: now also P108.4 (P4); no longer P108.16 (P16)
- net L2_PAIR_Q2/TR_X1_XLA_2o: now also P108.11 (P11); no longer P108.23 (P23)
- net L2_PAIR_Q2/TR_X1_XLA_3i: now also P108.3 (P3); no longer P108.15 (P15)
- net L2_PAIR_Q2/TR_X1_XLA_3o: now also P108.12 (P12); no longer P108.24 (P24)
- net L2_PAIR_Q2/TR_X1_XLA_4i: now also P108.2 (P2); no longer P108.14 (P14)
- net L2_PAIR_Q2/TR_X1_XLA_4o: now also P108.13 (P13); no longer P108.25 (P25)
- net RST_N_BUF_R: now also P108.22 (P22); no longer P108.8 (P8)
- net RST_N_L: now also P101.9 (P9); no longer P101.23 (P23)
- net TCK_BUF_R: now also P108.24 (P24); no longer P108.10 (P10)
- net TCK_L: now also P101.7 (P7); no longer P101.21 (P21)
- net TDI_L: now also P101.13 (P13); no longer P101.27 (P27)
- net TDI_R: now also P108.16 (P16); no longer P108.2 (P2)
- net TDO_L: now also P101.15 (P15); no longer P101.29 (P29)
- net TDO_R: now also P108.18 (P18); no longer P108.4 (P4)
- net TMS_BUF_R: now also P108.26 (P26); no longer P108.12 (P12)
- net TMS_L: now also P101.5 (P5); no longer P101.19 (P19)
- net TRST_N_BUF_R: now also P108.21 (P21); no longer P108.7 (P7)
- net TRST_N_L: now also P101.10 (P10); no longer P101.24 (P24)

Commit message: about to try add in new power island zones
Parts:
- added R130: 33R, symbol R
Connections:
- net CLK_20M: now also U124.3 (A2)
- net L1_TMS: no longer U124.3 (A2)
- net L1_TMS_BUF_R: no longer U124.4 (Y2)
- new net: R130.1, U124.4 (Y2)
- new net L1_CLK_20M: R130.2
Other:
- note added: "L1 TDI/TDO SELECTORS"

Commit message: headache...must...get...pills! Reset supervisors up and L1 mostly done
Connections:
- net CLK_20M: now also R121.1
Other:
- moved on the sheet: R121

Commit message: fixed buffer for DEBUG and TMS. Nets keep vanishing...KICAD!!!!
Connections:
- net DEBUG_N: now also U119.1 (A1); no longer U120.1 (A1)
- net DEBUG_N_BUF_R: now also U119.6 (Y1); no longer U120.6 (Y1)
- net L1_TMS: now also U120.3 (A2)
- net L1_TMS_BUF_R: now also U120.4 (Y2)
- net MSEL_N: now also U119.3 (A2); no longer U119.1 (A1)
- net RST_N: now also U118.1 (A1); no longer U119.3 (A2)
- net RST_N_BUF_R: now also U118.6 (Y1); no longer U119.4 (Y2)
- net TCK: now also U118.3 (A2); no longer U118.1 (A1)
- net TCK_BUF_R: now also U118.4 (Y2); no longer U118.6 (Y1)
- net TMS: now also U120.1 (A1); no longer U118.3 (A2)
- net TMS_BUF_R: now also U120.6 (Y1); no longer U118.4 (Y2)
- net TRST_N_BUF_R: now also U119.4 (Y2); no longer U119.6 (Y1)
Changed lines of the file:
@@
-EESchema Schematic File Version 2  date 25/08/2011 15:54:37
+EESchema Schematic File Version 2  date 25/08/2011 17:52:10
 LIBS:power
 LIBS:device
@@
 Comment4 ""
 $EndDescr
+Wire Wire Line
+	5710 6720 5830 6720
 Connection ~ 2400 17380
 Wire Wire Line
@@
 Wire Wire Line
 	1870 17290 1870 17380
+Wire Wire Line
+	7240 6720 7130 6720
+Text Label 5710 6720 2    39   ~ 0
+L1_TMS
+Text Label 7240 6720 0    39   ~ 0
+L1_TMS_BUF_R
 Text Label 4460 2510 2    39   ~ 0
 L1_CLK_20M
@@
 	1    0    0    -1
 $EndComp
-Text Label 7240 5630 0    39   ~ 0
-TRST_N_BUF_R
 Text Label 7240 5830 0    39   ~ 0
-RST_N_BUF_R
+TRST_N_BUF_R
 Text Label 7240 4730 0    39   ~ 0
-TCK_BUF_R
+RST_N_BUF_R
 Text Label 7240 4930 0    39   ~ 0
-TMS_BUF_R
+TCK_BUF_R
 Text Label 7240 6520 0    39   ~ 0
+TMS_BUF_R
+Text Label 7240 5630 0    39   ~ 0
 DEBUG_N_BUF_R
 Text Label 7240 7620 0    39   ~ 0
@@
 Text Label 7240 7420 0    39   ~ 0
 L1_RST_N_BUF_R
-Text Label 5720 5630 2    39   ~ 0
-MSEL_N
 Text Label 5720 5830 2    39   ~ 0
-RST_N
+MSEL_N
 Text Label 5720 4730 2    39   ~ 0
-TCK
+RST_N
 Text Label 5720 4930 2    39   ~ 0
-TMS
+TCK
 Text Label 5720 6520 2    39   ~ 0
+TMS
+Text Label 5720 5630 2    39   ~ 0
 DEBUG_N
 Text Label 5720 7620 2    39   ~ 0

Commit message: added pull ups for I2C bus, checking design over
Parts:
- added R? (x2): 3R3k, symbol R
Connections:
- net A0 is gone; now on net +3.3V: U132.7 (A0)
- net A1 is gone; now on net GND: U132.8 (A1)
- net +3.3V: now also R?.1, R?.1
- net CLK renamed I2C_SDA
- net I2C_SDA: now also R?.2
- net DATA renamed I2C_SCL
- net I2C_SCL: now also R?.2
Other:
- note added: "More Buffering!"

Commit message: save before adding in LEDs in Layout
Parts:
- R131, R132: renamed from R?; value 3R3k -> 1k
Other:
- note added: "I2C Bus Pull-ups"
