File: l2_dev_alternative/l2_dev_board.sch (KiCad schematic (older format))
At the start: 88 parts, among them P101 CONN_30, P102 CONN_30, P103 CONN_30, P104 CONN_30, P105 CONN_30, P106 CONN_30, P107 CONN_30, P108 CONN_30, P109 CONN_30, P110 CONN_30, U101 APX803-SR, U102 NC7SZ157, U103 A6RS-161RF, U104 SN74LVC1G18, U105 SN74LVC1G18, U106 SN74LVC1G18, U107 SN74LVC1G18, U108 SN74CBTD3861, U109 LT3480, U110 APX803-SR, U111 74AHC1GU04, U112 SN74LVC1G18, U113 SN74LVC1G18, U114 SN74LVC1G18, U115 SN74LVC1G18, U116 SN74CBTD3861, U117 NCP1529, U118 NC7WZ17, U119 NC7WZ17, U120 NC7WZ17, U121 NC7WZ17, U122 NC7WZ17, U123 ASE_CLK, U124 NC7WZ17, U125 NC7WZ17, U126 NC7WZ17, U127 NC7WZ17, U128 NC7WZ17, U129 NC7WZ17, U130 NC7WZ17, U131 NC7WZ17, U132 INA219, U133 NB3N551, U134 NB3N551

Commit message: replaced single I2C bus with individual busses for high speed conversions
Parts:
- added R133, R134, R135, R136: 1k, symbol R
Connections:
- net +3.3V: now also R133.1, R134.1, R135.1, R136.1
- new net I2C_SDA_0: R133.2
- new net I2C_SDA_1: R134.2
- new net I2C_SDA_2: R135.2
- new net I2C_SDA_3: R136.2
Other:
- moved on the sheet: R131, R132

Commit message: copied over new files from basic board
Parts:
- removed R118, R119, R120: 10k, symbol R
- removed R130: 33R, symbol R
- removed R132, R133, R134, R135: 1k, symbol R
- removed U102: NC7SZ157, symbol NC7SZ157
- removed U112, U113, U114, U115: SN74LVC1G18, symbol SN74LVC1G18
- removed U118, U121, U122, U124, U127, U129, U130: NC7WZ17, symbol NC7WZ17
- removed U132: INA219, symbol INA219
- removed U133, U134: NB3N551, symbol NB3N551
- added P111: PJ-044BH, symbol PJ-044BH
- added P112: CONN_7, symbol CONN_7
- added R141, R146, R151, R160, R165, R166, R171, R176, R181: 33R, 0603, symbol R
- added U102, U121, U122, U124, U129, U130, U132, U133, U134, U135, U136, U137: YC124, 4x0402, symbol YC124
- added U112, U113, U114, U115: NC7WZ17, SC70-6, symbol NC7WZ17
- added U119, U127: NC7WZ07, SC70-6, symbol NC7WZ07
- C101, C102, C105, C106, C107, R101, R102, R103, R104, R105, R106, R107, R108, R109, R110, R111, R112, R113, R121, R122, R123, R124, R125, R126, R127, R128, R129: footprint (none) -> 0603
- C103: value 0.47uF -> 0.22uF; footprint (none) -> 0603
- C104: value 47uF -> 10uF; footprint (none) -> 0603
- C108: value 0.1uF -> 0.01uF; footprint (none) -> 0603
- C109: value 0.1uF -> 10uF; footprint (none) -> 0603
- D101: footprint (none) -> DFLS240L
- L101: value 2.2uH -> 2u2H; footprint (none) -> LQH55P
- R114: value 10R -> 10k; footprint (none) -> 0603
- R115: value 0.05 -> 33R; footprint (none) -> 0603
- R116: value 10R -> 33R; footprint (none) -> 0603
- R117: value 10k -> 33R; footprint (none) -> 0603
- R131, R136: value 1k -> 33R; footprint (none) -> 0603
- U101, U110: footprint (none) -> SOT23-3
- U103: footprint (none) -> AR6S-SWT
- U104, U105, U106, U107: footprint (none) -> SOT23-6
- U108, U116: footprint (none) -> TSSOP-24
- U109: footprint (none) -> 10DFN
- U111: footprint (none) -> SOT25-5
- U117: footprint (none) -> SOT23-5
- U118: renamed from U119; footprint (none) -> SC70-6
- U120, U125, U126, U128, U131: footprint (none) -> SC70-6
- U123: footprint (none) -> SMD-4
Connections:
- net L1_DEBUG_N_BUF_B is gone; now on net GND: P107.15 (P15)
- net L1_DEBUG_N_BUF_R is gone; now on net GND: P109.17 (P17)
- net L1_RST_N_BUF_B is gone; now on net GND: P107.17 (P17)
- net L1_RST_N_BUF_R is gone; now on net GND: P109.19 (P19)
- net L1_TCK_BUF_B is gone; now on net GND: P107.19 (P19)
- net L1_TCK_BUF_R is gone; now on net GND: P109.20 (P20)
- net L1_TDI_B is gone; now on net GND: P105.2 (P2)
- net L1_TDI_L is gone; now on net GND: P102.16 (P16)
- net L1_TDI_R is gone; now on net GND: P109.13 (P13)
- net L1_TDO_B is gone; now on net L2_PAIR_Q4/B_X1_XLB_3i: P105.4 (P4)
- net L1_TDO_L is gone; now on net GND: P102.18 (P18)
- net L1_TDO_R is gone; now on net GND: P109.15 (P15)
- net L1_TDO_T is gone; now on net GND: P104.29 (P29)
- net L1_TRST_N_BUF_B is gone; now on net GND: P107.16 (P16)
- net L1_TRST_N_BUF_R is gone; now on net GND: P109.18 (P18)
- net L1_XLINK_0i_B is gone; now on net GND: P105.26 (P26)
- net L1_XLINK_0i_L is gone; now on net GND: P102.3 (P3)
- net L1_XLINK_0i_R is gone; now on net GND: P109.24 (P24)
- net L1_XLINK_0i_T is gone; now on net GND: P104.3 (P3)
- net L1_XLINK_0o_B is gone; now on net GND: P105.28 (P28)
- net L1_XLINK_0o_L is gone; now on net GND: P102.6 (P6)
- net L1_XLINK_0o_R is gone; now on net GND: P109.28 (P28)
- net L1_XLINK_0o_T is gone; now on net GND: P104.5 (P5)
- net L1_XLINK_1i_B is gone; now on net RST_N_BUF_B: P105.25 (P25)
- net L1_XLINK_1i_L is gone; now on net GND: P102.2 (P2)
- net L1_XLINK_1i_R is gone; now on net GND: P109.25 (P25)
- net L1_XLINK_1i_T is gone; now on net TMS_T: P104.2 (P2)
- net L1_XLINK_1o_B is gone; now on net TMS_BUF_B: P105.29 (P29)
- net L1_XLINK_1o_L is gone; now on net GND: P102.7 (P7)
- net L1_XLINK_1o_R is gone; now on net GND: P109.29 (P29)
- net L1_XLINK_1o_T is gone; now on net RST_N_T: P104.6 (P6)
- net L2_PAIR_Q1/T_X0_XLB_0i is gone; now on net GND: P104.13 (P13)
- net L2_PAIR_Q1/T_X0_XLB_0o is gone; now on net GND: P104.16 (P16)
- net L2_PAIR_Q1/T_X0_XLB_1i is gone; now on net GND: P104.12 (P12)
- net L2_PAIR_Q1/T_X0_XLB_2i is gone; now on net GND: P104.11 (P11)
- net L2_PAIR_Q1/T_X0_XLB_3i is gone; now on net GND: P104.10 (P10)
- net L2_PAIR_Q1/T_X0_XLB_4i is gone; now on net GND: P104.9 (P9)
- net +12V: now also P111.1 (PIN)
- net +3.3V: now also C106.1, C107.1, L102.2, R105.1, R110.1, R113.2, R114.1, U101.3 (VCC), U104.5 (VCC), U105.5 (VCC), U106.5 (VCC), U107.5 (VCC), U108.24 (VCC), U116.24 (VCC), U112.5 (VCC), U113.5 (VCC), U114.5 (VCC), U115.5 (VCC), U119.5 (VCC), U127.5 (VCC); no longer R113.1, R117.1, R131.1, R136.1
- net +5V: now also C109.1; no longer U104.5 (VCC), U105.5 (VCC), U106.5 (VCC), U107.5 (VCC), U108.24 (VCC), U116.24 (VCC)
- net CLK_20M: now also U112.1 (A1), U112.3 (A2), U113.1 (A1), U113.3 (A2), U114.1 (A1), U114.3 (A2), U115.1 (A1), U115.3 (A2)
- net DEBUG_N: now also U126.1 (A1), P112.3 (P3); no longer R117.2, U126.3 (A2)
- net DEBUG_N_BUF_B: now also P105.23 (P23), U126.6 (Y1); no longer P107.23 (P23), U126.4 (Y2)
- net DEBUG_N_BUF_R: now also P108.6 (P6); no longer P108.20 (P20)
- net DEBUG_N_L: now also P101.25 (P25); no longer P101.11 (P11)
- net DEBUG_N_T: now also P104.8 (P8); no longer P106.8 (P8)
- net GND: now also C109.2, D101.1 (A), P101.10 (P10), P101.11 (P11), P101.18 (P18), P101.20 (P20), P101.22 (P22), P101.26 (P26), P101.28 (P28), P102.11 (P11), P102.12 (P12), P102.13 (P13), P102.14 (P14), P102.9 (P9), P104.23 (P23), P105.15 (P15), P105.18 (P18), P105.19 (P19), P105.20 (P20), P105.21 (P21), P105.22 (P22), P105.8 (P8), P106.10 (P10), P106.12 (P12), P106.14 (P14), P106.15 (P15), P106.16 (P16), P106.2 (P2), P106.4 (P4), P106.6 (P6), P106.7 (P7), P106.8 (P8), P107.21 (P21), P107.23 (P23), P107.24 (P24), P107.25 (P25), P107.27 (P27), P107.29 (P29), P108.11 (P11), P108.13 (P13), P108.20 (P20), P108.21 (P21), P108.3 (P3), P108.5 (P5), P108.9 (P9), P109.22 (P22), P111.2, U112.2 (GND), U113.2 (GND), U114.2 (GND), U115.2 (GND), U119.2 (GND), U127.2 (GND); no longer D101.2 (K), P101.12 (P12), P101.14 (P14), P101.16 (P16), P101.23 (P23), P101.24 (P24), P101.6 (P6), P101.8 (P8), P104.21 (P21), P104.24 (P24), P104.26 (P26), P104.28 (P28), P104.4 (P4), P104.7 (P7), P104.8 (P8), P105.10 (P10), P105.23 (P23), P105.24 (P24), P105.27 (P27), P105.3 (P3), P105.5 (P5), P105.7 (P7), P106.3 (P3), P106.5 (P5), P107.26 (P26), P107.28 (P28), P108.15 (P15), P108.17 (P17), P108.19 (P19), P108.23 (P23), P108.25 (P25), P108.7 (P7), P108.8 (P8)
- net L2_PAIR_Q1/BL_X0_XLA_0o: now also U130.1; no longer P102.27 (P27)
- net L2_PAIR_Q1/BL_X0_XLA_1o: now also U130.2; no longer P102.28 (P28)
- net L2_PAIR_Q1/BL_X0_XLA_2o: now also U130.3; no longer P102.29 (P29)
- net L2_PAIR_Q1/BL_X0_XLA_3o: now also U130.4; no longer P101.2 (P2)
- net L2_PAIR_Q1/BL_X0_XLA_4o: now also R141.1; no longer P101.3 (P3)
- net L2_PAIR_Q1/TL_X0_XLA_0i: now also P101.9 (P9); no longer P101.22 (P22)
- net L2_PAIR_Q1/TL_X0_XLA_0o: now also U122.5; no longer P101.25 (P25)
- net L2_PAIR_Q1/TL_X0_XLA_1i: now also P101.8 (P8); no longer P101.21 (P21)
- net L2_PAIR_Q1/TL_X0_XLA_1o: now also U122.6; no longer P101.26 (P26)
- net L2_PAIR_Q1/TL_X0_XLA_2i: now also P101.7 (P7); no longer P101.20 (P20)
- net L2_PAIR_Q1/TL_X0_XLA_2o: now also U122.7; no longer P101.27 (P27)
- net L2_PAIR_Q1/TL_X0_XLA_3i: now also P101.6 (P6); no longer P101.19 (P19)
- net L2_PAIR_Q1/TL_X0_XLA_3o: now also U122.8; no longer P101.28 (P28)
- net L2_PAIR_Q1/TL_X0_XLA_4i: now also P101.5 (P5); no longer P101.18 (P18)
- net L2_PAIR_Q1/TL_X0_XLA_4o: now also R131.1; no longer P101.29 (P29)
- net L2_PAIR_Q2/TR_X1_XLA_0i: now also P108.19 (P19); no longer P108.6 (P6)
- net L2_PAIR_Q2/TR_X1_XLA_0o: now also R171.2; no longer P108.9 (P9)
- net L2_PAIR_Q2/TR_X1_XLA_1i: now also P108.18 (P18); no longer P108.5 (P5)
- net L2_PAIR_Q2/TR_X1_XLA_1o: now also U132.1; no longer P108.10 (P10)
- net L2_PAIR_Q2/TR_X1_XLA_2i: now also P108.17 (P17); no longer P108.4 (P4)
- net L2_PAIR_Q2/TR_X1_XLA_2o: now also U132.2; no longer P108.11 (P11)
- net L2_PAIR_Q2/TR_X1_XLA_3i: now also P108.16 (P16); no longer P108.3 (P3)
- net L2_PAIR_Q2/TR_X1_XLA_3o: now also U132.3; no longer P108.12 (P12)
- net L2_PAIR_Q2/TR_X1_XLA_4i: now also P108.15 (P15); no longer P108.2 (P2)
- net L2_PAIR_Q2/TR_X1_XLA_4o: now also U132.4; no longer P108.13 (P13)
- net L2_PAIR_Q3/B_X1_XLB_0o: now also R160.1; no longer P107.9 (P9)
- net L2_PAIR_Q3/B_X1_XLB_1o: now also U137.5; no longer P107.10 (P10)
- net L2_PAIR_Q3/B_X1_XLB_2o: now also U137.6; no longer P107.11 (P11)
- net L2_PAIR_Q3/B_X1_XLB_3o: now also U137.7; no longer P107.12 (P12)
- net L2_PAIR_Q3/B_X1_XLB_4o: now also U137.8; no longer P107.13 (P13)
- net L2_PAIR_Q3/TR_X1_XLA_0o: now also R181.2; no longer P110.10 (P10)
- net L2_PAIR_Q3/TR_X1_XLA_1o: now also U135.1; no longer P110.11 (P11)
- net L2_PAIR_Q3/TR_X1_XLA_2o: now also U135.2; no longer P110.12 (P12)
- net L2_PAIR_Q3/TR_X1_XLA_3o: now also U135.3; no longer P110.13 (P13)
- net L2_PAIR_Q3/TR_X1_XLA_4o: now also U135.4; no longer P110.14 (P14)
- net L2_PAIR_Q4/BL_X0_XLA_0o: now also U129.1; no longer P103.10 (P10)
- net L2_PAIR_Q4/BL_X0_XLA_1o: now also U129.2; no longer P103.11 (P11)
- net L2_PAIR_Q4/BL_X0_XLA_2o: now also U129.3; no longer P103.12 (P12)
- net L2_PAIR_Q4/BL_X0_XLA_3o: now also U129.4; no longer P103.13 (P13)
- net L2_PAIR_Q4/BL_X0_XLA_4o: now also R136.1; no longer P103.14 (P14)
- net L2_PAIR_Q4/B_X1_XLB_0i: now also P105.7 (P7); no longer P105.15 (P15)
- net L2_PAIR_Q4/B_X1_XLB_0o: now also R146.1; no longer P105.18 (P18)
- net L2_PAIR_Q4/B_X1_XLB_1i: now also P105.6 (P6); no longer P105.14 (P14)
- net L2_PAIR_Q4/B_X1_XLB_1o: now also U136.5; no longer P105.19 (P19)
- net L2_PAIR_Q4/B_X1_XLB_2i: now also P105.5 (P5); no longer P105.13 (P13)
- net L2_PAIR_Q4/B_X1_XLB_2o: now also U136.6; no longer P105.20 (P20)
- net L2_PAIR_Q4/B_X1_XLB_3i: no longer P105.12 (P12)
- net L2_PAIR_Q4/B_X1_XLB_3o: now also U136.7; no longer P105.21 (P21)
- net L2_PAIR_Q4/B_X1_XLB_4i: now also P105.3 (P3); no longer P105.11 (P11)
- net L2_PAIR_Q4/B_X1_XLB_4o: now also U136.8; no longer P105.22 (P22)
- net L2_PAIR_Q4/TL_X0_XLA_0o: now also U124.1; no longer P103.24 (P24)
- net L2_PAIR_Q4/TL_X0_XLA_1o: now also U124.2; no longer P103.25 (P25)
- net L2_PAIR_Q4/TL_X0_XLA_2o: now also U124.3; no longer P103.26 (P26)
- net L2_PAIR_Q4/TL_X0_XLA_3o: now also U124.4; no longer P103.27 (P27)
- net L2_PAIR_Q4/TL_X0_XLA_4o: now also R117.1; no longer P103.28 (P28)
- net MSEL_N: now also U126.3 (A2), P112.7 (P7); no longer R112.2
- net RST_N: now also R113.1, P112.1 (P1), U119.1 (A1), U127.3 (A2); no longer R113.2
- net RST_N_BUF_B: now also R112.2, U127.4 (Y2); no longer P107.25 (P25)
- net RST_N_BUF_R: now also P108.8 (P8), R114.2, U119.6 (Y1); no longer P108.22 (P22)
- net RST_N_L: now also P101.23 (P23); no longer P101.9 (P9)
- net RST_N_T: no longer P106.6 (P6)
- net SWT_4: now also U108.23 (OE), U111.2 (A)
- net TCK: now also U120.1 (A1), P112.4 (P4)
- net TCK_BUF_B: now also P105.27 (P27), R116.1; no longer P107.27 (P27), U128.6 (Y1)
- net TCK_BUF_R: now also P108.10 (P10), R115.1; no longer P108.24 (P24)
- net TCK_L: now also P101.21 (P21); no longer P101.7 (P7)
- net TCK_T: now also P104.4 (P4); no longer P106.4 (P4)
- net TDI_B: now also P107.26 (P26); no longer P105.6 (P6)
- net TDI_L: now also P101.27 (P27), P112.6 (P6); no longer P101.13 (P13)
- net TDI_R: now also P108.2 (P2); no longer P108.16 (P16)
- net TDI_T: now also P106.3 (P3); no longer P104.23 (P23)
- net TDO_B: now also P107.28 (P28); no longer P105.8 (P8)
- net TDO_L: now also P101.29 (P29), P112.2 (P2); no longer P101.15 (P15)
- net TDO_R: now also P108.4 (P4); no longer P108.18 (P18)
- net TDO_T: now also P106.5 (P5); no longer P104.25 (P25)
- net TMS: now also U120.3 (A2), P112.5 (P5); no longer U120.1 (A1)
- net TMS_BUF_B: no longer P107.29 (P29)
- net TMS_BUF_R: now also P108.12 (P12), U120.4 (Y2); no longer P108.26 (P26), U120.6 (Y1)
- net TMS_L: now also P101.19 (P19); no longer P101.5 (P5)
- net TMS_T: no longer P106.2 (P2)
- net TRST_N_BUF_B: now also P105.24 (P24), U126.4 (Y2); no longer P107.24 (P24)
- net TRST_N_BUF_R: now also P108.7 (P7); no longer P108.21 (P21)
- net TRST_N_L: now also P101.24 (P24); no longer P101.10 (P10)
- net TRST_N_T: now also P104.7 (P7); no longer P106.7 (P7)
- net at C103.2, L101.1, U109.3 (SW): now also D101.2 (K); no longer D101.1 (A)
- net at R109.2, U109.8 (FB): no longer R108.1
- net at R116.2: now also U128.6 (Y1); no longer C109.2
- net at R122.2: now also U112.6 (Y1)
- net at R123.2: now also U112.4 (Y2)
- net at R124.2: now also U113.6 (Y1)
- net at R125.2: now also U113.4 (Y2)
- net at R126.2: now also U114.6 (Y1)
- net at R127.2: now also U114.4 (Y2)
- net at R128.2: now also U115.6 (Y1)
- net at R129.2: now also U115.4 (Y2)
- removed net +3V3_L2: R105.1, R115.1, R116.1, U101.3 (VCC)
- removed net +3V3_L2_F: C106.1, C107.1, L102.2, R110.1, R114.1, R115.2
- net I2C_SCL: no longer names the net of R131.2
- net I2C_SCL: now also P101.16 (P16)
- net I2C_SDA_3: no longer names the net of R136.2
- net I2C_SDA_3: now also P103.14 (P14)
- net L1_DEBUG_N: no longer names the net of U108.17 (B6)
- net L1_DEBUG_N: no longer U116.22 (B1)
- net L1_DEBUG_N_L: no longer names the net of U108.7 (A6)
- net L1_DEBUG_N_L: no longer P102.14 (P14)
- net L1_DEBUG_N_T: no longer names the net of U116.2 (A1)
- net L1_DEBUG_N_T: no longer P106.16 (P16)
- net L1_MSEL_N: no longer names the net of U108.16 (B7)
- net L1_MSEL_N: no longer U116.21 (B2)
- net L1_RST_N: no longer names the net of U108.15 (B8)
- net L1_RST_N: no longer U116.20 (B3)
- net L1_RST_N_L: no longer names the net of U108.9 (A8)
- net L1_RST_N_L: no longer P102.12 (P12)
- net L1_RST_N_T: no longer names the net of U116.4 (A3)
- net L1_RST_N_T: no longer P106.14 (P14)
- net L1_TCK: no longer names the net of U108.14 (B9)
- net L1_TCK: no longer U116.19 (B4)
- net L1_TCK_L: no longer names the net of U108.10 (A9)
- net L1_TCK_L: no longer P102.11 (P11)
- net L1_TCK_T: no longer names the net of U116.5 (A4)
- net L1_TCK_T: no longer P106.12 (P12)
- net L1_TDI_T: no longer names the net of P104.27 (P27)
- net L1_TDI_T: now also U102.1
- removed net L1_TMS: U108.13 (B10), U116.18 (B5), U120.3 (A2), U126.1 (A1)
- removed net L1_TMS_BUF_B: P107.21 (P21), U126.6 (Y1)
- removed net L1_TMS_BUF_R: P109.22 (P22), U120.4 (Y2)
- net L1_TMS_L: no longer names the net of U108.11 (A10)
- net L1_TMS_L: no longer P102.9 (P9)
- net L1_TMS_T: no longer names the net of U116.6 (A5)
- net L1_TMS_T: no longer P106.10 (P10)
- net L1_TRST_N_L: no longer names the net of U108.8 (A7)
- net L1_TRST_N_L: no longer P102.13 (P13)
- net L1_TRST_N_T: no longer names the net of U116.3 (A2)
- net L1_TRST_N_T: no longer P106.15 (P15)
- net L2_PAIR_Q1/T_X0_XLB_1o renamed L2_PAIR_Q1/T_X1_XLA_4i
- net L2_PAIR_Q1/T_X0_XLB_2o renamed L2_PAIR_Q1/T_X1_XLA_3i
- net L2_PAIR_Q1/T_X0_XLB_3o renamed L2_PAIR_Q1/T_X1_XLA_2i
- net L2_PAIR_Q1/T_X0_XLB_4o renamed L2_PAIR_Q1/T_X1_XLA_1i
- net L2_PAIR_Q2/BR_X1_XLA_0i renamed L2_PAIR_Q2/BR_X0_XLB_0i
- net L2_PAIR_Q2/BR_X1_XLA_0o: no longer names the net of P109.7 (P7)
- net L2_PAIR_Q2/BR_X1_XLA_0o: now also R166.1
- net L2_PAIR_Q2/BR_X1_XLA_1i renamed L2_PAIR_Q2/BR_X0_XLB_1i
- net L2_PAIR_Q2/BR_X1_XLA_1o: no longer names the net of P109.8 (P8)
- net L2_PAIR_Q2/BR_X1_XLA_1o: now also U133.8
- net L2_PAIR_Q2/BR_X1_XLA_2i renamed L2_PAIR_Q2/BR_X0_XLB_2i
- net L2_PAIR_Q2/BR_X1_XLA_2o: no longer names the net of P109.9 (P9)
- net L2_PAIR_Q2/BR_X1_XLA_2o: now also U133.7
- net L2_PAIR_Q2/BR_X1_XLA_3i renamed L2_PAIR_Q2/BR_X0_XLB_3i
- net L2_PAIR_Q2/BR_X1_XLA_3o: no longer names the net of P109.10 (P10)
- net L2_PAIR_Q2/BR_X1_XLA_3o: now also U133.6
- net L2_PAIR_Q2/BR_X1_XLA_4i renamed L2_PAIR_Q2/BR_X0_XLB_4i
- net L2_PAIR_Q2/BR_X1_XLA_4o: no longer names the net of P109.11 (P11)
- net L2_PAIR_Q2/BR_X1_XLA_4o: now also U133.5
- net L2_PAIR_Q2/T_X0_XLB_0i renamed L2_PAIR_Q2/T_X1_XLA_0i
- net L2_PAIR_Q2/T_X0_XLB_0o: no longer names the net of P106.25 (P25)
- net L2_PAIR_Q2/T_X0_XLB_0o: now also U121.8
- net L2_PAIR_Q2/T_X0_XLB_1i renamed L2_PAIR_Q2/T_X1_XLA_1i
- net L2_PAIR_Q2/T_X0_XLB_1o: no longer names the net of P106.26 (P26)
- net L2_PAIR_Q2/T_X0_XLB_1o: now also U121.7
- net L2_PAIR_Q2/T_X0_XLB_2i renamed L2_PAIR_Q2/T_X1_XLA_2i
- net L2_PAIR_Q2/T_X0_XLB_2o: no longer names the net of P106.27 (P27)
- net L2_PAIR_Q2/T_X0_XLB_2o: now also U121.6
- net L2_PAIR_Q2/T_X0_XLB_3i renamed L2_PAIR_Q2/T_X1_XLA_3i
- net L2_PAIR_Q2/T_X0_XLB_3o: no longer names the net of P106.28 (P28)
- net L2_PAIR_Q2/T_X0_XLB_3o: now also U121.5
- net L2_PAIR_Q2/T_X0_XLB_4i renamed L2_PAIR_Q2/T_X1_XLA_4i
- net L2_PAIR_Q2/T_X0_XLB_4o: no longer names the net of P106.29 (P29)
- net L2_PAIR_Q2/T_X0_XLB_4o: now also R165.1
- net L2_PAIR_Q3/BR_X1_XLA_0i renamed L2_PAIR_Q3/BR_X0_XLB_0i
- net L2_PAIR_Q3/BR_X1_XLA_0o: no longer names the net of P110.24 (P24)
- net L2_PAIR_Q3/BR_X1_XLA_0o: now also R176.1
- net L2_PAIR_Q3/BR_X1_XLA_1i renamed L2_PAIR_Q3/BR_X0_XLB_1i
- net L2_PAIR_Q3/BR_X1_XLA_1o: no longer names the net of P110.25 (P25)
- net L2_PAIR_Q3/BR_X1_XLA_1o: now also U134.8
- net L2_PAIR_Q3/BR_X1_XLA_2i renamed L2_PAIR_Q3/BR_X0_XLB_2i
- net L2_PAIR_Q3/BR_X1_XLA_2o: no longer names the net of P110.26 (P26)
- net L2_PAIR_Q3/BR_X1_XLA_2o: now also U134.7
- net L2_PAIR_Q3/BR_X1_XLA_3i renamed L2_PAIR_Q3/BR_X0_XLB_3i
- net L2_PAIR_Q3/BR_X1_XLA_3o: no longer names the net of P110.27 (P27)
- net L2_PAIR_Q3/BR_X1_XLA_3o: now also U134.6
- net L2_PAIR_Q3/BR_X1_XLA_4i renamed L2_PAIR_Q3/BR_X0_XLB_4i
- net L2_PAIR_Q3/BR_X1_XLA_4o: no longer names the net of P110.28 (P28)
- net L2_PAIR_Q3/BR_X1_XLA_4o: now also U134.5
- new net: P101.12 (P12), U122.4
- new net: P101.13 (P13), U122.3
- new net: P101.14 (P14), U122.2
- new net: P101.15 (P15), U122.1
- new net: P101.2 (P2), U130.5
- new net: P101.3 (P3), R141.2
- new net: P102.27 (P27), U130.8
- new net: P102.28 (P28), U130.7
- new net: P102.29 (P29), U130.6
- new net: P104.24 (P24), U102.4
- new net: P104.25 (P25), U102.3
- new net: P104.26 (P26), U102.2
- new net: P104.28 (P28), R151.1
- new net: P103.10 (P10), U129.8
- new net: P103.11 (P11), U129.7
- new net: P103.12 (P12), U129.6
- new net: P103.13 (P13), U129.5
- new net: P103.24 (P24), U124.8
- new net: P103.25 (P25), U124.7
- new net: P103.26 (P26), U124.6
- new net: P103.27 (P27), U124.5
- new net: P103.28 (P28), R117.2
- new net: P110.10 (P10), R181.1
- new net: P110.11 (P11), U135.8
- new net: P110.12 (P12), U135.7
- new net: P110.13 (P13), U135.6
- new net: P110.14 (P14), U135.5
- new net: P108.22 (P22), R171.1
- new net: P108.23 (P23), U132.8
- new net: P108.24 (P24), U132.7
- new net: P108.25 (P25), U132.6
- new net: P108.26 (P26), U132.5
- new net: P107.10 (P10), U137.4
- new net: P107.11 (P11), U137.3
- new net: P107.12 (P12), U137.2
- new net: P107.13 (P13), U137.1
- new net: P107.9 (P9), R160.2
- new net: P105.10 (P10), R146.2
- new net: P105.11 (P11), U136.4
- new net: P105.12 (P12), U136.3
- new net: P105.13 (P13), U136.2
- new net: P105.14 (P14), U136.1
- new net: R115.2, U120.6 (Y1)
- new net L2_PAIR_Q1/T_X1_XLA_0i: P104.21 (P21)
- new net L2_PAIR_Q1/T_X1_XLA_0o: U102.5
- new net L2_PAIR_Q1/T_X1_XLA_1o: U102.6
- new net L2_PAIR_Q1/T_X1_XLA_2o: U102.7
- new net L2_PAIR_Q1/T_X1_XLA_3o: U102.8
- new net L2_PAIR_Q1/T_X1_XLA_4o: R151.2
- new net L2_PAIR_Q2/BR_X0_XLB_0o: R166.2
- new net L2_PAIR_Q2/BR_X0_XLB_1o: U133.1
- new net L2_PAIR_Q2/BR_X0_XLB_2o: U133.2
- new net L2_PAIR_Q2/BR_X0_XLB_3o: U133.3
- new net L2_PAIR_Q2/BR_X0_XLB_4o: U133.4
- new net L2_PAIR_Q2/T_X1_XLA_0o: U121.1
- new net L2_PAIR_Q2/T_X1_XLA_1o: U121.2
- new net L2_PAIR_Q2/T_X1_XLA_2o: U121.3
- new net L2_PAIR_Q2/T_X1_XLA_3o: U121.4
- new net L2_PAIR_Q2/T_X1_XLA_4o: R165.2
- new net L2_PAIR_Q3/BR_X0_XLB_0o: R176.2
- new net L2_PAIR_Q3/BR_X0_XLB_1o: U134.1
- new net L2_PAIR_Q3/BR_X0_XLB_2o: U134.2
- new net L2_PAIR_Q3/BR_X0_XLB_3o: U134.3
- new net L2_PAIR_Q3/BR_X0_XLB_4o: U134.4
Other:
- note added: "Nasty workaround for power\nsupplies layout\nwithout power sensing"
- note added: "Power Connector\n"
- note added: "TL- POS = 1\nML- POS = 8\nBL- POS = C\nMI- POS = 5\nRI- POS = 7"
- note removed: "Current Measurment\n"
- note removed: "I2C Bus Pull-ups"
- note removed: "L1 MODULE"
- note removed: "L1 TDI/TDO SELECTORS"
- note removed: "More Buffering!"
- note removed: "TL- POS = 1\nML- POS = 8\nBL- POS = 5\nMI- POS = C\nRI- POS = 7"
- moved on the sheet: C101, C102, C103, C104, C105, C106, C107, C108, D101, L101, L102, R101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

Commit message: almost done!
Parts:
- added C110: 220nF, symbol C
- added R118, R119, R120, R130, R132, R133, R134: 1k, symbol R
- added R135: 0R05, symbol R
- added R137, R138: 10R, symbol R
- added U138: INA219, symbol INA219
Connections:
- net +3.3V: now also R118.1, R119.1, R120.1, R130.1, R132.1, R133.1, R134.1, U138.4 (VS), U138.7 (A0); no longer C106.1, C107.1, L102.2, R105.1, R110.1, R113.2, U101.3 (VCC)
- net GND: now also U138.3 (GND), U138.8 (A1); no longer P102.10 (P10), P102.12 (P12), P102.13 (P13), P102.16 (P16), P102.18 (P18), P102.2 (P2), P102.3 (P3), P102.5 (P5), P102.6 (P6), P102.8 (P8), P104.10 (P10), P104.12 (P12), P104.14 (P14), P104.15 (P15), P105.16 (P16), P105.17 (P17), P105.19 (P19), P105.21 (P21), P106.11 (P11), P106.12 (P12), P106.15 (P15), P106.16 (P16), P106.7 (P7), P106.9 (P9), P107.15 (P15), P107.16 (P16), P107.19 (P19), P107.20 (P20), P107.22 (P22), P107.24 (P24), P109.13 (P13), P109.15 (P15), P109.18 (P18), P109.19 (P19), P109.21 (P21), P109.23 (P23), P109.25 (P25), P109.26 (P26), P109.28 (P28), P109.29 (P29)
- net L1_TCK_L: now reaches U108.10 (A9)
- net L1_TCK_L: now also P102.10 (P10)
- net L1_TMS_L: now reaches U108.11 (A10)
- net L1_TMS_L: now also P102.8 (P8)
- net L1_TMS: now reaches U108.13 (B10)
- net L1_TMS: now also U116.18 (B5)
- net L1_TCK: now reaches U108.14 (B9)
- net L1_TCK: now also U116.19 (B4)
- net L1_RST_N: now reaches U108.15 (B8)
- net L1_RST_N: now also U116.20 (B3)
- net L1_MSEL_N: now reaches U108.16 (B7)
- net L1_MSEL_N: now also U116.21 (B2)
- net L1_TRST_N_L: now reaches U108.8 (A7)
- net L1_TRST_N_L: now also P102.13 (P13)
- net L1_RST_N_L: now reaches U108.9 (A8)
- net L1_RST_N_L: now also P102.12 (P12)
- net L1_TRST_N_T: now reaches U116.3 (A2)
- net L1_TRST_N_T: now also P104.15 (P15)
- net L1_RST_N_T: now reaches U116.4 (A3)
- net L1_RST_N_T: now also P104.14 (P14)
- net L1_TCK_T: now reaches U116.5 (A4)
- net L1_TCK_T: now also P104.12 (P12)
- net L1_TMS_T: now reaches U116.6 (A5)
- net L1_TMS_T: now also P104.10 (P10)
- new net: C110.1, R138.1, U138.1 (VIN+)
- new net: C110.2, R137.1, U138.2 (VIN-)
- new net +3V3_L2: R135.1, R137.2
- new net +3V3_PWR: C106.1, C107.1, L102.2, R110.1, R135.2, R138.2
- new net +3V3_l2: R105.1, R113.2, U101.3 (VCC)
- new net I2C_SCL: U138.6 (DATA)
- new net I2C_SCL_0: R119.2
- new net I2C_SCL_1: R118.2
- new net I2C_SDA: R120.2, U138.5 (CLK)
- new net I2C_SDA_0: R134.2
- new net I2C_SDA_1: R133.2
- new net I2C_SDA_2: R132.2
- new net I2C_SDA_3: R130.2
- new net L1_MSEL_BUF_B: P105.16 (P16)
- new net L1_MSEL_BUF_R: P109.18 (P18)
- new net L1_RST_N_BUF_B: P105.17 (P17)
- new net L1_RST_N_BUF_R: P109.19 (P19)
- new net L1_TCK_BUF_B: P105.19 (P19)
- new net L1_TCK_BUF_R: P109.21 (P21)
- new net L1_TDI_B: P107.22 (P22)
- new net L1_TDI_L: P102.16 (P16)
- new net L1_TDI_R: P109.13 (P13)
- new net L1_TDI_T: P106.7 (P7)
- new net L1_TDO_B: P107.24 (P24)
- new net L1_TDO_L: P102.18 (P18)
- new net L1_TDO_R: P109.15 (P15)
- new net L1_TDO_T: P106.9 (P9)
- new net L1_TMS_BUF_B: P105.21 (P21)
- new net L1_TMS_BUF_R: P109.23 (P23)
- new net XLA_0i: P107.16 (P16)
- new net XLA_0o: P107.19 (P19)
- new net XLA_1i: P107.15 (P15)
- new net XLA_1o: P107.20 (P20)
- new net XLB_0i: P109.26 (P26)
- new net XLB_0o: P109.28 (P28)
- new net XLB_1i: P109.25 (P25)
- new net XLB_1o: P109.29 (P29)
- new net XLC_0i: P102.3 (P3)
- new net XLC_0o: P102.5 (P5)
- new net XLC_1i: P102.2 (P2)
- new net XLC_1o: P102.6 (P6)
- new net XLD_0i: P106.12 (P12)
- new net XLD_0o: P106.15 (P15)
- new net XLD_1i: P106.11 (P11)
- new net XLD_1o: P106.16 (P16)
Other:
- note added: "Nasty workaround for power\nsupplies layout"
- note added: "Nasty workaround for power\nsupplies layout\n"
- note added: "Power Sense for +3V3"
- note removed: "Nasty workaround for power\nsupplies layout\nwithout power sensing"

Commit message: done :)
Connections:
- net I2C_SCL is gone; now on net I2C_SCL_1: U138.6 (DATA)
