File: l2_dev_alternative/l2_pair.sch (KiCad schematic (older format))
At the start: 16 parts, among them U201 NC7WZ17, U202 NC7WZ07, U203 NCP1529, U204 INA219

Commit message: buffers are in and BOM started. Changed open drain buffers for normal buffers and added pull ups to the _N JTAG signals
Parts:
- removed R201, R202: 10k, symbol R
- removed U202: NC7WZ07, symbol NC7WZ07
- added U1102: NC7WZ17, symbol NC7WZ17
Connections:
- net +3.3V: now also U1102.5 (VCC)
- net GND: now also U1102.2 (GND)
- net MSEL_N: now also U1102.3 (A2)
- net MSEL_N_BUF: now also U1102.4 (Y2)
- net RST_N: now also U1102.1 (A1)
- net RST_N_BUF: now also U1102.6 (Y1)
