File: l2_dev_alternative/l2_pair.sch (KiCad schematic (older format))
At the start: 14 parts, among them U1102 NC7WZ17, U201 NC7WZ17, U203 NCP1529, U204 INA219

Commit message: save before adding in LEDs in Layout
Changed lines of the file:
@@
-EESchema Schematic File Version 2  date 30/08/2011 10:58:43
+EESchema Schematic File Version 2  date 30/08/2011 13:51:36
 LIBS:power
 LIBS:device
@@
 $Descr A4 11700 8267
 encoding utf-8
-Sheet 5 14
+Sheet 8 14
 Title ""
 Date "30 aug 2011"
@@
 AR Path="/4E36B777/4E5214B4" Ref="U502"  Part="1"
 AR Path="/4E36B760/4E5214B4" Ref="U802"  Part="1"
-F 0 "U202" H 1390 4450 60  0000 C CNN
+F 0 "U802" H 1390 4450 60  0000 C CNN
 F 1 "NC7WZ17" H 1540 3650 60  0000 C CNN
 	1    1690 4050
@@
 DATA
 $Comp
-L +5V #PWR0195
+L +5V #PWR0196
 U 1 1 4E4D4192
 P 1800 5700
-AR Path="/4E32CDCE/4E4D4192" Ref="#PWR0195"  Part="1"
-AR Path="/4E36B777/4E4D4192" Ref="#PWR0213"  Part="1"
-AR Path="/4E36B760/4E4D4192" Ref="#PWR0231"  Part="1"
-AR Path="/4E36B740/4E4D4192" Ref="#PWR0249"  Part="1"
-F 0 "#PWR0195" H 1800 5790 20  0001 C CNN
+AR Path="/4E32CDCE/4E4D4192" Ref="#PWR0196"  Part="1"
+AR Path="/4E36B777/4E4D4192" Ref="#PWR0222"  Part="1"
+AR Path="/4E36B760/4E4D4192" Ref="#PWR0248"  Part="1"
+AR Path="/4E36B740/4E4D4192" Ref="#PWR0274"  Part="1"
+F 0 "#PWR0274" H 1800 5790 20  0001 C CNN
 F 1 "+5V" H 1800 5790 30  0000 C CNN
 	1    1800 5700
@@
 AR Path="/4E36B760/4E4D4108" Ref="R806"  Part="1"
 AR Path="/4E36B740/4E4D4108" Ref="R1106"  Part="1"
-F 0 "R206" V 1450 4780 50  0000 C CNN
+F 0 "R806" V 1450 4780 50  0000 C CNN
 F 1 "0.05" V 1370 4780 50  0000 C CNN
 	1    1370 4780
@@
 AR Path="/4E36B760/4E4D40FB" Ref="C804"  Part="1"
 AR Path="/4E36B740/4E4D40FB" Ref="C1104"  Part="1"
-F 0 "C204" H 1430 5640 50  0000 L CNN
+F 0 "C804" H 1430 5640 50  0000 L CNN
 F 1 "0.1uF" H 1430 5440 50  0000 L CNN
 	1    1380 5540
@@
 AR Path="/4E36B760/4E4D40F6" Ref="R807"  Part="1"
 AR Path="/4E36B740/4E4D40F6" Ref="R1107"  Part="1"
-F 0 "R207" V 1700 5160 50  0000 C CNN
+F 0 "R807" V 1700 5160 50  0000 C CNN
 F 1 "10R" V 1620 5160 50  0000 C CNN
 	1    1620 5160
@@
 AR Path="/4E36B760/4E4D40F0" Ref="R805"  Part="1"
 AR Path="/4E36B740/4E4D40F0" Ref="R1105"  Part="1"
-F 0 "R205" V 1190 5160 50  0000 C CNN
+F 0 "R805" V 1190 5160 50  0000 C CNN
 F 1 "10R" V 1110 5160 50  0000 C CNN
 	1    1110 5160
@@
 $EndComp
 $Comp
-L GND #PWR0196
+L GND #PWR0197
 U 1 1 4E4D4061
 P 1110 7000
-AR Path="/4E32CDCE/4E4D4061" Ref="#PWR0196"  Part="1"
-AR Path="/4E36B777/4E4D4061" Ref="#PWR0214"  Part="1"
-AR Path="/4E36B760/4E4D4061" Ref="#PWR0232"  Part="1"
-AR Path="/4E36B740/4E4D4061" Ref="#PWR0250"  Part="1"
-F 0 "#PWR0196" H 1110 7000 30  0001 C CNN
+AR Path="/4E32CDCE/4E4D4061" Ref="#PWR0197"  Part="1"
+AR Path="/4E36B777/4E4D4061" Ref="#PWR0223"  Part="1"
+AR Path="/4E36B760/4E4D4061" Ref="#PWR0249"  Part="1"
+AR Path="/4E36B740/4E4D4061" Ref="#PWR0275"  Part="1"
+F 0 "#PWR0275" H 1110 7000 30  0001 C CNN
 F 1 "GND" H 1110 6930 30  0001 C CNN
 	1    1110 7000
@@
 AR Path="/4E36B760/4E4D4027" Ref="U804"  Part="1"
 AR Path="/4E36B740/4E4D4027" Ref="U1104"  Part="1"
-F 0 "U204" H 990 6860 60  0000 C CNN
+F 0 "U804" H 990 6860 60  0000 C CNN
 F 1 "INA219" H 1490 6140 60  0000 C CNN
 	1    1480 6420
@@
 TCK
 $Comp
-L GND #PWR0215
+L GND #PWR0224
 U 1 1 4E35D9C0
 P 2340 4500
-AR Path="/4E36B777/4E35D9C0" Ref="#PWR0215"  Part="1"
-AR Path="/4E36B760/4E35D9C0" Ref="#PWR0233"  Part="1"
-AR Path="/4E36B740/4E35D9C0" Ref="#PWR0251"  Part="1"
-AR Path="/4E32CDCE/4E35D9C0" Ref="#PWR0197"  Part="1"
-F 0 "#PWR0197" H 2340 4500 30  0001 C CNN
+AR Path="/4E36B777/4E35D9C0" Ref="#PWR0224"  Part="1"
+AR Path="/4E36B760/4E35D9C0" Ref="#PWR0250"  Part="1"
+AR Path="/4E36B740/4E35D9C0" Ref="#PWR0276"  Part="1"
+AR Path="/4E32CDCE/4E35D9C0" Ref="#PWR0198"  Part="1"
+F 0 "#PWR0276" H 2340 4500 30  0001 C CNN
 F 1 "GND" H 2340 4430 30  0001 C CNN
 	1    2340 4500
@@
 $EndComp
 $Comp
-L GND #PWR0216
+L GND #PWR0225
 U 1 1 4E35D9AA
 P 2340 3180
-AR Path="/4E36B777/4E35D9AA" Ref="#PWR0216"  Part="1"
-AR Path="/4E36B760/4E35D9AA" Ref="#PWR0234"  Part="1"
-AR Path="/4E36B740/4E35D9AA" Ref="#PWR0252"  Part="1"
-AR Path="/4E32CDCE/4E35D9AA" Ref="#PWR0198"  Part="1"
-F 0 "#PWR0198" H 2340 3180 30  0001 C CNN
+AR Path="/4E36B777/4E35D9AA" Ref="#PWR0225"  Part="1"
+AR Path="/4E36B760/4E35D9AA" Ref="#PWR0251"  Part="1"
+AR Path="/4E36B740/4E35D9AA" Ref="#PWR0277"  Part="1"
+AR Path="/4E32CDCE/4E35D9AA" Ref="#PWR0199"  Part="1"
+F 0 "#PWR0277" H 2340 3180 30  0001 C CNN
 F 1 "GND" H 2340 3110 30  0001 C CNN
 	1    2340 3180
@@
 $EndComp
 $Comp
-L +3.3V #PWR0217
+L +3.3V #PWR0226
 U 1 1 4E35D9A0
 P 2340 3570
-AR Path="/4E36B777/4E35D9A0" Ref="#PWR0217"  Part="1"
-AR Path="/4E36B760/4E35D9A0" Ref="#PWR0235"  Part="1"
-AR Path="/4E36B740/4E35D9A0" Ref="#PWR0253"  Part="1"
-AR Path="/4E32CDCE/4E35D9A0" Ref="#PWR0199"  Part="1"
-F 0 "#PWR0199" H 2340 3530 30  0001 C CNN
+AR Path="/4E36B777/4E35D9A0" Ref="#PWR0226"  Part="1"
+AR Path="/4E36B760/4E35D9A0" Ref="#PWR0252"  Part="1"
+AR Path="/4E36B740/4E35D9A0" Ref="#PWR0278"  Part="1"
+AR Path="/4E32CDCE/4E35D9A0" Ref="#PWR0200"  Part="1"
+F 0 "#PWR0278" H 2340 3530 30  0001 C CNN
 F 1 "+3.3V" H 2340 3680 30  0000 C CNN
 	1    2340 3570
@@
 $EndComp
 $Comp
-L +3.3V #PWR0218
+L +3.3V #PWR0227
 U 1 1 4E35D98B
 P 2340 2250
-AR Path="/4E36B777/4E35D98B" Ref="#PWR0218"  Part="1"
-AR Path="/4E36B760/4E35D98B" Ref="#PWR0236"  Part="1"
-AR Path="/4E36B740/4E35D98B" Ref="#PWR0254"  Part="1"
-AR Path="/4E32CDCE/4E35D98B" Ref="#PWR0200"  Part="1"
-F 0 "#PWR0200" H 2340 2210 30  0001 C CNN
+AR Path="/4E36B777/4E35D98B" Ref="#PWR0227"  Part="1"
+AR Path="/4E36B760/4E35D98B" Ref="#PWR0253"  Part="1"
+AR Path="/4E36B740/4E35D98B" Ref="#PWR0279"  Part="1"
+AR Path="/4E32CDCE/4E35D98B" Ref="#PWR0201"  Part="1"
+F 0 "#PWR0279" H 2340 2210 30  0001 C CNN
 F 1 "+3.3V" H 2340 2360 30  0000 C CNN
 	1    2340 2250
@@
 AR Path="/4E36B740/4E35D8BD" Ref="U801"  Part="1"
 AR Path="/4E32CDCE/4E35D8BD" Ref="U1101"  Part="1"
-F 0 "U1101" H 1390 3130 60  0000 C CNN
+F 0 "U501" H 1390 3130 60  0000 C CNN
 F 1 "NC7WZ17" H 1540 2330 60  0000 C CNN
 	1    1690 2730
@@
 AR Path="/4E36B740/4E35D6A2" Ref="C803"  Part="1"
 AR Path="/4E32CDCE/4E35D6A2" Ref="C1103"  Part="1"
-F 0 "C1103" H 3850 1290 50  0000 L CNN
+F 0 "C503" H 3850 1290 50  0000 L CNN
 F 1 "10uF" H 3850 1090 50  0000 L CNN
 	1    3800 1190
@@
 AR Path="/4E36B740/4E35D649" Ref="C802"  Part="1"
 AR Path="/4E32CDCE/4E35D649" Ref="C1102"  Part="1"
-F 0 "C1102" H 3510 1290 50  0000 L CNN
+F 0 "C502" H 3510 1290 50  0000 L CNN
 F 1 "33pF" H 3510 1100 50  0000 L CNN
 	1    3500 1190
@@
 AR Path="/4E36B740/4E35D5DA" Ref="R804"  Part="1"
 AR Path="/4E32CDCE/4E35D5DA" Ref="R1104"  Part="1"
-F 0 "R1104" V 3310 1700 50  0000 C CNN
+F 0 "R504" V 3310 1700 50  0000 C CNN
 F 1 "100k" V 3230 1700 50  0000 C CNN
 	1    3230 1700
@@
 AR Path="/4E36B740/4E35D5C1" Ref="R803"  Part="1"
 AR Path="/4E32CDCE/4E35D5C1" Ref="R1103"  Part="1"
-F 0 "R1103" V 3310 1170 50  0000 C CNN
+F 0 "R503" V 3310 1170 50  0000 C CNN
 F 1 "68k" V 3230 1170 50  0000 C CNN
 	1    3230 1170
@@
 AR Path="/4E36B740/4E35D5AC" Ref="L801"  Part="1"
 AR Path="/4E32CDCE/4E35D5AC" Ref="L1101"  Part="1"
-F 0 "L1101" V 2790 920 40  0000 C CNN
+F 0 "L501" V 2790 920 40  0000 C CNN
 F 1 "2u2H" V 2940 920 40  0000 C CNN
 	1    2840 920
@@
 $EndComp
 $Comp
-L GND #PWR0219
+L GND #PWR0228
 U 1 1 4E3545A6
 P 1740 1980
-AR Path="/4E36B777/4E3545A6" Ref="#PWR0219"  Part="1"
-AR Path="/4E36B760/4E3545A6" Ref="#PWR0237"  Part="1"
-AR Path="/4E36B740/4E3545A6" Ref="#PWR0255"  Part="1"
-AR Path="/4E32CDCE/4E3545A6" Ref="#PWR0201"  Part="1"
-F 0 "#PWR0201" H 1740 1980 30  0001 C CNN
+AR Path="/4E36B777/4E3545A6" Ref="#PWR0228"  Part="1"
+AR Path="/4E36B760/4E3545A6" Ref="#PWR0254"  Part="1"
+AR Path="/4E36B740/4E3545A6" Ref="#PWR0280"  Part="1"
+AR Path="/4E32CDCE/4E3545A6" Ref="#PWR0202"  Part="1"
+F 0 "#PWR0280" H 1740 1980 30  0001 C CNN
 F 1 "GND" H 1740 1910 30  0001 C CNN
 	1    1740 1980
@@
 AR Path="/4E36B740/4E354587" Ref="C801"  Part="1"
 AR Path="/4E32CDCE/4E354587" Ref="C1101"  Part="1"
-F 0 "C1101" H 740 1250 50  0000 L CNN
+F 0 "C501" H 740 1250 50  0000 L CNN
 F 1 "10uF" H 740 1050 50  0000 L CNN
 	1    690  1150
@@
 $EndComp
 $Comp
-L +5V #PWR0220
+L +5V #PWR0229
 U 1 1 4E35455A
 P 690 750
-AR Path="/4E36B777/4E35455A" Ref="#PWR0220"  Part="1"
-AR Path="/4E36B760/4E35455A" Ref="#PWR0238"  Part="1"
-AR Path="/4E36B740/4E35455A" Ref="#PWR0256"  Part="1"
-AR Path="/4E32CDCE/4E35455A" Ref="#PWR0202"  Part="1"
-F 0 "#PWR0202" H 690 840 20  0001 C CNN
+AR Path="/4E36B777/4E35455A" Ref="#PWR0229"  Part="1"
+AR Path="/4E36B760/4E35455A" Ref="#PWR0255"  Part="1"
+AR Path="/4E36B740/4E35455A" Ref="#PWR0281"  Part="1"
+AR Path="/4E32CDCE/4E35455A" Ref="#PWR0203"  Part="1"
+F 0 "#PWR0281" H 690 840 20  0001 C CNN
 F 1 "+5V" H 690 840 30  0000 C CNN
 	1    690  750
@@
 AR Path="/4E36B740/4E354532" Ref="U803"  Part="1"
 AR Path="/4E32CDCE/4E354532" Ref="U1103"  Part="1"
-F 0 "U1103" H 1740 1220 60  0000 C CNN
+F 0 "U503" H 1740 1220 60  0000 C CNN
 F 1 "NCP1529" H 1740 1320 60  0000 C CNN
 	1    1740 1270
