File: l2_dev_alternative/l1.sch (KiCad schematic (older format))
At the start: 35 parts, among them U1401 NC7WZ17, U1402 NC7WZ07, U1403 NCP1529, U1404 NCP1521B, U1405 APX803-SR, U1406 APX803-SR, U1407 XS1-L1-128

Commit message: Most of the components now in. About to try finalise the size!
Parts:
- removed R1401, R1402: 10k, symbol R
- removed U1402: NC7WZ07, symbol NC7WZ07
- added U1402: NC7WZ17, symbol NC7WZ17
Connections:
- wire segments 162 -> 159
Changed lines of the file:
@@
-EESchema Schematic File Version 2  date 22/08/2011 13:22:58
+EESchema Schematic File Version 2  date 23/08/2011 15:06:26
 LIBS:power
 LIBS:device
@@
 Sheet 14 14
 Title ""
-Date "22 aug 2011"
+Date "23 aug 2011"
 Rev ""
 Comp ""
@@
 Comment4 ""
 $EndDescr
+$Comp
+L NC7WZ17 U1402
+U 1 1 4E53B2A3
+P 1630 2490
+F 0 "U1402" H 1330 2890 60  0000 C CNN
+F 1 "NC7WZ17" H 1480 2090 60  0000 C CNN
+	1    1630 2490
+	1    0    0    -1
+$EndComp
 Wire Wire Line
 	8430 3700 8430 3720
@@
 Wire Notes Line
 	510  3090 510  4580
-Connection ~ 2650 1740
-Wire Wire Line
-	2470 1740 2830 1740
-Connection ~ 2650 2390
-Wire Wire Line
-	2650 2240 2650 2390
 Wire Notes Line
 	3060 3070 510  3070
@@
 Wire Notes Line
 	510  510  3060 510
-Wire Wire Line
-	2470 2240 2470 2590
-Connection ~ 2470 2590
 Wire Notes Line
 	6260 520  6260 5720
@@
 	8430 4220 8430 4250
 Connection ~ 8430 4250
-$Comp
-L +3.3V #PWR0256
+Text HLabel 6860 4250 0    60   Input ~ 0
+CLK_20M
+$Comp
+L +3.3V #PWR0260
 U 1 1 4E4BD358
 P 8430 3700
-F 0 "#PWR0256" H 8430 3660 30  0001 C CNN
+F 0 "#PWR0260" H 8430 3660 30  0001 C CNN
 F 1 "+3.3V" H 8430 3810 30  0000 C CNN
 	1    8430 3700
@@
 RST_N_BUF
 $Comp
-L +3.3V #PWR0257
+L +3.3V #PWR0261
 U 1 1 4E36A392
 P 6730 4620
-F 0 "#PWR0257" H 6730 4580 30  0001 C CNN
+F 0 "#PWR0261" H 6730 4580 30  0001 C CNN
 F 1 "+3.3V" H 6730 4730 30  0000 C CNN
 	1    6730 4620
@@
 NoConn ~ 7010 4600
 NoConn ~ 7010 4500
-Text GLabel 6860 4250 0    60   Input ~ 0
-CLK_20M
 $Comp
 L C C1411
@@
 $EndComp
 $Comp
-L +1V0 #PWR0258
+L +1V0 #PWR0262
 U 1 1 4E3688F5
 P 8950 2270
-F 0 "#PWR0258" H 8950 2230 30  0001 C CNN
+F 0 "#PWR0262" H 8950 2230 30  0001 C CNN
 F 1 "+1V0" H 8950 2400 30  0000 C CNN
 	1    8950 2270
@@
 $EndComp
 $Comp
-L GND #PWR0259
+L GND #PWR0263
 U 1 1 4E3688DC
 P 8260 3690
-F 0 "#PWR0259" H 8260 3690 30  0001 C CNN
+F 0 "#PWR0263" H 8260 3690 30  0001 C CNN
 F 1 "GND" H 8260 3620 30  0001 C CNN
 	1    8260 3690
@@
 $EndComp
 $Comp
-L +3.3V #PWR0260
+L +3.3V #PWR0264
 U 1 1 4E3688B7
 P 8690 3190
-F 0 "#PWR0260" H 8690 3150 30  0001 C CNN
+F 0 "#PWR0264" H 8690 3150 30  0001 C CNN
 F 1 "+3.3V" H 8690 3290 30  0000 C CNN
 	1    8690 3190
@@
 $EndComp
 $Comp
-L +1V0 #PWR0261
+L +1V0 #PWR0265
 U 1 1 4E36889D
 P 8530 3190
-F 0 "#PWR0261" H 8530 3150 30  0001 C CNN
+F 0 "#PWR0265" H 8530 3150 30  0001 C CNN
 F 1 "+1V0" H 8530 3290 30  0000 C CNN
 	1    8530 3190
@@
 NoConn ~ 8260 3110
 $Comp
-L +3.3V #PWR0262
+L +3.3V #PWR0266
 U 1 1 4E36886B
 P 8540 2920
-F 0 "#PWR0262" H 8540 2880 30  0001 C CNN
+F 0 "#PWR0266" H 8540 2880 30  0001 C CNN
 F 1 "+3.3V" H 8540 3030 30  0000 C CNN
 	1    8540 2920
@@
 $EndComp
 $Comp
-L GND #PWR0263
+L GND #PWR0267
 U 1 1 4E3687FE
 P 8350 2890
-F 0 "#PWR0263" H 8350 2890 30  0001 C CNN
+F 0 "#PWR0267" H 8350 2890 30  0001 C CNN
 F 1 "GND" H 8350 2820 30  0001 C CNN
 	1    8350 2890
@@
 $EndComp
 $Comp
-L +1V0 #PWR0264
+L +1V0 #PWR0268
 U 1 1 4E3687CA
 P 6880 810
-F 0 "#PWR0264" H 6880 770 30  0001 C CNN
+F 0 "#PWR0268" H 6880 770 30  0001 C CNN
 F 1 "+1V0" H 6880 940 30  0000 C CNN
 	1    6880 810
@@
 $EndComp
 $Comp
-L +1V0 #PWR0265
+L +1V0 #PWR0269
 U 1 1 4E3686DE
 P 7960 5960
-F 0 "#PWR0265" H 7960 5920 30  0001 C CNN
+F 0 "#PWR0269" H 7960 5920 30  0001 C CNN
 F 1 "+1V0" H 7960 6090 30  0000 C CNN
 	1    7960 5960
@@
 $EndComp
 $Comp
-L +3.3V #PWR0266
+L +3.3V #PWR0270
 U 1 1 4E3686D7
 P 9580 5960
-F 0 "#PWR0266" H 9580 5920 30  0001 C CNN
+F 0 "#PWR0270" H 9580 5920 30  0001 C CNN
 F 1 "+3.3V" H 9580 6070 30  0000 C CNN
 	1    9580 5960
@@
 $EndComp
 $Comp
-L GND #PWR0267
+L GND #PWR0271
 U 1 1 4E36868C
 P 8050 6570
-F 0 "#PWR0267" H 8050 6570 30  0001 C CNN
+F 0 "#PWR0271" H 8050 6570 30  0001 C CNN
 F 1 "GND" H 8050 6500 30  0001 C CNN
 	1    8050 6570
@@
 $EndComp
 $Comp
-L GND #PWR0268
+L GND #PWR0272
 U 1 1 4E36868B
 P 9670 6570
-F 0 "#PWR0268" H 9670 6570 30  0001 C CNN
+F 0 "#PWR0272" H 9670 6570 30  0001 C CNN
 F 1 "GND" H 9670 6500 30  0001 C CNN
 	1    9670 6570
@@
 $EndComp
 $Comp
-L +1V0 #PWR0269
+L +1V0 #PWR0273
 U 1 1 4E367E87
 P 3820 4880
-F 0 "#PWR0269" H 3820 4840 30  0001 C CNN
+F 0 "#PWR0273" H 3820 4840 30  0001 C CNN
 F 1 "+1V0" H 3820 5010 30  0000 C CNN
 	1    3820 4880
@@
 $EndComp
 $Comp
-L +3.3V #PWR0270
+L +3.3V #PWR0274
 U 1 1 4E367E10
 P 5220 600
-F 0 "#PWR0270" H 5220 560 30  0001 C CNN
+F 0 "#PWR0274" H 5220 560 30  0001 C CNN
 F 1 "+3.3V" H 5220 710 30  0000 C CNN
 	1    5220 600
@@
 $EndComp
 $Comp
-L +3.3V_PG #PWR0271
+L +3.3V_PG #PWR0275
 U 1 1 4E367DE3
 P 4480 680
-F 0 "#PWR0271" H 4480 640 30  0001 C CNN
+F 0 "#PWR0275" H 4480 640 30  0001 C CNN
 F 1 "+3.3V_PG" H 4480 810 30  0000 C CNN
 	1    4480 680
@@
 $EndComp
 $Comp
-L +3.3V #PWR0272
+L +3.3V #PWR0276
 U 1 1 4E367DD1
 P 3370 880
-F 0 "#PWR0272" H 3370 840 30  0001 C CNN
+F 0 "#PWR0276" H 3370 840 30  0001 C CNN
 F 1 "+3.3V" H 3370 990 30  0000 C CNN
 	1    3370 880
@@
 $EndComp
 $Comp
-L GND #PWR0273
+L GND #PWR0277
 U 1 1 4E367DC7
 P 3990 1460
-F 0 "#PWR0273" H 3990 1460 30  0001 C CNN
+F 0 "#PWR0277" H 3990 1460 30  0001 C CNN
 F 1 "GND" H 3990 1390 30  0001 C CNN
 	1    3990 1460
@@
 $EndComp
 $Comp
-L GND #PWR0274
+L GND #PWR0278
 U 1 1 4E367DC6
 P 5200 1460
-F 0 "#PWR0274" H 5200 1460 30  0001 C CNN
+F 0 "#PWR0278" H 5200 1460 30  0001 C CNN
 F 1 "GND" H 5200 1390 30  0001 C CNN
 	1    5200 1460
@@
 RST_N_SPVSR
 $Comp
-L +5V #PWR0275
+L +5V #PWR0279
 U 1 1 4E367507
 P 630 4800
-F 0 "#PWR0275" H 630 4890 20  0001 C CNN
+F 0 "#PWR0279" H 630 4890 20  0001 C CNN
 F 1 "+5V" H 630 4890 30  0000 C CNN
 	1    630  4800
@@
 $EndComp
 $Comp
-L GND #PWR0276
+L GND #PWR0280
 U 1 1 4E367505
 P 1680 6030
-F 0 "#PWR0276" H 1680 6030 30  0001 C CNN
+F 0 "#PWR0280" H 1680 6030 30  0001 C CNN
 F 1 "GND" H 1680 5960 30  0001 C CNN
 	1    1680 6030
@@
 5V to 1V0 @ 0.6A
 $Comp
-L +3.3V_PG #PWR0277
+L +3.3V_PG #PWR0281
 U 1 1 4E3674FF
 P 930 5510
-F 0 "#PWR0277" H 930 5470 30  0001 C CNN
+F 0 "#PWR0281" H 930 5470 30  0001 C CNN
 F 1 "+3.3V_PG" H 930 5640 30  0000 C CNN
 	1    930  5510
@@
 NoConn ~ 6960 3610
 $Comp
-L +3.3V #PWR0278
+L +3.3V #PWR0282
 U 1 1 4E3673AC
 P 6680 2020
-F 0 "#PWR0278" H 6680 1980 30  0001 C CNN
+F 0 "#PWR0282" H 6680 1980 30  0001 C CNN
 F 1 "+3.3V" H 6680 2130 30  0000 C CNN
 	1    6680 2020
@@
 $EndComp
 $Comp
-L +3.3V #PWR0279
+L +3.3V #PWR0283
 U 1 1 4E36736F
 P 3820 3360
-F 0 "#PWR0279" H 3820 3320 30  0001 C CNN
+F 0 "#PWR0283" H 3820 3320 30  0001 C CNN
 F 1 "+3.3V" H 3820 3470 30  0000 C CNN
 	1    3820 3360
@@
 $EndComp
 $Comp
-L +3.3V_PG #PWR0280
+L +3.3V_PG #PWR0284
 U 1 1 4E36735E
 P 930 3990
-F 0 "#PWR0280" H 930 3950 30  0001 C CNN
+F 0 "#PWR0284" H 930 3950 30  0001 C CNN
 F 1 "+3.3V_PG" H 930 4120 30  0000 C CNN
 	1    930  3990
@@
 $EndComp
 $Comp
-L GND #PWR0281
+L GND #PWR0285
 U 1 1 4E36734A
 P 1680 4510
-F 0 "#PWR0281" H 1680 4510 30  0001 C CNN
+F 0 "#PWR0285" H 1680 4510 30  0001 C CNN
 F 1 "GND" H 1680 4440 30  0001 C CNN
 	1    1680 4510
@@
 $EndComp
 $Comp
-L +5V #PWR0282
+L +5V #PWR0286
 U 1 1 4E367348
 P 630 3280
-F 0 "#PWR0282" H 630 3370 20  0001 C CNN
+F 0 "#PWR0286" H 630 3370 20  0001 C CNN
 F 1 "+5V" H 630 3370 30  0000 C CNN
 	1    630  3280
@@
 $EndComp
 $Comp
-L NC7WZ07 U1402
-U 1 1 4E366E41
-P 1630 2490
-F 0 "U1402" H 1330 2890 60  0000 C CNN
-F 1 "NC7WZ07" H 1480 2090 60  0000 C CNN
-	1    1630 2490
-	1    0    0    -1
-$EndComp
-$Comp
 L NC7WZ17 U1401
 U 1 1 4E366E40
@@
 $EndComp
 $Comp
-L +3.3V #PWR0283
+L +3.3V #PWR0287
 U 1 1 4E366E3F
 P 2280 690
-F 0 "#PWR0283" H 2280 650 30  0001 C CNN
+F 0 "#PWR0287" H 2280 650 30  0001 C CNN
 F 1 "+3.3V" H 2280 800 30  0000 C CNN
 	1    2280 690
@@
 $EndComp
 $Comp
-L +3.3V #PWR0284
+L +3.3V #PWR0288
 U 1 1 4E366E3E
 P 2280 2010
-F 0 "#PWR0284" H 2280 1970 30  0001 C CNN
+F 0 "#PWR0288" H 2280 1970 30  0001 C CNN
 F 1 "+3.3V" H 2280 2120 30  0000 C CNN
 	1    2280 2010
@@
 $EndComp
 $Comp
-L GND #PWR0285
+L GND #PWR0289
 U 1 1 4E366E3D
 P 2280 1620
-F 0 "#PWR0285" H 2280 1620 30  0001 C CNN
+F 0 "#PWR0289" H 2280 1620 30  0001 C CNN
 F 1 "GND" H 2280 1550 30  0001 C CNN
 	1    2280 1620
@@
 $EndComp
 $Comp
-L GND #PWR0286
+L GND #PWR0290
 U 1 1 4E366E3C
 P 2280 2940
-F 0 "#PWR0286" H 2280 2940 30  0001 C CNN
+F 0 "#PWR0290" H 2280 2940 30  0001 C CNN
 F 1 "GND" H 2280 2870 30  0001 C CNN
 	1    2280 2940
@@
 JTAG Buffering
 $Comp
-L R R1401
-U 1 1 4E366E3B
-P 2470 1990
-F 0 "R1401" V 2550 1990 50  0000 C CNN
-F 1 "10k" V 2470 1990 50  0000 C CNN
-	1    2470 1990
-	1    0    0    -1
-$EndComp
-$Comp
-L R R1402
-U 1 1 4E366E3A
-P 2650 1990
-F 0 "R1402" V 2730 1990 50  0000 C CNN
-F 1 "10k" V 2650 1990 50  0000 C CNN
-	1    2650 1990
-	1    0    0    -1
-$EndComp
-$Comp
-L +3.3V #PWR0287
-U 1 1 4E366E39
-P 2830 1740
-F 0 "#PWR0287" H 2830 1700 30  0001 C CNN
-F 1 "+3.3V" H 2830 1850 30  0000 C CNN
-	1    2830 1740
-	1    0    0    -1
-$EndComp
-$Comp
 L XS1-L1-128 U1407

Commit message: about to try add in new power island zones
Connections:
- net TCK: now also U1401.3 (A2); no longer U1401.1 (A1)
- net TCK_BUF: now also U1401.4 (Y2); no longer U1401.6 (Y1)
- net TMS: now also U1401.1 (A1); no longer U1401.3 (A2)
- net TMS_BUF: now also U1401.6 (Y1); no longer U1401.4 (Y2)
Changed lines of the file:
@@
-EESchema Schematic File Version 2  date 23/08/2011 16:52:50
+EESchema Schematic File Version 2  date 24/08/2011 15:41:50
 LIBS:power
 LIBS:device
@@
 Sheet 14 14
 Title ""
-Date "23 aug 2011"
+Date "24 aug 2011"
 Rev ""
 Comp ""
@@
 Comment4 ""
 $EndDescr
+Text HLabel 940  1070 0    39   Input ~ 0
+TMS
 $Comp
 L NC7WZ17 U1402
@@
 CLK_20M
 $Comp
-L +3.3V #PWR0260
+L +3.3V #PWR1425
 U 1 1 4E4BD358
 P 8430 3700
-F 0 "#PWR0260" H 8430 3660 30  0001 C CNN
+F 0 "#PWR1425" H 8430 3660 30  0001 C CNN
 F 1 "+3.3V" H 8430 3810 30  0000 C CNN
 	1    8430 3700
@@
 RST_N_BUF
 $Comp
-L +3.3V #PWR0261
+L +3.3V #PWR1419
 U 1 1 4E36A392
 P 6730 4620
-F 0 "#PWR0261" H 6730 4580 30  0001 C CNN
+F 0 "#PWR1419" H 6730 4580 30  0001 C CNN
 F 1 "+3.3V" H 6730 4730 30  0000 C CNN
 	1    6730 4620
@@
 $EndComp
 $Comp
-L +1V0 #PWR0262
+L +1V0 #PWR1429
 U 1 1 4E3688F5
 P 8950 2270
-F 0 "#PWR0262" H 8950 2230 30  0001 C CNN
+F 0 "#PWR1429" H 8950 2230 30  0001 C CNN
 F 1 "+1V0" H 8950 2400 30  0000 C CNN
 	1    8950 2270
@@
 $EndComp
 $Comp
-L GND #PWR0263
+L GND #PWR1423
 U 1 1 4E3688DC
 P 8260 3690
-F 0 "#PWR0263" H 8260 3690 30  0001 C CNN
+F 0 "#PWR1423" H 8260 3690 30  0001 C CNN
 F 1 "GND" H 8260 3620 30  0001 C CNN
 	1    8260 3690
@@
 $EndComp
 $Comp
-L +3.3V #PWR0264
+L +3.3V #PWR1428
 U 1 1 4E3688B7
 P 8690 3190
-F 0 "#PWR0264" H 8690 3150 30  0001 C CNN
+F 0 "#PWR1428" H 8690 3150 30  0001 C CNN
 F 1 "+3.3V" H 8690 3290 30  0000 C CNN
 	1    8690 3190
@@
 $EndComp
 $Comp
-L +1V0 #PWR0265
+L +1V0 #PWR1426
 U 1 1 4E36889D
 P 8530 3190
-F 0 "#PWR0265" H 8530 3150 30  0001 C CNN
+F 0 "#PWR1426" H 8530 3150 30  0001 C CNN
 F 1 "+1V0" H 8530 3290 30  0000 C CNN
 	1    8530 3190
@@
 NoConn ~ 8260 3110
 $Comp
-L +3.3V #PWR0266
+L +3.3V #PWR1427
 U 1 1 4E36886B
 P 8540 2920
-F 0 "#PWR0266" H 8540 2880 30  0001 C CNN
+F 0 "#PWR1427" H 8540 2880 30  0001 C CNN
 F 1 "+3.3V" H 8540 3030 30  0000 C CNN
 	1    8540 2920
@@
 $EndComp
 $Comp
-L GND #PWR0267
+L GND #PWR1424
 U 1 1 4E3687FE
 P 8350 2890
-F 0 "#PWR0267" H 8350 2890 30  0001 C CNN
+F 0 "#PWR1424" H 8350 2890 30  0001 C CNN
 F 1 "GND" H 8350 2820 30  0001 C CNN
 	1    8350 2890
@@
 $EndComp
 $Comp
-L +1V0 #PWR0268
+L +1V0 #PWR1420
 U 1 1 4E3687CA
 P 6880 810
-F 0 "#PWR0268" H 6880 770 30  0001 C CNN
+F 0 "#PWR1420" H 6880 770 30  0001 C CNN
 F 1 "+1V0" H 6880 940 30  0000 C CNN
 	1    6880 810
@@
 $EndComp
 $Comp
-L +1V0 #PWR0269
+L +1V0 #PWR1421
 U 1 1 4E3686DE
 P 7960 5960
-F 0 "#PWR0269" H 7960 5920 30  0001 C CNN
+F 0 "#PWR1421" H 7960 5920 30  0001 C CNN
 F 1 "+1V0" H 7960 6090 30  0000 C CNN
 	1    7960 5960
@@
 $EndComp
 $Comp
-L +3.3V #PWR0270
+L +3.3V #PWR1430
 U 1 1 4E3686D7
 P 9580 5960
-F 0 "#PWR0270" H 9580 5920 30  0001 C CNN
+F 0 "#PWR1430" H 9580 5920 30  0001 C CNN
 F 1 "+3.3V" H 9580 6070 30  0000 C CNN
 	1    9580 5960
@@
 $EndComp
 $Comp
-L GND #PWR0271
+L GND #PWR1422
 U 1 1 4E36868C
 P 8050 6570
-F 0 "#PWR0271" H 8050 6570 30  0001 C CNN
+F 0 "#PWR1422" H 8050 6570 30  0001 C CNN
 F 1 "GND" H 8050 6500 30  0001 C CNN
 	1    8050 6570
@@
 $EndComp
 $Comp
-L GND #PWR0272
+L GND #PWR1431
 U 1 1 4E36868B
 P 9670 6570
-F 0 "#PWR0272" H 9670 6570 30  0001 C CNN
+F 0 "#PWR1431" H 9670 6570 30  0001 C CNN
 F 1 "GND" H 9670 6500 30  0001 C CNN
 	1    9670 6570
@@
 $EndComp
 $Comp
-L +1V0 #PWR0273
+L +1V0 #PWR1413
 U 1 1 4E367E87
 P 3820 4880
-F 0 "#PWR0273" H 3820 4840 30  0001 C CNN
+F 0 "#PWR1413" H 3820 4840 30  0001 C CNN
 F 1 "+1V0" H 3820 5010 30  0000 C CNN
 	1    3820 4880
@@
 $EndComp
 $Comp
-L +3.3V #PWR0274
+L +3.3V #PWR1417
 U 1 1 4E367E10
 P 5220 600
-F 0 "#PWR0274" H 5220 560 30  0001 C CNN
+F 0 "#PWR1417" H 5220 560 30  0001 C CNN
 F 1 "+3.3V" H 5220 710 30  0000 C CNN
 	1    5220 600
@@
 $EndComp
 $Comp
-L +3.3V_PG #PWR0275
+L +3.3V_PG #PWR1415
 U 1 1 4E367DE3
 P 4480 680
-F 0 "#PWR0275" H 4480 640 30  0001 C CNN
+F 0 "#PWR1415" H 4480 640 30  0001 C CNN
 F 1 "+3.3V_PG" H 4480 810 30  0000 C CNN
 	1    4480 680
@@
 $EndComp
 $Comp
-L +3.3V #PWR0276
+L +3.3V #PWR1411
 U 1 1 4E367DD1
 P 3370 880
-F 0 "#PWR0276" H 3370 840 30  0001 C CNN
+F 0 "#PWR1411" H 3370 840 30  0001 C CNN
 F 1 "+3.3V" H 3370 990 30  0000 C CNN
 	1    3370 880
@@
 $EndComp
 $Comp
-L GND #PWR0277
+L GND #PWR1414
 U 1 1 4E367DC7
 P 3990 1460
-F 0 "#PWR0277" H 3990 1460 30  0001 C CNN
+F 0 "#PWR1414" H 3990 1460 30  0001 C CNN
 F 1 "GND" H 3990 1390 30  0001 C CNN
 	1    3990 1460
@@
 $EndComp
 $Comp
-L GND #PWR0278
+L GND #PWR1416
 U 1 1 4E367DC6
 P 5200 1460
-F 0 "#PWR0278" H 5200 1460 30  0001 C CNN
+F 0 "#PWR1416" H 5200 1460 30  0001 C CNN
 F 1 "GND" H 5200 1390 30  0001 C CNN
 	1    5200 1460
@@
 RST_N_SPVSR
 $Comp
-L +5V #PWR0279
+L +5V #PWR1402
 U 1 1 4E367507
 P 630 4800
-F 0 "#PWR0279" H 630 4890 20  0001 C CNN
+F 0 "#PWR1402" H 630 4890 20  0001 C CNN
 F 1 "+5V" H 630 4890 30  0000 C CNN
 	1    630  4800
@@
 $EndComp
 $Comp
-L GND #PWR0280
+L GND #PWR1406
 U 1 1 4E367505
 P 1680 6030
-F 0 "#PWR0280" H 1680 6030 30  0001 C CNN
+F 0 "#PWR1406" H 1680 6030 30  0001 C CNN
 F 1 "GND" H 1680 5960 30  0001 C CNN
 	1    1680 6030
@@
 5V to 1V0 @ 0.6A
 $Comp
-L +3.3V_PG #PWR0281
+L +3.3V_PG #PWR1404
 U 1 1 4E3674FF
 P 930 5510
-F 0 "#PWR0281" H 930 5470 30  0001 C CNN
+F 0 "#PWR1404" H 930 5470 30  0001 C CNN
 F 1 "+3.3V_PG" H 930 5640 30  0000 C CNN
 	1    930  5510
@@
 NoConn ~ 6960 3610
 $Comp
-L +3.3V #PWR0282
+L +3.3V #PWR1418
 U 1 1 4E3673AC
 P 6680 2020
-F 0 "#PWR0282" H 6680 1980 30  0001 C CNN
+F 0 "#PWR1418" H 6680 1980 30  0001 C CNN
 F 1 "+3.3V" H 6680 2130 30  0000 C CNN
 	1    6680 2020
@@
 $EndComp
 $Comp
-L +3.3V #PWR0283
+L +3.3V #PWR1412
 U 1 1 4E36736F
 P 3820 3360
-F 0 "#PWR0283" H 3820 3320 30  0001 C CNN
+F 0 "#PWR1412" H 3820 3320 30  0001 C CNN
 F 1 "+3.3V" H 3820 3470 30  0000 C CNN
 	1    3820 3360
@@
 $EndComp
 $Comp
-L +3.3V_PG #PWR0284
+L +3.3V_PG #PWR1403
 U 1 1 4E36735E
 P 930 3990
-F 0 "#PWR0284" H 930 3950 30  0001 C CNN
+F 0 "#PWR1403" H 930 3950 30  0001 C CNN
 F 1 "+3.3V_PG" H 930 4120 30  0000 C CNN
 	1    930  3990
@@
 $EndComp
 $Comp
-L GND #PWR0285
+L GND #PWR1405
 U 1 1 4E36734A
 P 1680 4510
-F 0 "#PWR0285" H 1680 4510 30  0001 C CNN
+F 0 "#PWR1405" H 1680 4510 30  0001 C CNN
 F 1 "GND" H 1680 4440 30  0001 C CNN
 	1    1680 4510
@@
 $EndComp
 $Comp
-L +5V #PWR0286
+L +5V #PWR1401
 U 1 1 4E367348
 P 630 3280
-F 0 "#PWR0286" H 630 3370 20  0001 C CNN
+F 0 "#PWR1401" H 630 3370 20  0001 C CNN
 F 1 "+5V" H 630 3370 30  0000 C CNN
 	1    630  3280
@@
 $EndComp
 $Comp
-L +3.3V #PWR0287
+L +3.3V #PWR1407
 U 1 1 4E366E3F
 P 2280 690
-F 0 "#PWR0287" H 2280 650 30  0001 C CNN
+F 0 "#PWR1407" H 2280 650 30  0001 C CNN
 F 1 "+3.3V" H 2280 800 30  0000 C CNN
 	1    2280 690
@@
 $EndComp
 $Comp
-L +3.3V #PWR0288
+L +3.3V #PWR1409
 U 1 1 4E366E3E
 P 2280 2010
-F 0 "#PWR0288" H 2280 1970 30  0001 C CNN
+F 0 "#PWR1409" H 2280 1970 30  0001 C CNN
 F 1 "+3.3V" H 2280 2120 30  0000 C CNN
 	1    2280 2010
@@
 $EndComp
 $Comp
-L GND #PWR0289
+L GND #PWR1408
 U 1 1 4E366E3D
 P 2280 1620
-F 0 "#PWR0289" H 2280 1620 30  0001 C CNN
+F 0 "#PWR1408" H 2280 1620 30  0001 C CNN
 F 1 "GND" H 2280 1550 30  0001 C CNN
 	1    2280 1620
@@
 $EndComp
 $Comp
-L GND #PWR0290
+L GND #PWR1410
 U 1 1 4E366E3C
 P 2280 2940
-F 0 "#PWR0290" H 2280 2940 30  0001 C CNN
+F 0 "#PWR1410" H 2280 2940 30  0001 C CNN
 F 1 "GND" H 2280 2870 30  0001 C CNN
 	1    2280 2940
 	1    0    0    -1
 $EndComp
-Text HLabel 940  1070 0    39   Input ~ 0
+Text HLabel 940  1270 0    39   Input ~ 0
 TCK
-Text HLabel 940  1270 0    39   Input ~ 0
-TMS
+Text Label 2340 1270 0    39   ~ 0
+TCK_BUF
 Text Label 2340 1070 0    39   ~ 0
-TCK_BUF
-Text Label 2340 1270 0    39   ~ 0
 TMS_BUF
 Text HLabel 940  2590 0    39   Input ~ 0
