File: l2_dev_alternative/l1.sch (KiCad schematic (older format))
At the start: 33 parts, among them U1401 NC7WZ17, U1402 NC7WZ17, U1403 NCP1529, U1404 NCP1521B, U1405 APX803-SR, U1406 APX803-SR, U1407 XS1-L1-128

Commit message: need to check if L1 X-linkks need buffering
Parts:
- R1408: value 4.7 -> 4R7
- R1409: value R -> 10k
Changed lines of the file:
@@
-EESchema Schematic File Version 2  date 24/08/2011 17:10:00
+EESchema Schematic File Version 2  date 25/08/2011 15:54:37
 LIBS:power
 LIBS:device
@@
 Sheet 14 14
 Title ""
-Date "24 aug 2011"
+Date "25 aug 2011"
 Rev ""
 Comp ""
@@
 CLK_20M
 $Comp
-L +3.3V #PWR0260
+L +3.3V #PWR0264
 U 1 1 4E4BD358
 P 8430 3700
-F 0 "#PWR0260" H 8430 3660 30  0001 C CNN
+F 0 "#PWR0264" H 8430 3660 30  0001 C CNN
 F 1 "+3.3V" H 8430 3810 30  0000 C CNN
 	1    8430 3700
@@
 P 8430 3970
 F 0 "R1409" V 8510 3970 50  0000 C CNN
-F 1 "R" V 8430 3970 50  0000 C CNN
+F 1 "10k" V 8430 3970 50  0000 C CNN
 	1    8430 3970
 	1    0    0    -1
@@
 RST_N_BUF
 $Comp
-L +3.3V #PWR0261
+L +3.3V #PWR0265
 U 1 1 4E36A392
 P 6730 4620
-F 0 "#PWR0261" H 6730 4580 30  0001 C CNN
+F 0 "#PWR0265" H 6730 4580 30  0001 C CNN
 F 1 "+3.3V" H 6730 4730 30  0000 C CNN
 	1    6730 4620
@@
 P 8950 2600
 F 0 "R1408" V 9030 2600 50  0000 C CNN
-F 1 "4.7" V 8950 2600 50  0000 C CNN
+F 1 "4R7" V 8950 2600 50  0000 C CNN
 	1    8950 2600
 	1    0    0    -1
 $EndComp
 $Comp
-L +1V0 #PWR0262
+L +1V0 #PWR0266
 U 1 1 4E3688F5
 P 8950 2270
-F 0 "#PWR0262" H 8950 2230 30  0001 C CNN
+F 0 "#PWR0266" H 8950 2230 30  0001 C CNN
 F 1 "+1V0" H 8950 2400 30  0000 C CNN
 	1    8950 2270
@@
 $EndComp
 $Comp
-L GND #PWR0263
+L GND #PWR0267
 U 1 1 4E3688DC
 P 8260 3690
-F 0 "#PWR0263" H 8260 3690 30  0001 C CNN
+F 0 "#PWR0267" H 8260 3690 30  0001 C CNN
 F 1 "GND" H 8260 3620 30  0001 C CNN
 	1    8260 3690
@@
 $EndComp
 $Comp
-L +3.3V #PWR0264
+L +3.3V #PWR0268
 U 1 1 4E3688B7
 P 8690 3190
-F 0 "#PWR0264" H 8690 3150 30  0001 C CNN
+F 0 "#PWR0268" H 8690 3150 30  0001 C CNN
 F 1 "+3.3V" H 8690 3290 30  0000 C CNN
 	1    8690 3190
@@
 $EndComp
 $Comp
-L +1V0 #PWR0265
+L +1V0 #PWR0269
 U 1 1 4E36889D
 P 8530 3190
-F 0 "#PWR0265" H 8530 3150 30  0001 C CNN
+F 0 "#PWR0269" H 8530 3150 30  0001 C CNN
 F 1 "+1V0" H 8530 3290 30  0000 C CNN
 	1    8530 3190
@@
 NoConn ~ 8260 3110
 $Comp
-L +3.3V #PWR0266
+L +3.3V #PWR0270
 U 1 1 4E36886B
 P 8540 2920
-F 0 "#PWR0266" H 8540 2880 30  0001 C CNN
+F 0 "#PWR0270" H 8540 2880 30  0001 C CNN
 F 1 "+3.3V" H 8540 3030 30  0000 C CNN
 	1    8540 2920
@@
 $EndComp
 $Comp
-L GND #PWR0267
+L GND #PWR0271
 U 1 1 4E3687FE
 P 8350 2890
-F 0 "#PWR0267" H 8350 2890 30  0001 C CNN
+F 0 "#PWR0271" H 8350 2890 30  0001 C CNN
 F 1 "GND" H 8350 2820 30  0001 C CNN
 	1    8350 2890
@@
 $EndComp
 $Comp
-L +1V0 #PWR0268
+L +1V0 #PWR0272
 U 1 1 4E3687CA
 P 6880 810
-F 0 "#PWR0268" H 6880 770 30  0001 C CNN
+F 0 "#PWR0272" H 6880 770 30  0001 C CNN
 F 1 "+1V0" H 6880 940 30  0000 C CNN
 	1    6880 810
@@
 $EndComp
 $Comp
-L +1V0 #PWR0269
+L +1V0 #PWR0273
 U 1 1 4E3686DE
 P 7960 5960
-F 0 "#PWR0269" H 7960 5920 30  0001 C CNN
+F 0 "#PWR0273" H 7960 5920 30  0001 C CNN
 F 1 "+1V0" H 7960 6090 30  0000 C CNN
 	1    7960 5960
@@
 $EndComp
 $Comp
-L +3.3V #PWR0270
+L +3.3V #PWR0274
 U 1 1 4E3686D7
 P 9580 5960
-F 0 "#PWR0270" H 9580 5920 30  0001 C CNN
+F 0 "#PWR0274" H 9580 5920 30  0001 C CNN
 F 1 "+3.3V" H 9580 6070 30  0000 C CNN
 	1    9580 5960
@@
 $EndComp
 $Comp
-L GND #PWR0271
+L GND #PWR0275
 U 1 1 4E36868C
 P 8050 6570
-F 0 "#PWR0271" H 8050 6570 30  0001 C CNN
+F 0 "#PWR0275" H 8050 6570 30  0001 C CNN
 F 1 "GND" H 8050 6500 30  0001 C CNN
 	1    8050 6570
@@
 $EndComp
 $Comp
-L GND #PWR0272
+L GND #PWR0276
 U 1 1 4E36868B
 P 9670 6570
-F 0 "#PWR0272" H 9670 6570 30  0001 C CNN
+F 0 "#PWR0276" H 9670 6570 30  0001 C CNN
 F 1 "GND" H 9670 6500 30  0001 C CNN
 	1    9670 6570
@@
 $EndComp
 $Comp
-L +1V0 #PWR0273
+L +1V0 #PWR0277
 U 1 1 4E367E87
 P 3820 4880
-F 0 "#PWR0273" H 3820 4840 30  0001 C CNN
+F 0 "#PWR0277" H 3820 4840 30  0001 C CNN
 F 1 "+1V0" H 3820 5010 30  0000 C CNN
 	1    3820 4880
@@
 $EndComp
 $Comp
-L +3.3V #PWR0274
+L +3.3V #PWR0278
 U 1 1 4E367E10
 P 5220 600
-F 0 "#PWR0274" H 5220 560 30  0001 C CNN
+F 0 "#PWR0278" H 5220 560 30  0001 C CNN
 F 1 "+3.3V" H 5220 710 30  0000 C CNN
 	1    5220 600
@@
 $EndComp
 $Comp
-L +3.3V_PG #PWR0275
+L +3.3V_PG #PWR0279
 U 1 1 4E367DE3
 P 4480 680
-F 0 "#PWR0275" H 4480 640 30  0001 C CNN
+F 0 "#PWR0279" H 4480 640 30  0001 C CNN
 F 1 "+3.3V_PG" H 4480 810 30  0000 C CNN
 	1    4480 680
@@
 $EndComp
 $Comp
-L +3.3V #PWR0276
+L +3.3V #PWR0280
 U 1 1 4E367DD1
 P 3370 880
-F 0 "#PWR0276" H 3370 840 30  0001 C CNN
+F 0 "#PWR0280" H 3370 840 30  0001 C CNN
 F 1 "+3.3V" H 3370 990 30  0000 C CNN
 	1    3370 880
@@
 $EndComp
 $Comp
-L GND #PWR0277
+L GND #PWR0281
 U 1 1 4E367DC7
 P 3990 1460
-F 0 "#PWR0277" H 3990 1460 30  0001 C CNN
+F 0 "#PWR0281" H 3990 1460 30  0001 C CNN
 F 1 "GND" H 3990 1390 30  0001 C CNN
 	1    3990 1460
@@
 $EndComp
 $Comp
-L GND #PWR0278
+L GND #PWR0282
 U 1 1 4E367DC6
 P 5200 1460
-F 0 "#PWR0278" H 5200 1460 30  0001 C CNN
+F 0 "#PWR0282" H 5200 1460 30  0001 C CNN
 F 1 "GND" H 5200 1390 30  0001 C CNN
 	1    5200 1460
@@
 RST_N_SPVSR
 $Comp
-L +5V #PWR0279
+L +5V #PWR0283
 U 1 1 4E367507
 P 630 4800
-F 0 "#PWR0279" H 630 4890 20  0001 C CNN
+F 0 "#PWR0283" H 630 4890 20  0001 C CNN
 F 1 "+5V" H 630 4890 30  0000 C CNN
 	1    630  4800
@@
 $EndComp
 $Comp
-L GND #PWR0280
+L GND #PWR0284
 U 1 1 4E367505
 P 1680 6030
-F 0 "#PWR0280" H 1680 6030 30  0001 C CNN
+F 0 "#PWR0284" H 1680 6030 30  0001 C CNN
 F 1 "GND" H 1680 5960 30  0001 C CNN
 	1    1680 6030
@@
 F 0 "L1402" V 2730 4970 40  0000 C CNN
 F 1 "2u2H" V 2880 4970 40  0000 C CNN
+F 3 "http://www.tdk.co.jp/tefe02/e533_mlz2012.pdf" H 2780 4970 60  0001 C CNN
 	1    2780 4970
 	0    -1   -1   0
@@
 5V to 1V0 @ 0.6A
 $Comp
-L +3.3V_PG #PWR0281
+L +3.3V_PG #PWR0285
 U 1 1 4E3674FF
 P 930 5510
-F 0 "#PWR0281" H 930 5470 30  0001 C CNN
+F 0 "#PWR0285" H 930 5470 30  0001 C CNN
 F 1 "+3.3V_PG" H 930 5640 30  0000 C CNN
 	1    930  5510
@@
 NoConn ~ 6960 3610
 $Comp
-L +3.3V #PWR0282
+L +3.3V #PWR0286
 U 1 1 4E3673AC
 P 6680 2020
-F 0 "#PWR0282" H 6680 1980 30  0001 C CNN
+F 0 "#PWR0286" H 6680 1980 30  0001 C CNN
 F 1 "+3.3V" H 6680 2130 30  0000 C CNN
 	1    6680 2020
@@
 $EndComp
 $Comp
-L +3.3V #PWR0283
+L +3.3V #PWR0287
 U 1 1 4E36736F
 P 3820 3360
-F 0 "#PWR0283" H 3820 3320 30  0001 C CNN
+F 0 "#PWR0287" H 3820 3320 30  0001 C CNN
 F 1 "+3.3V" H 3820 3470 30  0000 C CNN
 	1    3820 3360
@@
 $EndComp
 $Comp
-L +3.3V_PG #PWR0284
+L +3.3V_PG #PWR0288
 U 1 1 4E36735E
 P 930 3990
-F 0 "#PWR0284" H 930 3950 30  0001 C CNN
+F 0 "#PWR0288" H 930 3950 30  0001 C CNN
 F 1 "+3.3V_PG" H 930 4120 30  0000 C CNN
 	1    930  3990
@@
 $EndComp
 $Comp
-L GND #PWR0285
+L GND #PWR0289
 U 1 1 4E36734A
 P 1680 4510
-F 0 "#PWR0285" H 1680 4510 30  0001 C CNN
+F 0 "#PWR0289" H 1680 4510 30  0001 C CNN
 F 1 "GND" H 1680 4440 30  0001 C CNN
 	1    1680 4510
@@
 $EndComp
 $Comp
-L +5V #PWR0286
+L +5V #PWR0290
 U 1 1 4E367348
 P 630 3280
-F 0 "#PWR0286" H 630 3370 20  0001 C CNN
+F 0 "#PWR0290" H 630 3370 20  0001 C CNN
 F 1 "+5V" H 630 3370 30  0000 C CNN
 	1    630  3280
@@
 $EndComp
 $Comp
-L +3.3V #PWR0287
+L +3.3V #PWR0291
 U 1 1 4E366E3F
 P 2280 690
-F 0 "#PWR0287" H 2280 650 30  0001 C CNN
+F 0 "#PWR0291" H 2280 650 30  0001 C CNN
 F 1 "+3.3V" H 2280 800 30  0000 C CNN
 	1    2280 690
@@
 $EndComp
 $Comp
-L +3.3V #PWR0288
+L +3.3V #PWR0292
 U 1 1 4E366E3E
 P 2280 2010
-F 0 "#PWR0288" H 2280 1970 30  0001 C CNN
+F 0 "#PWR0292" H 2280 1970 30  0001 C CNN
 F 1 "+3.3V" H 2280 2120 30  0000 C CNN
 	1    2280 2010
@@
 $EndComp
 $Comp
-L GND #PWR0289
+L GND #PWR0293
 U 1 1 4E366E3D
 P 2280 1620
-F 0 "#PWR0289" H 2280 1620 30  0001 C CNN
+F 0 "#PWR0293" H 2280 1620 30  0001 C CNN
 F 1 "GND" H 2280 1550 30  0001 C CNN
 	1    2280 1620
@@
 $EndComp
 $Comp
-L GND #PWR0290
+L GND #PWR0294
 U 1 1 4E366E3C
 P 2280 2940
-F 0 "#PWR0290" H 2280 2940 30  0001 C CNN
+F 0 "#PWR0294" H 2280 2940 30  0001 C CNN
 F 1 "GND" H 2280 2870 30  0001 C CNN
 	1    2280 2940

Commit message: added pull ups for I2C bus, checking design over
Connections:
- net I2C_DATA: now reaches U1407.2 (X0D11)
- net I2C_CLK: now reaches U1407.37 (X0D0)
- no-connect marks 52 -> 50
Changed lines of the file:
@@
-EESchema Schematic File Version 2  date 25/08/2011 17:52:10
+EESchema Schematic File Version 2  date 30/08/2011 10:58:43
 LIBS:power
 LIBS:device
@@
 Sheet 14 14
 Title ""
-Date "25 aug 2011"
+Date "30 aug 2011"
 Rev ""
 Comp ""
@@
 Comment4 ""
 $EndDescr
+Wire Wire Line
+	10390 780  10520 780
+Text HLabel 10520 780  2    60   Input ~ 0
+I2C_CLK
+Text HLabel 10520 1880 2    60   Input ~ 0
+I2C_DATA
+Wire Wire Line
+	10390 1880 10520 1880
 Text HLabel 940  1070 0    39   Input ~ 0
 TMS
@@
 CLK_20M
 $Comp
-L +3.3V #PWR0260
+L +3.3V #PWR0267
 U 1 1 4E4BD358
 P 8430 3700
-F 0 "#PWR0260" H 8430 3660 30  0001 C CNN
+F 0 "#PWR0267" H 8430 3660 30  0001 C CNN
 F 1 "+3.3V" H 8430 3810 30  0000 C CNN
 	1    8430 3700
@@
 NoConn ~ 10390 3280
 NoConn ~ 10390 1980
-NoConn ~ 10390 1880
-NoConn ~ 10390 780
 NoConn ~ 9300 2480
 NoConn ~ 9300 2380
@@
 RST_N_BUF
 $Comp
-L +3.3V #PWR0261
+L +3.3V #PWR0268
 U 1 1 4E36A392
 P 6730 4620
-F 0 "#PWR0261" H 6730 4580 30  0001 C CNN
+F 0 "#PWR0268" H 6730 4580 30  0001 C CNN
 F 1 "+3.3V" H 6730 4730 30  0000 C CNN
 	1    6730 4620
@@
 $EndComp
 $Comp
-L +1V0 #PWR0262
+L +1V0 #PWR0269
 U 1 1 4E3688F5
 P 8950 2270
-F 0 "#PWR0262" H 8950 2230 30  0001 C CNN
+F 0 "#PWR0269" H 8950 2230 30  0001 C CNN
 F 1 "+1V0" H 8950 2400 30  0000 C CNN
 	1    8950 2270
@@
 $EndComp
 $Comp
-L GND #PWR0263
+L GND #PWR0270
 U 1 1 4E3688DC
 P 8260 3690
-F 0 "#PWR0263" H 8260 3690 30  0001 C CNN
+F 0 "#PWR0270" H 8260 3690 30  0001 C CNN
 F 1 "GND" H 8260 3620 30  0001 C CNN
 	1    8260 3690
@@
 $EndComp
 $Comp
-L +3.3V #PWR0264
+L +3.3V #PWR0271
 U 1 1 4E3688B7
 P 8690 3190
-F 0 "#PWR0264" H 8690 3150 30  0001 C CNN
+F 0 "#PWR0271" H 8690 3150 30  0001 C CNN
 F 1 "+3.3V" H 8690 3290 30  0000 C CNN
 	1    8690 3190
@@
 $EndComp
 $Comp
-L +1V0 #PWR0265
+L +1V0 #PWR0272
 U 1 1 4E36889D
 P 8530 3190
-F 0 "#PWR0265" H 8530 3150 30  0001 C CNN
+F 0 "#PWR0272" H 8530 3150 30  0001 C CNN
 F 1 "+1V0" H 8530 3290 30  0000 C CNN
 	1    8530 3190
@@
 NoConn ~ 8260 3110
 $Comp
-L +3.3V #PWR0266
+L +3.3V #PWR0273
 U 1 1 4E36886B
 P 8540 2920
-F 0 "#PWR0266" H 8540 2880 30  0001 C CNN
+F 0 "#PWR0273" H 8540 2880 30  0001 C CNN
 F 1 "+3.3V" H 8540 3030 30  0000 C CNN
 	1    8540 2920
@@
 $EndComp
 $Comp
-L GND #PWR0267
+L GND #PWR0274
 U 1 1 4E3687FE
 P 8350 2890
-F 0 "#PWR0267" H 8350 2890 30  0001 C CNN
+F 0 "#PWR0274" H 8350 2890 30  0001 C CNN
 F 1 "GND" H 8350 2820 30  0001 C CNN
 	1    8350 2890
@@
 $EndComp
 $Comp
-L +1V0 #PWR0268
+L +1V0 #PWR0275
 U 1 1 4E3687CA
 P 6880 810
-F 0 "#PWR0268" H 6880 770 30  0001 C CNN
+F 0 "#PWR0275" H 6880 770 30  0001 C CNN
 F 1 "+1V0" H 6880 940 30  0000 C CNN
 	1    6880 810
@@
 $EndComp
 $Comp
-L +1V0 #PWR0269
+L +1V0 #PWR0276
 U 1 1 4E3686DE
 P 7960 5960
-F 0 "#PWR0269" H 7960 5920 30  0001 C CNN
+F 0 "#PWR0276" H 7960 5920 30  0001 C CNN
 F 1 "+1V0" H 7960 6090 30  0000 C CNN
 	1    7960 5960
@@
 $EndComp
 $Comp
-L +3.3V #PWR0270
+L +3.3V #PWR0277
 U 1 1 4E3686D7
 P 9580 5960
-F 0 "#PWR0270" H 9580 5920 30  0001 C CNN
+F 0 "#PWR0277" H 9580 5920 30  0001 C CNN
 F 1 "+3.3V" H 9580 6070 30  0000 C CNN
 	1    9580 5960
@@
 $EndComp
 $Comp
-L GND #PWR0271
+L GND #PWR0278
 U 1 1 4E36868C
 P 8050 6570
-F 0 "#PWR0271" H 8050 6570 30  0001 C CNN
+F 0 "#PWR0278" H 8050 6570 30  0001 C CNN
 F 1 "GND" H 8050 6500 30  0001 C CNN
 	1    8050 6570
@@
 $EndComp
 $Comp
-L GND #PWR0272
+L GND #PWR0279
 U 1 1 4E36868B
 P 9670 6570
-F 0 "#PWR0272" H 9670 6570 30  0001 C CNN
+F 0 "#PWR0279" H 9670 6570 30  0001 C CNN
 F 1 "GND" H 9670 6500 30  0001 C CNN
 	1    9670 6570
@@
 $EndComp
 $Comp
-L +1V0 #PWR0273
+L +1V0 #PWR0280
 U 1 1 4E367E87
 P 3820 4880
-F 0 "#PWR0273" H 3820 4840 30  0001 C CNN
+F 0 "#PWR0280" H 3820 4840 30  0001 C CNN
 F 1 "+1V0" H 3820 5010 30  0000 C CNN
 	1    3820 4880
@@
 $EndComp
 $Comp
-L +3.3V #PWR0274
+L +3.3V #PWR0281
 U 1 1 4E367E10
 P 5220 600
-F 0 "#PWR0274" H 5220 560 30  0001 C CNN
+F 0 "#PWR0281" H 5220 560 30  0001 C CNN
 F 1 "+3.3V" H 5220 710 30  0000 C CNN
 	1    5220 600
@@
 $EndComp
 $Comp
-L +3.3V_PG #PWR0275
+L +3.3V_PG #PWR0282
 U 1 1 4E367DE3
 P 4480 680
-F 0 "#PWR0275" H 4480 640 30  0001 C CNN
+F 0 "#PWR0282" H 4480 640 30  0001 C CNN
 F 1 "+3.3V_PG" H 4480 810 30  0000 C CNN
 	1    4480 680
@@
 $EndComp
 $Comp
-L +3.3V #PWR0276
+L +3.3V #PWR0283
 U 1 1 4E367DD1
 P 3370 880
-F 0 "#PWR0276" H 3370 840 30  0001 C CNN
+F 0 "#PWR0283" H 3370 840 30  0001 C CNN
 F 1 "+3.3V" H 3370 990 30  0000 C CNN
 	1    3370 880
@@
 $EndComp
 $Comp
-L GND #PWR0277
+L GND #PWR0284
 U 1 1 4E367DC7
 P 3990 1460
-F 0 "#PWR0277" H 3990 1460 30  0001 C CNN
+F 0 "#PWR0284" H 3990 1460 30  0001 C CNN
 F 1 "GND" H 3990 1390 30  0001 C CNN
 	1    3990 1460
@@
 $EndComp
 $Comp
-L GND #PWR0278
+L GND #PWR0285
 U 1 1 4E367DC6
 P 5200 1460
-F 0 "#PWR0278" H 5200 1460 30  0001 C CNN
+F 0 "#PWR0285" H 5200 1460 30  0001 C CNN
 F 1 "GND" H 5200 1390 30  0001 C CNN
 	1    5200 1460
@@
 RST_N_SPVSR
 $Comp
-L +5V #PWR0279
+L +5V #PWR0286
 U 1 1 4E367507
 P 630 4800
-F 0 "#PWR0279" H 630 4890 20  0001 C CNN
+F 0 "#PWR0286" H 630 4890 20  0001 C CNN
 F 1 "+5V" H 630 4890 30  0000 C CNN
 	1    630  4800
@@
 $EndComp
 $Comp
-L GND #PWR0280
+L GND #PWR0287
 U 1 1 4E367505
 P 1680 6030
-F 0 "#PWR0280" H 1680 6030 30  0001 C CNN
+F 0 "#PWR0287" H 1680 6030 30  0001 C CNN
 F 1 "GND" H 1680 5960 30  0001 C CNN
 	1    1680 6030
@@
 5V to 1V0 @ 0.6A
 $Comp
-L +3.3V_PG #PWR0281
+L +3.3V_PG #PWR0288
 U 1 1 4E3674FF
 P 930 5510
-F 0 "#PWR0281" H 930 5470 30  0001 C CNN
+F 0 "#PWR0288" H 930 5470 30  0001 C CNN
 F 1 "+3.3V_PG" H 930 5640 30  0000 C CNN
 	1    930  5510
@@
 NoConn ~ 6960 3610
 $Comp
-L +3.3V #PWR0282
+L +3.3V #PWR0289
 U 1 1 4E3673AC
 P 6680 2020
-F 0 "#PWR0282" H 6680 1980 30  0001 C CNN
+F 0 "#PWR0289" H 6680 1980 30  0001 C CNN
 F 1 "+3.3V" H 6680 2130 30  0000 C CNN
 	1    6680 2020
@@
 $EndComp
 $Comp
-L +3.3V #PWR0283
+L +3.3V #PWR0290
 U 1 1 4E36736F
 P 3820 3360
-F 0 "#PWR0283" H 3820 3320 30  0001 C CNN
+F 0 "#PWR0290" H 3820 3320 30  0001 C CNN
 F 1 "+3.3V" H 3820 3470 30  0000 C CNN
 	1    3820 3360
@@
 $EndComp
 $Comp
-L +3.3V_PG #PWR0284
+L +3.3V_PG #PWR0291
 U 1 1 4E36735E
 P 930 3990
-F 0 "#PWR0284" H 930 3950 30  0001 C CNN
+F 0 "#PWR0291" H 930 3950 30  0001 C CNN
 F 1 "+3.3V_PG" H 930 4120 30  0000 C CNN
 	1    930  3990
@@
 $EndComp
 $Comp
-L GND #PWR0285
+L GND #PWR0292
 U 1 1 4E36734A
 P 1680 4510
-F 0 "#PWR0285" H 1680 4510 30  0001 C CNN
+F 0 "#PWR0292" H 1680 4510 30  0001 C CNN
 F 1 "GND" H 1680 4440 30  0001 C CNN
 	1    1680 4510
@@
 $EndComp
 $Comp
-L +5V #PWR0286
+L +5V #PWR0293
 U 1 1 4E367348
 P 630 3280
-F 0 "#PWR0286" H 630 3370 20  0001 C CNN
+F 0 "#PWR0293" H 630 3370 20  0001 C CNN
 F 1 "+5V" H 630 3370 30  0000 C CNN
 	1    630  3280
@@
 $EndComp
 $Comp
-L +3.3V #PWR0287
+L +3.3V #PWR0294
 U 1 1 4E366E3F
 P 2280 690
-F 0 "#PWR0287" H 2280 650 30  0001 C CNN
+F 0 "#PWR0294" H 2280 650 30  0001 C CNN
 F 1 "+3.3V" H 2280 800 30  0000 C CNN
 	1    2280 690
@@
 $EndComp
 $Comp
-L +3.3V #PWR0288
+L +3.3V #PWR0295
 U 1 1 4E366E3E
 P 2280 2010
-F 0 "#PWR0288" H 2280 1970 30  0001 C CNN
+F 0 "#PWR0295" H 2280 1970 30  0001 C CNN
 F 1 "+3.3V" H 2280 2120 30  0000 C CNN
 	1    2280 2010
@@
 $EndComp
 $Comp
-L GND #PWR0289
+L GND #PWR0296
 U 1 1 4E366E3D
 P 2280 1620
-F 0 "#PWR0289" H 2280 1620 30  0001 C CNN
+F 0 "#PWR0296" H 2280 1620 30  0001 C CNN
 F 1 "GND" H 2280 1550 30  0001 C CNN
 	1    2280 1620
@@
 $EndComp
 $Comp
-L GND #PWR0290
+L GND #PWR0297
 U 1 1 4E366E3C
 P 2280 2940
-F 0 "#PWR0290" H 2280 2940 30  0001 C CNN
+F 0 "#PWR0297" H 2280 2940 30  0001 C CNN
 F 1 "GND" H 2280 2870 30  0001 C CNN
 	1    2280 2940
