File: l2_dev_alternative/l1.sch (KiCad schematic (older format))
At the start: 33 parts, among them U1401 NC7WZ17, U1402 NC7WZ17, U1403 NCP1529, U1404 NCP1521B, U1405 APX803-SR, U1406 APX803-SR, U1407 XS1-L1-128

Commit message: replaced single I2C bus with individual busses for high speed conversions
Connections:
- net I2C_DATA_1: now reaches U1407.115 (X0D15)
- net I2C_DATA_0: now reaches U1407.118 (X0D14)
- net I2C_DATA_3: now reaches U1407.90 (X0D21)
- net I2C_DATA_2: now reaches U1407.96 (X0D20)
- no-connect marks 50 -> 46
Changed lines of the file:
@@
-EESchema Schematic File Version 2  date 30/08/2011 13:51:36
+EESchema Schematic File Version 2  date 30/08/2011 17:05:00
 LIBS:power
 LIBS:device
@@
 $EndDescr
 Wire Wire Line
+	10390 1880 10520 1880
+Text HLabel 10520 1880 2    60   Input ~ 0
+I2C_DATA
+Wire Wire Line
+	10390 2780 10520 2780
+Text HLabel 10520 2780 2    60   Input ~ 0
+I2C_DATA_2
+Text HLabel 10520 2880 2    60   Input ~ 0
+I2C_DATA_3
+Wire Wire Line
+	10390 2880 10520 2880
+Wire Wire Line
+	10390 2280 10520 2280
+Text HLabel 10520 2280 2    60   Input ~ 0
+I2C_DATA_1
+Text HLabel 10520 2180 2    60   Input ~ 0
+I2C_DATA_0
+Wire Wire Line
 	10390 780  10520 780
 Text HLabel 10520 780  2    60   Input ~ 0
 I2C_CLK
-Text HLabel 10520 1880 2    60   Input ~ 0
-I2C_DATA
-Wire Wire Line
-	10390 1880 10520 1880
+Wire Wire Line
+	10390 2180 10520 2180
 Text HLabel 940  1070 0    39   Input ~ 0
 TMS
@@
 CLK_20M
 $Comp
-L +3.3V #PWR0300
+L +3.3V #PWR0299
 U 1 1 4E4BD358
 P 8430 3700
-F 0 "#PWR0300" H 8430 3660 30  0001 C CNN
+F 0 "#PWR0299" H 8430 3660 30  0001 C CNN
 F 1 "+3.3V" H 8430 3810 30  0000 C CNN
 	1    8430 3700
@@
 XLC_1o
 NoConn ~ 10390 2980
-NoConn ~ 10390 2880
-NoConn ~ 10390 2780
 Text HLabel 10520 2380 2    60   Input ~ 0
 XLB_1o
@@
 XLB_1i
 NoConn ~ 10390 2080
-NoConn ~ 10390 2180
-NoConn ~ 10390 2280
 NoConn ~ 10390 1780
 NoConn ~ 10390 1680
@@
 RST_N_BUF
 $Comp
-L +3.3V #PWR0301
+L +3.3V #PWR0300
 U 1 1 4E36A392
 P 6730 4620
-F 0 "#PWR0301" H 6730 4580 30  0001 C CNN
+F 0 "#PWR0300" H 6730 4580 30  0001 C CNN
 F 1 "+3.3V" H 6730 4730 30  0000 C CNN
 	1    6730 4620
@@
 $EndComp
 $Comp
-L +1V0 #PWR0302
+L +1V0 #PWR0301
 U 1 1 4E3688F5
 P 8950 2270
-F 0 "#PWR0302" H 8950 2230 30  0001 C CNN
+F 0 "#PWR0301" H 8950 2230 30  0001 C CNN
 F 1 "+1V0" H 8950 2400 30  0000 C CNN
 	1    8950 2270
@@
 $EndComp
 $Comp
-L GND #PWR0303
+L GND #PWR0302
 U 1 1 4E3688DC
 P 8260 3690
-F 0 "#PWR0303" H 8260 3690 30  0001 C CNN
+F 0 "#PWR0302" H 8260 3690 30  0001 C CNN
 F 1 "GND" H 8260 3620 30  0001 C CNN
 	1    8260 3690
@@
 $EndComp
 $Comp
-L +3.3V #PWR0304
+L +3.3V #PWR0303
 U 1 1 4E3688B7
 P 8690 3190
-F 0 "#PWR0304" H 8690 3150 30  0001 C CNN
+F 0 "#PWR0303" H 8690 3150 30  0001 C CNN
 F 1 "+3.3V" H 8690 3290 30  0000 C CNN
 	1    8690 3190
@@
 $EndComp
 $Comp
-L +1V0 #PWR0305
+L +1V0 #PWR0304
 U 1 1 4E36889D
 P 8530 3190
-F 0 "#PWR0305" H 8530 3150 30  0001 C CNN
+F 0 "#PWR0304" H 8530 3150 30  0001 C CNN
 F 1 "+1V0" H 8530 3290 30  0000 C CNN
 	1    8530 3190
@@
 NoConn ~ 8260 3110
 $Comp
-L +3.3V #PWR0306
+L +3.3V #PWR0305
 U 1 1 4E36886B
 P 8540 2920
-F 0 "#PWR0306" H 8540 2880 30  0001 C CNN
+F 0 "#PWR0305" H 8540 2880 30  0001 C CNN
 F 1 "+3.3V" H 8540 3030 30  0000 C CNN
 	1    8540 2920
@@
 $EndComp
 $Comp
-L GND #PWR0307
+L GND #PWR0306
 U 1 1 4E3687FE
 P 8350 2890
-F 0 "#PWR0307" H 8350 2890 30  0001 C CNN
+F 0 "#PWR0306" H 8350 2890 30  0001 C CNN
 F 1 "GND" H 8350 2820 30  0001 C CNN
 	1    8350 2890
@@
 $EndComp
 $Comp
-L +1V0 #PWR0308
+L +1V0 #PWR0307
 U 1 1 4E3687CA
 P 6880 810
-F 0 "#PWR0308" H 6880 770 30  0001 C CNN
+F 0 "#PWR0307" H 6880 770 30  0001 C CNN
 F 1 "+1V0" H 6880 940 30  0000 C CNN
 	1    6880 810
@@
 $EndComp
 $Comp
-L +1V0 #PWR0309
+L +1V0 #PWR0308
 U 1 1 4E3686DE
 P 7960 5960
-F 0 "#PWR0309" H 7960 5920 30  0001 C CNN
+F 0 "#PWR0308" H 7960 5920 30  0001 C CNN
 F 1 "+1V0" H 7960 6090 30  0000 C CNN
 	1    7960 5960
@@
 $EndComp
 $Comp
-L +3.3V #PWR0310
+L +3.3V #PWR0309
 U 1 1 4E3686D7
 P 9580 5960
-F 0 "#PWR0310" H 9580 5920 30  0001 C CNN
+F 0 "#PWR0309" H 9580 5920 30  0001 C CNN
 F 1 "+3.3V" H 9580 6070 30  0000 C CNN
 	1    9580 5960
@@
 $EndComp
 $Comp
-L GND #PWR0311
+L GND #PWR0310
 U 1 1 4E36868C
 P 8050 6570
-F 0 "#PWR0311" H 8050 6570 30  0001 C CNN
+F 0 "#PWR0310" H 8050 6570 30  0001 C CNN
 F 1 "GND" H 8050 6500 30  0001 C CNN
 	1    8050 6570
@@
 $EndComp
 $Comp
-L GND #PWR0312
+L GND #PWR0311
 U 1 1 4E36868B
 P 9670 6570
-F 0 "#PWR0312" H 9670 6570 30  0001 C CNN
+F 0 "#PWR0311" H 9670 6570 30  0001 C CNN
 F 1 "GND" H 9670 6500 30  0001 C CNN
 	1    9670 6570
@@
 $EndComp
 $Comp
-L +1V0 #PWR0313
+L +1V0 #PWR0312
 U 1 1 4E367E87
 P 3820 4880
-F 0 "#PWR0313" H 3820 4840 30  0001 C CNN
+F 0 "#PWR0312" H 3820 4840 30  0001 C CNN
 F 1 "+1V0" H 3820 5010 30  0000 C CNN
 	1    3820 4880
@@
 $EndComp
 $Comp
-L +3.3V #PWR0314
+L +3.3V #PWR0313
 U 1 1 4E367E10
 P 5220 600
-F 0 "#PWR0314" H 5220 560 30  0001 C CNN
+F 0 "#PWR0313" H 5220 560 30  0001 C CNN
 F 1 "+3.3V" H 5220 710 30  0000 C CNN
 	1    5220 600
@@
 $EndComp
 $Comp
-L +3.3V_PG #PWR0315
+L +3.3V_PG #PWR0314
 U 1 1 4E367DE3
 P 4480 680
-F 0 "#PWR0315" H 4480 640 30  0001 C CNN
+F 0 "#PWR0314" H 4480 640 30  0001 C CNN
 F 1 "+3.3V_PG" H 4480 810 30  0000 C CNN
 	1    4480 680
@@
 $EndComp
 $Comp
-L +3.3V #PWR0316
+L +3.3V #PWR0315
 U 1 1 4E367DD1
 P 3370 880
-F 0 "#PWR0316" H 3370 840 30  0001 C CNN
+F 0 "#PWR0315" H 3370 840 30  0001 C CNN
 F 1 "+3.3V" H 3370 990 30  0000 C CNN
 	1    3370 880
@@
 $EndComp
 $Comp
-L GND #PWR0317
+L GND #PWR0316
 U 1 1 4E367DC7
 P 3990 1460
-F 0 "#PWR0317" H 3990 1460 30  0001 C CNN
+F 0 "#PWR0316" H 3990 1460 30  0001 C CNN
 F 1 "GND" H 3990 1390 30  0001 C CNN
 	1    3990 1460
@@
 $EndComp
 $Comp
-L GND #PWR0318
+L GND #PWR0317
 U 1 1 4E367DC6
 P 5200 1460
-F 0 "#PWR0318" H 5200 1460 30  0001 C CNN
+F 0 "#PWR0317" H 5200 1460 30  0001 C CNN
 F 1 "GND" H 5200 1390 30  0001 C CNN
 	1    5200 1460
@@
 RST_N_SPVSR
 $Comp
-L +5V #PWR0319
+L +5V #PWR0318
 U 1 1 4E367507
 P 630 4800
-F 0 "#PWR0319" H 630 4890 20  0001 C CNN
+F 0 "#PWR0318" H 630 4890 20  0001 C CNN
 F 1 "+5V" H 630 4890 30  0000 C CNN
 	1    630  4800
@@
 $EndComp
 $Comp
-L GND #PWR0320
+L GND #PWR0319
 U 1 1 4E367505
 P 1680 6030
-F 0 "#PWR0320" H 1680 6030 30  0001 C CNN
+F 0 "#PWR0319" H 1680 6030 30  0001 C CNN
 F 1 "GND" H 1680 5960 30  0001 C CNN
 	1    1680 6030
@@
 5V to 1V0 @ 0.6A
 $Comp
-L +3.3V_PG #PWR0321
+L +3.3V_PG #PWR0320
 U 1 1 4E3674FF
 P 930 5510
-F 0 "#PWR0321" H 930 5470 30  0001 C CNN
+F 0 "#PWR0320" H 930 5470 30  0001 C CNN
 F 1 "+3.3V_PG" H 930 5640 30  0000 C CNN
 	1    930  5510
@@
 NoConn ~ 6960 3610
 $Comp
-L +3.3V #PWR0322
+L +3.3V #PWR0321
 U 1 1 4E3673AC
 P 6680 2020
-F 0 "#PWR0322" H 6680 1980 30  0001 C CNN
+F 0 "#PWR0321" H 6680 1980 30  0001 C CNN
 F 1 "+3.3V" H 6680 2130 30  0000 C CNN
 	1    6680 2020
@@
 $EndComp
 $Comp
-L +3.3V #PWR0323
+L +3.3V #PWR0322
 U 1 1 4E36736F
 P 3820 3360
-F 0 "#PWR0323" H 3820 3320 30  0001 C CNN
+F 0 "#PWR0322" H 3820 3320 30  0001 C CNN
 F 1 "+3.3V" H 3820 3470 30  0000 C CNN
 	1    3820 3360
@@
 $EndComp
 $Comp
-L +3.3V_PG #PWR0324
+L +3.3V_PG #PWR0323
 U 1 1 4E36735E
 P 930 3990
-F 0 "#PWR0324" H 930 3950 30  0001 C CNN
+F 0 "#PWR0323" H 930 3950 30  0001 C CNN
 F 1 "+3.3V_PG" H 930 4120 30  0000 C CNN
 	1    930  3990
@@
 $EndComp
 $Comp
-L GND #PWR0325
+L GND #PWR0324
 U 1 1 4E36734A
 P 1680 4510
-F 0 "#PWR0325" H 1680 4510 30  0001 C CNN
+F 0 "#PWR0324" H 1680 4510 30  0001 C CNN
 F 1 "GND" H 1680 4440 30  0001 C CNN
 	1    1680 4510
@@
 $EndComp
 $Comp
-L +5V #PWR0326
+L +5V #PWR0325
 U 1 1 4E367348
 P 630 3280
-F 0 "#PWR0326" H 630 3370 20  0001 C CNN
+F 0 "#PWR0325" H 630 3370 20  0001 C CNN
 F 1 "+5V" H 630 3370 30  0000 C CNN
 	1    630  3280
@@
 $EndComp
 $Comp
-L +3.3V #PWR0327
+L +3.3V #PWR0326
 U 1 1 4E366E3F
 P 2280 690
-F 0 "#PWR0327" H 2280 650 30  0001 C CNN
+F 0 "#PWR0326" H 2280 650 30  0001 C CNN
 F 1 "+3.3V" H 2280 800 30  0000 C CNN
 	1    2280 690
@@
 $EndComp
 $Comp
-L +3.3V #PWR0328
+L +3.3V #PWR0327
 U 1 1 4E366E3E
 P 2280 2010
-F 0 "#PWR0328" H 2280 1970 30  0001 C CNN
+F 0 "#PWR0327" H 2280 1970 30  0001 C CNN
 F 1 "+3.3V" H 2280 2120 30  0000 C CNN
 	1    2280 2010
@@
 $EndComp
 $Comp
-L GND #PWR0329
+L GND #PWR0328
 U 1 1 4E366E3D
 P 2280 1620
-F 0 "#PWR0329" H 2280 1620 30  0001 C CNN
+F 0 "#PWR0328" H 2280 1620 30  0001 C CNN
 F 1 "GND" H 2280 1550 30  0001 C CNN
 	1    2280 1620
@@
 $EndComp
 $Comp
-L GND #PWR0330
+L GND #PWR0329
 U 1 1 4E366E3C
 P 2280 2940
-F 0 "#PWR0330" H 2280 2940 30  0001 C CNN
+F 0 "#PWR0329" H 2280 2940 30  0001 C CNN
 F 1 "GND" H 2280 2870 30  0001 C CNN
 	1    2280 2940
