File: l2_dev_alternative/l2.sch (KiCad schematic (older format))
At the start: 13 parts, among them U301 XS1_L2-QFN124

Commit message: save before adding in LEDs in Layout
Parts:
- added D302, D303, D304, D401: LED, symbol LED
- added R303, R304, R305, R402: 1k, symbol R
Connections:
- net GND: now also D302.2 (K), D303.2 (K), D304.2 (K), D401.2 (K)
- net LED_0: now reaches U301.B18 (X1D28)
- net LED_0: now also R305.1
- net LED_1: now reaches U301.B19 (X1D29)
- net LED_1: now also R304.1
- net LED_2: now reaches U301.B20 (X1D30)
- net LED_2: now also R303.1
- net LED_3: now reaches U301.B21 (X1D31)
- net LED_3: now also R402.1
- new net: D401.1 (A), R402.2
- new net: D302.1 (A), R303.2
- new net: D303.1 (A), R304.2
- new net: D304.1 (A), R305.2
- no-connect marks 50 -> 46
Other:
- note added: "LED_ARRAY"
