File: l2_dev_alternative/l2.sch (KiCad schematic (older format))
At the start: 21 parts, among them U301 XS1_L2-QFN124

Commit message: copied over new files from basic board
Parts:
- C301: value 1uF -> 0.1uF; footprint (none) -> 0603
- C302, C303, C304, C305, C307, C308, C309, C310: footprint (none) -> 0402
- C306, C311, D302, D303, D304, D401, R301, R303, R304, R305, R402: footprint (none) -> 0603
- U301: footprint (none) -> QFN124

Commit message: done :)
Connections:
- net GND: now also U301.B35 (MODE2)
- net MSEL: no longer U301.B35 (MODE2)
