File: l2_dev_alternative _nopwrsense/l2.sch (KiCad schematic (older format))
At the start: 21 parts, among them U301 XS1_L2-QFN124

Commit message: logic error! remove the mux and put SW_4 instead
Changed lines of the file:
@@
-EESchema Schematic File Version 2  date 01/09/2011 14:48:10
+EESchema Schematic File Version 2  date 01/09/2011 16:24:27
 LIBS:power
 LIBS:device
@@
 AR Path="/4E36B740/4E3470E5/4E5CC072" Ref="R1205"  Part="1"
 AR Path="/4E36B740/4E32CE0C/4E5CC072" Ref="R1305"  Part="1"
-F 0 "R1305" V 5470 5920 50  0000 C CNN
+F 0 "R1005" V 5470 5920 50  0000 C CNN
 F 1 "1k" V 5390 5920 50  0000 C CNN
 	1    5390 5920
@@
 AR Path="/4E36B740/4E3470E5/4E5CC071" Ref="D1204"  Part="1"
 AR Path="/4E36B740/4E32CE0C/4E5CC071" Ref="D1304"  Part="1"
-F 0 "D1304" H 5390 6570 50  0000 C CNN
+F 0 "D1004" H 5390 6570 50  0000 C CNN
 F 1 "LED" H 5390 6370 50  0000 C CNN
 	1    5390 6470
@@
 AR Path="/4E36B740/4E3470E5/4E5CC058" Ref="D1203"  Part="1"
 AR Path="/4E36B740/4E32CE0C/4E5CC058" Ref="D1303"  Part="1"
-F 0 "D1303" H 5090 6570 50  0000 C CNN
+F 0 "D1003" H 5090 6570 50  0000 C CNN
 F 1 "LED" H 5090 6370 50  0000 C CNN
 	1    5090 6470
@@
 AR Path="/4E36B740/4E3470E5/4E5CC057" Ref="R1204"  Part="1"
 AR Path="/4E36B740/4E32CE0C/4E5CC057" Ref="R1304"  Part="1"
-F 0 "R1304" V 5170 5920 50  0000 C CNN
+F 0 "R1004" V 5170 5920 50  0000 C CNN
 F 1 "1k" V 5090 5920 50  0000 C CNN
 	1    5090 5920
@@
 AR Path="/4E36B740/4E3470E5/4E5CC032" Ref="R1203"  Part="1"
 AR Path="/4E36B740/4E32CE0C/4E5CC032" Ref="R1303"  Part="1"
-F 0 "R1303" V 4880 5920 50  0000 C CNN
+F 0 "R1003" V 4880 5920 50  0000 C CNN
 F 1 "1k" V 4800 5920 50  0000 C CNN
 	1    4800 5920
@@
 AR Path="/4E36B740/4E3470E5/4E5CC031" Ref="D1202"  Part="1"
 AR Path="/4E36B740/4E32CE0C/4E5CC031" Ref="D1302"  Part="1"
-F 0 "D1302" H 4800 6570 50  0000 C CNN
+F 0 "D1002" H 4800 6570 50  0000 C CNN
 F 1 "LED" H 4800 6370 50  0000 C CNN
 	1    4800 6470
@@
 AR Path="/4E36B740/4E3470E5/4E5CC004" Ref="D1201"  Part="1"
 AR Path="/4E36B740/4E32CE0C/4E5CC004" Ref="D1301"  Part="1"
-F 0 "D1301" H 4490 6570 50  0000 C CNN
+F 0 "D1001" H 4490 6570 50  0000 C CNN
 F 1 "LED" H 4490 6370 50  0000 C CNN
 	1    4490 6470
@@
 AR Path="/4E36B740/4E3470E5/4E5CBFFC" Ref="R1202"  Part="1"
 AR Path="/4E36B740/4E32CE0C/4E5CBFFC" Ref="R1302"  Part="1"
-F 0 "R1302" V 4570 5920 50  0000 C CNN
+F 0 "R1002" V 4570 5920 50  0000 C CNN
 F 1 "1k" V 4490 5920 50  0000 C CNN
 	1    4490 5920
@@
 AR Path="/4E32CDCE/4E3470E5/4E32CE3D" Ref="U1201"  Part="3"
 AR Path="/4E32CDCE/4E32CE0C/4E32CE3D" Ref="U1301"  Part="3"
-F 0 "U1001" H 7740 2480 60  0000 C CNN
+F 0 "U701" H 7740 2480 60  0000 C CNN
 F 1 "XS1_L2-QFN124" H 8030 2360 60  0000 C CNN
 	3    8060 1630
@@
 AR Path="/4E32CDCE/4E3470E5/4E32D8E0" Ref="C1207"  Part="1"
 AR Path="/4E32CDCE/4E32CE0C/4E32D8E0" Ref="C1307"  Part="1"
-F 0 "C1007" H 9720 5790 50  0000 L CNN
+F 0 "C707" H 9720 5790 50  0000 L CNN
 F 1 "100nF" H 9680 5590 50  0000 L CNN
 	1    9670 5690
@@
 AR Path="/4E32CDCE/4E3470E5/4E32D8DF" Ref="C1208"  Part="1"
 AR Path="/4E32CDCE/4E32CE0C/4E32D8DF" Ref="C1308"  Part="1"
-F 0 "C1008" H 9980 5790 50  0000 L CNN
+F 0 "C708" H 9980 5790 50  0000 L CNN
 F 1 "100nF" H 9940 5590 50  0000 L CNN
 	1    9930 5690
@@
 AR Path="/4E32CDCE/4E3470E5/4E32D8DE" Ref="C1209"  Part="1"
 AR Path="/4E32CDCE/4E32CE0C/4E32D8DE" Ref="C1309"  Part="1"
-F 0 "C1009" H 10240 5790 50  0000 L CNN
+F 0 "C709" H 10240 5790 50  0000 L CNN
 F 1 "100nF" H 10200 5590 50  0000 L CNN
 	1    10190 5690
@@
 AR Path="/4E32CDCE/4E3470E5/4E32D8DD" Ref="C1210"  Part="1"
 AR Path="/4E32CDCE/4E32CE0C/4E32D8DD" Ref="C1310"  Part="1"
-F 0 "C1010" H 10500 5790 50  0000 L CNN
+F 0 "C710" H 10500 5790 50  0000 L CNN
 F 1 "100nF" H 10460 5590 50  0000 L CNN
 	1    10450 5690
@@
 AR Path="/4E32CDCE/4E3470E5/4E32D8DC" Ref="C1211"  Part="1"
 AR Path="/4E32CDCE/4E32CE0C/4E32D8DC" Ref="C1311"  Part="1"
-F 0 "C1011" H 10760 5790 50  0000 L CNN
+F 0 "C711" H 10760 5790 50  0000 L CNN
 F 1 "10uF" H 10720 5590 50  0000 L CNN
 	1    10710 5690
@@
 AR Path="/4E32CDCE/4E3470E5/4E32D84E" Ref="C1206"  Part="1"
 AR Path="/4E32CDCE/4E32CE0C/4E32D84E" Ref="C1306"  Part="1"
-F 0 "C1006" H 9140 5790 50  0000 L CNN
+F 0 "C706" H 9140 5790 50  0000 L CNN
 F 1 "10uF" H 9100 5590 50  0000 L CNN
 	1    9090 5690
@@
 AR Path="/4E32CDCE/4E3470E5/4E32D828" Ref="C1205"  Part="1"
 AR Path="/4E32CDCE/4E32CE0C/4E32D828" Ref="C1305"  Part="1"
-F 0 "C1005" H 8880 5790 50  0000 L CNN
+F 0 "C705" H 8880 5790 50  0000 L CNN
 F 1 "100nF" H 8840 5590 50  0000 L CNN
 	1    8830 5690
@@
 AR Path="/4E32CDCE/4E3470E5/4E32D822" Ref="C1204"  Part="1"
 AR Path="/4E32CDCE/4E32CE0C/4E32D822" Ref="C1304"  Part="1"
-F 0 "C1004" H 8620 5790 50  0000 L CNN
+F 0 "C704" H 8620 5790 50  0000 L CNN
 F 1 "100nF" H 8580 5590 50  0000 L CNN
 	1    8570 5690
@@
 AR Path="/4E32CDCE/4E3470E5/4E32D7FC" Ref="C1203"  Part="1"
 AR Path="/4E32CDCE/4E32CE0C/4E32D7FC" Ref="C1303"  Part="1"
-F 0 "C1003" H 8360 5790 50  0000 L CNN
+F 0 "C703" H 8360 5790 50  0000 L CNN
 F 1 "100nF" H 8320 5590 50  0000 L CNN
 	1    8310 5690
@@
 AR Path="/4E32CDCE/4E3470E5/4E32D7F4" Ref="C1202"  Part="1"
 AR Path="/4E32CDCE/4E32CE0C/4E32D7F4" Ref="C1302"  Part="1"
-F 0 "C1002" H 8100 5790 50  0000 L CNN
+F 0 "C702" H 8100 5790 50  0000 L CNN
 F 1 "100nF" H 8060 5590 50  0000 L CNN
 	1    8050 5690
@@
 AR Path="/4E32CDCE/4E3470E5/4E32D1CA" Ref="C1201"  Part="1"
 AR Path="/4E32CDCE/4E32CE0C/4E32D1CA" Ref="C1301"  Part="1"
-F 0 "C1001" H 7300 4560 50  0000 L CNN
+F 0 "C701" H 7300 4560 50  0000 L CNN
 F 1 "1uF" H 7300 4360 50  0000 L CNN
 	1    7250 4460
@@
 AR Path="/4E32CDCE/4E3470E5/4E32D1C4" Ref="R1201"  Part="1"
 AR Path="/4E32CDCE/4E32CE0C/4E32D1C4" Ref="R1301"  Part="1"
-F 0 "R1001" V 7330 3870 50  0000 C CNN
+F 0 "R701" V 7330 3870 50  0000 C CNN
 F 1 "2R2" V 7250 3870 50  0000 C CNN
 	1    7250 3870
@@
 AR Path="/4E32CDCE/4E3470E5/4E32CE40" Ref="U1201"  Part="4"
 AR Path="/4E32CDCE/4E32CE0C/4E32CE40" Ref="U1301"  Part="4"
-F 0 "U1001" H 9520 2480 60  0000 C CNN
+F 0 "U701" H 9520 2480 60  0000 C CNN
 F 1 "XS1_L2-QFN124" H 9810 2360 60  0000 C CNN
 	4    9840 1630
@@
 AR Path="/4E32CDCE/4E3470E5/4E32CE3B" Ref="U1201"  Part="1"
 AR Path="/4E32CDCE/4E32CE0C/4E32CE3B" Ref="U1301"  Part="1"
-F 0 "U1001" H 5350 2640 60  0000 C CNN
+F 0 "U701" H 5350 2640 60  0000 C CNN
 F 1 "XS1_L2-QFN124" H 5640 2520 60  0000 C CNN
 	1    5670 1790
@@
 AR Path="/4E32CDCE/4E3470E5/4E32CE36" Ref="U1201"  Part="2"
 AR Path="/4E32CDCE/4E32CE0C/4E32CE36" Ref="U1301"  Part="2"
-F 0 "U1001" H 5400 4690 60  0000 C CNN
+F 0 "U701" H 5400 4690 60  0000 C CNN
 F 1 "XS1_L2-QFN124" H 5690 4570 60  0000 C CNN
 	2    5720 3840

Commit message: added term resistors for xlinks and changed RST buffers to open drain
Changed lines of the file:
@@
-EESchema Schematic File Version 2  date 01/09/2011 16:28:35
+EESchema Schematic File Version 2  date 02/09/2011 13:05:35
 LIBS:power
 LIBS:device
@@
 Sheet 13 13
 Title ""
-Date "1 sep 2011"
+Date "2 sep 2011"
 Rev ""
 Comp ""
@@
 AR Path="/4E36B740/4E3470E5/4E5CC072" Ref="R1205"  Part="1"
 AR Path="/4E36B740/4E32CE0C/4E5CC072" Ref="R1305"  Part="1"
-F 0 "R1005" V 5470 5920 50  0000 C CNN
+F 0 "R1305" V 5470 5920 50  0000 C CNN
 F 1 "1k" V 5390 5920 50  0000 C CNN
 	1    5390 5920
@@
 AR Path="/4E36B740/4E3470E5/4E5CC071" Ref="D1204"  Part="1"
 AR Path="/4E36B740/4E32CE0C/4E5CC071" Ref="D1304"  Part="1"
-F 0 "D1004" H 5390 6570 50  0000 C CNN
+F 0 "D1304" H 5390 6570 50  0000 C CNN
 F 1 "LED" H 5390 6370 50  0000 C CNN
 	1    5390 6470
@@
 AR Path="/4E36B740/4E3470E5/4E5CC058" Ref="D1203"  Part="1"
 AR Path="/4E36B740/4E32CE0C/4E5CC058" Ref="D1303"  Part="1"
-F 0 "D1003" H 5090 6570 50  0000 C CNN
+F 0 "D1303" H 5090 6570 50  0000 C CNN
 F 1 "LED" H 5090 6370 50  0000 C CNN
 	1    5090 6470
@@
 AR Path="/4E36B740/4E3470E5/4E5CC057" Ref="R1204"  Part="1"
 AR Path="/4E36B740/4E32CE0C/4E5CC057" Ref="R1304"  Part="1"
-F 0 "R1004" V 5170 5920 50  0000 C CNN
+F 0 "R1304" V 5170 5920 50  0000 C CNN
 F 1 "1k" V 5090 5920 50  0000 C CNN
 	1    5090 5920
@@
 AR Path="/4E36B740/4E3470E5/4E5CC032" Ref="R1203"  Part="1"
 AR Path="/4E36B740/4E32CE0C/4E5CC032" Ref="R1303"  Part="1"
-F 0 "R1003" V 4880 5920 50  0000 C CNN
+F 0 "R1303" V 4880 5920 50  0000 C CNN
 F 1 "1k" V 4800 5920 50  0000 C CNN
 	1    4800 5920
@@
 AR Path="/4E36B740/4E3470E5/4E5CC031" Ref="D1202"  Part="1"
 AR Path="/4E36B740/4E32CE0C/4E5CC031" Ref="D1302"  Part="1"
-F 0 "D1002" H 4800 6570 50  0000 C CNN
+F 0 "D1302" H 4800 6570 50  0000 C CNN
 F 1 "LED" H 4800 6370 50  0000 C CNN
 	1    4800 6470
@@
 AR Path="/4E36B740/4E3470E5/4E5CC004" Ref="D1201"  Part="1"
 AR Path="/4E36B740/4E32CE0C/4E5CC004" Ref="D1301"  Part="1"
-F 0 "D1001" H 4490 6570 50  0000 C CNN
+F 0 "D1301" H 4490 6570 50  0000 C CNN
 F 1 "LED" H 4490 6370 50  0000 C CNN
 	1    4490 6470
@@
 AR Path="/4E36B740/4E3470E5/4E5CBFFC" Ref="R1202"  Part="1"
 AR Path="/4E36B740/4E32CE0C/4E5CBFFC" Ref="R1302"  Part="1"
-F 0 "R1002" V 4570 5920 50  0000 C CNN
+F 0 "R1302" V 4570 5920 50  0000 C CNN
 F 1 "1k" V 4490 5920 50  0000 C CNN
 	1    4490 5920
@@
 AR Path="/4E32CDCE/4E3470E5/4E32CE3D" Ref="U1201"  Part="3"
 AR Path="/4E32CDCE/4E32CE0C/4E32CE3D" Ref="U1301"  Part="3"
-F 0 "U701" H 7740 2480 60  0000 C CNN
+F 0 "U1001" H 7740 2480 60  0000 C CNN
 F 1 "XS1_L2-QFN124" H 8030 2360 60  0000 C CNN
 	3    8060 1630
@@
 AR Path="/4E32CDCE/4E3470E5/4E32D8E0" Ref="C1207"  Part="1"
 AR Path="/4E32CDCE/4E32CE0C/4E32D8E0" Ref="C1307"  Part="1"
-F 0 "C707" H 9720 5790 50  0000 L CNN
+F 0 "C1007" H 9720 5790 50  0000 L CNN
 F 1 "100nF" H 9680 5590 50  0000 L CNN
 	1    9670 5690
@@
 AR Path="/4E32CDCE/4E3470E5/4E32D8DF" Ref="C1208"  Part="1"
 AR Path="/4E32CDCE/4E32CE0C/4E32D8DF" Ref="C1308"  Part="1"
-F 0 "C708" H 9980 5790 50  0000 L CNN
+F 0 "C1008" H 9980 5790 50  0000 L CNN
 F 1 "100nF" H 9940 5590 50  0000 L CNN
 	1    9930 5690
@@
 AR Path="/4E32CDCE/4E3470E5/4E32D8DE" Ref="C1209"  Part="1"
 AR Path="/4E32CDCE/4E32CE0C/4E32D8DE" Ref="C1309"  Part="1"
-F 0 "C709" H 10240 5790 50  0000 L CNN
+F 0 "C1009" H 10240 5790 50  0000 L CNN
 F 1 "100nF" H 10200 5590 50  0000 L CNN
 	1    10190 5690
@@
 AR Path="/4E32CDCE/4E3470E5/4E32D8DD" Ref="C1210"  Part="1"
 AR Path="/4E32CDCE/4E32CE0C/4E32D8DD" Ref="C1310"  Part="1"
-F 0 "C710" H 10500 5790 50  0000 L CNN
+F 0 "C1010" H 10500 5790 50  0000 L CNN
 F 1 "100nF" H 10460 5590 50  0000 L CNN
 	1    10450 5690
@@
 AR Path="/4E32CDCE/4E3470E5/4E32D8DC" Ref="C1211"  Part="1"
 AR Path="/4E32CDCE/4E32CE0C/4E32D8DC" Ref="C1311"  Part="1"
-F 0 "C711" H 10760 5790 50  0000 L CNN
+F 0 "C1011" H 10760 5790 50  0000 L CNN
 F 1 "10uF" H 10720 5590 50  0000 L CNN
 	1    10710 5690
@@
 AR Path="/4E32CDCE/4E3470E5/4E32D84E" Ref="C1206"  Part="1"
 AR Path="/4E32CDCE/4E32CE0C/4E32D84E" Ref="C1306"  Part="1"
-F 0 "C706" H 9140 5790 50  0000 L CNN
+F 0 "C1006" H 9140 5790 50  0000 L CNN
 F 1 "10uF" H 9100 5590 50  0000 L CNN
 	1    9090 5690
@@
 AR Path="/4E32CDCE/4E3470E5/4E32D828" Ref="C1205"  Part="1"
 AR Path="/4E32CDCE/4E32CE0C/4E32D828" Ref="C1305"  Part="1"
-F 0 "C705" H 8880 5790 50  0000 L CNN
+F 0 "C1005" H 8880 5790 50  0000 L CNN
 F 1 "100nF" H 8840 5590 50  0000 L CNN
 	1    8830 5690
@@
 AR Path="/4E32CDCE/4E3470E5/4E32D822" Ref="C1204"  Part="1"
 AR Path="/4E32CDCE/4E32CE0C/4E32D822" Ref="C1304"  Part="1"
-F 0 "C704" H 8620 5790 50  0000 L CNN
+F 0 "C1004" H 8620 5790 50  0000 L CNN
 F 1 "100nF" H 8580 5590 50  0000 L CNN
 	1    8570 5690
@@
 AR Path="/4E32CDCE/4E3470E5/4E32D7FC" Ref="C1203"  Part="1"
 AR Path="/4E32CDCE/4E32CE0C/4E32D7FC" Ref="C1303"  Part="1"
-F 0 "C703" H 8360 5790 50  0000 L CNN
+F 0 "C1003" H 8360 5790 50  0000 L CNN
 F 1 "100nF" H 8320 5590 50  0000 L CNN
 	1    8310 5690
@@
 AR Path="/4E32CDCE/4E3470E5/4E32D7F4" Ref="C1202"  Part="1"
 AR Path="/4E32CDCE/4E32CE0C/4E32D7F4" Ref="C1302"  Part="1"
-F 0 "C702" H 8100 5790 50  0000 L CNN
+F 0 "C1002" H 8100 5790 50  0000 L CNN
 F 1 "100nF" H 8060 5590 50  0000 L CNN
 	1    8050 5690
@@
 AR Path="/4E32CDCE/4E3470E5/4E32D1CA" Ref="C1201"  Part="1"
 AR Path="/4E32CDCE/4E32CE0C/4E32D1CA" Ref="C1301"  Part="1"
-F 0 "C701" H 7300 4560 50  0000 L CNN
+F 0 "C1001" H 7300 4560 50  0000 L CNN
 F 1 "1uF" H 7300 4360 50  0000 L CNN
 	1    7250 4460
@@
 AR Path="/4E32CDCE/4E3470E5/4E32D1C4" Ref="R1201"  Part="1"
 AR Path="/4E32CDCE/4E32CE0C/4E32D1C4" Ref="R1301"  Part="1"
-F 0 "R701" V 7330 3870 50  0000 C CNN
+F 0 "R1001" V 7330 3870 50  0000 C CNN
 F 1 "2R2" V 7250 3870 50  0000 C CNN
 	1    7250 3870
@@
 AR Path="/4E32CDCE/4E3470E5/4E32CE40" Ref="U1201"  Part="4"
 AR Path="/4E32CDCE/4E32CE0C/4E32CE40" Ref="U1301"  Part="4"
-F 0 "U701" H 9520 2480 60  0000 C CNN
+F 0 "U1001" H 9520 2480 60  0000 C CNN
 F 1 "XS1_L2-QFN124" H 9810 2360 60  0000 C CNN
 	4    9840 1630
@@
 AR Path="/4E32CDCE/4E3470E5/4E32CE3B" Ref="U1201"  Part="1"
 AR Path="/4E32CDCE/4E32CE0C/4E32CE3B" Ref="U1301"  Part="1"
-F 0 "U701" H 5350 2640 60  0000 C CNN
+F 0 "U1001" H 5350 2640 60  0000 C CNN
 F 1 "XS1_L2-QFN124" H 5640 2520 60  0000 C CNN
 	1    5670 1790
@@
 AR Path="/4E32CDCE/4E3470E5/4E32CE36" Ref="U1201"  Part="2"
 AR Path="/4E32CDCE/4E32CE0C/4E32CE36" Ref="U1301"  Part="2"
-F 0 "U701" H 5400 4690 60  0000 C CNN
+F 0 "U1001" H 5400 4690 60  0000 C CNN
 F 1 "XS1_L2-QFN124" H 5690 4570 60  0000 C CNN
 	2    5720 3840

Commit message: almost all the links in, some of the JTAG in. Surprisingly nice :)
Changed lines of the file:
@@
-EESchema Schematic File Version 2  date 05/09/2011 16:29:32
+EESchema Schematic File Version 2  date 06/09/2011 18:50:43
 LIBS:power
 LIBS:device
@@
 Sheet 4 13
 Title ""
-Date "5 sep 2011"
+Date "6 sep 2011"
 Rev ""
 Comp ""
@@
 Comment4 ""
 $EndDescr
-Text Notes 5490 5310 0    30   ~ 0
-LED_ARRAY
 Wire Notes Line
 	3750 5200 3750 6840
@@
 Wire Wire Line
 	5390 5360 4150 5360
+Text Notes 5490 5310 0    30   ~ 0
+LED_ARRAY
 $Comp
 L R R305
@@
 AR Path="/4E36B740/4E3470E5/4E5CC072" Ref="R1205"  Part="1"
 AR Path="/4E36B740/4E32CE0C/4E5CC072" Ref="R1305"  Part="1"
-F 0 "R405" V 5470 5920 50  0000 C CNN
+F 0 "R1305" V 5470 5920 50  0000 C CNN
 F 1 "1k" V 5390 5920 50  0000 C CNN
 	1    5390 5920
@@
 AR Path="/4E36B740/4E3470E5/4E5CC071" Ref="D1204"  Part="1"
 AR Path="/4E36B740/4E32CE0C/4E5CC071" Ref="D1304"  Part="1"
-F 0 "D404" H 5390 6570 50  0000 C CNN
+F 0 "D1304" H 5390 6570 50  0000 C CNN
 F 1 "LED" H 5390 6370 50  0000 C CNN
 	1    5390 6470
@@
 AR Path="/4E36B740/4E3470E5/4E5CC058" Ref="D1203"  Part="1"
 AR Path="/4E36B740/4E32CE0C/4E5CC058" Ref="D1303"  Part="1"
-F 0 "D403" H 5090 6570 50  0000 C CNN
+F 0 "D1303" H 5090 6570 50  0000 C CNN
 F 1 "LED" H 5090 6370 50  0000 C CNN
 	1    5090 6470
@@
 AR Path="/4E36B740/4E3470E5/4E5CC057" Ref="R1204"  Part="1"
 AR Path="/4E36B740/4E32CE0C/4E5CC057" Ref="R1304"  Part="1"
-F 0 "R404" V 5170 5920 50  0000 C CNN
+F 0 "R1304" V 5170 5920 50  0000 C CNN
 F 1 "1k" V 5090 5920 50  0000 C CNN
 	1    5090 5920
@@
 AR Path="/4E36B740/4E3470E5/4E5CC032" Ref="R1203"  Part="1"
 AR Path="/4E36B740/4E32CE0C/4E5CC032" Ref="R1303"  Part="1"
-F 0 "R403" V 4880 5920 50  0000 C CNN
+F 0 "R1303" V 4880 5920 50  0000 C CNN
 F 1 "1k" V 4800 5920 50  0000 C CNN
 	1    4800 5920
@@
 AR Path="/4E36B740/4E3470E5/4E5CC031" Ref="D1202"  Part="1"
 AR Path="/4E36B740/4E32CE0C/4E5CC031" Ref="D1302"  Part="1"
-F 0 "D402" H 4800 6570 50  0000 C CNN
+F 0 "D1302" H 4800 6570 50  0000 C CNN
 F 1 "LED" H 4800 6370 50  0000 C CNN
 	1    4800 6470
@@
 AR Path="/4E36B740/4E3470E5/4E5CC004" Ref="D1201"  Part="1"
 AR Path="/4E36B740/4E32CE0C/4E5CC004" Ref="D1301"  Part="1"
-F 0 "D401" H 4490 6570 50  0000 C CNN
+F 0 "D1301" H 4490 6570 50  0000 C CNN
 F 1 "LED" H 4490 6370 50  0000 C CNN
 	1    4490 6470
@@
 AR Path="/4E36B740/4E3470E5/4E5CBFFC" Ref="R1202"  Part="1"
 AR Path="/4E36B740/4E32CE0C/4E5CBFFC" Ref="R1302"  Part="1"
-F 0 "R402" V 4570 5920 50  0000 C CNN
+F 0 "R1302" V 4570 5920 50  0000 C CNN
 F 1 "1k" V 4490 5920 50  0000 C CNN
 	1    4490 5920
@@
 AR Path="/4E32CDCE/4E3470E5/4E32CE3D" Ref="U1201"  Part="3"
 AR Path="/4E32CDCE/4E32CE0C/4E32CE3D" Ref="U1301"  Part="3"
-F 0 "U1301" H 7740 2480 60  0000 C CNN
+F 0 "U1001" H 7740 2480 60  0000 C CNN
 F 1 "XS1_L2-QFN124" H 8030 2360 60  0000 C CNN
 	3    8060 1630
@@
 AR Path="/4E32CDCE/4E3470E5/4E32D8E0" Ref="C1207"  Part="1"
 AR Path="/4E32CDCE/4E32CE0C/4E32D8E0" Ref="C1307"  Part="1"
-F 0 "C1307" H 9720 5790 50  0000 L CNN
+F 0 "C1007" H 9720 5790 50  0000 L CNN
 F 1 "100nF" H 9680 5590 50  0000 L CNN
 	1    9670 5690
@@
 AR Path="/4E32CDCE/4E3470E5/4E32D8DF" Ref="C1208"  Part="1"
 AR Path="/4E32CDCE/4E32CE0C/4E32D8DF" Ref="C1308"  Part="1"
-F 0 "C1308" H 9980 5790 50  0000 L CNN
+F 0 "C1008" H 9980 5790 50  0000 L CNN
 F 1 "100nF" H 9940 5590 50  0000 L CNN
 	1    9930 5690
@@
 AR Path="/4E32CDCE/4E3470E5/4E32D8DE" Ref="C1209"  Part="1"
 AR Path="/4E32CDCE/4E32CE0C/4E32D8DE" Ref="C1309"  Part="1"
-F 0 "C1309" H 10240 5790 50  0000 L CNN
+F 0 "C1009" H 10240 5790 50  0000 L CNN
 F 1 "100nF" H 10200 5590 50  0000 L CNN
 	1    10190 5690
@@
 AR Path="/4E32CDCE/4E3470E5/4E32D8DD" Ref="C1210"  Part="1"
 AR Path="/4E32CDCE/4E32CE0C/4E32D8DD" Ref="C1310"  Part="1"
-F 0 "C1310" H 10500 5790 50  0000 L CNN
+F 0 "C1010" H 10500 5790 50  0000 L CNN
 F 1 "100nF" H 10460 5590 50  0000 L CNN
 	1    10450 5690
@@
 AR Path="/4E32CDCE/4E3470E5/4E32D8DC" Ref="C1211"  Part="1"
 AR Path="/4E32CDCE/4E32CE0C/4E32D8DC" Ref="C1311"  Part="1"
-F 0 "C1311" H 10760 5790 50  0000 L CNN
+F 0 "C1011" H 10760 5790 50  0000 L CNN
 F 1 "10uF" H 10720 5590 50  0000 L CNN
 	1    10710 5690
@@
 AR Path="/4E32CDCE/4E3470E5/4E32D84E" Ref="C1206"  Part="1"
 AR Path="/4E32CDCE/4E32CE0C/4E32D84E" Ref="C1306"  Part="1"
-F 0 "C1306" H 9140 5790 50  0000 L CNN
+F 0 "C1006" H 9140 5790 50  0000 L CNN
 F 1 "10uF" H 9100 5590 50  0000 L CNN
 	1    9090 5690
@@
 AR Path="/4E32CDCE/4E3470E5/4E32D828" Ref="C1205"  Part="1"
 AR Path="/4E32CDCE/4E32CE0C/4E32D828" Ref="C1305"  Part="1"
-F 0 "C1305" H 8880 5790 50  0000 L CNN
+F 0 "C1005" H 8880 5790 50  0000 L CNN
 F 1 "100nF" H 8840 5590 50  0000 L CNN
 	1    8830 5690
@@
 AR Path="/4E32CDCE/4E3470E5/4E32D822" Ref="C1204"  Part="1"
 AR Path="/4E32CDCE/4E32CE0C/4E32D822" Ref="C1304"  Part="1"
-F 0 "C1304" H 8620 5790 50  0000 L CNN
+F 0 "C1004" H 8620 5790 50  0000 L CNN
 F 1 "100nF" H 8580 5590 50  0000 L CNN
 	1    8570 5690
@@
 AR Path="/4E32CDCE/4E3470E5/4E32D7FC" Ref="C1203"  Part="1"
 AR Path="/4E32CDCE/4E32CE0C/4E32D7FC" Ref="C1303"  Part="1"
-F 0 "C1303" H 8360 5790 50  0000 L CNN
+F 0 "C1003" H 8360 5790 50  0000 L CNN
 F 1 "100nF" H 8320 5590 50  0000 L CNN
 	1    8310 5690
@@
 AR Path="/4E32CDCE/4E3470E5/4E32D7F4" Ref="C1202"  Part="1"
 AR Path="/4E32CDCE/4E32CE0C/4E32D7F4" Ref="C1302"  Part="1"
-F 0 "C1302" H 8100 5790 50  0000 L CNN
+F 0 "C1002" H 8100 5790 50  0000 L CNN
 F 1 "100nF" H 8060 5590 50  0000 L CNN
 	1    8050 5690
@@
 AR Path="/4E32CDCE/4E3470E5/4E32D1CA" Ref="C1201"  Part="1"
 AR Path="/4E32CDCE/4E32CE0C/4E32D1CA" Ref="C1301"  Part="1"
-F 0 "C1301" H 7300 4560 50  0000 L CNN
+F 0 "C1001" H 7300 4560 50  0000 L CNN
 F 1 "1uF" H 7300 4360 50  0000 L CNN
 	1    7250 4460
@@
 AR Path="/4E32CDCE/4E3470E5/4E32D1C4" Ref="R1201"  Part="1"
 AR Path="/4E32CDCE/4E32CE0C/4E32D1C4" Ref="R1301"  Part="1"
-F 0 "R1301" V 7330 3870 50  0000 C CNN
+F 0 "R1001" V 7330 3870 50  0000 C CNN
 F 1 "2R2" V 7250 3870 50  0000 C CNN
 	1    7250 3870
@@
 AR Path="/4E32CDCE/4E3470E5/4E32CE40" Ref="U1201"  Part="4"
 AR Path="/4E32CDCE/4E32CE0C/4E32CE40" Ref="U1301"  Part="4"
-F 0 "U1301" H 9520 2480 60  0000 C CNN
+F 0 "U1001" H 9520 2480 60  0000 C CNN
 F 1 "XS1_L2-QFN124" H 9810 2360 60  0000 C CNN
 	4    9840 1630
@@
 AR Path="/4E32CDCE/4E3470E5/4E32CE3B" Ref="U1201"  Part="1"
 AR Path="/4E32CDCE/4E32CE0C/4E32CE3B" Ref="U1301"  Part="1"
-F 0 "U1301" H 5350 2640 60  0000 C CNN
+F 0 "U1001" H 5350 2640 60  0000 C CNN
 F 1 "XS1_L2-QFN124" H 5640 2520 60  0000 C CNN
 	1    5670 1790
@@
 AR Path="/4E32CDCE/4E3470E5/4E32CE36" Ref="U1201"  Part="2"
 AR Path="/4E32CDCE/4E32CE0C/4E32CE36" Ref="U1301"  Part="2"
-F 0 "U1301" H 5400 4690 60  0000 C CNN
+F 0 "U1001" H 5400 4690 60  0000 C CNN
 F 1 "XS1_L2-QFN124" H 5690 4570 60  0000 C CNN
 	2    5720 3840
