File: l2_dev_alternative _nopwrsense/l2.sch (KiCad schematic (older format))
At the start: 21 parts, among them U301 XS1_L2-QFN124

Commit message: going to flood the top!
Parts:
- C301, C306, C311, D302, D303, D304, D401, R301, R303, R304, R305, R402: footprint (none) -> 0603
- C302, C303, C304, C305, C307, C308, C309, C310: footprint (none) -> 0402
- U301: footprint (none) -> QFN124
