File: l2_dev_alternative _nopwrsense/l2.sch (KiCad schematic (older format))
At the start: 21 parts, among them U301 XS1_L2-QFN124

Commit message: working on power sense again now. The normal board should be more or less done!
Parts:
- C301: value 1uF -> 0.1uF
