File: l2_dev_alternative _nopwrsense/l2_dev_board.sch (KiCad schematic (older format))
At the start: 69 parts, among them P101 CONN_30, P102 CONN_30, P103 CONN_30, P104 CONN_30, P105 CONN_30, P106 CONN_30, P107 CONN_30, P108 CONN_30, P109 CONN_30, P110 CONN_30, U101 APX803-SR, U103 A6RS-161RF, U104 SN74LVC1G18, U105 SN74LVC1G18, U106 SN74LVC1G18, U107 SN74LVC1G18, U108 SN74CBTD3861, U109 LT3480, U110 APX803-SR, U111 74AHC1GU04, U112 NC7WZ17, U113 NC7WZ17, U114 NC7WZ17, U115 NC7WZ17, U116 SN74CBTD3861, U117 NCP1529, U118 NC7WZ17, U119 NC7WZ17, U120 NC7WZ17, U123 ASE_CLK, U125 NC7WZ17, U126 NC7WZ17, U127 NC7WZ17, U128 NC7WZ17, U131 NC7WZ17

Commit message: added term resistors for xlinks and changed RST buffers to open drain
Parts:
- removed R112, R117: 10k, symbol R
- removed U118, U127: NC7WZ17, symbol NC7WZ17
- added R? (x124): 33R, symbol R
- added U118, U127: NC7WZ07, symbol NC7WZ07
- C103: value 0.47uF -> 0.22uF
- C104: value 47uF -> 15uF
Connections:
- net +3.3V: now also R113.2, U108.24 (VCC), U116.24 (VCC), U118.5 (VCC), U127.5 (VCC); no longer R113.1
- net +5V: no longer U108.24 (VCC), U116.24 (VCC)
- net DEBUG_N: now also U119.3 (A2), U126.1 (A1); no longer U119.1 (A1), U126.3 (A2)
- net DEBUG_N_BUF_B: now also U126.6 (Y1); no longer U126.4 (Y2)
- net DEBUG_N_BUF_R: now also U119.4 (Y2); no longer U119.6 (Y1)
- net GND: now also D101.1 (A), U118.2 (GND), U127.2 (GND); no longer D101.2 (K)
- net L2_PAIR_Q1/BL_X0_XLA_0i: now also R?.1; no longer P102.24 (P24)
- net L2_PAIR_Q1/BL_X0_XLA_0o: now also R?.1; no longer P102.27 (P27)
- net L2_PAIR_Q1/BL_X0_XLA_1i: now also R?.1; no longer P102.23 (P23)
- net L2_PAIR_Q1/BL_X0_XLA_1o: now also R?.1; no longer P102.28 (P28)
- net L2_PAIR_Q1/BL_X0_XLA_2i: now also R?.1; no longer P102.22 (P22)
- net L2_PAIR_Q1/BL_X0_XLA_2o: now also R?.1; no longer P102.29 (P29)
- net L2_PAIR_Q1/BL_X0_XLA_3i: now also R?.1; no longer P102.21 (P21)
- net L2_PAIR_Q1/BL_X0_XLA_3o: now also R?.1; no longer P101.2 (P2)
- net L2_PAIR_Q1/BL_X0_XLA_4i: now also R?.1; no longer P102.20 (P20)
- net L2_PAIR_Q1/BL_X0_XLA_4o: now also R?.1; no longer P101.3 (P3)
- net L2_PAIR_Q1/TL_X0_XLA_0i: now also R?.1; no longer P101.22 (P22)
- net L2_PAIR_Q1/TL_X0_XLA_0o: now also R?.1; no longer P101.25 (P25)
- net L2_PAIR_Q1/TL_X0_XLA_1i: now also R?.1; no longer P101.21 (P21)
- net L2_PAIR_Q1/TL_X0_XLA_1o: now also R?.1; no longer P101.26 (P26)
- net L2_PAIR_Q1/TL_X0_XLA_2i: now also R?.1; no longer P101.20 (P20)
- net L2_PAIR_Q1/TL_X0_XLA_2o: now also R?.1; no longer P101.27 (P27)
- net L2_PAIR_Q1/TL_X0_XLA_3i: now also R?.1; no longer P101.19 (P19)
- net L2_PAIR_Q1/TL_X0_XLA_3o: now also R?.1; no longer P101.28 (P28)
- net L2_PAIR_Q1/TL_X0_XLA_4i: now also R?.1; no longer P101.18 (P18)
- net L2_PAIR_Q1/TL_X0_XLA_4o: now also R?.1; no longer P101.29 (P29)
- net L2_PAIR_Q1/T_X0_XLB_0i: now also R?.2; no longer P104.13 (P13)
- net L2_PAIR_Q1/T_X0_XLB_0o: now also R?.2; no longer P104.16 (P16)
- net L2_PAIR_Q1/T_X0_XLB_1i: now also R?.2; no longer P104.12 (P12)
- net L2_PAIR_Q1/T_X0_XLB_1o: now also R?.2; no longer P104.17 (P17)
- net L2_PAIR_Q1/T_X0_XLB_2i: now also R?.2; no longer P104.11 (P11)
- net L2_PAIR_Q1/T_X0_XLB_2o: now also R?.2; no longer P104.18 (P18)
- net L2_PAIR_Q1/T_X0_XLB_3i: now also R?.2; no longer P104.10 (P10)
- net L2_PAIR_Q1/T_X0_XLB_3o: now also R?.2; no longer P104.19 (P19)
- net L2_PAIR_Q1/T_X0_XLB_4i: now also R?.2; no longer P104.9 (P9)
- net L2_PAIR_Q1/T_X0_XLB_4o: now also R?.2; no longer P104.20 (P20)
- net L2_PAIR_Q2/BR_X1_XLA_0i: now also R?.2; no longer P109.4 (P4)
- net L2_PAIR_Q2/BR_X1_XLA_0o: now also R?.2; no longer P109.7 (P7)
- net L2_PAIR_Q2/BR_X1_XLA_1i: now also R?.2; no longer P109.3 (P3)
- net L2_PAIR_Q2/BR_X1_XLA_1o: now also R?.2; no longer P109.8 (P8)
- net L2_PAIR_Q2/BR_X1_XLA_2i: now also R?.2; no longer P109.2 (P2)
- net L2_PAIR_Q2/BR_X1_XLA_2o: now also R?.2; no longer P109.9 (P9)
- net L2_PAIR_Q2/BR_X1_XLA_3i: now also R?.2; no longer P108.29 (P29)
- net L2_PAIR_Q2/BR_X1_XLA_3o: now also R?.2; no longer P109.10 (P10)
- net L2_PAIR_Q2/BR_X1_XLA_4i: now also R?.2; no longer P108.28 (P28)
- net L2_PAIR_Q2/BR_X1_XLA_4o: now also R?.2; no longer P109.11 (P11)
- net L2_PAIR_Q2/TR_X1_XLA_0i: now also R?.2; no longer P108.6 (P6)
- net L2_PAIR_Q2/TR_X1_XLA_0o: now also R?.2; no longer P108.9 (P9)
- net L2_PAIR_Q2/TR_X1_XLA_1i: now also R?.2; no longer P108.5 (P5)
- net L2_PAIR_Q2/TR_X1_XLA_1o: now also R?.2; no longer P108.10 (P10)
- net L2_PAIR_Q2/TR_X1_XLA_2i: now also R?.2; no longer P108.4 (P4)
- net L2_PAIR_Q2/TR_X1_XLA_2o: now also R?.2; no longer P108.11 (P11)
- net L2_PAIR_Q2/TR_X1_XLA_3i: now also R?.2; no longer P108.3 (P3)
- net L2_PAIR_Q2/TR_X1_XLA_3o: now also R?.2; no longer P108.12 (P12)
- net L2_PAIR_Q2/TR_X1_XLA_4i: now also R?.2; no longer P108.2 (P2)
- net L2_PAIR_Q2/TR_X1_XLA_4o: now also R?.2; no longer P108.13 (P13)
- net L2_PAIR_Q2/T_X0_XLB_0i: now also R?.2; no longer P106.22 (P22)
- net L2_PAIR_Q2/T_X0_XLB_0o: now also R?.2; no longer P106.25 (P25)
- net L2_PAIR_Q2/T_X0_XLB_1i: now also R?.2; no longer P106.21 (P21)
- net L2_PAIR_Q2/T_X0_XLB_1o: now also R?.2; no longer P106.26 (P26)
- net L2_PAIR_Q2/T_X0_XLB_2i: now also R?.2; no longer P106.20 (P20)
- net L2_PAIR_Q2/T_X0_XLB_2o: now also R?.2; no longer P106.27 (P27)
- net L2_PAIR_Q2/T_X0_XLB_3i: now also R?.2; no longer P106.19 (P19)
- net L2_PAIR_Q2/T_X0_XLB_3o: now also R?.2; no longer P106.28 (P28)
- net L2_PAIR_Q2/T_X0_XLB_4i: now also R?.2; no longer P106.18 (P18)
- net L2_PAIR_Q2/T_X0_XLB_4o: now also R?.2; no longer P106.29 (P29)
- net L2_PAIR_Q3/BR_X1_XLA_0i: now also R?.2; no longer P110.21 (P21)
- net L2_PAIR_Q3/BR_X1_XLA_0o: now also R?.2; no longer P110.24 (P24)
- net L2_PAIR_Q3/BR_X1_XLA_1i: now also R?.2; no longer P110.20 (P20)
- net L2_PAIR_Q3/BR_X1_XLA_1o: now also R?.2; no longer P110.25 (P25)
- net L2_PAIR_Q3/BR_X1_XLA_2i: now also R?.2; no longer P110.19 (P19)
- net L2_PAIR_Q3/BR_X1_XLA_2o: now also R?.2; no longer P110.26 (P26)
- net L2_PAIR_Q3/BR_X1_XLA_3i: now also R?.2; no longer P110.18 (P18)
- net L2_PAIR_Q3/BR_X1_XLA_3o: now also R?.2; no longer P110.27 (P27)
- net L2_PAIR_Q3/BR_X1_XLA_4i: now also R?.2; no longer P110.17 (P17)
- net L2_PAIR_Q3/BR_X1_XLA_4o: now also R?.2; no longer P110.28 (P28)
- net L2_PAIR_Q3/B_X1_XLB_0i: now also R?.1; no longer P107.6 (P6)
- net L2_PAIR_Q3/B_X1_XLB_0o: now also R?.1; no longer P107.9 (P9)
- net L2_PAIR_Q3/B_X1_XLB_1i: now also R?.1; no longer P107.5 (P5)
- net L2_PAIR_Q3/B_X1_XLB_1o: now also R?.1; no longer P107.10 (P10)
- net L2_PAIR_Q3/B_X1_XLB_2i: now also R?.1; no longer P107.4 (P4)
- net L2_PAIR_Q3/B_X1_XLB_2o: now also R?.1; no longer P107.11 (P11)
- net L2_PAIR_Q3/B_X1_XLB_3i: now also R?.1; no longer P107.3 (P3)
- net L2_PAIR_Q3/B_X1_XLB_3o: now also R?.1; no longer P107.12 (P12)
- net L2_PAIR_Q3/B_X1_XLB_4i: now also R?.1; no longer P107.2 (P2)
- net L2_PAIR_Q3/B_X1_XLB_4o: now also R?.1; no longer P107.13 (P13)
- net L2_PAIR_Q3/TR_X1_XLA_0i: now also R?.2; no longer P110.7 (P7)
- net L2_PAIR_Q3/TR_X1_XLA_0o: now also R?.2; no longer P110.10 (P10)
- net L2_PAIR_Q3/TR_X1_XLA_1i: now also R?.2; no longer P110.6 (P6)
- net L2_PAIR_Q3/TR_X1_XLA_1o: now also R?.2; no longer P110.11 (P11)
- net L2_PAIR_Q3/TR_X1_XLA_2i: now also R?.2; no longer P110.5 (P5)
- net L2_PAIR_Q3/TR_X1_XLA_2o: now also R?.2; no longer P110.12 (P12)
- net L2_PAIR_Q3/TR_X1_XLA_3i: now also R?.2; no longer P110.4 (P4)
- net L2_PAIR_Q3/TR_X1_XLA_3o: now also R?.2; no longer P110.13 (P13)
- net L2_PAIR_Q3/TR_X1_XLA_4i: now also R?.2; no longer P110.3 (P3)
- net L2_PAIR_Q3/TR_X1_XLA_4o: now also R?.2; no longer P110.14 (P14)
- net L2_PAIR_Q4/BL_X0_XLA_0i: now also R?.1; no longer P103.7 (P7)
- net L2_PAIR_Q4/BL_X0_XLA_0o: now also R?.1; no longer P103.10 (P10)
- net L2_PAIR_Q4/BL_X0_XLA_1i: now also R?.1; no longer P103.6 (P6)
- net L2_PAIR_Q4/BL_X0_XLA_1o: now also R?.1; no longer P103.11 (P11)
- net L2_PAIR_Q4/BL_X0_XLA_2i: now also R?.1; no longer P103.5 (P5)
- net L2_PAIR_Q4/BL_X0_XLA_2o: now also R?.1; no longer P103.12 (P12)
- net L2_PAIR_Q4/BL_X0_XLA_3i: now also R?.1; no longer P103.4 (P4)
- net L2_PAIR_Q4/BL_X0_XLA_3o: now also R?.1; no longer P103.13 (P13)
- net L2_PAIR_Q4/BL_X0_XLA_4i: now also R?.1; no longer P103.3 (P3)
- net L2_PAIR_Q4/BL_X0_XLA_4o: now also R?.1; no longer P103.14 (P14)
- net L2_PAIR_Q4/B_X1_XLB_0i: now also R?.1; no longer P105.15 (P15)
- net L2_PAIR_Q4/B_X1_XLB_0o: now also R?.1; no longer P105.18 (P18)
- net L2_PAIR_Q4/B_X1_XLB_1i: now also R?.1; no longer P105.14 (P14)
- net L2_PAIR_Q4/B_X1_XLB_1o: now also R?.1; no longer P105.19 (P19)
- net L2_PAIR_Q4/B_X1_XLB_2i: now also R?.1; no longer P105.13 (P13)
- net L2_PAIR_Q4/B_X1_XLB_2o: now also R?.1; no longer P105.20 (P20)
- net L2_PAIR_Q4/B_X1_XLB_3i: now also R?.1; no longer P105.12 (P12)
- net L2_PAIR_Q4/B_X1_XLB_3o: now also R?.1; no longer P105.21 (P21)
- net L2_PAIR_Q4/B_X1_XLB_4i: now also R?.1; no longer P105.11 (P11)
- net L2_PAIR_Q4/B_X1_XLB_4o: now also R?.1; no longer P105.22 (P22)
- net L2_PAIR_Q4/TL_X0_XLA_0i: now also R?.1; no longer P103.21 (P21)
- net L2_PAIR_Q4/TL_X0_XLA_0o: now also R?.1; no longer P103.24 (P24)
- net L2_PAIR_Q4/TL_X0_XLA_1i: now also R?.1; no longer P103.20 (P20)
- net L2_PAIR_Q4/TL_X0_XLA_1o: now also R?.1; no longer P103.25 (P25)
- net L2_PAIR_Q4/TL_X0_XLA_2i: now also R?.1; no longer P103.19 (P19)
- net L2_PAIR_Q4/TL_X0_XLA_2o: now also R?.1; no longer P103.26 (P26)
- net L2_PAIR_Q4/TL_X0_XLA_3i: now also R?.1; no longer P103.18 (P18)
- net L2_PAIR_Q4/TL_X0_XLA_3o: now also R?.1; no longer P103.27 (P27)
- net L2_PAIR_Q4/TL_X0_XLA_4i: now also R?.1; no longer P103.17 (P17)
- net L2_PAIR_Q4/TL_X0_XLA_4o: now also R?.1; no longer P103.28 (P28)
- net MSEL_N: now also U120.1 (A1), U126.3 (A2); no longer U119.3 (A2)
- net RST_N: now also R113.1, U118.1 (A1), U127.3 (A2); no longer R113.2
- net RST_N_BUF_B: now also U127.4 (Y2)
- net RST_N_BUF_R: now also U118.6 (Y1)
- net TCK: now also U119.1 (A1)
- net TCK_BUF_B: now also R?.1; no longer U128.6 (Y1)
- net TCK_BUF_R: now also R?.1
- net TCK_L: now also R?.2; no longer U108.5 (A4)
- net TCK_T: now also R?.2; no longer U116.10 (A9)
- net TMS: now also U120.3 (A2); no longer U120.1 (A1)
- net TMS_BUF_R: now also U120.4 (Y2); no longer U120.6 (Y1)
- net TRST_N_BUF_B: now also U126.4 (Y2)
- net TRST_N_BUF_R: now also U120.6 (Y1); no longer U119.4 (Y2)
- net at C103.2, L101.1, U109.3 (SW): now also D101.2 (K); no longer D101.1 (A)
- new net: P101.18 (P18), R?.2
- new net: P101.19 (P19), R?.2
- new net: P101.2 (P2), R?.2
- new net: P101.20 (P20), R?.2
- new net: P101.21 (P21), R?.2
- new net: P101.22 (P22), R?.2
- new net: P101.25 (P25), R?.2
- new net: P101.26 (P26), R?.2
- new net: P101.27 (P27), R?.2
- new net: P101.28 (P28), R?.2
- new net: P101.29 (P29), R?.2
- new net: P101.3 (P3), R?.2
- new net: P102.20 (P20), R?.2
- new net: P102.21 (P21), R?.2
- new net: P102.22 (P22), R?.2
- new net: P102.23 (P23), R?.2
- new net: P102.24 (P24), R?.2
- new net: P102.27 (P27), R?.2
- new net: P102.28 (P28), R?.2
- new net: P102.29 (P29), R?.2
- new net: P104.10 (P10), R?.1
- new net: P104.11 (P11), R?.1
- new net: P104.12 (P12), R?.1
- new net: P104.13 (P13), R?.1
- new net: P104.16 (P16), R?.1
- new net: P104.17 (P17), R?.1
- new net: P104.18 (P18), R?.1
- new net: P104.19 (P19), R?.1
- new net: P104.20 (P20), R?.1
- new net: P104.9 (P9), R?.1
- new net: P106.18 (P18), R?.1
- new net: P106.19 (P19), R?.1
- new net: P106.20 (P20), R?.1
- new net: P106.21 (P21), R?.1
- new net: P106.22 (P22), R?.1
- new net: P106.25 (P25), R?.1
- new net: P106.26 (P26), R?.1
- new net: P106.27 (P27), R?.1
- new net: P106.28 (P28), R?.1
- new net: P106.29 (P29), R?.1
- new net: P103.10 (P10), R?.2
- new net: P103.11 (P11), R?.2
- new net: P103.12 (P12), R?.2
- new net: P103.13 (P13), R?.2
- new net: P103.14 (P14), R?.2
- new net: P103.17 (P17), R?.2
- new net: P103.18 (P18), R?.2
- new net: P103.19 (P19), R?.2
- new net: P103.20 (P20), R?.2
- new net: P103.21 (P21), R?.2
- new net: P103.24 (P24), R?.2
- new net: P103.25 (P25), R?.2
- new net: P103.26 (P26), R?.2
- new net: P103.27 (P27), R?.2
- new net: P103.28 (P28), R?.2
- new net: P103.3 (P3), R?.2
- new net: P103.4 (P4), R?.2
- new net: P103.5 (P5), R?.2
- new net: P103.6 (P6), R?.2
- new net: P103.7 (P7), R?.2
- new net: P110.10 (P10), R?.1
- new net: P110.11 (P11), R?.1
- new net: P110.12 (P12), R?.1
- new net: P110.13 (P13), R?.1
- new net: P110.14 (P14), R?.1
- new net: P110.3 (P3), R?.1
- new net: P110.4 (P4), R?.1
- new net: P110.5 (P5), R?.1
- new net: P110.6 (P6), R?.1
- new net: P110.7 (P7), R?.1
- new net: P109.10 (P10), R?.1
- new net: P109.11 (P11), R?.1
- new net: P109.2 (P2), R?.1
- new net: P109.3 (P3), R?.1
- new net: P109.4 (P4), R?.1
- new net: P109.7 (P7), R?.1
- new net: P109.8 (P8), R?.1
- new net: P109.9 (P9), R?.1
- new net: P108.10 (P10), R?.1
- new net: P108.11 (P11), R?.1
- new net: P108.12 (P12), R?.1
- new net: P108.13 (P13), R?.1
- new net: P108.2 (P2), R?.1
- new net: P108.28 (P28), R?.1
- new net: P108.29 (P29), R?.1
- new net: P108.3 (P3), R?.1
- new net: P108.4 (P4), R?.1
- new net: P108.5 (P5), R?.1
- new net: P108.6 (P6), R?.1
- new net: P108.9 (P9), R?.1
- new net: P107.10 (P10), R?.2
- new net: P107.11 (P11), R?.2
- new net: P107.12 (P12), R?.2
- new net: P107.13 (P13), R?.2
- new net: P107.2 (P2), R?.2
- new net: P107.3 (P3), R?.2
- new net: P107.4 (P4), R?.2
- new net: P107.5 (P5), R?.2
- new net: P107.6 (P6), R?.2
- new net: P107.9 (P9), R?.2
- new net: P105.11 (P11), R?.2
- new net: P105.12 (P12), R?.2
- new net: P105.13 (P13), R?.2
- new net: P105.14 (P14), R?.2
- new net: P105.15 (P15), R?.2
- new net: P105.18 (P18), R?.2
- new net: P105.19 (P19), R?.2
- new net: P105.20 (P20), R?.2
- new net: P105.21 (P21), R?.2
- new net: P105.22 (P22), R?.2
- new net: R?.1, U108.5 (A4)
- new net: R?.1, U116.10 (A9)
- new net: R?.2, U119.6 (Y1)
- new net: R?.2, U128.6 (Y1)
Other:
- moved on the sheet: R113

Commit message: monumental cockup- re-design point here!
Parts:
- removed R? (x60): 33R, symbol R
Connections:
- net L2_PAIR_Q1/BL_X0_XLA_0i: now also P102.24 (P24)
- net L2_PAIR_Q1/BL_X0_XLA_1i: now also P102.23 (P23)
- net L2_PAIR_Q1/BL_X0_XLA_2i: now also P102.22 (P22)
- net L2_PAIR_Q1/BL_X0_XLA_3i: now also P102.21 (P21)
- net L2_PAIR_Q1/BL_X0_XLA_4i: now also P102.20 (P20)
- net L2_PAIR_Q1/TL_X0_XLA_0i: now also P101.22 (P22)
- net L2_PAIR_Q1/TL_X0_XLA_1i: now also P101.21 (P21)
- net L2_PAIR_Q1/TL_X0_XLA_2i: now also P101.20 (P20)
- net L2_PAIR_Q1/TL_X0_XLA_3i: now also P101.19 (P19)
- net L2_PAIR_Q1/TL_X0_XLA_4i: now also P101.18 (P18)
- net L2_PAIR_Q1/T_X0_XLB_0i: now also P104.13 (P13)
- net L2_PAIR_Q1/T_X0_XLB_1i: now also P104.12 (P12)
- net L2_PAIR_Q1/T_X0_XLB_2i: now also P104.11 (P11)
- net L2_PAIR_Q1/T_X0_XLB_3i: now also P104.10 (P10)
- net L2_PAIR_Q1/T_X0_XLB_4i: now also P104.9 (P9)
- net L2_PAIR_Q2/BR_X1_XLA_0i: now also P109.4 (P4)
- net L2_PAIR_Q2/BR_X1_XLA_1i: now also P109.3 (P3)
- net L2_PAIR_Q2/BR_X1_XLA_2i: now also P109.2 (P2)
- net L2_PAIR_Q2/BR_X1_XLA_3i: now also P108.29 (P29)
- net L2_PAIR_Q2/BR_X1_XLA_4i: now also P108.28 (P28)
- net L2_PAIR_Q2/TR_X1_XLA_0i: now also P108.6 (P6)
- net L2_PAIR_Q2/TR_X1_XLA_1i: now also P108.5 (P5)
- net L2_PAIR_Q2/TR_X1_XLA_2i: now also P108.4 (P4)
- net L2_PAIR_Q2/TR_X1_XLA_3i: now also P108.3 (P3)
- net L2_PAIR_Q2/TR_X1_XLA_4i: now also P108.2 (P2)
- net L2_PAIR_Q2/T_X0_XLB_0i: now also P106.22 (P22)
- net L2_PAIR_Q2/T_X0_XLB_1i: now also P106.21 (P21)
- net L2_PAIR_Q2/T_X0_XLB_2i: now also P106.20 (P20)
- net L2_PAIR_Q2/T_X0_XLB_3i: now also P106.19 (P19)
- net L2_PAIR_Q2/T_X0_XLB_4i: now also P106.18 (P18)
- net L2_PAIR_Q3/BR_X1_XLA_0i: now also P110.21 (P21)
- net L2_PAIR_Q3/BR_X1_XLA_1i: now also P110.20 (P20)
- net L2_PAIR_Q3/BR_X1_XLA_2i: now also P110.19 (P19)
- net L2_PAIR_Q3/BR_X1_XLA_3i: now also P110.18 (P18)
- net L2_PAIR_Q3/BR_X1_XLA_4i: now also P110.17 (P17)
- net L2_PAIR_Q3/B_X1_XLB_0i: now also P107.6 (P6)
- net L2_PAIR_Q3/B_X1_XLB_1i: now also P107.5 (P5)
- net L2_PAIR_Q3/B_X1_XLB_2i: now also P107.4 (P4)
- net L2_PAIR_Q3/B_X1_XLB_3i: now also P107.3 (P3)
- net L2_PAIR_Q3/B_X1_XLB_4i: now also P107.2 (P2)
- net L2_PAIR_Q3/TR_X1_XLA_0i: now also P110.7 (P7)
- net L2_PAIR_Q3/TR_X1_XLA_1i: now also P110.6 (P6)
- net L2_PAIR_Q3/TR_X1_XLA_2i: now also P110.5 (P5)
- net L2_PAIR_Q3/TR_X1_XLA_3i: now also P110.4 (P4)
- net L2_PAIR_Q3/TR_X1_XLA_4i: now also P110.3 (P3)
- net L2_PAIR_Q4/BL_X0_XLA_0i: now also P103.7 (P7)
- net L2_PAIR_Q4/BL_X0_XLA_1i: now also P103.6 (P6)
- net L2_PAIR_Q4/BL_X0_XLA_2i: now also P103.5 (P5)
- net L2_PAIR_Q4/BL_X0_XLA_3i: now also P103.4 (P4)
- net L2_PAIR_Q4/BL_X0_XLA_4i: now also P103.3 (P3)
- net L2_PAIR_Q4/B_X1_XLB_0i: now also P105.15 (P15)
- net L2_PAIR_Q4/B_X1_XLB_1i: now also P105.14 (P14)
- net L2_PAIR_Q4/B_X1_XLB_2i: now also P105.13 (P13)
- net L2_PAIR_Q4/B_X1_XLB_3i: now also P105.12 (P12)
- net L2_PAIR_Q4/B_X1_XLB_4i: now also P105.11 (P11)
- net L2_PAIR_Q4/TL_X0_XLA_0i: now also P103.21 (P21)
- net L2_PAIR_Q4/TL_X0_XLA_1i: now also P103.20 (P20)
- net L2_PAIR_Q4/TL_X0_XLA_2i: now also P103.19 (P19)
- net L2_PAIR_Q4/TL_X0_XLA_3i: now also P103.18 (P18)
- net L2_PAIR_Q4/TL_X0_XLA_4i: now also P103.17 (P17)
- net at P110.24 (P24): now also R?.1
- net at P110.25 (P25): now also R?.1
- net at P110.26 (P26): now also R?.1
- net at P110.27 (P27): now also R?.1
- net at P110.28 (P28): now also R?.1

Commit message: ugh, this is painful!
Parts:
- gave numbers to parts that had none: 64
Connections:
- net L2_PAIR_Q1/T_X0_XLB_0i renamed L2_PAIR_Q1/T_X1_XLA_0i
- net L2_PAIR_Q1/T_X0_XLB_0o renamed L2_PAIR_Q1/T_X1_XLA_0o
- net L2_PAIR_Q1/T_X0_XLB_1i renamed L2_PAIR_Q1/T_X1_XLA_1i
- net L2_PAIR_Q1/T_X0_XLB_1o renamed L2_PAIR_Q1/T_X1_XLA_1o
- net L2_PAIR_Q1/T_X0_XLB_2i renamed L2_PAIR_Q1/T_X1_XLA_2i
- net L2_PAIR_Q1/T_X0_XLB_2o renamed L2_PAIR_Q1/T_X1_XLA_2o
- net L2_PAIR_Q1/T_X0_XLB_3i renamed L2_PAIR_Q1/T_X1_XLA_3i
- net L2_PAIR_Q1/T_X0_XLB_3o renamed L2_PAIR_Q1/T_X1_XLA_3o
- net L2_PAIR_Q1/T_X0_XLB_4i renamed L2_PAIR_Q1/T_X1_XLA_4i
- net L2_PAIR_Q1/T_X0_XLB_4o renamed L2_PAIR_Q1/T_X1_XLA_4o
- net L2_PAIR_Q2/BR_X1_XLA_0i renamed L2_PAIR_Q2/BR_X0_XLB_0i
- net L2_PAIR_Q2/BR_X1_XLA_0o renamed L2_PAIR_Q2/BR_X0_XLB_0o
- net L2_PAIR_Q2/BR_X1_XLA_1i renamed L2_PAIR_Q2/BR_X0_XLB_1i
- net L2_PAIR_Q2/BR_X1_XLA_1o renamed L2_PAIR_Q2/BR_X0_XLB_1o
- net L2_PAIR_Q2/BR_X1_XLA_2i renamed L2_PAIR_Q2/BR_X0_XLB_2i
- net L2_PAIR_Q2/BR_X1_XLA_2o renamed L2_PAIR_Q2/BR_X0_XLB_2o
- net L2_PAIR_Q2/BR_X1_XLA_3i renamed L2_PAIR_Q2/BR_X0_XLB_3i
- net L2_PAIR_Q2/BR_X1_XLA_3o renamed L2_PAIR_Q2/BR_X0_XLB_3o
- net L2_PAIR_Q2/BR_X1_XLA_4i renamed L2_PAIR_Q2/BR_X0_XLB_4i
- net L2_PAIR_Q2/BR_X1_XLA_4o renamed L2_PAIR_Q2/BR_X0_XLB_4o
- net L2_PAIR_Q2/T_X0_XLB_0i renamed L2_PAIR_Q2/T_X1_XLA_0i
- net L2_PAIR_Q2/T_X0_XLB_0o renamed L2_PAIR_Q2/T_X1_XLA_0o
- net L2_PAIR_Q2/T_X0_XLB_1i renamed L2_PAIR_Q2/T_X1_XLA_1i
- net L2_PAIR_Q2/T_X0_XLB_1o renamed L2_PAIR_Q2/T_X1_XLA_1o
- net L2_PAIR_Q2/T_X0_XLB_2i renamed L2_PAIR_Q2/T_X1_XLA_2i
- net L2_PAIR_Q2/T_X0_XLB_2o renamed L2_PAIR_Q2/T_X1_XLA_2o
- net L2_PAIR_Q2/T_X0_XLB_3i renamed L2_PAIR_Q2/T_X1_XLA_3i
- net L2_PAIR_Q2/T_X0_XLB_3o renamed L2_PAIR_Q2/T_X1_XLA_3o
- net L2_PAIR_Q2/T_X0_XLB_4i renamed L2_PAIR_Q2/T_X1_XLA_4i
- net L2_PAIR_Q2/T_X0_XLB_4o renamed L2_PAIR_Q2/T_X1_XLA_4o
- net L2_PAIR_Q3/BR_X1_XLA_0i renamed L2_PAIR_Q3/BR_X0_XLB_0i
- net L2_PAIR_Q3/BR_X1_XLA_0o renamed L2_PAIR_Q3/BR_X0_XLB_0o
- net L2_PAIR_Q3/BR_X1_XLA_1i renamed L2_PAIR_Q3/BR_X0_XLB_1i
- net L2_PAIR_Q3/BR_X1_XLA_1o renamed L2_PAIR_Q3/BR_X0_XLB_1o
- net L2_PAIR_Q3/BR_X1_XLA_2i renamed L2_PAIR_Q3/BR_X0_XLB_2i
- net L2_PAIR_Q3/BR_X1_XLA_2o renamed L2_PAIR_Q3/BR_X0_XLB_2o
- net L2_PAIR_Q3/BR_X1_XLA_3i renamed L2_PAIR_Q3/BR_X0_XLB_3i
- net L2_PAIR_Q3/BR_X1_XLA_3o renamed L2_PAIR_Q3/BR_X0_XLB_3o
- net L2_PAIR_Q3/BR_X1_XLA_4i renamed L2_PAIR_Q3/BR_X0_XLB_4i
- net L2_PAIR_Q3/BR_X1_XLA_4o renamed L2_PAIR_Q3/BR_X0_XLB_4o

Commit message: almost all the links in, some of the JTAG in. Surprisingly nice :)
Parts:
- removed R118, R119, R120, R130, R132, R133, R134, R135, R137, R138, R139, R140, R142, R143, R144, R145, R152, R153, R154, R155, R161, R162, R163, R164, R167, R168, R169, R170, R172, R173, R174, R175, R177, R178, R179, R180, R182, R183, R184, R185: 33R, symbol R
- added U102, U121, U122, U124, U129, U130, U132, U133, U134, U135: YC124, symbol YC124
Connections:
- net DEBUG_N_BUF_B: now also P105.23 (P23); no longer P107.23 (P23)
- net DEBUG_N_BUF_R: now also P108.6 (P6); no longer P108.20 (P20)
- net DEBUG_N_L: now also P101.25 (P25); no longer P101.11 (P11)
- net DEBUG_N_T: now also P104.8 (P8); no longer P106.8 (P8)
- net GND: now also P101.10 (P10), P101.11 (P11), P101.18 (P18), P101.20 (P20), P101.22 (P22), P101.26 (P26), P101.28 (P28), P104.10 (P10), P104.11 (P11), P104.12 (P12), P104.13 (P13), P104.16 (P16), P104.23 (P23), P104.9 (P9), P105.15 (P15), P105.18 (P18), P105.19 (P19), P105.20 (P20), P105.21 (P21), P105.22 (P22), P105.8 (P8), P106.2 (P2), P106.4 (P4), P106.6 (P6), P106.7 (P7), P106.8 (P8), P107.23 (P23), P107.24 (P24), P107.25 (P25), P107.27 (P27), P107.29 (P29), P108.11 (P11), P108.13 (P13), P108.20 (P20), P108.21 (P21), P108.3 (P3), P108.5 (P5), P108.9 (P9); no longer P101.12 (P12), P101.14 (P14), P101.16 (P16), P101.23 (P23), P101.24 (P24), P101.6 (P6), P101.8 (P8), P104.2 (P2), P104.21 (P21), P104.24 (P24), P104.26 (P26), P104.27 (P27), P104.28 (P28), P104.4 (P4), P104.6 (P6), P104.7 (P7), P104.8 (P8), P105.10 (P10), P105.23 (P23), P105.24 (P24), P105.25 (P25), P105.27 (P27), P105.29 (P29), P105.3 (P3), P105.4 (P4), P105.5 (P5), P105.7 (P7), P106.3 (P3), P106.5 (P5), P107.26 (P26), P107.28 (P28), P108.15 (P15), P108.17 (P17), P108.19 (P19), P108.23 (P23), P108.25 (P25), P108.7 (P7), P108.8 (P8)
- net L2_PAIR_Q1/BL_X0_XLA_0o: now also U130.1
- net L2_PAIR_Q1/BL_X0_XLA_1o: now also U130.2
- net L2_PAIR_Q1/BL_X0_XLA_2o: now also U130.3
- net L2_PAIR_Q1/BL_X0_XLA_3o: now also U130.4
- net L2_PAIR_Q1/TL_X0_XLA_0i: now also P101.9 (P9); no longer P101.22 (P22)
- net L2_PAIR_Q1/TL_X0_XLA_0o: now also U122.5
- net L2_PAIR_Q1/TL_X0_XLA_1i: now also P101.8 (P8); no longer P101.21 (P21)
- net L2_PAIR_Q1/TL_X0_XLA_1o: now also U122.6
- net L2_PAIR_Q1/TL_X0_XLA_2i: now also P101.7 (P7); no longer P101.20 (P20)
- net L2_PAIR_Q1/TL_X0_XLA_2o: now also U122.7
- net L2_PAIR_Q1/TL_X0_XLA_3i: now also P101.6 (P6); no longer P101.19 (P19)
- net L2_PAIR_Q1/TL_X0_XLA_3o: now also U122.8
- net L2_PAIR_Q1/TL_X0_XLA_4i: now also P101.5 (P5); no longer P101.18 (P18)
- net L2_PAIR_Q1/T_X1_XLA_0i: now also P104.21 (P21); no longer P104.13 (P13)
- net L2_PAIR_Q1/T_X1_XLA_0o: now also U102.5; no longer R151.2
- net L2_PAIR_Q1/T_X1_XLA_1i: now also P104.20 (P20); no longer P104.12 (P12)
- net L2_PAIR_Q1/T_X1_XLA_1o: now also U102.6
- net L2_PAIR_Q1/T_X1_XLA_2i: now also P104.19 (P19); no longer P104.11 (P11)
- net L2_PAIR_Q1/T_X1_XLA_2o: now also U102.7
- net L2_PAIR_Q1/T_X1_XLA_3i: now also P104.18 (P18); no longer P104.10 (P10)
- net L2_PAIR_Q1/T_X1_XLA_3o: now also U102.8
- net L2_PAIR_Q1/T_X1_XLA_4i: now also P104.17 (P17); no longer P104.9 (P9)
- net L2_PAIR_Q1/T_X1_XLA_4o: now also R151.2
- net L2_PAIR_Q2/BR_X0_XLB_1o: now also U133.1
- net L2_PAIR_Q2/BR_X0_XLB_2o: now also U133.2
- net L2_PAIR_Q2/BR_X0_XLB_3o: now also U133.3
- net L2_PAIR_Q2/BR_X0_XLB_4o: now also U133.4
- net L2_PAIR_Q2/TR_X1_XLA_0i: now also P108.19 (P19); no longer P108.6 (P6)
- net L2_PAIR_Q2/TR_X1_XLA_1i: now also P108.18 (P18); no longer P108.5 (P5)
- net L2_PAIR_Q2/TR_X1_XLA_1o: now also U132.1
- net L2_PAIR_Q2/TR_X1_XLA_2i: now also P108.17 (P17); no longer P108.4 (P4)
- net L2_PAIR_Q2/TR_X1_XLA_2o: now also U132.2
- net L2_PAIR_Q2/TR_X1_XLA_3i: now also P108.16 (P16); no longer P108.3 (P3)
- net L2_PAIR_Q2/TR_X1_XLA_3o: now also U132.3
- net L2_PAIR_Q2/TR_X1_XLA_4i: now also P108.15 (P15); no longer P108.2 (P2)
- net L2_PAIR_Q2/TR_X1_XLA_4o: now also U132.4
- net L2_PAIR_Q2/T_X1_XLA_1o: now also U121.2
- net L2_PAIR_Q2/T_X1_XLA_2o: now also U121.3
- net L2_PAIR_Q2/T_X1_XLA_3o: now also U121.4
- net L2_PAIR_Q3/BR_X0_XLB_1o: now also U134.1
- net L2_PAIR_Q3/BR_X0_XLB_2o: now also U134.2
- net L2_PAIR_Q3/BR_X0_XLB_3o: now also U134.3
- net L2_PAIR_Q3/BR_X0_XLB_4o: now also U134.4
- net L2_PAIR_Q3/TR_X1_XLA_1o: now also U135.1
- net L2_PAIR_Q3/TR_X1_XLA_2o: now also U135.2
- net L2_PAIR_Q3/TR_X1_XLA_3o: now also U135.3
- net L2_PAIR_Q3/TR_X1_XLA_4o: now also U135.4
- net L2_PAIR_Q4/BL_X0_XLA_0o: now also U129.1
- net L2_PAIR_Q4/BL_X0_XLA_1o: now also U129.2
- net L2_PAIR_Q4/BL_X0_XLA_2o: now also U129.3
- net L2_PAIR_Q4/BL_X0_XLA_3o: now also U129.4
- net L2_PAIR_Q4/B_X1_XLB_0i: now also P105.7 (P7); no longer P105.15 (P15)
- net L2_PAIR_Q4/B_X1_XLB_1i: now also P105.6 (P6); no longer P105.14 (P14)
- net L2_PAIR_Q4/B_X1_XLB_2i: now also P105.5 (P5); no longer P105.13 (P13)
- net L2_PAIR_Q4/B_X1_XLB_3i: now also P105.4 (P4); no longer P105.12 (P12)
- net L2_PAIR_Q4/B_X1_XLB_4i: now also P105.3 (P3); no longer P105.11 (P11)
- net L2_PAIR_Q4/TL_X0_XLA_0o: now also U124.1
- net L2_PAIR_Q4/TL_X0_XLA_1o: now also U124.2
- net L2_PAIR_Q4/TL_X0_XLA_2o: now also U124.3
- net L2_PAIR_Q4/TL_X0_XLA_3o: now also U124.4
- net RST_N_BUF_B: now also P105.25 (P25); no longer P107.25 (P25)
- net RST_N_BUF_R: now also P108.8 (P8); no longer P108.22 (P22)
- net RST_N_L: now also P101.23 (P23); no longer P101.9 (P9)
- net RST_N_T: now also P104.6 (P6); no longer P106.6 (P6)
- net TCK_BUF_B: now also P105.27 (P27); no longer P107.27 (P27)
- net TCK_BUF_R: now also P108.10 (P10); no longer P108.24 (P24)
- net TCK_L: now also P101.21 (P21); no longer P101.7 (P7)
- net TCK_T: now also P104.4 (P4); no longer P106.4 (P4)
- net TDI_B: now also P107.26 (P26); no longer P105.6 (P6)
- net TDI_L: now also P101.27 (P27); no longer P101.13 (P13)
- net TDI_R: now also P108.2 (P2); no longer P108.16 (P16)
- net TDI_T: now also P106.3 (P3); no longer P104.23 (P23)
- net TDO_B: now also P107.28 (P28); no longer P105.8 (P8)
- net TDO_L: now also P101.29 (P29); no longer P101.15 (P15)
- net TDO_R: now also P108.4 (P4); no longer P108.18 (P18)
- net TDO_T: now also P106.5 (P5); no longer P104.25 (P25)
- net TMS_BUF_B: now also P105.29 (P29); no longer P107.29 (P29)
- net TMS_BUF_R: now also P108.12 (P12); no longer P108.26 (P26)
- net TMS_L: now also P101.19 (P19); no longer P101.5 (P5)
- net TMS_T: now also P104.2 (P2); no longer P106.2 (P2)
- net TRST_N_BUF_B: now also P105.24 (P24); no longer P107.24 (P24)
- net TRST_N_BUF_R: now also P108.7 (P7); no longer P108.21 (P21)
- net TRST_N_L: now also P101.24 (P24); no longer P101.10 (P10)
- net TRST_N_T: now also P104.7 (P7); no longer P106.7 (P7)
- net at P101.2 (P2): now also U130.5
- net at R131.2: now also P101.16 (P16); no longer P101.29 (P29)
- net at P102.27 (P27): now also U130.8
- net at P102.28 (P28): now also U130.7
- net at P102.29 (P29): now also U130.6
- net at R151.1: now also P104.28 (P28); no longer P104.16 (P16)
- net at P106.25 (P25): now also U121.8
- net at P106.26 (P26): now also U121.7
- net at P106.27 (P27): now also U121.6
- net at P106.28 (P28): now also U121.5
- net at P103.10 (P10): now also U129.8
- net at P103.11 (P11): now also U129.7
- net at P103.12 (P12): now also U129.6
- net at P103.13 (P13): now also U129.5
- net at P103.24 (P24): now also U124.8
- net at P103.25 (P25): now also U124.7
- net at P103.26 (P26): now also U124.6
- net at P103.27 (P27): now also U124.5
- net at P110.11 (P11): now also U135.8
- net at P110.12 (P12): now also U135.7
- net at P110.13 (P13): now also U135.6
- net at P110.14 (P14): now also U135.5
- net at P110.25 (P25): now also U134.8
- net at P110.26 (P26): now also U134.7
- net at P110.27 (P27): now also U134.6
- net at P110.28 (P28): now also U134.5
- net at P109.10 (P10): now also U133.6
- net at P109.11 (P11): now also U133.5
- net at P109.8 (P8): now also U133.8
- net at P109.9 (P9): now also U133.7
- net at R171.1: now also P108.22 (P22); no longer P108.9 (P9)
- net at R150.2: now also P105.10 (P10); no longer P105.18 (P18)
- net at R149.2: now also P105.11 (P11); no longer P105.19 (P19)
- net at R148.2: now also P105.12 (P12); no longer P105.20 (P20)
- net at R147.2: now also P105.13 (P13); no longer P105.21 (P21)
- net at R146.2: now also P105.14 (P14); no longer P105.22 (P22)
- new net: P101.12 (P12), U122.4
- new net: P101.13 (P13), U122.3
- new net: P101.14 (P14), U122.2
- new net: P101.15 (P15), U122.1
- new net: P104.24 (P24), U102.4
- new net: P104.25 (P25), U102.3
- new net: P104.26 (P26), U102.2
- new net: P104.27 (P27), U102.1
- new net: P108.23 (P23), U132.8
- new net: P108.24 (P24), U132.7
- new net: P108.25 (P25), U132.6
- new net: P108.26 (P26), U132.5
Other:
- moved on the sheet: R131, R146, R147, R148, R149, R150, R151, R171
