File: l2_dev_alternative _nopwrsense/l2_dev_board.sch (KiCad schematic (older format))
At the start: 101 parts, among them P101 CONN_30, P102 CONN_30, P103 CONN_30, P104 CONN_30, P105 CONN_30, P106 CONN_30, P107 CONN_30, P108 CONN_30, P109 CONN_30, P110 CONN_30, U101 APX803-SR, U102 YC124, U103 A6RS-161RF, U104 SN74LVC1G18, U105 SN74LVC1G18, U106 SN74LVC1G18, U107 SN74LVC1G18, U108 SN74CBTD3861, U109 LT3480, U110 APX803-SR, U111 74AHC1GU04, U112 NC7WZ17, U113 NC7WZ17, U114 NC7WZ17, U115 NC7WZ17, U116 SN74CBTD3861, U117 NCP1529, U118 NC7WZ07, U119 NC7WZ17, U120 NC7WZ17, U121 YC124, U122 YC124, U123 ASE_CLK, U124 YC124, U125 NC7WZ17, U126 NC7WZ17, U127 NC7WZ07, U128 NC7WZ17, U129 YC124, U130 YC124, U131 NC7WZ17, U132 YC124, U133 YC124, U134 YC124, U135 YC124

Commit message: almost done. adding cutouts for power islands
Parts:
- removed R147, R148, R149, R150, R156, R157, R158, R159: 33R, symbol R
- added U136, U137: YC124, symbol YC124
Connections:
- net DEBUG_N: now also U118.1 (A1), U126.3 (A2); no longer U119.3 (A2), U126.1 (A1)
- net DEBUG_N_BUF_B: now also U126.4 (Y2); no longer U126.6 (Y1)
- net DEBUG_N_BUF_R: now also U118.6 (Y1); no longer U119.4 (Y2)
- net L2_PAIR_Q3/B_X1_XLB_1o: now also U137.5
- net L2_PAIR_Q3/B_X1_XLB_2o: now also U137.6
- net L2_PAIR_Q3/B_X1_XLB_3o: now also U137.7
- net L2_PAIR_Q3/B_X1_XLB_4o: now also U137.8
- net L2_PAIR_Q4/B_X1_XLB_0o: now also R146.1
- net L2_PAIR_Q4/B_X1_XLB_1o: now also U136.5
- net L2_PAIR_Q4/B_X1_XLB_2o: now also U136.6
- net L2_PAIR_Q4/B_X1_XLB_3o: now also U136.7
- net L2_PAIR_Q4/B_X1_XLB_4o: now also U136.8; no longer R146.1
- net MSEL_N: now also U118.3 (A2), U127.1 (A1); no longer U120.1 (A1), U126.3 (A2)
- net RST_N: now also U119.1 (A1); no longer U118.1 (A1)
- net RST_N_BUF_R: now also U119.6 (Y1); no longer U118.6 (Y1)
- net TCK: now also U119.3 (A2); no longer U119.1 (A1)
- net TMS: now also U120.1 (A1); no longer U120.3 (A2)
- net TMS_BUF_R: now also U120.6 (Y1); no longer U120.4 (Y2)
- net TRST_N_BUF_B: now also U127.6 (Y1); no longer U126.4 (Y2)
- net TRST_N_BUF_R: now also U118.4 (Y2); no longer U120.6 (Y1)
- net at P107.10 (P10): now also U137.4
- net at P107.11 (P11): now also U137.3
- net at P107.12 (P12): now also U137.2
- net at P107.13 (P13): now also U137.1
- net at P105.10 (P10): now also R146.2
- net at P105.11 (P11): now also U136.4
- net at P105.12 (P12): now also U136.3
- net at P105.13 (P13): now also U136.2
- net at P105.14 (P14): now also U136.1; no longer R146.2
- net at R115.2: now also U119.4 (Y2); no longer U119.6 (Y1)
Other:
- moved on the sheet: R115, R146
Changed lines of the file:
@@
-EESchema Schematic File Version 2  date 06/09/2011 20:03:42
+EESchema Schematic File Version 2  date 07/09/2011 23:31:18
 LIBS:power
 LIBS:device
@@
 Sheet 1 13
 Title ""
-Date "6 sep 2011"
+Date "7 sep 2011"
 Rev ""
 Comp ""
@@
 Comment4 ""
 $EndDescr
+Text Label 7970 4840 0    39   ~ 0
+TRST_N_BUF_B
+Wire Wire Line
+	7970 2120 7860 2120
+Wire Wire Line
+	7980 1420 7860 1420
+Wire Wire Line
+	18580 13630 18580 13150
+Wire Wire Line
+	18380 13630 18380 13250
+Wire Wire Line
+	14070 14030 14070 13750
+Wire Wire Line
+	13870 13970 13870 13870
 Wire Wire Line
 	21360 12750 20160 12750
@@
 	21160 5410 21160 5530
 Wire Wire Line
-	11390 13980 13670 13980
-Wire Wire Line
-	11490 13870 13870 13870
+	13870 13870 11490 13870
 Wire Wire Line
-	11610 13750 14070 13750
+	14070 13750 11610 13750
 Wire Wire Line
 	11730 13630 14470 13630
@@
 	12970 11730 11390 11730
 Wire Wire Line
-	11390 11730 11390 13980
-Wire Wire Line
 	12970 12370 11850 12370
 Wire Wire Line
@@
 	8520 5570 8520 5730
 Wire Wire Line
-	8500 1930 8500 2120
-Wire Wire Line
-	8500 2120 8470 2120
+	8470 2320 8500 2320
 Wire Notes Line
 	5970 5540 1240 5540
@@
 	21510 10950 21280 10950
 Wire Wire Line
-	18280 13690 18280 13300
-Wire Wire Line
-	18480 13690 18480 13200
-Wire Wire Line
 	18680 13690 18680 13100
 Wire Wire Line
@@
 	18680 14720 18680 14190
 Wire Wire Line
-	13670 13980 13670 14030
-Wire Wire Line
-	13870 13870 13870 14030
-Wire Wire Line
-	14070 13750 14070 14030
-Wire Wire Line
 	13770 14720 13770 14530
 Wire Wire Line
@@
 	7860 4380 7860 4340
 Wire Wire Line
-	7860 3940 7970 3940
+	7860 4140 7970 4140
 Wire Wire Line
 	7860 5040 7970 5040
 Wire Wire Line
-	7860 4140 7970 4140
+	7860 4840 7970 4840
 Wire Wire Line
 	7860 5930 7970 5930
@@
 	7860 5730 7970 5730
 Wire Wire Line
-	6560 4140 6450 4140
+	6560 4840 6450 4840
 Wire Wire Line
 	6560 5040 6450 5040
 Wire Wire Line
-	6560 3940 6450 3940
+	6560 4140 6450 4140
 Wire Wire Line
 	6560 5930 6450 5930
@@
 	7950 6890 7860 6890
 Wire Wire Line
-	6560 6690 6460 6690
+	6460 6690 6560 6690
 Wire Wire Line
 	7860 6420 7860 6490
@@
 Connection ~ 7810 11820
 Wire Wire Line
-	8050 11820 7570 11820
+	7570 11820 8050 11820
 Connection ~ 7890 11820
 Connection ~ 8050 11260
@@
 	7730 11320 7730 10860
 Wire Wire Line
-	7490 11060 8180 11060
+	8180 11060 7490 11060
 Wire Wire Line
-	7490 11260 8180 11260
+	8180 11260 7490 11260
 Wire Wire Line
-	7490 10860 8180 10860
+	8180 10860 7490 10860
 Wire Wire Line
-	7490 10660 8180 10660
+	8180 10660 7490 10660
 Wire Wire Line
 	4740 4320 4740 4360
@@
 Connection ~ 7620 9170
 Wire Wire Line
-	7620 9700 7620 9670
+	7620 9670 7620 9700
 Wire Wire Line
 	6930 9170 6880 9170
 Wire Wire Line
-	6130 10170 6130 10230
+	6130 10230 6130 10170
 Wire Wire Line
 	5080 9170 5380 9170
 Wire Wire Line
-	5080 9000 5080 9200
+	5080 9200 5080 9000
 Connection ~ 5080 9170
 Wire Wire Line
@@
 	1840 1050 650  1050
 Wire Wire Line
-	2040 3030 2040 3130
+	2040 3130 2040 3030
 Wire Wire Line
 	1190 3070 1190 2890
@@
 Connection ~ 2880 3070
 Wire Wire Line
-	2790 2530 2930 2530
+	2930 2530 2790 2530
 Connection ~ 2880 2530
 Wire Wire Line
-	2850 2130 2790 2130
+	2790 2130 2850 2130
 Connection ~ 2820 2130
 Wire Wire Line
 	2840 1780 2790 1780
 Wire Wire Line
-	2160 3750 1950 3750
+	1950 3750 2160 3750
 Wire Wire Line
 	2680 3420 2630 3420
@@
 	7860 2320 7970 2320
 Wire Wire Line
-	7860 2120 7970 2120
-Wire Wire Line
 	7860 3010 7970 3010
 Wire Wire Line
@@
 	7860 7340 7860 7410
 Wire Wire Line
-	6560 7610 6460 7610
+	6460 7610 6560 7610
 Wire Wire Line
 	7950 6690 7860 6690
@@
 	18680 13100 15610 13100
 Wire Wire Line
-	18480 13200 15490 13200
+	15490 13200 18480 13200
 Wire Wire Line
-	18280 13300 15380 13300
+	15380 13300 18280 13300
 Wire Wire Line
 	2100 10070 2100 10020
@@
 Connection ~ 2370 10180
 Wire Wire Line
-	2510 10180 2340 10180
+	2340 10180 2510 10180
 Wire Wire Line
 	2370 11300 2510 11300
@@
 	13670 14530 13670 14720
 Wire Wire Line
-	13970 14030 13970 13810
-Wire Wire Line
-	13770 14030 13770 13930
-Wire Wire Line
 	18580 14190 18580 14720
 Wire Wire Line
 	18380 14190 18380 14720
 Wire Wire Line
-	18580 13150 18580 13690
-Wire Wire Line
-	18380 13250 18380 13690
-Wire Wire Line
 	20640 11100 20640 11950
 Wire Wire Line
@@
 Wire Wire Line
 	20240 12650 21360 12650
+Wire Wire Line
+	13770 13930 13770 13970
+Wire Wire Line
+	13970 13810 13970 13970
+Wire Wire Line
+	13670 13970 11390 13970
+Wire Wire Line
+	11390 13970 11390 11730
+Wire Wire Line
+	18280 13300 18280 13630
+Wire Wire Line
+	18480 13200 18480 13630
+Wire Wire Line
+	6440 1420 6560 1420
+Wire Wire Line
+	8500 2320 8500 2470
+$Comp
+L YC124 U137
+U 1 1 4E672AD0
+P 18430 13910
+F 0 "U137" H 18460 13720 60  0000 C CNN
+F 1 "YC124" H 18470 14090 60  0000 C CNN
+	1    18430 13910
+	1    0    0    -1
+$EndComp
+$Comp
+L YC124 U136
+U 1 1 4E672949
+P 13820 14250
+F 0 "U136" H 13850 14060 60  0000 C CNN
+F 1 "YC124" H 13860 14430 60  0000 C CNN
+	1    13820 14250
+	1    0    0    -1
+$EndComp
 $Comp
 L YC124 U134
@@
 L R R115
 U 1 1 4E60C5E9
-P 8220 2120
-F 0 "R115" V 8180 2320 50  0000 C CNN
-F 1 "33R" V 8220 2120 50  0000 C CNN
-	1    8220 2120
+P 8220 2320
+F 0 "R115" V 8180 2520 50  0000 C CNN
+F 1 "33R" V 8220 2320 50  0000 C CNN
+	1    8220 2320
 	0    1    1    0
 $EndComp
@@
 L R R146
 U 1 1 4E60B46A
-P 13670 14280
-F 0 "R146" V 13640 14480 50  0000 C CNN
-F 1 "33R" V 13670 14280 50  0000 C CNN
-	1    13670 14280
-	1    0    0    -1
-$EndComp
-$Comp
-L R R147
-U 1 1 4E60B469
-P 13770 14280
-F 0 "R147" V 13740 14480 50  0000 C CNN
-F 1 "33R" V 13770 14280 50  0000 C CNN
-	1    13770 14280
-	1    0    0    -1
-$EndComp
-$Comp
-L R R148
-U 1 1 4E60B468
-P 13870 14280
-F 0 "R148" V 13840 14480 50  0000 C CNN
-F 1 "33R" V 13870 14280 50  0000 C CNN
-	1    13870 14280
-	1    0    0    -1
-$EndComp
-$Comp
-L R R149
-U 1 1 4E60B467
-P 13970 14280
-F 0 "R149" V 13940 14480 50  0000 C CNN
-F 1 "33R" V 13970 14280 50  0000 C CNN
-	1    13970 14280
-	1    0    0    -1
-$EndComp
-$Comp
-L R R150
-U 1 1 4E60B466
 P 14070 14280
-F 0 "R150" V 14040 14480 50  0000 C CNN
+F 0 "R146" V 14040 14480 50  0000 C CNN
 F 1 "33R" V 14070 14280 50  0000 C CNN
 	1    14070 14280
@@
 $EndComp
 $Comp
-L R R156
-U 1 1 4E60B463
-P 18280 13940
-F 0 "R156" V 18250 14140 50  0000 C CNN
-F 1 "33R" V 18280 13940 50  0000 C CNN
-	1    18280 13940
-	1    0    0    -1
-$EndComp
-$Comp
-L R R157
-U 1 1 4E60B462
-P 18380 13940
-F 0 "R157" V 18350 14140 50  0000 C CNN
-F 1 "33R" V 18380 13940 50  0000 C CNN
-	1    18380 13940
-	1    0    0    -1
-$EndComp
-$Comp
-L R R158
-U 1 1 4E60B461
-P 18480 13940
-F 0 "R158" V 18450 14140 50  0000 C CNN
-F 1 "33R" V 18480 13940 50  0000 C CNN
-	1    18480 13940
-	1    0    0    -1
-$EndComp
-$Comp
-L R R159
-U 1 1 4E60B460
-P 18580 13940
-F 0 "R159" V 18550 14140 50  0000 C CNN
-F 1 "33R" V 18580 13940 50  0000 C CNN
-	1    18580 13940
-	1    0    0    -1
-$EndComp
-$Comp
 L R R160
 U 1 1 4E60B45F
@@
 CLK_20M_BUF_3
 Text Label 12890 8820 2    30   ~ 0
-CLK_20M_BUF_2
+CLK_20M_BUF_7
 Text Label 12880 3600 2    30   ~ 0
 CLK_20M_BUF_1
@@
 CLK_20M_BUF_4
 Text Label 12890 8740 2    30   ~ 0
-CLK_20M_BUF_1
+CLK_20M_BUF_8
 Text Label 12880 3520 2    30   ~ 0
 CLK_20M_BUF_2
-Text Label 16560 8790 2    30   ~ 0
-CLK_20M_BUF_6
 Text Label 16560 8700 2    30   ~ 0
+CLK_20M_BUF_6
+Text Label 16560 8790 2    30   ~ 0
 CLK_20M_BUF_5
 Text Label 2370 9870 2    30   ~ 0
@@
 	1    0    0    -1
 $EndComp
-Text Notes 8070 2400 0    60   ~ 0
+Text Notes 8070 2600 0    60   ~ 0
 \n
 $Comp
@@
 	1    0    0    -1
 $EndComp
-Text Label 6450 3940 2    39   ~ 0
+Text Label 6450 4140 2    39   ~ 0
 DEBUG_N
 Text Label 6450 5930 2    39   ~ 0
@@
 Text Label 6450 5040 2    39   ~ 0
 RST_N
-Text Label 6450 4140 2    39   ~ 0
+Text Label 6450 4840 2    39   ~ 0
 MSEL_N
-Text Label 7970 3940 0    39   ~ 0
+Text Label 7970 4140 0    39   ~ 0
 DEBUG_N_BUF_B
 Text Label 7970 5930 0    39   ~ 0
@@
 Text Label 7970 5040 0    39   ~ 0
 RST_N_BUF_B
-Text Label 7970 4140 0    39   ~ 0
-TRST_N_BUF_B
 $Comp
 L +3.3V #PWR067
@@
 	1    0    0    -1
 $EndComp
-Text Label 7970 3010 0    39   ~ 0
+Text Label 7980 1420 0    39   ~ 0
 TRST_N_BUF_R
-Text Label 7970 1220 0    39   ~ 0
+Text Label 7970 2120 0    39   ~ 0
 RST_N_BUF_R
-Text Label 8500 1930 2    39   ~ 0
+Text Label 8500 2470 2    39   ~ 0
 TCK_BUF_R
-Text Label 7970 3210 0    39   ~ 0
+Text Label 7970 3010 0    39   ~ 0
 TMS_BUF_R
-Text Label 7970 2320 0    39   ~ 0
+Text Label 7970 1220 0    39   ~ 0
 DEBUG_N_BUF_R
-Text Label 6450 3010 2    39   ~ 0
+Text Label 6440 1420 2    39   ~ 0
 MSEL_N
-Text Label 6450 1220 2    39   ~ 0
-RST_N
 Text Label 6450 2120 2    39   ~ 0
+RST_N
+Text Label 6450 2320 2    39   ~ 0
 TCK
-Text Label 6450 3210 2    39   ~ 0
+Text Label 6450 3010 2    39   ~ 0
 TMS
-Text Label 6450 2320 2    39   ~ 0
+Text Label 6450 1220 2    39   ~ 0
 DEBUG_N
 $Comp

Commit message: going to flood the top!
Parts:
- C101, C102, C103, C104, C105, C106, C107, C108, R101, R102, R103, R104, R105, R106, R107, R108, R109, R110, R111, R113, R115, R116, R117, R121, R122, R123, R124, R125, R126, R127, R128, R129, R131, R136, R141, R146, R151, R160, R165, R166, R171, R176, R181: footprint (none) -> 0603
- D101: footprint (none) -> DFLS240L
- L101: value 2.2uH -> 2u2H; footprint (none) -> LQH55P
- R112, R114: value 33R -> 10k; footprint (none) -> 0603
- U101, U110: footprint (none) -> SOT23-3
- U102, U121, U122, U124, U129, U130, U132, U133, U134, U135, U136, U137: footprint (none) -> 4x0402
- U103: footprint (none) -> AR6S-SWT
- U104, U105, U106, U107: footprint (none) -> SOT23-6
- U108, U116: footprint (none) -> TSSOP-24
- U109: footprint (none) -> 10DFN
- U111: footprint (none) -> SOT25-5
- U112, U113, U114, U115, U120, U125, U126, U127, U128, U131: footprint (none) -> SC70-6
- U117: footprint (none) -> SOT23-5
- U118: renamed from U119; footprint (none) -> SC70-6
- U119: renamed from U118; footprint (none) -> SC70-6
- U123: footprint (none) -> SMD-4
Connections:
- net +3.3V: now also R112.1, R114.1, U104.5 (VCC), U105.5 (VCC), U106.5 (VCC), U107.5 (VCC)
- net +5V: no longer U104.5 (VCC), U105.5 (VCC), U106.5 (VCC), U107.5 (VCC)
- net DEBUG_N: now also U118.1 (A1), U126.1 (A1); no longer U119.1 (A1), U126.3 (A2)
- net DEBUG_N_BUF_B: now also U126.6 (Y1); no longer U126.4 (Y2)
- net DEBUG_N_BUF_R: now also U118.6 (Y1); no longer U119.6 (Y1)
- net MSEL_N: now also U118.3 (A2), U126.3 (A2); no longer U119.3 (A2), U127.1 (A1)
- net RST_N: now also U119.1 (A1); no longer U118.1 (A1)
- net RST_N_BUF_B: now also R112.2
- net RST_N_BUF_R: now also R114.2, U119.6 (Y1); no longer U118.6 (Y1)
- net TCK: now also U120.1 (A1); no longer U118.3 (A2)
- net TCK_L: now also U108.5 (A4); no longer R112.2
- net TCK_T: now also U116.10 (A9); no longer R114.2
- net TMS: now also U120.3 (A2); no longer U120.1 (A1)
- net TMS_BUF_R: now also U120.4 (Y2); no longer U120.6 (Y1)
- net TRST_N_BUF_B: now also U126.4 (Y2); no longer U127.6 (Y1)
- net TRST_N_BUF_R: now also U118.4 (Y2); no longer U119.4 (Y2)
- net at R115.2: now also U120.6 (Y1); no longer U118.4 (Y2)
Other:
- moved on the sheet: R115, U118, U119
