File: l2_dev_alternative _nopwrsense/l2_dev_board.sch (KiCad schematic (older format))
At the start: 95 parts, among them P101 CONN_30, P102 CONN_30, P103 CONN_30, P104 CONN_30, P105 CONN_30, P106 CONN_30, P107 CONN_30, P108 CONN_30, P109 CONN_30, P110 CONN_30, U101 APX803-SR, U102 YC124, U103 A6RS-161RF, U104 SN74LVC1G18, U105 SN74LVC1G18, U106 SN74LVC1G18, U107 SN74LVC1G18, U108 SN74CBTD3861, U109 LT3480, U110 APX803-SR, U111 74AHC1GU04, U112 NC7WZ17, U113 NC7WZ17, U114 NC7WZ17, U115 NC7WZ17, U116 SN74CBTD3861, U117 NCP1529, U118 NC7WZ17, U119 NC7WZ07, U120 NC7WZ17, U121 YC124, U122 YC124, U123 ASE_CLK, U124 YC124, U125 NC7WZ17, U126 NC7WZ17, U127 NC7WZ07, U128 NC7WZ17, U129 YC124, U130 YC124, U131 NC7WZ17, U132 YC124, U133 YC124, U134 YC124, U135 YC124, U136 YC124, U137 YC124

Commit message: working on power sense again now. The normal board should be more or less done!
Parts:
- added C109: 10uF, 0603, symbol C
- added P111: PJ-044BH, symbol PJ-044BH
- added P112: CONN_7, symbol CONN_7
- C104: value 15uF -> 10uF
- C108: value 0.1uF -> 0.01uF
Connections:
- net +12V: now also P111.1 (PIN)
- net +5V: now also C109.1
- net DEBUG_N: now also P112.3 (P3)
- net GND: now also C109.2, P111.2
- net MSEL_N: now also P112.7 (P7)
- net RST_N: now also P112.1 (P1)
- net TCK: now also P112.4 (P4)
- net TDI_L: now also P112.6 (P6)
- net TDO_L: now also P112.2 (P2)
- net TMS: now also P112.5 (P5)
- net at R109.2, U109.8 (FB): no longer R108.1
- no-connect marks 2 -> 4
Other:
- note added: "Power Connector\n"
- moved on the sheet: C104, R108, R109
