File: l2_dev_alternative _nopwrsense/l2_pair.sch (KiCad schematic (older format))
At the start: 14 parts, among them U1102 NC7WZ17, U201 NC7WZ17, U203 NCP1529, U204 INA219

Commit message: doing the l2s alone
Parts:
- removed C204: 0.1uF, symbol C
- removed R205, R207: 10R, symbol R
- removed R206: 0.05, symbol R
- removed U204: INA219, symbol INA219
Connections:
- net labels removed: A0, A1, CLK, DATA
- wire segments 139 -> 119
Other:
- note removed: "Current Measurment\n"

Commit message: +1V0 power islands ready
Connections:
- net +1V0_F is gone; now on net +1V0: C202.1, C203.1, L201.2, R203.1
Changed lines of the file:
@@
-EESchema Schematic File Version 2  date 31/08/2011 14:36:59
+EESchema Schematic File Version 2  date 01/09/2011 14:48:10
 LIBS:power
 LIBS:device
@@
 $Descr A4 11700 8267
 encoding utf-8
-Sheet 5 13
+Sheet 11 13
 Title ""
-Date "31 aug 2011"
+Date "1 sep 2011"
 Rev ""
 Comp ""
@@
 Comment4 ""
 $EndDescr
+Text HLabel 3880 830  1    39   Input ~ 0
++1V0
+Text HLabel 8110 1230 0    60   Input ~ 0
++1V0_B
+Text HLabel 5470 1230 0    60   Input ~ 0
++1V0_T
 Wire Wire Line
 	10350 3760 10140 3760
@@
 AR Path="/4E36B777/4E5214B4" Ref="U502"  Part="1"
 AR Path="/4E36B760/4E5214B4" Ref="U802"  Part="1"
-F 0 "U502" H 1390 4450 60  0000 C CNN
+F 0 "U1102" H 1390 4450 60  0000 C CNN
 F 1 "NC7WZ17" H 1540 3650 60  0000 C CNN
 	1    1690 4050
@@
 Text Label 5390 3580 2    39   ~ 0
 TCK_BUF
-Text Label 8110 1230 2    60   ~ 0
-+1V0
-Text Label 5470 1230 2    60   ~ 0
-+1V0
 Text Notes 730  3420 0    60   ~ 0
 JTAG Buffering
@@
 TCK
 $Comp
-L GND #PWR506
+L GND #PWR0248
 U 1 1 4E35D9C0
 P 2340 4500
-AR Path="/4E36B777/4E35D9C0" Ref="#PWR506"  Part="1"
-AR Path="/4E36B760/4E35D9C0" Ref="#PWR806"  Part="1"
-AR Path="/4E36B740/4E35D9C0" Ref="#PWR1106"  Part="1"
-AR Path="/4E32CDCE/4E35D9C0" Ref="#PWR323"  Part="1"
-F 0 "#PWR506" H 2340 4500 30  0001 C CNN
+AR Path="/4E36B777/4E35D9C0" Ref="#PWR0248"  Part="1"
+AR Path="/4E36B760/4E35D9C0" Ref="#PWR0272"  Part="1"
+AR Path="/4E36B740/4E35D9C0" Ref="#PWR0296"  Part="1"
+AR Path="/4E32CDCE/4E35D9C0" Ref="#PWR0224"  Part="1"
+F 0 "#PWR0296" H 2340 4500 30  0001 C CNN
 F 1 "GND" H 2340 4430 30  0001 C CNN
 	1    2340 4500
@@
 $EndComp
 $Comp
-L GND #PWR504
+L GND #PWR0249
 U 1 1 4E35D9AA
 P 2340 3180
-AR Path="/4E36B777/4E35D9AA" Ref="#PWR504"  Part="1"
-AR Path="/4E36B760/4E35D9AA" Ref="#PWR804"  Part="1"
-AR Path="/4E36B740/4E35D9AA" Ref="#PWR1104"  Part="1"
-AR Path="/4E32CDCE/4E35D9AA" Ref="#PWR321"  Part="1"
-F 0 "#PWR504" H 2340 3180 30  0001 C CNN
+AR Path="/4E36B777/4E35D9AA" Ref="#PWR0249"  Part="1"
+AR Path="/4E36B760/4E35D9AA" Ref="#PWR0273"  Part="1"
+AR Path="/4E36B740/4E35D9AA" Ref="#PWR0297"  Part="1"
+AR Path="/4E32CDCE/4E35D9AA" Ref="#PWR0225"  Part="1"
+F 0 "#PWR0297" H 2340 3180 30  0001 C CNN
 F 1 "GND" H 2340 3110 30  0001 C CNN
 	1    2340 3180
@@
 $EndComp
 $Comp
-L +3.3V #PWR505
+L +3.3V #PWR0250
 U 1 1 4E35D9A0
 P 2340 3570
-AR Path="/4E36B777/4E35D9A0" Ref="#PWR505"  Part="1"
-AR Path="/4E36B760/4E35D9A0" Ref="#PWR805"  Part="1"
-AR Path="/4E36B740/4E35D9A0" Ref="#PWR1105"  Part="1"
-AR Path="/4E32CDCE/4E35D9A0" Ref="#PWR322"  Part="1"
-F 0 "#PWR505" H 2340 3530 30  0001 C CNN
+AR Path="/4E36B777/4E35D9A0" Ref="#PWR0250"  Part="1"
+AR Path="/4E36B760/4E35D9A0" Ref="#PWR0274"  Part="1"
+AR Path="/4E36B740/4E35D9A0" Ref="#PWR0298"  Part="1"
+AR Path="/4E32CDCE/4E35D9A0" Ref="#PWR0226"  Part="1"
+F 0 "#PWR0298" H 2340 3530 30  0001 C CNN
 F 1 "+3.3V" H 2340 3680 30  0000 C CNN
 	1    2340 3570
@@
 $EndComp
 $Comp
-L +3.3V #PWR503
+L +3.3V #PWR0251
 U 1 1 4E35D98B
 P 2340 2250
-AR Path="/4E36B777/4E35D98B" Ref="#PWR503"  Part="1"
-AR Path="/4E36B760/4E35D98B" Ref="#PWR803"  Part="1"
-AR Path="/4E36B740/4E35D98B" Ref="#PWR1103"  Part="1"
-AR Path="/4E32CDCE/4E35D98B" Ref="#PWR320"  Part="1"
-F 0 "#PWR503" H 2340 2210 30  0001 C CNN
+AR Path="/4E36B777/4E35D98B" Ref="#PWR0251"  Part="1"
+AR Path="/4E36B760/4E35D98B" Ref="#PWR0275"  Part="1"
+AR Path="/4E36B740/4E35D98B" Ref="#PWR0299"  Part="1"
+AR Path="/4E32CDCE/4E35D98B" Ref="#PWR0227"  Part="1"
+F 0 "#PWR0299" H 2340 2210 30  0001 C CNN
 F 1 "+3.3V" H 2340 2360 30  0000 C CNN
 	1    2340 2250
@@
 AR Path="/4E36B740/4E35D8BD" Ref="U801"  Part="1"
 AR Path="/4E32CDCE/4E35D8BD" Ref="U1101"  Part="1"
-F 0 "U201" H 1390 3130 60  0000 C CNN
+F 0 "U801" H 1390 3130 60  0000 C CNN
 F 1 "NC7WZ17" H 1540 2330 60  0000 C CNN
 	1    1690 2730
@@
 Text Notes 1320 720  0    60   ~ 0
 5V to 1V @ 1A
-Text Label 3880 830  1    39   ~ 0
-+1V0_F
 $Comp
 L C C203
@@
 AR Path="/4E36B740/4E35D6A2" Ref="C803"  Part="1"
 AR Path="/4E32CDCE/4E35D6A2" Ref="C1103"  Part="1"
-F 0 "C203" H 3850 1290 50  0000 L CNN
+F 0 "C803" H 3850 1290 50  0000 L CNN
 F 1 "10uF" H 3850 1090 50  0000 L CNN
 	1    3800 1190
@@
 AR Path="/4E36B740/4E35D649" Ref="C802"  Part="1"
 AR Path="/4E32CDCE/4E35D649" Ref="C1102"  Part="1"
-F 0 "C202" H 3510 1290 50  0000 L CNN
+F 0 "C802" H 3510 1290 50  0000 L CNN
 F 1 "33pF" H 3510 1100 50  0000 L CNN
 	1    3500 1190
@@
 AR Path="/4E36B740/4E35D5DA" Ref="R804"  Part="1"
 AR Path="/4E32CDCE/4E35D5DA" Ref="R1104"  Part="1"
-F 0 "R204" V 3310 1700 50  0000 C CNN
+F 0 "R804" V 3310 1700 50  0000 C CNN
 F 1 "100k" V 3230 1700 50  0000 C CNN
 	1    3230 1700
@@
 AR Path="/4E36B740/4E35D5C1" Ref="R803"  Part="1"
 AR Path="/4E32CDCE/4E35D5C1" Ref="R1103"  Part="1"
-F 0 "R203" V 3310 1170 50  0000 C CNN
+F 0 "R803" V 3310 1170 50  0000 C CNN
 F 1 "68k" V 3230 1170 50  0000 C CNN
 	1    3230 1170
@@
 AR Path="/4E36B740/4E35D5AC" Ref="L801"  Part="1"
 AR Path="/4E32CDCE/4E35D5AC" Ref="L1101"  Part="1"
-F 0 "L201" V 2790 920 40  0000 C CNN
+F 0 "L801" V 2790 920 40  0000 C CNN
 F 1 "2u2H" V 2940 920 40  0000 C CNN
 	1    2840 920
@@
 $EndComp
 $Comp
-L GND #PWR502
+L GND #PWR0252
 U 1 1 4E3545A6
 P 1740 1980
-AR Path="/4E36B777/4E3545A6" Ref="#PWR502"  Part="1"
-AR Path="/4E36B760/4E3545A6" Ref="#PWR802"  Part="1"
-AR Path="/4E36B740/4E3545A6" Ref="#PWR1102"  Part="1"
-AR Path="/4E32CDCE/4E3545A6" Ref="#PWR319"  Part="1"
-F 0 "#PWR502" H 1740 1980 30  0001 C CNN
+AR Path="/4E36B777/4E3545A6" Ref="#PWR0252"  Part="1"
+AR Path="/4E36B760/4E3545A6" Ref="#PWR0276"  Part="1"
+AR Path="/4E36B740/4E3545A6" Ref="#PWR0300"  Part="1"
+AR Path="/4E32CDCE/4E3545A6" Ref="#PWR0228"  Part="1"
+F 0 "#PWR0300" H 1740 1980 30  0001 C CNN
 F 1 "GND" H 1740 1910 30  0001 C CNN
 	1    1740 1980
@@
 AR Path="/4E36B740/4E354587" Ref="C801"  Part="1"
 AR Path="/4E32CDCE/4E354587" Ref="C1101"  Part="1"
-F 0 "C201" H 740 1250 50  0000 L CNN
+F 0 "C801" H 740 1250 50  0000 L CNN
 F 1 "10uF" H 740 1050 50  0000 L CNN
 	1    690  1150
@@
 $EndComp
 $Comp
-L +5V #PWR501
+L +5V #PWR0253
 U 1 1 4E35455A
 P 690 750
-AR Path="/4E36B777/4E35455A" Ref="#PWR501"  Part="1"
-AR Path="/4E36B760/4E35455A" Ref="#PWR801"  Part="1"
-AR Path="/4E36B740/4E35455A" Ref="#PWR1101"  Part="1"
-AR Path="/4E32CDCE/4E35455A" Ref="#PWR318"  Part="1"
-F 0 "#PWR501" H 690 840 20  0001 C CNN
+AR Path="/4E36B777/4E35455A" Ref="#PWR0253"  Part="1"
+AR Path="/4E36B760/4E35455A" Ref="#PWR0277"  Part="1"
+AR Path="/4E36B740/4E35455A" Ref="#PWR0301"  Part="1"
+AR Path="/4E32CDCE/4E35455A" Ref="#PWR0229"  Part="1"
+F 0 "#PWR0301" H 690 840 20  0001 C CNN
 F 1 "+5V" H 690 840 30  0000 C CNN
 	1    690  750
@@
 AR Path="/4E36B740/4E354532" Ref="U803"  Part="1"
 AR Path="/4E32CDCE/4E354532" Ref="U1103"  Part="1"
-F 0 "U203" H 1740 1220 60  0000 C CNN
+F 0 "U803" H 1740 1220 60  0000 C CNN
 F 1 "NCP1529" H 1740 1320 60  0000 C CNN
 	1    1740 1270

Commit message: logic error! remove the mux and put SW_4 instead
Changed lines of the file:
@@
-EESchema Schematic File Version 2  date 01/09/2011 14:48:10
+EESchema Schematic File Version 2  date 01/09/2011 16:24:27
 LIBS:power
 LIBS:device
@@
 $Descr A4 11700 8267
 encoding utf-8
-Sheet 11 13
+Sheet 8 13
 Title ""
 Date "1 sep 2011"
@@
 AR Path="/4E36B777/4E5214B4" Ref="U502"  Part="1"
 AR Path="/4E36B760/4E5214B4" Ref="U802"  Part="1"
-F 0 "U1102" H 1390 4450 60  0000 C CNN
+F 0 "U802" H 1390 4450 60  0000 C CNN
 F 1 "NC7WZ17" H 1540 3650 60  0000 C CNN
 	1    1690 4050
@@
 AR Path="/4E36B740/4E35D8BD" Ref="U801"  Part="1"
 AR Path="/4E32CDCE/4E35D8BD" Ref="U1101"  Part="1"
-F 0 "U801" H 1390 3130 60  0000 C CNN
+F 0 "U501" H 1390 3130 60  0000 C CNN
 F 1 "NC7WZ17" H 1540 2330 60  0000 C CNN
 	1    1690 2730
@@
 AR Path="/4E36B740/4E35D6A2" Ref="C803"  Part="1"
 AR Path="/4E32CDCE/4E35D6A2" Ref="C1103"  Part="1"
-F 0 "C803" H 3850 1290 50  0000 L CNN
+F 0 "C503" H 3850 1290 50  0000 L CNN
 F 1 "10uF" H 3850 1090 50  0000 L CNN
 	1    3800 1190
@@
 AR Path="/4E36B740/4E35D649" Ref="C802"  Part="1"
 AR Path="/4E32CDCE/4E35D649" Ref="C1102"  Part="1"
-F 0 "C802" H 3510 1290 50  0000 L CNN
+F 0 "C502" H 3510 1290 50  0000 L CNN
 F 1 "33pF" H 3510 1100 50  0000 L CNN
 	1    3500 1190
@@
 AR Path="/4E36B740/4E35D5DA" Ref="R804"  Part="1"
 AR Path="/4E32CDCE/4E35D5DA" Ref="R1104"  Part="1"
-F 0 "R804" V 3310 1700 50  0000 C CNN
+F 0 "R504" V 3310 1700 50  0000 C CNN
 F 1 "100k" V 3230 1700 50  0000 C CNN
 	1    3230 1700
@@
 AR Path="/4E36B740/4E35D5C1" Ref="R803"  Part="1"
 AR Path="/4E32CDCE/4E35D5C1" Ref="R1103"  Part="1"
-F 0 "R803" V 3310 1170 50  0000 C CNN
+F 0 "R503" V 3310 1170 50  0000 C CNN
 F 1 "68k" V 3230 1170 50  0000 C CNN
 	1    3230 1170
@@
 AR Path="/4E36B740/4E35D5AC" Ref="L801"  Part="1"
 AR Path="/4E32CDCE/4E35D5AC" Ref="L1101"  Part="1"
-F 0 "L801" V 2790 920 40  0000 C CNN
+F 0 "L501" V 2790 920 40  0000 C CNN
 F 1 "2u2H" V 2940 920 40  0000 C CNN
 	1    2840 920
@@
 AR Path="/4E36B740/4E354587" Ref="C801"  Part="1"
 AR Path="/4E32CDCE/4E354587" Ref="C1101"  Part="1"
-F 0 "C801" H 740 1250 50  0000 L CNN
+F 0 "C501" H 740 1250 50  0000 L CNN
 F 1 "10uF" H 740 1050 50  0000 L CNN
 	1    690  1150
@@
 AR Path="/4E36B740/4E354532" Ref="U803"  Part="1"
 AR Path="/4E32CDCE/4E354532" Ref="U1103"  Part="1"
-F 0 "U803" H 1740 1220 60  0000 C CNN
+F 0 "U503" H 1740 1220 60  0000 C CNN
 F 1 "NCP1529" H 1740 1320 60  0000 C CNN
 	1    1740 1270

Commit message: added term resistors for xlinks and changed RST buffers to open drain
Changed lines of the file:
@@
-EESchema Schematic File Version 2  date 01/09/2011 16:28:35
+EESchema Schematic File Version 2  date 02/09/2011 13:05:35
 LIBS:power
 LIBS:device
@@
 $Descr A4 11700 8267
 encoding utf-8
-Sheet 8 13
+Sheet 2 13
 Title ""
-Date "1 sep 2011"
+Date "2 sep 2011"
 Rev ""
 Comp ""
@@
 AR Path="/4E36B777/4E5214B4" Ref="U502"  Part="1"
 AR Path="/4E36B760/4E5214B4" Ref="U802"  Part="1"
-F 0 "U802" H 1390 4450 60  0000 C CNN
+F 0 "U202" H 1390 4450 60  0000 C CNN
 F 1 "NC7WZ17" H 1540 3650 60  0000 C CNN
 	1    1690 4050
@@
 AR Path="/4E36B740/4E35D9C0" Ref="#PWR0296"  Part="1"
 AR Path="/4E32CDCE/4E35D9C0" Ref="#PWR0224"  Part="1"
-F 0 "#PWR0296" H 2340 4500 30  0001 C CNN
+F 0 "#PWR0224" H 2340 4500 30  0001 C CNN
 F 1 "GND" H 2340 4430 30  0001 C CNN
 	1    2340 4500
@@
 AR Path="/4E36B740/4E35D9AA" Ref="#PWR0297"  Part="1"
 AR Path="/4E32CDCE/4E35D9AA" Ref="#PWR0225"  Part="1"
-F 0 "#PWR0297" H 2340 3180 30  0001 C CNN
+F 0 "#PWR0225" H 2340 3180 30  0001 C CNN
 F 1 "GND" H 2340 3110 30  0001 C CNN
 	1    2340 3180
@@
 AR Path="/4E36B740/4E35D9A0" Ref="#PWR0298"  Part="1"
 AR Path="/4E32CDCE/4E35D9A0" Ref="#PWR0226"  Part="1"
-F 0 "#PWR0298" H 2340 3530 30  0001 C CNN
+F 0 "#PWR0226" H 2340 3530 30  0001 C CNN
 F 1 "+3.3V" H 2340 3680 30  0000 C CNN
 	1    2340 3570
@@
 AR Path="/4E36B740/4E35D98B" Ref="#PWR0299"  Part="1"
 AR Path="/4E32CDCE/4E35D98B" Ref="#PWR0227"  Part="1"
-F 0 "#PWR0299" H 2340 2210 30  0001 C CNN
+F 0 "#PWR0227" H 2340 2210 30  0001 C CNN
 F 1 "+3.3V" H 2340 2360 30  0000 C CNN
 	1    2340 2250
@@
 AR Path="/4E36B740/4E35D8BD" Ref="U801"  Part="1"
 AR Path="/4E32CDCE/4E35D8BD" Ref="U1101"  Part="1"
-F 0 "U501" H 1390 3130 60  0000 C CNN
+F 0 "U1101" H 1390 3130 60  0000 C CNN
 F 1 "NC7WZ17" H 1540 2330 60  0000 C CNN
 	1    1690 2730
@@
 AR Path="/4E36B740/4E35D6A2" Ref="C803"  Part="1"
 AR Path="/4E32CDCE/4E35D6A2" Ref="C1103"  Part="1"
-F 0 "C503" H 3850 1290 50  0000 L CNN
+F 0 "C1103" H 3850 1290 50  0000 L CNN
 F 1 "10uF" H 3850 1090 50  0000 L CNN
 	1    3800 1190
@@
 AR Path="/4E36B740/4E35D649" Ref="C802"  Part="1"
 AR Path="/4E32CDCE/4E35D649" Ref="C1102"  Part="1"
-F 0 "C502" H 3510 1290 50  0000 L CNN
+F 0 "C1102" H 3510 1290 50  0000 L CNN
 F 1 "33pF" H 3510 1100 50  0000 L CNN
 	1    3500 1190
@@
 AR Path="/4E36B740/4E35D5DA" Ref="R804"  Part="1"
 AR Path="/4E32CDCE/4E35D5DA" Ref="R1104"  Part="1"
-F 0 "R504" V 3310 1700 50  0000 C CNN
+F 0 "R1104" V 3310 1700 50  0000 C CNN
 F 1 "100k" V 3230 1700 50  0000 C CNN
 	1    3230 1700
@@
 AR Path="/4E36B740/4E35D5C1" Ref="R803"  Part="1"
 AR Path="/4E32CDCE/4E35D5C1" Ref="R1103"  Part="1"
-F 0 "R503" V 3310 1170 50  0000 C CNN
+F 0 "R1103" V 3310 1170 50  0000 C CNN
 F 1 "68k" V 3230 1170 50  0000 C CNN
 	1    3230 1170
@@
 AR Path="/4E36B740/4E35D5AC" Ref="L801"  Part="1"
 AR Path="/4E32CDCE/4E35D5AC" Ref="L1101"  Part="1"
-F 0 "L501" V 2790 920 40  0000 C CNN
+F 0 "L1101" V 2790 920 40  0000 C CNN
 F 1 "2u2H" V 2940 920 40  0000 C CNN
 	1    2840 920
@@
 AR Path="/4E36B740/4E3545A6" Ref="#PWR0300"  Part="1"
 AR Path="/4E32CDCE/4E3545A6" Ref="#PWR0228"  Part="1"
-F 0 "#PWR0300" H 1740 1980 30  0001 C CNN
+F 0 "#PWR0228" H 1740 1980 30  0001 C CNN
 F 1 "GND" H 1740 1910 30  0001 C CNN
 	1    1740 1980
@@
 AR Path="/4E36B740/4E354587" Ref="C801"  Part="1"
 AR Path="/4E32CDCE/4E354587" Ref="C1101"  Part="1"
-F 0 "C501" H 740 1250 50  0000 L CNN
+F 0 "C1101" H 740 1250 50  0000 L CNN
 F 1 "10uF" H 740 1050 50  0000 L CNN
 	1    690  1150
@@
 AR Path="/4E36B740/4E35455A" Ref="#PWR0301"  Part="1"
 AR Path="/4E32CDCE/4E35455A" Ref="#PWR0229"  Part="1"
-F 0 "#PWR0301" H 690 840 20  0001 C CNN
+F 0 "#PWR0229" H 690 840 20  0001 C CNN
 F 1 "+5V" H 690 840 30  0000 C CNN
 	1    690  750
@@
 AR Path="/4E36B740/4E354532" Ref="U803"  Part="1"
 AR Path="/4E32CDCE/4E354532" Ref="U1103"  Part="1"
-F 0 "U503" H 1740 1220 60  0000 C CNN
+F 0 "U1103" H 1740 1220 60  0000 C CNN
 F 1 "NCP1529" H 1740 1320 60  0000 C CNN
 	1    1740 1270

Commit message: almost all the links in, some of the JTAG in. Surprisingly nice :)
Changed lines of the file:
@@
-EESchema Schematic File Version 2  date 05/09/2011 16:29:32
+EESchema Schematic File Version 2  date 06/09/2011 18:50:43
 LIBS:power
 LIBS:device
@@
 $Descr A4 11700 8267
 encoding utf-8
-Sheet 8 13
+Sheet 5 13
 Title ""
-Date "5 sep 2011"
+Date "6 sep 2011"
 Rev ""
 Comp ""
@@
 AR Path="/4E36B777/4E5214B4" Ref="U502"  Part="1"
 AR Path="/4E36B760/4E5214B4" Ref="U802"  Part="1"
-F 0 "U802" H 1390 4450 60  0000 C CNN
+F 0 "U1102" H 1390 4450 60  0000 C CNN
 F 1 "NC7WZ17" H 1540 3650 60  0000 C CNN
 	1    1690 4050
@@
 AR Path="/4E36B740/4E35D8BD" Ref="U801"  Part="1"
 AR Path="/4E32CDCE/4E35D8BD" Ref="U1101"  Part="1"
-F 0 "U501" H 1390 3130 60  0000 C CNN
+F 0 "U801" H 1390 3130 60  0000 C CNN
 F 1 "NC7WZ17" H 1540 2330 60  0000 C CNN
 	1    1690 2730
@@
 AR Path="/4E36B740/4E35D6A2" Ref="C803"  Part="1"
 AR Path="/4E32CDCE/4E35D6A2" Ref="C1103"  Part="1"
-F 0 "C503" H 3850 1290 50  0000 L CNN
+F 0 "C803" H 3850 1290 50  0000 L CNN
 F 1 "10uF" H 3850 1090 50  0000 L CNN
 	1    3800 1190
@@
 AR Path="/4E36B740/4E35D649" Ref="C802"  Part="1"
 AR Path="/4E32CDCE/4E35D649" Ref="C1102"  Part="1"
-F 0 "C502" H 3510 1290 50  0000 L CNN
+F 0 "C802" H 3510 1290 50  0000 L CNN
 F 1 "33pF" H 3510 1100 50  0000 L CNN
 	1    3500 1190
@@
 AR Path="/4E36B740/4E35D5DA" Ref="R804"  Part="1"
 AR Path="/4E32CDCE/4E35D5DA" Ref="R1104"  Part="1"
-F 0 "R504" V 3310 1700 50  0000 C CNN
+F 0 "R804" V 3310 1700 50  0000 C CNN
 F 1 "100k" V 3230 1700 50  0000 C CNN
 	1    3230 1700
@@
 AR Path="/4E36B740/4E35D5C1" Ref="R803"  Part="1"
 AR Path="/4E32CDCE/4E35D5C1" Ref="R1103"  Part="1"
-F 0 "R503" V 3310 1170 50  0000 C CNN
+F 0 "R803" V 3310 1170 50  0000 C CNN
 F 1 "68k" V 3230 1170 50  0000 C CNN
 	1    3230 1170
@@
 AR Path="/4E36B740/4E35D5AC" Ref="L801"  Part="1"
 AR Path="/4E32CDCE/4E35D5AC" Ref="L1101"  Part="1"
-F 0 "L501" V 2790 920 40  0000 C CNN
+F 0 "L801" V 2790 920 40  0000 C CNN
 F 1 "2u2H" V 2940 920 40  0000 C CNN
 	1    2840 920
@@
 AR Path="/4E36B740/4E354587" Ref="C801"  Part="1"
 AR Path="/4E32CDCE/4E354587" Ref="C1101"  Part="1"
-F 0 "C501" H 740 1250 50  0000 L CNN
+F 0 "C801" H 740 1250 50  0000 L CNN
 F 1 "10uF" H 740 1050 50  0000 L CNN
 	1    690  1150
@@
 AR Path="/4E36B740/4E354532" Ref="U803"  Part="1"
 AR Path="/4E32CDCE/4E354532" Ref="U1103"  Part="1"
-F 0 "U503" H 1740 1220 60  0000 C CNN
+F 0 "U803" H 1740 1220 60  0000 C CNN
 F 1 "NCP1529" H 1740 1320 60  0000 C CNN
 	1    1740 1270
