File: l2_dev_alternative _nopwrsense/l2_pair.sch (KiCad schematic (older format))
At the start: 9 parts, among them U1102 NC7WZ17, U201 NC7WZ17, U203 NCP1529

Commit message: almost done. adding cutouts for power islands
Changed lines of the file:
@@
-EESchema Schematic File Version 2  date 06/09/2011 20:03:42
+EESchema Schematic File Version 2  date 07/09/2011 23:31:18
 LIBS:power
 LIBS:device
@@
 $Descr A4 11700 8267
 encoding utf-8
-Sheet 5 13
+Sheet 2 13
 Title ""
-Date "6 sep 2011"
+Date "7 sep 2011"
 Rev ""
 Comp ""
@@
 AR Path="/4E36B777/4E5214B4" Ref="U502"  Part="1"
 AR Path="/4E36B760/4E5214B4" Ref="U802"  Part="1"
-F 0 "U1102" H 1390 4450 60  0000 C CNN
+F 0 "U502" H 1390 4450 60  0000 C CNN
 F 1 "NC7WZ17" H 1540 3650 60  0000 C CNN
 	1    1690 4050
@@
 AR Path="/4E36B740/4E35D8BD" Ref="U801"  Part="1"
 AR Path="/4E32CDCE/4E35D8BD" Ref="U1101"  Part="1"
-F 0 "U801" H 1390 3130 60  0000 C CNN
+F 0 "U201" H 1390 3130 60  0000 C CNN
 F 1 "NC7WZ17" H 1540 2330 60  0000 C CNN
 	1    1690 2730
@@
 AR Path="/4E36B740/4E35D6A2" Ref="C803"  Part="1"
 AR Path="/4E32CDCE/4E35D6A2" Ref="C1103"  Part="1"
-F 0 "C803" H 3850 1290 50  0000 L CNN
+F 0 "C203" H 3850 1290 50  0000 L CNN
 F 1 "10uF" H 3850 1090 50  0000 L CNN
 	1    3800 1190
@@
 AR Path="/4E36B740/4E35D649" Ref="C802"  Part="1"
 AR Path="/4E32CDCE/4E35D649" Ref="C1102"  Part="1"
-F 0 "C802" H 3510 1290 50  0000 L CNN
+F 0 "C202" H 3510 1290 50  0000 L CNN
 F 1 "33pF" H 3510 1100 50  0000 L CNN
 	1    3500 1190
@@
 AR Path="/4E36B740/4E35D5DA" Ref="R804"  Part="1"
 AR Path="/4E32CDCE/4E35D5DA" Ref="R1104"  Part="1"
-F 0 "R804" V 3310 1700 50  0000 C CNN
+F 0 "R204" V 3310 1700 50  0000 C CNN
 F 1 "100k" V 3230 1700 50  0000 C CNN
 	1    3230 1700
@@
 AR Path="/4E36B740/4E35D5C1" Ref="R803"  Part="1"
 AR Path="/4E32CDCE/4E35D5C1" Ref="R1103"  Part="1"
-F 0 "R803" V 3310 1170 50  0000 C CNN
+F 0 "R203" V 3310 1170 50  0000 C CNN
 F 1 "68k" V 3230 1170 50  0000 C CNN
 	1    3230 1170
@@
 AR Path="/4E36B740/4E35D5AC" Ref="L801"  Part="1"
 AR Path="/4E32CDCE/4E35D5AC" Ref="L1101"  Part="1"
-F 0 "L801" V 2790 920 40  0000 C CNN
+F 0 "L201" V 2790 920 40  0000 C CNN
 F 1 "2u2H" V 2940 920 40  0000 C CNN
 	1    2840 920
@@
 AR Path="/4E36B740/4E354587" Ref="C801"  Part="1"
 AR Path="/4E32CDCE/4E354587" Ref="C1101"  Part="1"
-F 0 "C801" H 740 1250 50  0000 L CNN
+F 0 "C201" H 740 1250 50  0000 L CNN
 F 1 "10uF" H 740 1050 50  0000 L CNN
 	1    690  1150
@@
 AR Path="/4E36B740/4E354532" Ref="U803"  Part="1"
 AR Path="/4E32CDCE/4E354532" Ref="U1103"  Part="1"
-F 0 "U803" H 1740 1220 60  0000 C CNN
+F 0 "U203" H 1740 1220 60  0000 C CNN
 F 1 "NCP1529" H 1740 1320 60  0000 C CNN
 	1    1740 1270

Commit message: going to flood the top!
Parts:
- added R501: 33R, 0603, symbol R
- C201, C202, C203, R203, R204: footprint (none) -> 0603
- L201: footprint (none) -> NCLV
- U1102, U201: footprint (none) -> SC70-6
- U203: footprint (none) -> SOT23-5
Connections:
- net TCK_BUF: now also R501.1; no longer U201.6 (Y1)
- new net: R501.2, U201.6 (Y1)
