File: l2_dev_alternative _nopwrsense/l2_pair.sch (KiCad schematic (older format))
At the start: 10 parts, among them U1102 NC7WZ17, U201 NC7WZ17, U203 NCP1529

Commit message: working on power sense again now. The normal board should be more or less done!
Changed lines of the file:
@@
-EESchema Schematic File Version 2  date 09/09/2011 00:11:47
+EESchema Schematic File Version 2  date 12/09/2011 21:13:56
 LIBS:power
 LIBS:device
@@
 Sheet 5 13
 Title ""
-Date "8 sep 2011"
+Date "12 sep 2011"
 Rev ""
 Comp ""
@@
 AR Path="/4E36B760/4E688FDA" Ref="R801"  Part="1"
 AR Path="/4E36B740/4E688FDA" Ref="R1101"  Part="1"
-F 0 "R501" V 2730 2630 50  0000 C CNN
+F 0 "R201" V 2730 2630 50  0000 C CNN
 F 1 "33R" V 2650 2630 50  0000 C CNN
 F 2 "0603" H 2650 2630 60  0001 C CNN
@@
 AR Path="/4E36B777/4E5214B4" Ref="U502"  Part="1"
 AR Path="/4E36B760/4E5214B4" Ref="U802"  Part="1"
-F 0 "U202" H 1390 4450 60  0000 C CNN
+F 0 "U502" H 1390 4450 60  0000 C CNN
 F 1 "NC7WZ17" H 1540 3650 60  0000 C CNN
 F 2 "SC70-6" H 1690 4050 60  0001 C CNN
@@
 TCK
 $Comp
-L GND #PWR0222
+L GND #PWR0224
 U 1 1 4E35D9C0
 P 2340 4500
-AR Path="/4E36B777/4E35D9C0" Ref="#PWR0222"  Part="1"
-AR Path="/4E36B760/4E35D9C0" Ref="#PWR0270"  Part="1"
-AR Path="/4E36B740/4E35D9C0" Ref="#PWR0294"  Part="1"
-AR Path="/4E32CDCE/4E35D9C0" Ref="#PWR0246"  Part="1"
-F 0 "#PWR0246" H 2340 4500 30  0001 C CNN
+AR Path="/4E36B777/4E35D9C0" Ref="#PWR0224"  Part="1"
+AR Path="/4E36B760/4E35D9C0" Ref="#PWR0272"  Part="1"
+AR Path="/4E36B740/4E35D9C0" Ref="#PWR0296"  Part="1"
+AR Path="/4E32CDCE/4E35D9C0" Ref="#PWR0248"  Part="1"
+F 0 "#PWR0224" H 2340 4500 30  0001 C CNN
 F 1 "GND" H 2340 4430 30  0001 C CNN
 	1    2340 4500
@@
 $EndComp
 $Comp
-L GND #PWR0223
+L GND #PWR0225
 U 1 1 4E35D9AA
 P 2340 3180
-AR Path="/4E36B777/4E35D9AA" Ref="#PWR0223"  Part="1"
-AR Path="/4E36B760/4E35D9AA" Ref="#PWR0271"  Part="1"
-AR Path="/4E36B740/4E35D9AA" Ref="#PWR0295"  Part="1"
-AR Path="/4E32CDCE/4E35D9AA" Ref="#PWR0247"  Part="1"
-F 0 "#PWR0247" H 2340 3180 30  0001 C CNN
+AR Path="/4E36B777/4E35D9AA" Ref="#PWR0225"  Part="1"
+AR Path="/4E36B760/4E35D9AA" Ref="#PWR0273"  Part="1"
+AR Path="/4E36B740/4E35D9AA" Ref="#PWR0297"  Part="1"
+AR Path="/4E32CDCE/4E35D9AA" Ref="#PWR0249"  Part="1"
+F 0 "#PWR0225" H 2340 3180 30  0001 C CNN
 F 1 "GND" H 2340 3110 30  0001 C CNN
 	1    2340 3180
@@
 $EndComp
 $Comp
-L +3.3V #PWR0224
+L +3.3V #PWR0226
 U 1 1 4E35D9A0
 P 2340 3570
-AR Path="/4E36B777/4E35D9A0" Ref="#PWR0224"  Part="1"
-AR Path="/4E36B760/4E35D9A0" Ref="#PWR0272"  Part="1"
-AR Path="/4E36B740/4E35D9A0" Ref="#PWR0296"  Part="1"
-AR Path="/4E32CDCE/4E35D9A0" Ref="#PWR0248"  Part="1"
-F 0 "#PWR0248" H 2340 3530 30  0001 C CNN
+AR Path="/4E36B777/4E35D9A0" Ref="#PWR0226"  Part="1"
+AR Path="/4E36B760/4E35D9A0" Ref="#PWR0274"  Part="1"
+AR Path="/4E36B740/4E35D9A0" Ref="#PWR0298"  Part="1"
+AR Path="/4E32CDCE/4E35D9A0" Ref="#PWR0250"  Part="1"
+F 0 "#PWR0226" H 2340 3530 30  0001 C CNN
 F 1 "+3.3V" H 2340 3680 30  0000 C CNN
 	1    2340 3570
@@
 $EndComp
 $Comp
-L +3.3V #PWR0225
+L +3.3V #PWR0227
 U 1 1 4E35D98B
 P 2340 2250
-AR Path="/4E36B777/4E35D98B" Ref="#PWR0225"  Part="1"
-AR Path="/4E36B760/4E35D98B" Ref="#PWR0273"  Part="1"
-AR Path="/4E36B740/4E35D98B" Ref="#PWR0297"  Part="1"
-AR Path="/4E32CDCE/4E35D98B" Ref="#PWR0249"  Part="1"
-F 0 "#PWR0249" H 2340 2210 30  0001 C CNN
+AR Path="/4E36B777/4E35D98B" Ref="#PWR0227"  Part="1"
+AR Path="/4E36B760/4E35D98B" Ref="#PWR0275"  Part="1"
+AR Path="/4E36B740/4E35D98B" Ref="#PWR0299"  Part="1"
+AR Path="/4E32CDCE/4E35D98B" Ref="#PWR0251"  Part="1"
+F 0 "#PWR0227" H 2340 2210 30  0001 C CNN
 F 1 "+3.3V" H 2340 2360 30  0000 C CNN
 	1    2340 2250
@@
 AR Path="/4E36B740/4E35D8BD" Ref="U801"  Part="1"
 AR Path="/4E32CDCE/4E35D8BD" Ref="U1101"  Part="1"
-F 0 "U1101" H 1390 3130 60  0000 C CNN
+F 0 "U201" H 1390 3130 60  0000 C CNN
 F 1 "NC7WZ17" H 1540 2330 60  0000 C CNN
 F 2 "SC70-6" H 1690 2730 60  0001 C CNN
@@
 AR Path="/4E36B740/4E35D6A2" Ref="C803"  Part="1"
 AR Path="/4E32CDCE/4E35D6A2" Ref="C1103"  Part="1"
-F 0 "C1103" H 3850 1290 50  0000 L CNN
+F 0 "C203" H 3850 1290 50  0000 L CNN
 F 1 "10uF" H 3850 1090 50  0000 L CNN
 F 2 "0603" H 3800 1190 60  0001 C CNN
@@
 AR Path="/4E36B740/4E35D649" Ref="C802"  Part="1"
 AR Path="/4E32CDCE/4E35D649" Ref="C1102"  Part="1"
-F 0 "C1102" H 3510 1290 50  0000 L CNN
+F 0 "C202" H 3510 1290 50  0000 L CNN
 F 1 "33pF" H 3510 1100 50  0000 L CNN
 F 2 "0603" H 3500 1190 60  0001 C CNN
@@
 AR Path="/4E36B740/4E35D5DA" Ref="R804"  Part="1"
 AR Path="/4E32CDCE/4E35D5DA" Ref="R1104"  Part="1"
-F 0 "R1104" V 3310 1700 50  0000 C CNN
+F 0 "R204" V 3310 1700 50  0000 C CNN
 F 1 "100k" V 3230 1700 50  0000 C CNN
 F 2 "0603" H 3230 1700 60  0001 C CNN
@@
 AR Path="/4E36B740/4E35D5C1" Ref="R803"  Part="1"
 AR Path="/4E32CDCE/4E35D5C1" Ref="R1103"  Part="1"
-F 0 "R1103" V 3310 1170 50  0000 C CNN
+F 0 "R203" V 3310 1170 50  0000 C CNN
 F 1 "68k" V 3230 1170 50  0000 C CNN
 F 2 "0603" H 3230 1170 60  0001 C CNN
@@
 AR Path="/4E36B740/4E35D5AC" Ref="L801"  Part="1"
 AR Path="/4E32CDCE/4E35D5AC" Ref="L1101"  Part="1"
-F 0 "L1101" V 2790 920 40  0000 C CNN
+F 0 "L201" V 2790 920 40  0000 C CNN
 F 1 "2u2H" V 2940 920 40  0000 C CNN
 F 2 "NCLV" H 2840 920 60  0001 C CNN
@@
 $EndComp
 $Comp
-L GND #PWR0226
+L GND #PWR0228
 U 1 1 4E3545A6
 P 1740 1980
-AR Path="/4E36B777/4E3545A6" Ref="#PWR0226"  Part="1"
-AR Path="/4E36B760/4E3545A6" Ref="#PWR0274"  Part="1"
-AR Path="/4E36B740/4E3545A6" Ref="#PWR0298"  Part="1"
-AR Path="/4E32CDCE/4E3545A6" Ref="#PWR0250"  Part="1"
-F 0 "#PWR0250" H 1740 1980 30  0001 C CNN
+AR Path="/4E36B777/4E3545A6" Ref="#PWR0228"  Part="1"
+AR Path="/4E36B760/4E3545A6" Ref="#PWR0276"  Part="1"
+AR Path="/4E36B740/4E3545A6" Ref="#PWR0300"  Part="1"
+AR Path="/4E32CDCE/4E3545A6" Ref="#PWR0252"  Part="1"
+F 0 "#PWR0228" H 1740 1980 30  0001 C CNN
 F 1 "GND" H 1740 1910 30  0001 C CNN
 	1    1740 1980
@@
 AR Path="/4E36B740/4E354587" Ref="C801"  Part="1"
 AR Path="/4E32CDCE/4E354587" Ref="C1101"  Part="1"
-F 0 "C1101" H 740 1250 50  0000 L CNN
+F 0 "C201" H 740 1250 50  0000 L CNN
 F 1 "10uF" H 740 1050 50  0000 L CNN
 F 2 "0603" H 690 1150 60  0001 C CNN
@@
 $EndComp
 $Comp
-L +5V #PWR0227
+L +5V #PWR0229
 U 1 1 4E35455A
 P 690 750
-AR Path="/4E36B777/4E35455A" Ref="#PWR0227"  Part="1"
-AR Path="/4E36B760/4E35455A" Ref="#PWR0275"  Part="1"
-AR Path="/4E36B740/4E35455A" Ref="#PWR0299"  Part="1"
-AR Path="/4E32CDCE/4E35455A" Ref="#PWR0251"  Part="1"
-F 0 "#PWR0251" H 690 840 20  0001 C CNN
+AR Path="/4E36B777/4E35455A" Ref="#PWR0229"  Part="1"
+AR Path="/4E36B760/4E35455A" Ref="#PWR0277"  Part="1"
+AR Path="/4E36B740/4E35455A" Ref="#PWR0301"  Part="1"
+AR Path="/4E32CDCE/4E35455A" Ref="#PWR0253"  Part="1"
+F 0 "#PWR0229" H 690 840 20  0001 C CNN
 F 1 "+5V" H 690 840 30  0000 C CNN
 	1    690  750
@@
 AR Path="/4E36B740/4E354532" Ref="U803"  Part="1"
 AR Path="/4E32CDCE/4E354532" Ref="U1103"  Part="1"
-F 0 "U1103" H 1740 1220 60  0000 C CNN
+F 0 "U203" H 1740 1220 60  0000 C CNN
 F 1 "NCP1529" H 1740 1320 60  0000 C CNN
 F 2 "SOT23-5" H 1740 1270 60  0001 C CNN
